Commit message: renamed .stl files

File: lbr_description/urdf/iiwa14.urdf (robot description, URDF)
Before this commit: robot iiwa, 8 links, 7 joints
Links:
- removed link link_1_1
- removed link link_2_1
- removed link link_3_1
- removed link link_4_1
- removed link link_5_1
- removed link link_6_1
- removed link link_7_1
- added link link_1, mass 32.252499792432545; collision mesh filename=package://fusion2urdf/lbr_description/meshes/iiwa14/link_1.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; visual mesh filename=package://fusion2urdf/lbr_description/meshes/iiwa14/link_1.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
- added link link_2, mass 31.020446759849573; collision mesh filename=package://fusion2urdf/lbr_description/meshes/iiwa14/link_2.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; visual mesh filename=package://fusion2urdf/lbr_description/meshes/iiwa14/link_2.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
- added link link_3, mass 0.0; collision mesh filename=package://fusion2urdf/lbr_description/meshes/iiwa14/link_3.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; visual mesh filename=package://fusion2urdf/lbr_description/meshes/iiwa14/link_3.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
- added link link_4, mass 21.50439908415142; collision mesh filename=package://fusion2urdf/lbr_description/meshes/iiwa14/link_4.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; visual mesh filename=package://fusion2urdf/lbr_description/meshes/iiwa14/link_4.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
- added link link_5, mass 13.294575666066379; collision mesh filename=package://fusion2urdf/lbr_description/meshes/iiwa14/link_5.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; visual mesh filename=package://fusion2urdf/lbr_description/meshes/iiwa14/link_5.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
- added link link_6, mass 14.198362583652283; collision mesh filename=package://fusion2urdf/lbr_description/meshes/iiwa14/link_6.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; visual mesh filename=package://fusion2urdf/lbr_description/meshes/iiwa14/link_6.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
- added link link_7, mass 2.4182992945540933; collision mesh filename=package://fusion2urdf/lbr_description/meshes/iiwa14/link_7.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; visual mesh filename=package://fusion2urdf/lbr_description/meshes/iiwa14/link_7.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
Joints:
- joint A1: child link_1_1 -> link_1
- joint A2: child link_2_1 -> link_2; parent link_1_1 -> link_1
- joint A3: child link_3_1 -> link_3; parent link_2_1 -> link_2
- joint A4: child link_4_1 -> link_4; parent link_3_1 -> link_3
- joint A5: child link_5_1 -> link_5; parent link_4_1 -> link_4
- joint A6: child link_6_1 -> link_6; parent link_5_1 -> link_5
- joint A7: child link_7_1 -> link_7; parent link_6_1 -> link_6

File: lbr_description/urdf/iiwa7.urdf (robot description, URDF)
Before this commit: robot iiwa7, 8 links, 7 joints
Links:
- removed link link_1_1
- removed link link_2_1
- removed link link_3_1
- removed link link_4_1
- removed link link_5_1
- removed link link_6_1
- removed link link_7_1
- added link link_1, mass 21.213926420791886; collision mesh filename=package://fusion2urdf/lbr_description/meshes/iiwa7/link_1.s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; visual mesh filename=package://fusion2urdf/lbr_description/meshes/iiwa7/link_1.s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
- added link link_2, mass 21.39756651772542; collision mesh filename=package://fusion2urdf/lbr_description/meshes/iiwa7/link_2.s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; visual mesh filename=package://fusion2urdf/lbr_description/meshes/iiwa7/link_2.s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
- added link link_3, mass 24.923667110884463; collision mesh filename=package://fusion2urdf/lbr_description/meshes/iiwa7/link_3.s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; visual mesh filename=package://fusion2urdf/lbr_description/meshes/iiwa7/link_3.s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
- added link link_4, mass 21.39755453189086; collision mesh filename=package://fusion2urdf/lbr_description/meshes/iiwa7/link_4.s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; visual mesh filename=package://fusion2urdf/lbr_description/meshes/iiwa7/link_4.s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
- added link link_5, mass 13.296700832855965; collision mesh filename=package://fusion2urdf/lbr_description/meshes/iiwa7/link_5.s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; visual mesh filename=package://fusion2urdf/lbr_description/meshes/iiwa7/link_5.s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
- added link link_6, mass 14.421451173118493; collision mesh filename=package://fusion2urdf/lbr_description/meshes/iiwa7/link_6.s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; visual mesh filename=package://fusion2urdf/lbr_description/meshes/iiwa7/link_6.s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
- added link link_7, mass 2.113113203151399; collision mesh filename=package://fusion2urdf/lbr_description/meshes/iiwa7/link_7.s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; visual mesh filename=package://fusion2urdf/lbr_description/meshes/iiwa7/link_7.s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
Joints:
- joint A1: child link_1_1 -> link_1
- joint A2: child link_2_1 -> link_2; parent link_1_1 -> link_1
- joint A3: child link_3_1 -> link_3; parent link_2_1 -> link_2
- joint A4: child link_4_1 -> link_4; parent link_3_1 -> link_3
- joint A5: child link_5_1 -> link_5; parent link_4_1 -> link_4
- joint A6: child link_6_1 -> link_6; parent link_5_1 -> link_5
- joint A7: child link_7_1 -> link_7; parent link_6_1 -> link_6

File: lbr_description/urdf/med14.urdf (robot description, URDF)
Before this commit: robot med14, 8 links, 7 joints
Links:
- removed link link_1_1
- removed link link_2_1
- removed link link_3_1
- removed link link_4_1
- removed link link_5_1
- removed link link_6_1
- removed link link_7_1
- added link link_1, mass 32.252499792432545; collision mesh filename=package://fusion2urdf/lbr_description/meshes/med14/link_1.s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; visual mesh filename=package://fusion2urdf/lbr_description/meshes/med14/link_1.s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
- added link link_2, mass 34.68757984100769; collision mesh filename=package://fusion2urdf/lbr_description/meshes/med14/link_2.s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; visual mesh filename=package://fusion2urdf/lbr_description/meshes/med14/link_2.s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
- added link link_3, mass 21.104680740321076; collision mesh filename=package://fusion2urdf/lbr_description/meshes/med14/link_3.s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; visual mesh filename=package://fusion2urdf/lbr_description/meshes/med14/link_3.s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
- added link link_4, mass 25.13964883334753; collision mesh filename=package://fusion2urdf/lbr_description/meshes/med14/link_4.s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; visual mesh filename=package://fusion2urdf/lbr_description/meshes/med14/link_4.s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
- added link link_5, mass 9.534880920206561; collision mesh filename=package://fusion2urdf/lbr_description/meshes/med14/link_5.s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; visual mesh filename=package://fusion2urdf/lbr_description/meshes/med14/link_5.s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
- added link link_6, mass 14.987109331085524; collision mesh filename=package://fusion2urdf/lbr_description/meshes/med14/link_6.s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; visual mesh filename=package://fusion2urdf/lbr_description/meshes/med14/link_6.s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
- added link link_7, mass 1.617833997596271; collision mesh filename=package://fusion2urdf/lbr_description/meshes/med14/link_7.s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; visual mesh filename=package://fusion2urdf/lbr_description/meshes/med14/link_7.s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
Joints:
- joint A1: child link_1_1 -> link_1
- joint A2: child link_2_1 -> link_2; parent link_1_1 -> link_1
- joint A3: child link_3_1 -> link_3; parent link_2_1 -> link_2
- joint A4: child link_4_1 -> link_4; parent link_3_1 -> link_3
- joint A5: child link_5_1 -> link_5; parent link_4_1 -> link_4
- joint A6: child link_6_1 -> link_6; parent link_5_1 -> link_5
- joint A7: child link_7_1 -> link_7; parent link_6_1 -> link_6

File: lbr_description/urdf/med7.urdf (robot description, URDF)
Before this commit: robot med7, 8 links, 7 joints
Links:
- removed link link_1_1
- removed link link_2_1
- removed link link_3_1
- removed link link_4_1
- removed link link_5_1
- removed link link_6_1
- removed link link_7_1
- added link link_1, mass 21.161828997118327; collision mesh filename=package://fusion2urdf/lbr_description/meshes/med7/link_1.stl; visual mesh filename=package://fusion2urdf/lbr_description/meshes/med7/link_1.stl
- added link link_2, mass 25.13966081800886; collision mesh filename=package://fusion2urdf/lbr_description/meshes/med7/link_2.stl; visual mesh filename=package://fusion2urdf/lbr_description/meshes/med7/link_2.stl
- added link link_3, mass 21.1618289971097; collision mesh filename=package://fusion2urdf/lbr_description/meshes/med7/link_3.stl; visual mesh filename=package://fusion2urdf/lbr_description/meshes/med7/link_3.stl
- added link link_4, mass 25.139648831600116; collision mesh filename=package://fusion2urdf/lbr_description/meshes/med7/link_4.stl; visual mesh filename=package://fusion2urdf/lbr_description/meshes/med7/link_4.stl
- added link link_5, mass 9.534880920206515; collision mesh filename=package://fusion2urdf/lbr_description/meshes/med7/link_5.stl; visual mesh filename=package://fusion2urdf/lbr_description/meshes/med7/link_5.stl
- added link link_6, mass 14.987109331100873; collision mesh filename=package://fusion2urdf/lbr_description/meshes/med7/link_6.stl; visual mesh filename=package://fusion2urdf/lbr_description/meshes/med7/link_6.stl
- added link link_7, mass 1.6178339975962697; collision mesh filename=package://fusion2urdf/lbr_description/meshes/med7/link_7.stl; visual mesh filename=package://fusion2urdf/lbr_description/meshes/med7/link_7.stl
Joints:
- joint A1: child link_1_1 -> link_1
- joint A2: child link_2_1 -> link_2; parent link_1_1 -> link_1
- joint A3: child link_3_1 -> link_3; parent link_2_1 -> link_2
- joint A4: child link_4_1 -> link_4; parent link_3_1 -> link_3
- joint A5: child link_5_1 -> link_5; parent link_4_1 -> link_4
- joint A6: child link_6_1 -> link_6; parent link_5_1 -> link_5
- joint A7: child link_7_1 -> link_7; parent link_6_1 -> link_6

Commit message: visualizations launching for ros1

File: lbr_description/urdf/iiwa14.urdf (robot description, URDF)
Before this commit: robot iiwa, 8 links, 7 joints
Links:
- link link_3: mass 0.0 -> 24.923667076480577
- link link_5: mass 13.294575666066379 -> 13.29457566606638
Joints:
- joint A1: limit lower=-2.96706 upper=2.96706 effort=100 velocity=1.48352986 -> lower=-2.96706 upper=2.96706 effort=100 velocity=100
- joint A2: limit lower=-2.094395 upper=2.094395 effort=100 velocity=1.48352986 -> lower=-2.094395 upper=2.094395 effort=100 velocity=100
- joint A3: limit lower=-2.96706 upper=2.96706 effort=100 velocity=1.74532925 -> lower=-2.96706 upper=2.96706 effort=100 velocity=100; origin xyz=-0.0 0.01 0.1945 rpy=0 0 0 -> xyz=0.0 0.01 0.1945 rpy=0 0 0
- joint A4: limit lower=-2.094395 upper=2.094395 effort=100 velocity=1.30899694 -> lower=-2.094395 upper=2.094395 effort=100 velocity=100; origin xyz=0.0 0.0105 0.2255 rpy=0 0 0 -> xyz=-0.0 0.0105 0.2255 rpy=0 0 0
- joint A5: limit lower=-2.96706 upper=2.96706 effort=100 velocity=2.26892803 -> lower=-2.96706 upper=2.96706 effort=100 velocity=100
- joint A6: limit lower=-2.094395 upper=2.094395 effort=100 velocity=2.35619449 -> lower=-2.094395 upper=2.094395 effort=100 velocity=100
- joint A7: limit lower=-3.054326 upper=3.054326 effort=100 velocity=2.35619449 -> lower=-3.054326 upper=3.054326 effort=100 velocity=100

Commit message: added fixed world frame to urdf files

File: lbr_description/urdf/iiwa14.urdf (robot description, URDF)
Before this commit: robot iiwa14, 8 links, 7 joints
Links:
- added link world
Joints:
- added joint world_iiwa7_joint: type fixed, parent world, child base_link, origin xyz=0.0 0.0 0.0 rpy=0 0 0

File: lbr_description/urdf/iiwa7.urdf (robot description, URDF)
Before this commit: robot iiwa7, 8 links, 7 joints
Links:
- added link world
Joints:
- added joint world_iiwa7_joint: type fixed, parent world, child base_link, origin xyz=0.0 0.0 0.0 rpy=0 0 0

File: lbr_description/urdf/med14.urdf (robot description, URDF)
Before this commit: robot med14, 8 links, 7 joints
Links:
- added link world
Joints:
- added joint world_iiwa7_joint: type fixed, parent world, child base_link, origin xyz=0.0 0.0 0.0 rpy=0 0 0

File: lbr_description/urdf/med7.urdf (robot description, URDF)
Before this commit: robot med7, 8 links, 7 joints
Links:
- added link world
Joints:
- added joint world_iiwa7_joint: type fixed, parent world, child base_link, origin xyz=0.0 0.0 0.0 rpy=0 0 0

Commit message: corrected maximum velocity

File: lbr_description/urdf/iiwa14.urdf (robot description, URDF)
Before this commit: robot iiwa14, 9 links, 8 joints
Joints:
- joint A1: limit lower=-2.96706 upper=2.96706 effort=100 velocity=100 -> lower=-2.96706 upper=2.96706 effort=100 velocity=1.48352986
- joint A2: limit lower=-2.094395 upper=2.094395 effort=100 velocity=100 -> lower=-2.094395 upper=2.094395 effort=100 velocity=1.48352986
- joint A3: limit lower=-2.96706 upper=2.96706 effort=100 velocity=100 -> lower=-2.96706 upper=2.96706 effort=100 velocity=1.74532925
- joint A4: limit lower=-2.094395 upper=2.094395 effort=100 velocity=100 -> lower=-2.094395 upper=2.094395 effort=100 velocity=1.30899694
- joint A5: limit lower=-2.96706 upper=2.96706 effort=100 velocity=100 -> lower=-2.96706 upper=2.96706 effort=100 velocity=2.26892803
- joint A6: limit lower=-2.094395 upper=2.094395 effort=100 velocity=100 -> lower=-2.094395 upper=2.094395 effort=100 velocity=2.35619449
- joint A7: limit lower=-3.054326 upper=3.054326 effort=100 velocity=100 -> lower=-3.054326 upper=3.054326 effort=100 velocity=2.35619449

Commit message: add med res stl

File: lbr_description/urdf/iiwa14.urdf (robot description, URDF)
Before this commit: robot iiwa14, 9 links, 8 joints
Links:
- link base_link: geometry collision mesh filename=package://lbr_description/meshes/iiwa14/collision/base_link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; visual mesh filename=package://lbr_description/meshes/iiwa14/visual/base_link.stl
- link link_1: geometry collision mesh filename=package://lbr_description/meshes/iiwa14/collisionink_1.stl; visual mesh filename=package://lbr_description/meshes/iiwa14/visual/link_1.stl
- link link_2: geometry collision mesh filename=package://lbr_description/meshes/iiwa14/collisionink_2.stl; visual mesh filename=package://lbr_description/meshes/iiwa14/visual/link_2.stl
- link link_3: geometry collision mesh filename=package://lbr_description/meshes/iiwa14/collisionink_3.stl; visual mesh filename=package://lbr_description/meshes/iiwa14/visual/link_3.stl
- link link_4: geometry collision mesh filename=package://lbr_description/meshes/iiwa14/collisionink_4.stl; visual mesh filename=package://lbr_description/meshes/iiwa14/visual/link_4.stl
- link link_5: geometry collision mesh filename=package://lbr_description/meshes/iiwa14/collisionink_5.stl; visual mesh filename=package://lbr_description/meshes/iiwa14/visual/link_5.stl
- link link_6: geometry collision mesh filename=package://lbr_description/meshes/iiwa14/collisionink_6.stl; visual mesh filename=package://lbr_description/meshes/iiwa14/visual/link_6.stl
- link link_7: geometry collision mesh filename=package://lbr_description/meshes/iiwa14/collisionink_7.stl; visual mesh filename=package://lbr_description/meshes/iiwa14/visual/link_7.stl

File: lbr_description/urdf/iiwa7.urdf (robot description, URDF)
Before this commit: robot iiwa7, 9 links, 8 joints
Links:
- link base_link: geometry collision mesh filename=package://lbr_description/meshes/iiwa7/collision/base_link.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; visual mesh filename=package://lbr_description/meshes/iiwa7/visual/base_link.stl
- link link_1: geometry collision mesh filename=package://lbr_description/meshes/iiwa7/collision/link_1.stl; visual mesh filename=package://lbr_description/meshes/iiwa7/visual/link_1.stl
- link link_2: geometry collision mesh filename=package://lbr_description/meshes/iiwa7/collision/link_2.stl; visual mesh filename=package://lbr_description/meshes/iiwa7/visual/link_2.stl
- link link_3: geometry collision mesh filename=package://lbr_description/meshes/iiwa7/collision/link_3.stl; visual mesh filename=package://lbr_description/meshes/iiwa7/visual/link_3.stl
- link link_4: geometry collision mesh filename=package://lbr_description/meshes/iiwa7/collision/link_4.stl; visual mesh filename=package://lbr_description/meshes/iiwa7/visual/link_4.stl
- link link_5: geometry collision mesh filename=package://lbr_description/meshes/iiwa7/collision/link_5.stl; visual mesh filename=package://lbr_description/meshes/iiwa7/visual/link_5.stl
- link link_6: geometry collision mesh filename=package://lbr_description/meshes/iiwa7/collision/link_6.stl; visual mesh filename=package://lbr_description/meshes/iiwa7/visual/link_6.stl
- link link_7: geometry collision mesh filename=package://lbr_description/meshes/iiwa7/collision/link_7.stl; visual mesh filename=package://lbr_description/meshes/iiwa7/visual/link_7.stl

File: lbr_description/urdf/med14.urdf (robot description, URDF)
Before this commit: robot med14, 9 links, 8 joints
Links:
- link base_link: geometry collision mesh filename=package://lbr_description/meshes/med14/collision/base_link.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; visual mesh filename=package://lbr_description/meshes/med14/visual/base_link.stl
- link link_1: geometry collision mesh filename=package://lbr_description/meshes/med14/collision/link_1.stl; visual mesh filename=package://lbr_description/meshes/med14/visual/link_1.stl
- link link_2: geometry collision mesh filename=package://lbr_description/meshes/med14/collision/link_2.stl; visual mesh filename=package://lbr_description/meshes/med14/visual/link_2.stl
- link link_3: geometry collision mesh filename=package://lbr_description/meshes/med14/collision/link_3.stl; visual mesh filename=package://lbr_description/meshes/med14/visual/link_3.stl
- link link_4: geometry collision mesh filename=package://lbr_description/meshes/med14/collision/link_4.stl; visual mesh filename=package://lbr_description/meshes/med14/visual/link_4.stl
- link link_5: geometry collision mesh filename=package://lbr_description/meshes/med14/collision/link_5.stl; visual mesh filename=package://lbr_description/meshes/med14/visual/link_5.stl
- link link_6: geometry collision mesh filename=package://lbr_description/meshes/med14/collision/link_6.stl; visual mesh filename=package://lbr_description/meshes/med14/visual/link_6.stl
- link link_7: geometry collision mesh filename=package://lbr_description/meshes/med14/collision/link_7.stl; visual mesh filename=package://lbr_description/meshes/med14/visual/link_7.stl

File: lbr_description/urdf/med7.urdf (robot description, URDF)
Before this commit: robot med7, 9 links, 8 joints
Links:
- link base_link: geometry collision mesh filename=package://lbr_description/meshes/med7/collision/base_link.s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; visual mesh filename=package://lbr_description/meshes/med7/visual/base_link.stl
- link link_1: geometry collision mesh filename=package://lbr_description/meshes/med7/collisionink_1.stl; visual mesh filename=package://lbr_description/meshes/med7/visual/link_1.stl
- link link_2: geometry collision mesh filename=package://lbr_description/meshes/med7/collisionink_2.stl; visual mesh filename=package://lbr_description/meshes/med7/visual/link_2.stl
- link link_3: geometry collision mesh filename=package://lbr_description/meshes/med7/collisionink_3.stl; visual mesh filename=package://lbr_description/meshes/med7/visual/link_3.stl
- link link_4: geometry collision mesh filename=package://lbr_description/meshes/med7/collisionink_4.stl; visual mesh filename=package://lbr_description/meshes/med7/visual/link_4.stl
- link link_5: geometry collision mesh filename=package://lbr_description/meshes/med7/collisionink_5.stl; visual mesh filename=package://lbr_description/meshes/med7/visual/link_5.stl
- link link_6: geometry collision mesh filename=package://lbr_description/meshes/med7/collisionink_6.stl; visual mesh filename=package://lbr_description/meshes/med7/visual/link_6.stl
- link link_7: geometry collision mesh filename=package://lbr_description/meshes/med7/collisionink_7.stl; visual mesh filename=package://lbr_description/meshes/med7/visual/link_7.stl

Commit message: added joint state publisher

File: lbr_description/urdf/iiwa14.urdf (robot description, URDF)
Before this commit: robot iiwa14, 9 links, 8 joints
Links:
- link link_1: geometry collision mesh filename=package://lbr_description/meshes/iiwa14/collision/link_1.stl; visual mesh filename=package://lbr_description/meshes/iiwa14/visual/link_1.stl
- link link_2: geometry collision mesh filename=package://lbr_description/meshes/iiwa14/collision/link_2.stl; visual mesh filename=package://lbr_description/meshes/iiwa14/visual/link_2.stl
- link link_3: geometry collision mesh filename=package://lbr_description/meshes/iiwa14/collision/link_3.stl; visual mesh filename=package://lbr_description/meshes/iiwa14/visual/link_3.stl
- link link_4: geometry collision mesh filename=package://lbr_description/meshes/iiwa14/collision/link_4.stl; visual mesh filename=package://lbr_description/meshes/iiwa14/visual/link_4.stl
- link link_5: geometry collision mesh filename=package://lbr_description/meshes/iiwa14/collision/link_5.stl; visual mesh filename=package://lbr_description/meshes/iiwa14/visual/link_5.stl
- link link_6: geometry collision mesh filename=package://lbr_description/meshes/iiwa14/collision/link_6.stl; visual mesh filename=package://lbr_description/meshes/iiwa14/visual/link_6.stl
- link link_7: geometry collision mesh filename=package://lbr_description/meshes/iiwa14/collision/link_7.stl; visual mesh filename=package://lbr_description/meshes/iiwa14/visual/link_7.stl

File: lbr_description/urdf/med7.urdf (robot description, URDF)
Before this commit: robot med7, 9 links, 8 joints
Links:
- link link_1: geometry collision mesh filename=package://lbr_description/meshes/med7/collision/link_1.stl; visual mesh filename=package://lbr_description/meshes/med7/visual/link_1.stl
- link link_2: geometry collision mesh filename=package://lbr_description/meshes/med7/collision/link_2.stl; visual mesh filename=package://lbr_description/meshes/med7/visual/link_2.stl
- link link_3: geometry collision mesh filename=package://lbr_description/meshes/med7/collision/link_3.stl; visual mesh filename=package://lbr_description/meshes/med7/visual/link_3.stl
- link link_4: geometry collision mesh filename=package://lbr_description/meshes/med7/collision/link_4.stl; visual mesh filename=package://lbr_description/meshes/med7/visual/link_4.stl
- link link_5: geometry collision mesh filename=package://lbr_description/meshes/med7/collision/link_5.stl; visual mesh filename=package://lbr_description/meshes/med7/visual/link_5.stl
- link link_6: geometry collision mesh filename=package://lbr_description/meshes/med7/collision/link_6.stl; visual mesh filename=package://lbr_description/meshes/med7/visual/link_6.stl
- link link_7: geometry collision mesh filename=package://lbr_description/meshes/med7/collision/link_7.stl; visual mesh filename=package://lbr_description/meshes/med7/visual/link_7.stl
