Commit message: updated materials

File: lbr_description/urdf/iiwa14.urdf.xacro (robot description, xacro)
@@ -2,4 +2,6 @@
 <!-- top level -->
 <robot name="iiwa14" xmlns:xacro="http://www.ros.org/wiki/xacro">
+    <!-- include materials -->
+    <xacro:include filename="$(find lbr_description)/urdf/materials.xacro"/>
     <!-- include the lbr iiwa macro -->
     <xacro:include filename="$(find lbr_description)/urdf/iiwa14.xacro"/>

File: lbr_description/urdf/iiwa14.xacro (robot description, xacro)
@@ -32,7 +32,5 @@
                 <mesh filename="package://lbr_description/meshes/iiwa14/visual/link_0.stl"/>
             </geometry>
-            <material name="silver">
-                <color rgba="1 0 0 1"/>
-            </material>
+            <material name="silver"/>
             </visual>
             <collision>
@@ -68,7 +66,5 @@
                 <mesh filename="package://lbr_description/meshes/iiwa14/visual/link_1.stl"/>
             </geometry>
-            <material name="silver">
-                <color rgba="1 0 0 1"/>
-            </material>
+            <material name="orange"/>
             </visual>
             <collision>
@@ -104,7 +100,5 @@
                 <mesh filename="package://lbr_description/meshes/iiwa14/visual/link_2.stl"/>
             </geometry>
-            <material name="silver">
-                <color rgba="1 0 0 1"/>
-            </material>
+            <material name="orange"/>
             </visual>
             <collision>
@@ -140,7 +134,5 @@
                 <mesh filename="package://lbr_description/meshes/iiwa14/visual/link_3.stl"/>
             </geometry>
-            <material name="silver">
-                <color rgba="1 0 0 1"/>
-            </material>
+            <material name="orange"/>
             </visual>
             <collision>
@@ -176,7 +168,5 @@
                 <mesh filename="package://lbr_description/meshes/iiwa14/visual/link_4.stl"/>
             </geometry>
-            <material name="silver">
-                <color rgba="1 0 0 1"/>
-            </material>
+            <material name="orange"/>
             </visual>
             <collision>
@@ -212,7 +202,5 @@
                 <mesh filename="package://lbr_description/meshes/iiwa14/visual/link_5.stl"/>
             </geometry>
-            <material name="silver">
-                <color rgba="1 0 0 1"/>
-            </material>
+            <material name="orange"/>
             </visual>
             <collision>
@@ -248,7 +236,5 @@
                 <mesh filename="package://lbr_description/meshes/iiwa14/visual/link_6.stl"/>
             </geometry>
-            <material name="silver">
-                <color rgba="1 0 0 1"/>
-            </material>
+            <material name="orange"/>
             </visual>
             <collision>
@@ -284,7 +270,5 @@
                 <mesh filename="package://lbr_description/meshes/iiwa14/visual/link_7.stl"/>
             </geometry>
-            <material name="silver">
-                <color rgba="1 0 0 1"/>
-            </material>
+            <material name="silver"/>
             </visual>
             <collision>

File: lbr_description/urdf/iiwa7.urdf.xacro (robot description, xacro)
@@ -2,4 +2,6 @@
 <!-- top level -->
 <robot name="iiwa7" xmlns:xacro="http://www.ros.org/wiki/xacro">
+    <!-- include materials -->
+    <xacro:include filename="$(find lbr_description)/urdf/materials.xacro"/>
     <!-- include the lbr iiwa macro -->
     <xacro:include filename="$(find lbr_description)/urdf/iiwa7.xacro"/>

File: lbr_description/urdf/iiwa7.xacro (robot description, xacro)
@@ -32,7 +32,5 @@
                 <mesh filename="package://lbr_description/meshes/iiwa7/visual/link_0.stl"/>
             </geometry>
-            <material name="silver">
-                <color rgba="1 0 0 1"/>
-            </material>
+            <material name="silver"/>
             </visual>
             <collision>
@@ -68,7 +66,5 @@
                 <mesh filename="package://lbr_description/meshes/iiwa7/visual/link_1.stl"/>
             </geometry>
-            <material name="silver">
-                <color rgba="1 0 0 1"/>
-            </material>
+            <material name="orange"/>
             </visual>
             <collision>
@@ -104,7 +100,5 @@
                 <mesh filename="package://lbr_description/meshes/iiwa7/visual/link_2.stl"/>
             </geometry>
-            <material name="silver">
-                <color rgba="1 0 0 1"/>
-            </material>
+            <material name="orange"/>
             </visual>
             <collision>
@@ -140,7 +134,5 @@
                 <mesh filename="package://lbr_description/meshes/iiwa7/visual/link_3.stl"/>
             </geometry>
-            <material name="silver">
-                <color rgba="1 0 0 1"/>
-            </material>
+            <material name="orange"/>
             </visual>
             <collision>
@@ -176,7 +168,5 @@
                 <mesh filename="package://lbr_description/meshes/iiwa7/visual/link_4.stl"/>
             </geometry>
-            <material name="silver">
-                <color rgba="1 0 0 1"/>
-            </material>
+            <material name="orange"/>
             </visual>
             <collision>
@@ -212,7 +202,5 @@
                 <mesh filename="package://lbr_description/meshes/iiwa7/visual/link_5.stl"/>
             </geometry>
-            <material name="silver">
-                <color rgba="1 0 0 1"/>
-            </material>
+            <material name="orange"/>
             </visual>
             <collision>
@@ -248,7 +236,5 @@
                 <mesh filename="package://lbr_description/meshes/iiwa7/visual/link_6.stl"/>
             </geometry>
-            <material name="silver">
-                <color rgba="1 0 0 1"/>
-            </material>
+            <material name="orange"/>
             </visual>
             <collision>
@@ -284,7 +270,5 @@
                 <mesh filename="package://lbr_description/meshes/iiwa7/visual/link_7.stl"/>
             </geometry>
-            <material name="silver">
-                <color rgba="1 0 0 1"/>
-            </material>
+            <material name="silver"/>
             </visual>
             <collision>

File: lbr_description/urdf/med14.urdf.xacro (robot description, xacro)
@@ -2,4 +2,6 @@
 <!-- top level -->
 <robot name="med14" xmlns:xacro="http://www.ros.org/wiki/xacro">
+    <!-- include materials -->
+    <xacro:include filename="$(find lbr_description)/urdf/materials.xacro"/>
     <!-- include the lbr med macro -->
     <xacro:include filename="$(find lbr_description)/urdf/med14.xacro"/>

File: lbr_description/urdf/med14.xacro (robot description, xacro)
@@ -32,7 +32,5 @@
                 <mesh filename="package://lbr_description/meshes/med14/visual/link_0.stl"/>
             </geometry>
-            <material name="white">
-                <color rgba="1.0 1.0 1.0 1.0"/>
-            </material>
+            <material name="white"/>
             </visual>
             <collision>
@@ -68,7 +66,5 @@
                 <mesh filename="package://lbr_description/meshes/med14/visual/link_1.stl"/>
             </geometry>
-            <material name="white">
-                <color rgba="1.0 1.0 1.0 1.0"/>
-            </material>
+            <material name="white"/>
             </visual>
             <collision>
@@ -104,7 +100,5 @@
                 <mesh filename="package://lbr_description/meshes/med14/visual/link_2.stl"/>
             </geometry>
-            <material name="white">
-                <color rgba="1.0 1.0 1.0 1.0"/>
-            </material>
+            <material name="white"/>
             </visual>
             <collision>
@@ -140,7 +134,5 @@
                 <mesh filename="package://lbr_description/meshes/med14/visual/link_3.stl"/>
             </geometry>
-            <material name="white">
-                <color rgba="1.0 1.0 1.0 1.0"/>
-            </material>
+            <material name="white"/>
             </visual>
             <collision>
@@ -176,7 +168,5 @@
                 <mesh filename="package://lbr_description/meshes/med14/visual/link_4.stl"/>
             </geometry>
-            <material name="white">
-                <color rgba="1.0 1.0 1.0 1.0"/>
-            </material>
+            <material name="white"/>
             </visual>
             <collision>
@@ -212,7 +202,5 @@
                 <mesh filename="package://lbr_description/meshes/med14/visual/link_5.stl"/>
             </geometry>
-            <material name="white">
-                <color rgba="1.0 1.0 1.0 1.0"/>
-            </material>
+            <material name="white"/>
             </visual>
             <collision>
@@ -248,7 +236,5 @@
                 <mesh filename="package://lbr_description/meshes/med14/visual/link_6.stl"/>
             </geometry>
-            <material name="white">
-                <color rgba="1.0 1.0 1.0 1.0"/>
-            </material>
+            <material name="white"/>
             </visual>
             <collision>
@@ -284,7 +270,5 @@
                 <mesh filename="package://lbr_description/meshes/med14/visual/link_7.stl"/>
             </geometry>
-            <material name="silver">
-                <color rgba="0.7 0.7 0.7 1.0"/>
-            </material>
+            <material name="silver"/>
             </visual>
             <collision>

File: lbr_description/urdf/med7.urdf.xacro (robot description, xacro)
@@ -2,4 +2,6 @@
 <!-- top level -->
 <robot name="med7" xmlns:xacro="http://www.ros.org/wiki/xacro">
+    <!-- include materials -->
+    <xacro:include filename="$(find lbr_description)/urdf/materials.xacro"/>
     <!-- include the lbr med macro -->
     <xacro:include filename="$(find lbr_description)/urdf/med7.xacro"/>

File: lbr_description/urdf/med7.xacro (robot description, xacro)
@@ -32,7 +32,5 @@
                 <mesh filename="package://lbr_description/meshes/med7/visual/link_0.stl"/>
             </geometry>
-            <material name="white">
-                <color rgba="1.0 1.0 1.0 1.0"/>
-            </material>
+            <material name="white"/>
             </visual>
             <collision>
@@ -68,7 +66,5 @@
                 <mesh filename="package://lbr_description/meshes/med7/visual/link_1.stl"/>
             </geometry>
-            <material name="white">
-                <color rgba="1.0 1.0 1.0 1.0"/>
-            </material>
+            <material name="white"/>
             </visual>
             <collision>
@@ -104,7 +100,5 @@
                 <mesh filename="package://lbr_description/meshes/med7/visual/link_2.stl"/>
             </geometry>
-            <material name="white">
-                <color rgba="1.0 1.0 1.0 1.0"/>
-            </material>
+            <material name="white"/>
             </visual>
             <collision>
@@ -140,7 +134,5 @@
                 <mesh filename="package://lbr_description/meshes/med7/visual/link_3.stl"/>
             </geometry>
-            <material name="white">
-                <color rgba="1.0 1.0 1.0 1.0"/>
-            </material>
+            <material name="white"/>
             </visual>
             <collision>
@@ -176,7 +168,5 @@
                 <mesh filename="package://lbr_description/meshes/med7/visual/link_4.stl"/>
             </geometry>
-            <material name="white">
-                <color rgba="1.0 1.0 1.0 1.0"/>
-            </material>
+            <material name="white"/>
             </visual>
             <collision>
@@ -212,7 +202,5 @@
                 <mesh filename="package://lbr_description/meshes/med7/visual/link_5.stl"/>
             </geometry>
-            <material name="white">
-                <color rgba="1.0 1.0 1.0 1.0"/>
-            </material>
+            <material name="white"/>
             </visual>
             <collision>
@@ -248,7 +236,5 @@
                 <mesh filename="package://lbr_description/meshes/med7/visual/link_6.stl"/>
             </geometry>
-            <material name="white">
-                <color rgba="1.0 1.0 1.0 1.0"/>
-            </material>
+            <material name="white"/>
             </visual>
             <collision>
@@ -284,7 +270,5 @@
                 <mesh filename="package://lbr_description/meshes/med7/visual/link_7.stl"/>
             </geometry>
-            <material name="silver">
-                <color rgba="0.7 0.7 0.7 1.0"/>
-            </material>
+            <material name="silver"/>
             </visual>
             <collision>
