Commit message: added end effector to robots

File: lbr_description/urdf/iiwa14.xacro (robot description, xacro)
@@ -294,4 +294,11 @@
             </collision>
         </link>
+        <joint name="joint_ee" type="fixed">
+            <parent link="$link_7"/>
+            <child link="$link_ee"/>
+            <origin xyz="0 0 0.045" rpy="0 0 0"/>
+        </joint>
+        <link name="$link_ee">
+        </link>
         <!-- extensions -->
         <xacro:iiwa_gazebo robot_name="${robot_name}"/>

File: lbr_description/urdf/iiwa7.xacro (robot description, xacro)
@@ -294,4 +294,11 @@
             </collision>
         </link>
+        <joint name="joint_ee" type="fixed">
+            <parent link="$link_7"/>
+            <child link="$link_ee"/>
+            <origin xyz="0 0 0.045" rpy="0 0 0"/>
+        </joint>
+        <link name="$link_ee">
+        </link>
         <!-- extensions -->
         <xacro:iiwa_gazebo robot_name="${robot_name}"/>

File: lbr_description/urdf/med14.xacro (robot description, xacro)
@@ -294,4 +294,11 @@
             </collision>
         </link>
+        <joint name="joint_ee" type="fixed">
+            <parent link="$link_7"/>
+            <child link="$link_ee"/>
+            <origin xyz="0 0 0.045" rpy="0 0 0"/>
+        </joint>
+        <link name="$link_ee">
+        </link>
         <!-- extensions -->
         <xacro:med_gazebo robot_name="${robot_name}"/>

File: lbr_description/urdf/med7.xacro (robot description, xacro)
@@ -294,4 +294,11 @@
             </collision>
         </link>
+        <joint name="joint_ee" type="fixed">
+            <parent link="$link_7"/>
+            <child link="$link_ee"/>
+            <origin xyz="0 0 0.045" rpy="0 0 0"/>
+        </joint>
+        <link name="$link_ee">
+        </link>
         <!-- extensions -->
         <xacro:med_gazebo robot_name="${robot_name}"/>

Commit message: changed ee offset

File: lbr_description/urdf/iiwa14.xacro (robot description, xacro)
@@ -297,5 +297,5 @@
             <parent link="${robot_name}_link_7"/>
             <child link="${robot_name}_link_ee"/>
-            <origin xyz="0 0 0.045" rpy="0 0 0"/>
+            <origin xyz="0 0 0.035" rpy="0 0 0"/>
         </joint>
         <link name="${robot_name}_link_ee">

File: lbr_description/urdf/iiwa7.xacro (robot description, xacro)
@@ -297,5 +297,5 @@
             <parent link="${robot_name}_link_7"/>
             <child link="${robot_name}_link_ee"/>
-            <origin xyz="0 0 0.045" rpy="0 0 0"/>
+            <origin xyz="0 0 0.035" rpy="0 0 0"/>
         </joint>
         <link name="${robot_name}_link_ee">

File: lbr_description/urdf/med14.xacro (robot description, xacro)
@@ -297,5 +297,5 @@
             <parent link="${robot_name}_link_7"/>
             <child link="${robot_name}_link_ee"/>
-            <origin xyz="0 0 0.045" rpy="0 0 0"/>
+            <origin xyz="0 0 0.035" rpy="0 0 0"/>
         </joint>
         <link name="${robot_name}_link_ee">

File: lbr_description/urdf/med7.xacro (robot description, xacro)
@@ -297,5 +297,5 @@
             <parent link="${robot_name}_link_7"/>
             <child link="${robot_name}_link_ee"/>
-            <origin xyz="0 0 0.045" rpy="0 0 0"/>
+            <origin xyz="0 0 0.035" rpy="0 0 0"/>
         </joint>
         <link name="${robot_name}_link_ee">

Commit message: increased damping, added friction

File: lbr_description/urdf/iiwa14.xacro (robot description, xacro)
@@ -9,5 +9,6 @@
     <xacro:property name="safety_controller_k_pos" value="100"/>
     <xacro:property name="safety_controller_k_vel" value="2"/>
-    <xacro:property name="joint_damping" value="0.5"/>
+    <xacro:property name="joint_damping" value="10.0"/>
+    <xacro:property name="joint_friction" value="0.1"/>
     <xacro:property name="max_effort" value="300"/>
     <xacro:property name="max_velocity" value="10"/>
@@ -54,5 +55,5 @@
                 k_velocity="${safety_controller_k_vel}"
             />
-            <dynamics damping="${joint_damping}"/>
+            <dynamics damping="${joint_damping}" friction="${joint_friction}"/>
         </joint>
         <link name="${robot_name}_link_1">
@@ -90,5 +91,5 @@
                 k_velocity="${safety_controller_k_vel}"
             />
-            <dynamics damping="${joint_damping}"/>
+            <dynamics damping="${joint_damping}" friction="${joint_friction}"/>
         </joint>
         <link name="${robot_name}_link_2">
@@ -126,5 +127,5 @@
                 k_velocity="${safety_controller_k_vel}"
             />
-            <dynamics damping="${joint_damping}"/>
+            <dynamics damping="${joint_damping}" friction="${joint_friction}"/>
         </joint>
         <link name="${robot_name}_link_3">
@@ -162,5 +163,5 @@
                 k_velocity="${safety_controller_k_vel}"
             />
-            <dynamics damping="${joint_damping}"/>
+            <dynamics damping="${joint_damping}" friction="${joint_friction}"/>
         </joint>
         <link name="${robot_name}_link_4">
@@ -198,5 +199,5 @@
                 k_velocity="${safety_controller_k_vel}"
             />
-            <dynamics damping="${joint_damping}"/>
+            <dynamics damping="${joint_damping}" friction="${joint_friction}"/>
         </joint>
         <link name="${robot_name}_link_5">
@@ -234,5 +235,5 @@
                 k_velocity="${safety_controller_k_vel}"
             />
-            <dynamics damping="${joint_damping}"/>
+            <dynamics damping="${joint_damping}" friction="${joint_friction}"/>
         </joint>
         <link name="${robot_name}_link_6">
@@ -270,5 +271,5 @@
                 k_velocity="${safety_controller_k_vel}"
             />
-            <dynamics damping="${joint_damping}"/>
+            <dynamics damping="${joint_damping}" friction="${joint_friction}"/>
         </joint>
         <link name="${robot_name}_link_7">

File: lbr_description/urdf/iiwa7.xacro (robot description, xacro)
@@ -9,5 +9,6 @@
     <xacro:property name="safety_controller_k_pos" value="100"/>
     <xacro:property name="safety_controller_k_vel" value="2"/>
-    <xacro:property name="joint_damping" value="0.5"/>
+    <xacro:property name="joint_damping" value="10.0"/>
+    <xacro:property name="joint_friction" value="0.1"/>
     <xacro:property name="max_effort" value="300"/>
     <xacro:property name="max_velocity" value="10"/>
@@ -54,5 +55,5 @@
                 k_velocity="${safety_controller_k_vel}"
             />
-            <dynamics damping="${joint_damping}"/>
+            <dynamics damping="${joint_damping}" friction="${joint_friction}"/>
         </joint>
         <link name="${robot_name}_link_1">
@@ -90,5 +91,5 @@
                 k_velocity="${safety_controller_k_vel}"
             />
-            <dynamics damping="${joint_damping}"/>
+            <dynamics damping="${joint_damping}" friction="${joint_friction}"/>
         </joint>
         <link name="${robot_name}_link_2">
@@ -126,5 +127,5 @@
                 k_velocity="${safety_controller_k_vel}"
             />
-            <dynamics damping="${joint_damping}"/>
+            <dynamics damping="${joint_damping}" friction="${joint_friction}"/>
         </joint>
         <link name="${robot_name}_link_3">
@@ -162,5 +163,5 @@
                 k_velocity="${safety_controller_k_vel}"
             />
-            <dynamics damping="${joint_damping}"/>
+            <dynamics damping="${joint_damping}" friction="${joint_friction}"/>
         </joint>
         <link name="${robot_name}_link_4">
@@ -198,5 +199,5 @@
                 k_velocity="${safety_controller_k_vel}"
             />
-            <dynamics damping="${joint_damping}"/>
+            <dynamics damping="${joint_damping}" friction="${joint_friction}"/>
         </joint>
         <link name="${robot_name}_link_5">
@@ -234,5 +235,5 @@
                 k_velocity="${safety_controller_k_vel}"
             />
-            <dynamics damping="${joint_damping}"/>
+            <dynamics damping="${joint_damping}" friction="${joint_friction}"/>
         </joint>
         <link name="${robot_name}_link_6">
@@ -270,5 +271,5 @@
                 k_velocity="${safety_controller_k_vel}"
             />
-            <dynamics damping="${joint_damping}"/>
+            <dynamics damping="${joint_damping}" friction="${joint_friction}"/>
         </joint>
         <link name="${robot_name}_link_7">

File: lbr_description/urdf/med14.xacro (robot description, xacro)
@@ -9,5 +9,6 @@
     <xacro:property name="safety_controller_k_pos" value="100"/>
     <xacro:property name="safety_controller_k_vel" value="2"/>
-    <xacro:property name="joint_damping" value="0.5"/>
+    <xacro:property name="joint_damping" value="10.0"/>
+    <xacro:property name="joint_friction" value="0.1"/>
     <xacro:property name="max_effort" value="300"/>
     <xacro:property name="max_velocity" value="10"/>
@@ -54,5 +55,5 @@
                 k_velocity="${safety_controller_k_vel}"
             />
-            <dynamics damping="${joint_damping}"/>
+            <dynamics damping="${joint_damping}" friction="${joint_friction}"/>
         </joint>
         <link name="${robot_name}_link_1">
@@ -90,5 +91,5 @@
                 k_velocity="${safety_controller_k_vel}"
             />
-            <dynamics damping="${joint_damping}"/>
+            <dynamics damping="${joint_damping}" friction="${joint_friction}"/>
         </joint>
         <link name="${robot_name}_link_2">
@@ -126,5 +127,5 @@
                 k_velocity="${safety_controller_k_vel}"
             />
-            <dynamics damping="${joint_damping}"/>
+            <dynamics damping="${joint_damping}" friction="${joint_friction}"/>
         </joint>
         <link name="${robot_name}_link_3">
@@ -162,5 +163,5 @@
                 k_velocity="${safety_controller_k_vel}"
             />
-            <dynamics damping="${joint_damping}"/>
+            <dynamics damping="${joint_damping}" friction="${joint_friction}"/>
         </joint>
         <link name="${robot_name}_link_4">
@@ -198,5 +199,5 @@
                 k_velocity="${safety_controller_k_vel}"
             />
-            <dynamics damping="${joint_damping}"/>
+            <dynamics damping="${joint_damping}" friction="${joint_friction}"/>
         </joint>
         <link name="${robot_name}_link_5">
@@ -234,5 +235,5 @@
                 k_velocity="${safety_controller_k_vel}"
             />
-            <dynamics damping="${joint_damping}"/>
+            <dynamics damping="${joint_damping}" friction="${joint_friction}"/>
         </joint>
         <link name="${robot_name}_link_6">
@@ -270,5 +271,5 @@
                 k_velocity="${safety_controller_k_vel}"
             />
-            <dynamics damping="${joint_damping}"/>
+            <dynamics damping="${joint_damping}" friction="${joint_friction}"/>
         </joint>
         <link name="${robot_name}_link_7">

File: lbr_description/urdf/med7.xacro (robot description, xacro)
@@ -9,5 +9,6 @@
     <xacro:property name="safety_controller_k_pos" value="100"/>
     <xacro:property name="safety_controller_k_vel" value="2"/>
-    <xacro:property name="joint_damping" value="0.5"/>
+    <xacro:property name="joint_damping" value="10.0"/>
+    <xacro:property name="joint_friction" value="0.1"/>
     <xacro:property name="max_effort" value="300"/>
     <xacro:property name="max_velocity" value="10"/>
@@ -18,5 +19,5 @@
             <xacro:insert_block name="origin"/>
             <parent link="${parent}"/>
-            <child link="${robot_name}_link_0"/>
+            <child link="${robot_name}_link_0"/>=
         </joint>
         <link name="${robot_name}_link_0">
@@ -54,5 +55,5 @@
                 k_velocity="${safety_controller_k_vel}"
             />
-            <dynamics damping="${joint_damping}"/>
+            <dynamics damping="${joint_damping}" friction="${joint_friction}"/>
         </joint>
         <link name="${robot_name}_link_1">
@@ -90,5 +91,5 @@
                 k_velocity="${safety_controller_k_vel}"
             />
-            <dynamics damping="${joint_damping}"/>
+            <dynamics damping="${joint_damping}" friction="${joint_friction}"/>
         </joint>
         <link name="${robot_name}_link_2">
@@ -126,5 +127,5 @@
                 k_velocity="${safety_controller_k_vel}"
             />
-            <dynamics damping="${joint_damping}"/>
+            <dynamics damping="${joint_damping}" friction="${joint_friction}"/>
         </joint>
         <link name="${robot_name}_link_3">
@@ -162,5 +163,5 @@
                 k_velocity="${safety_controller_k_vel}"
             />
-            <dynamics damping="${joint_damping}"/>
+            <dynamics damping="${joint_damping}" friction="${joint_friction}"/>
         </joint>
         <link name="${robot_name}_link_4">
@@ -198,5 +199,5 @@
                 k_velocity="${safety_controller_k_vel}"
             />
-            <dynamics damping="${joint_damping}"/>
+            <dynamics damping="${joint_damping}" friction="${joint_friction}"/>
         </joint>
         <link name="${robot_name}_link_5">
@@ -234,5 +235,5 @@
                 k_velocity="${safety_controller_k_vel}"
             />
-            <dynamics damping="${joint_damping}"/>
+            <dynamics damping="${joint_damping}" friction="${joint_friction}"/>
         </joint>
         <link name="${robot_name}_link_6">
@@ -270,5 +271,5 @@
                 k_velocity="${safety_controller_k_vel}"
             />
-            <dynamics damping="${joint_damping}"/>
+            <dynamics damping="${joint_damping}" friction="${joint_friction}"/>
         </joint>
         <link name="${robot_name}_link_7">
