Commit message: fixed masses

File: lbr_description/urdf/iiwa14.xacro (robot description, xacro)
@@ -26,6 +26,6 @@
             <inertial>
             <origin rpy="0 0 0" xyz="-0.0128215344957798 -7.86364415362405e-08 0.07150661827888387"/>
-            <mass value="42.98914417363736"/>
-            <inertia ixx="0.190401" ixy="0.0" ixz="0.005312" iyy="0.242047" iyz="0.0" izz="0.262814"/>
+            <mass value="7.039242"/>
+            <inertia ixx="0.031177" ixy="0.000000" ixz="0.000870" iyy="0.039634" iyz="0.000000" izz="0.043034"/>
             </inertial>
             <visual>
@@ -60,6 +60,6 @@
             <inertial>
             <origin rpy="0 0 0" xyz="9.307232415315581e-08 -0.03379543155079102 0.13240370669453902"/>
-            <mass value="32.252499792432545"/>
-            <inertia ixx="0.258906" ixy="-0.0" ixz="-0.0" iyy="0.261201" iyz="0.038666" izz="0.096765"/>
+            <mass value="5.281174"/>
+            <inertia ixx="0.042394" ixy="-0.000000" ixz="-0.000000" iyy="0.042770" iyz="0.006331" izz="0.015845"/>
             </inertial>
             <visual>
@@ -94,6 +94,6 @@
             <inertial>
             <origin rpy="0 0 0" xyz="0.00015188022518878674 0.051987109728758904 0.05880129877994178"/>
-            <mass value="31.020446759849573"/>
-            <inertia ixx="0.240168" ixy="-0.000179" ixz="0.000259" iyy="0.238795" iyz="0.038362" izz="0.086485"/>
+            <mass value="5.079432"/>
+            <inertia ixx="0.039326" ixy="-0.000029" ixz="0.000042" iyy="0.039101" iyz="0.006282" izz="0.014161"/>
             </inertial>
             <visual>
@@ -128,6 +128,6 @@
             <inertial>
             <origin rpy="0 0 0" xyz="-5.974614313346012e-09 0.029563618732667742 0.13650341869763982"/>
-            <mass value="24.923667076480577"/>
-            <inertia ixx="0.196866" ixy="-0.0" ixz="0.0" iyy="0.186889" iyz="-0.038259" izz="0.059722"/>
+            <mass value="4.0811177"/>
+            <inertia ixx="0.032236" ixy="-0.000000" ixz="0.000000" iyy="0.030602" iyz="-0.006265" izz="0.009779"/>
             </inertial>
             <visual>
@@ -162,6 +162,6 @@
             <inertial>
             <origin rpy="0 0 0" xyz="-2.09625967727708e-08 -0.04476439079596513 0.06741903952954653"/>
-            <mass value="21.50439908415142"/>
-            <inertia ixx="0.135049" ixy="-0.0" ixz="-0.0" iyy="0.128699" iyz="-0.022352" izz="0.048185"/>
+            <mass value="3.521230"/>
+            <inertia ixx="0.022114" ixy="-0.000000" ixz="-0.000000" iyy="0.021074" iyz="-0.003660" izz="0.007890"/>
             </inertial>
             <visual>
@@ -196,6 +196,6 @@
             <inertial>
             <origin rpy="0 0 0" xyz="-0.00012008657208039079 -0.021390023245727908 0.0854754261653966"/>
-            <mass value="13.29457566606638"/>
-            <inertia ixx="0.079116" ixy="1.2e-05" ixz="-6e-06" iyy="0.06831" iyz="0.024259" izz="0.035078"/>
+            <mass value="2.176916"/>
+            <inertia ixx="0.012955" ixy="0.000002" ixz="-0.000001" iyy="0.011185" iyz="0.003972" izz="0.005744"/>
             </inertial>
             <visual>
@@ -230,6 +230,6 @@
             <inertial>
             <origin rpy="0 0 0" xyz="-6.000032555678588e-08 0.07103825551434698 0.000565530522845803"/>
-            <mass value="14.198362583652283"/>
-            <inertia ixx="0.038424" ixy="-0.0" ixz="-0.0" iyy="0.036784" iyz="0.001919" izz="0.027998"/>
+            <mass value="2.324906"/>
+            <inertia ixx="0.006292" ixy="-0.000000" ixz="-0.000000" iyy="0.006023" iyz="0.000314" izz="0.004585"/>
             </inertial>
             <visual>
@@ -264,6 +264,6 @@
             <inertial>
             <origin rpy="0 0 0" xyz="3.963019849314055e-06 -1.5392768444664745e-08 0.027186686478491096"/>
-            <mass value="2.4182992945540933"/>
-            <inertia ixx="0.001719" ixy="-0.0" ixz="-0.0" iyy="0.001692" iyz="0.0" izz="0.002627"/>
+            <mass value="0.395984"/>
+            <inertia ixx="0.000281" ixy="-0.000000" ixz="-0.000000" iyy="0.000277" iyz="0.000000" izz="0.000430"/>
             </inertial>
             <visual>

File: lbr_description/urdf/iiwa7.xacro (robot description, xacro)
@@ -26,6 +26,6 @@
             <inertial>
             <origin rpy="0 0 0" xyz="-0.01283618494463161 4.904567390585061e-08 0.07010682239932087"/>
-            <mass value="30.324767682917948"/>
-            <inertia ixx="0.111667" ixy="0.0" ixz="0.004812" iyy="0.139457" iyz="-0.0" izz="0.133156"/>
+            <mass value="4.861279"/>
+            <inertia ixx="0.017901" ixy="0.000000" ixz="0.000771" iyy="0.022356" iyz="-0.000000" izz="0.021346"/>
             </inertial>
             <visual>
@@ -60,6 +60,6 @@
             <inertial>
             <origin rpy="0 0 0" xyz="4.9980243666546455e-08 -0.0347335291089292 0.12351608478142942"/>
-            <mass value="21.213926420791886"/>
-            <inertia ixx="0.134131" ixy="-0.0" ixz="0.0" iyy="0.127957" iyz="0.023881" izz="0.047328"/>
+            <mass value="3.400745"/>
+            <inertia ixx="0.021502" ixy="-0.000000" ixz="0.000000" iyy="0.020512" iyz="0.003828" izz="0.007587"/>
             </inertial>
             <visual>
@@ -94,6 +94,6 @@
             <inertial>
             <origin rpy="0 0 0" xyz="4.0558428502019873e-08 0.04491581578298656 0.06732515284873997"/>
-            <mass value="21.39756651772542"/>
-            <inertia ixx="0.133839" ixy="-0.0" ixz="0.0" iyy="0.12753" iyz="0.022271" izz="0.047853"/>
+            <mass value="3.430184"/>
+            <inertia ixx="0.021455" ixy="-0.000000" ixz="0.000000" iyy="0.020444" iyz="0.003570" izz="0.007671"/>
             </inertial>
             <visual>
@@ -128,6 +128,6 @@
             <inertial>
             <origin rpy="0 0 0" xyz="-5.881068064938613e-09 0.02956361869175564 0.1365034185434154"/>
-            <mass value="24.923667110884463"/>
-            <inertia ixx="0.196866" ixy="-0.0" ixz="0.0" iyy="0.186889" iyz="-0.038259" izz="0.059722"/>
+            <mass value="3.995443"/>
+            <inertia ixx="0.031559" ixy="-0.000000" ixz="0.000000" iyy="0.029960" iyz="-0.006133" izz="0.009574"/>
             </inertial>
             <visual>
@@ -162,6 +162,6 @@
             <inertial>
             <origin rpy="0 0 0" xyz="-4.1344813497116265e-08 -0.044916218629510306 0.06732501840381"/>
-            <mass value="21.39755453189086"/>
-            <inertia ixx="0.13383" ixy="0.0" ixz="-0.0" iyy="0.127527" iyz="-0.022269" izz="0.047848"/>
+            <mass value="3.430182"/>
+            <inertia ixx="0.021454" ixy="0.000000" ixz="-0.000000" iyy="0.020443" iyz="-0.003570" izz="0.007670"/>
             </inertial>
             <visual>
@@ -196,6 +196,6 @@
             <inertial>
             <origin rpy="0 0 0" xyz="2.416002990197734e-08 -0.021386601078580914 0.085468591256322"/>
-            <mass value="13.296700832855965"/>
-            <inertia ixx="0.079123" ixy="-0.0" ixz="-0.0" iyy="0.068318" iyz="0.024261" izz="0.035085"/>
+            <mass value="2.131557"/>
+            <inertia ixx="0.012684" ixy="-0.000000" ixz="-0.000000" iyy="0.010952" iyz="0.003889" izz="0.005624"/>
             </inertial>
             <visual>
@@ -230,6 +230,6 @@
             <inertial>
             <origin rpy="0 0 0" xyz="-9.07120004240837e-08 0.0709871260349443 0.002115721730276743"/>
-            <mass value="14.421451173118493"/>
-            <inertia ixx="0.040001" ixy="-0.0" ixz="-0.0" iyy="0.038461" iyz="0.00196" izz="0.027816"/>
+            <mass value="2.311862"/>
+            <inertia ixx="0.006412" ixy="-0.000000" ixz="-0.000000" iyy="0.006166" iyz="0.000314" izz="0.004459"/>
             </inertial>
             <visual>
@@ -264,6 +264,6 @@
             <inertial>
             <origin rpy="0 0 0" xyz="4.535378460217862e-06 -1.7615872956281168e-08 0.009883270430701696"/>
-            <mass value="2.113113203151399"/>
-            <inertia ixx="0.001557" ixy="-0.0" ixz="-0.0" iyy="0.00153" iyz="0.0" izz="0.002532"/>
+            <mass value="0.338747"/>
+            <inertia ixx="0.000250" ixy="-0.000000" ixz="-0.000000" iyy="0.000245" iyz="0.000000" izz="0.000406"/>
             </inertial>
             <visual>

File: lbr_description/urdf/med14.xacro (robot description, xacro)
@@ -26,6 +26,6 @@
             <inertial>
             <origin rpy="0 0 0" xyz="-0.0018642104260720833 -9.120393625716289e-09 0.07751683665104403"/>
-            <mass value="46.99016031984989"/>
-            <inertia ixx="0.257284" ixy="-0.0" ixz="-0.004545" iyy="0.262253" iyz="0.0" izz="0.357074"/>
+            <mass value="8.146350"/>
+            <inertia ixx="0.044603" ixy="-0.000000" ixz="-0.000788" iyy="0.045465" iyz="0.000000" izz="0.061903"/>
             </inertial>
             <visual>
@@ -60,6 +60,6 @@
             <inertial>
             <origin rpy="0 0 0" xyz="9.307232415315581e-08 -0.033795431550791004 0.13240370669453896"/>
-            <mass value="32.252499792432545"/>
-            <inertia ixx="0.258906" ixy="-0.0" ixz="-0.0" iyy="0.261201" iyz="0.038666" izz="0.096765"/>
+            <mass value="5.591386"/>
+            <inertia ixx="0.044885" ixy="-0.000000" ixz="-0.000000" iyy="0.045283" iyz="0.006703" izz="0.016775"/>
             </inertial>
             <visual>
@@ -94,6 +94,6 @@
             <inertial>
             <origin rpy="0 0 0" xyz="0.0001358226533474577 0.0475476440926152 0.07632205850106144"/>
-            <mass value="34.68757984100769"/>
-            <inertia ixx="0.336472" ixy="-0.0002" ixz="0.000342" iyy="0.329156" iyz="0.06118" izz="0.100748"/>
+            <mass value="6.013539"/>
+            <inertia ixx="0.058332" ixy="-0.000035" ixz="0.000059" iyy="0.057063" iyz="0.010606" izz="0.017466"/>
             </inertial>
             <visual>
@@ -128,6 +128,6 @@
             <inertial>
             <origin rpy="0 0 0" xyz="5.689213978259012e-08 0.03491265072974692 0.12310820658934007"/>
-            <mass value="21.104680740321076"/>
-            <inertia ixx="0.132439" ixy="-0.0" ixz="0.0" iyy="0.126397" iyz="-0.023446" izz="0.046954"/>
+            <mass value="3.658768"/>
+            <inertia ixx="0.022960" ixy="-0.000000" ixz="0.000000" iyy="0.021913" iyz="-0.004065" izz="0.008140"/>
             </inertial>
             <visual>
@@ -162,6 +162,6 @@
             <inertial>
             <origin rpy="0 0 0" xyz="-3.025185496951432e-08 -0.03979329512420171 0.08694364647762443"/>
-            <mass value="25.13964883334753"/>
-            <inertia ixx="0.197617" ixy="-0.0" ixz="-0.0" iyy="0.187546" iyz="-0.036716" izz="0.060263"/>
+            <mass value="4.358282"/>
+            <inertia ixx="0.034259" ixy="-0.000000" ixz="-0.000000" iyy="0.032514" iyz="-0.006365" izz="0.010447"/>
             </inertial>
             <visual>
@@ -196,6 +196,6 @@
             <inertial>
             <origin rpy="0 0 0" xyz="3.8871741664391765e-08 -0.029824284088761824 0.07626701716135809"/>
-            <mass value="9.534880920206561"/>
-            <inertia ixx="0.052905" ixy="0.0" ixz="-0.0" iyy="0.044495" iyz="0.017493" izz="0.023991"/>
+            <mass value="1.652994"/>
+            <inertia ixx="0.009172" ixy="0.000000" ixz="-0.000000" iyy="0.007714" iyz="0.003033" izz="0.004159"/>
             </inertial>
             <visual>
@@ -230,6 +230,6 @@
             <inertial>
             <origin rpy="0 0 0" xyz="-7.073221484902805e-07 0.07101990943401978 0.004952526180380223"/>
-            <mass value="14.987109331085524"/>
-            <inertia ixx="0.044068" ixy="-0.0" ixz="1e-06" iyy="0.042427" iyz="0.001941" izz="0.028865"/>
+            <mass value="2.598208"/>
+            <inertia ixx="0.007640" ixy="-0.000000" ixz="0.000000" iyy="0.007355" iyz="0.000336" izz="0.005004"/>
             </inertial>
             <visual>
@@ -264,6 +264,6 @@
             <inertial>
             <origin rpy="0 0 0" xyz="3.121827460016089e-06 -1.635815563460264e-06 0.0137822955218736"/>
-            <mass value="1.617833997596271"/>
-            <inertia ixx="0.001066" ixy="0.0" ixz="-0.0" iyy="0.001066" iyz="0.0" izz="0.001864"/>
+            <mass value="0.280472"/>
+            <inertia ixx="0.000185" ixy="0.000000" ixz="-0.000000" iyy="0.000185" iyz="0.000000" izz="0.000323"/>
             </inertial>
             <visual>

File: lbr_description/urdf/med7.xacro (robot description, xacro)
@@ -21,11 +21,11 @@
             <xacro:insert_block name="origin"/>
             <parent link="${parent}"/>
-            <child link="${robot_name}_link_0"/>=
+            <child link="${robot_name}_link_0"/>
         </joint>
         <link name="${robot_name}_link_0">
             <inertial>
             <origin rpy="0 0 0" xyz="-0.0018958727522859222 -8.736009549202623e-09 0.07626305487275586"/>
-            <mass value="46.20540698229506"/>
-            <inertia ixx="0.250291" ixy="-0.0" ixz="-0.004435" iyy="0.255257" iyz="-0.0" izz="0.351803"/>
+            <mass value="7.143078"/>
+            <inertia ixx="0.038693" ixy="-0.000000" ixz="-0.000686" iyy="0.039461" iyz="-0.000000" izz="0.054387"/>
             </inertial>
             <visual>
@@ -60,6 +60,6 @@
             <inertial>
             <origin rpy="0 0 0" xyz="5.010328793588479e-08 -0.03481903813472808 0.12329857163085542"/>
-            <mass value="21.161828997118327"/>
-            <inertia ixx="0.133324" ixy="-0.0" ixz="0.0" iyy="0.127214" iyz="0.023673" izz="0.047155"/>
+            <mass value="3.271492"/>
+            <inertia ixx="0.020611" ixy="-0.000000" ixz="0.000000" iyy="0.019667" iyz="0.003660" izz="0.007290"/>
             </inertial>
             <visual>
@@ -94,6 +94,6 @@
             <inertial>
             <origin rpy="0 0 0" xyz="2.958275959973659e-08 0.03979295468456965 0.08694361150855662"/>
-            <mass value="25.13966081800886"/>
-            <inertia ixx="0.19763" ixy="-0.0" ixz="0.0" iyy="0.187553" iyz="0.036718" izz="0.060269"/>
+            <mass value="3.886440"/>
+            <inertia ixx="0.030552" ixy="-0.000000" ixz="0.000000" iyy="0.028995" iyz="0.005676" izz="0.009317"/>
             </inertial>
             <visual>
@@ -128,6 +128,6 @@
             <inertial>
             <origin rpy="0 0 0" xyz="-5.010330962930412e-08 0.03481903813473644 0.1232985716309013"/>
-            <mass value="21.1618289971097"/>
-            <inertia ixx="0.133324" ixy="-0.0" ixz="-0.0" iyy="0.127214" iyz="-0.023673" izz="0.047155"/>
+            <mass value="3.271492"/>
+            <inertia ixx="0.020611" ixy="-0.000000" ixz="-0.000000" iyy="0.019667" iyz="-0.003660" izz="0.007290"/>
             </inertial>
             <visual>
@@ -162,6 +162,6 @@
             <inertial>
             <origin rpy="0 0 0" xyz="-3.025230048709993e-08 -0.03979329512443697 0.08694363375610437"/>
-            <mass value="25.139648831600116"/>
-            <inertia ixx="0.197618" ixy="-0.0" ixz="-0.0" iyy="0.187546" iyz="-0.036716" izz="0.060263"/>
+            <mass value="3.886439"/>
+            <inertia ixx="0.030551" ixy="-0.000000" ixz="-0.000000" iyy="0.028993" iyz="-0.005676" izz="0.009316"/>
             </inertial>
             <visual>
@@ -196,6 +196,6 @@
             <inertial>
             <origin rpy="0 0 0" xyz="3.887174133882675e-08 -0.02982428408876193 0.07626701716135398"/>
-            <mass value="9.534880920206515"/>
-            <inertia ixx="0.052905" ixy="0.0" ixz="-0.0" iyy="0.044495" iyz="0.017493" izz="0.023991"/>
+            <mass value="1.474035"/>
+            <inertia ixx="0.008179" ixy="0.000000" ixz="-0.000000" iyy="0.006879" iyz="0.002704" izz="0.003709"/>
             </inertial>
             <visual>
@@ -230,6 +230,6 @@
             <inertial>
             <origin rpy="0 0 0" xyz="-7.073221144775636e-07 0.07101990943401648 0.004952526180360017"/>
-            <mass value="14.987109331100873"/>
-            <inertia ixx="0.044068" ixy="-0.0" ixz="1e-06" iyy="0.042427" iyz="0.001941" izz="0.028865"/>
+            <mass value="2.316917"/>
+            <inertia ixx="0.006813" ixy="-0.000000" ixz="0.000000" iyy="0.006559" iyz="0.000300" izz="0.004462"/>
             </inertial>
             <visual>
@@ -264,6 +264,6 @@
             <inertial>
             <origin rpy="0 0 0" xyz="3.1218274599808524e-06 -1.6358155634513969e-06 0.013782295521067356"/>
-            <mass value="1.6178339975962697"/>
-            <inertia ixx="0.001066" ixy="0.0" ixz="-0.0" iyy="0.001066" iyz="0.0" izz="0.001864"/>
+            <mass value="0.250107"/>
+            <inertia ixx="0.000165" ixy="0.000000" ixz="-0.000000" iyy="0.000165" iyz="0.000000" izz="0.000288"/>
             </inertial>
             <visual>

Commit message: ee fix #125

File: lbr_description/urdf/iiwa14.xacro (robot description, xacro)
@@ -284,5 +284,5 @@
             <parent link="${robot_name}_link_7"/>
             <child link="${robot_name}_link_ee"/>
-            <origin xyz="0 0 0.035" rpy="0 0 0"/>
+            <origin xyz="0 0 0.045" rpy="0 0 0"/>
         </joint>
         <link name="${robot_name}_link_ee">

File: lbr_description/urdf/med14.xacro (robot description, xacro)
@@ -284,5 +284,5 @@
             <parent link="${robot_name}_link_7"/>
             <child link="${robot_name}_link_ee"/>
-            <origin xyz="0 0 0.035" rpy="0 0 0"/>
+            <origin xyz="0 0 0.045" rpy="0 0 0"/>
         </joint>
         <link name="${robot_name}_link_ee">

Commit message: revert tf

File: lbr_description/urdf/iiwa14.xacro (robot description, xacro)
@@ -284,5 +284,5 @@
             <parent link="${robot_name}_link_7"/>
             <child link="${robot_name}_link_ee"/>
-            <origin xyz="0 0 0.045" rpy="0 0 0"/>
+            <origin xyz="0 0 0.035" rpy="0 0 0"/>
         </joint>
         <link name="${robot_name}_link_ee">

File: lbr_description/urdf/med14.xacro (robot description, xacro)
@@ -284,5 +284,5 @@
             <parent link="${robot_name}_link_7"/>
             <child link="${robot_name}_link_ee"/>
-            <origin xyz="0 0 0.045" rpy="0 0 0"/>
+            <origin xyz="0 0 0.035" rpy="0 0 0"/>
         </joint>
         <link name="${robot_name}_link_ee">
