Commit message: removed robot name from joints

File: lbr_description/urdf/med14.xacro (robot description, xacro)
@@ -18,7 +18,7 @@
             <xacro:insert_block name="origin"/>
             <parent link="${parent}"/>
-            <child link="${robot_name}_link_0"/>
-        </joint>
-        <link name="${robot_name}_link_0">
+            <child link="link_0"/>
+        </joint>
+        <link name="link_0">
             <inertial>
             <origin rpy="0 0 0" xyz="-0.0018642104260720833 -9.120393625716289e-09 0.07751683665104403"/>
@@ -42,8 +42,8 @@
             </collision>
         </link>
-        <joint name="${robot_name}_joint_1" type="revolute">
+        <joint name="joint_1" type="revolute">
             <origin rpy="0 0 0" xyz="0.0 0.0 0.147"/>
-            <parent link="${robot_name}_link_0"/>
-            <child link="${robot_name}_link_1"/>
+            <parent link="link_0"/>
+            <child link="link_1"/>
             <axis xyz="0.0 0.0 0.01"/>
             <limit effort="${max_effort}" lower="${-170 * PI / 180}" upper="${170 * PI / 180}" velocity="${max_velocity}"/>
@@ -56,5 +56,5 @@
             <dynamics damping="${joint_damping}"/>
         </joint>
-        <link name="${robot_name}_link_1">
+        <link name="link_1">
             <inertial>
             <origin rpy="0 0 0" xyz="9.307232415315581e-08 -0.033795431550791004 0.13240370669453896"/>
@@ -78,8 +78,8 @@
             </collision>
         </link>
-        <joint name="${robot_name}_joint_2" type="revolute">
+        <joint name="joint_2" type="revolute">
             <origin rpy="0 0 0" xyz="0.0 -0.01 0.2125"/>
-            <parent link="${robot_name}_link_1"/>
-            <child link="${robot_name}_link_2"/>
+            <parent link="link_1"/>
+            <child link="link_2"/>
             <axis xyz="0.0 0.01 0.0"/>
             <limit effort="${max_effort}" lower="${-120 * PI / 180}" upper="${120 * PI / 180}" velocity="${max_velocity}"/>
@@ -92,5 +92,5 @@
             <dynamics damping="${joint_damping}"/>
         </joint>
-        <link name="${robot_name}_link_2">
+        <link name="link_2">
             <inertial>
             <origin rpy="0 0 0" xyz="0.0001358226533474577 0.0475476440926152 0.07632205850106144"/>
@@ -114,8 +114,8 @@
             </collision>
         </link>
-        <joint name="${robot_name}_joint_3" type="revolute">
+        <joint name="joint_3" type="revolute">
             <origin rpy="0 0 0" xyz="-0.0 0.01 0.228"/>
-            <parent link="${robot_name}_link_2"/>
-            <child link="${robot_name}_link_3"/>
+            <parent link="link_2"/>
+            <child link="link_3"/>
             <axis xyz="0.0 0.0 0.01"/>
             <limit effort="${max_effort}" lower="${-170 * PI / 180}" upper="${170 * PI / 180}" velocity="${max_velocity}"/>
@@ -128,5 +128,5 @@
             <dynamics damping="${joint_damping}"/>
         </joint>
-        <link name="${robot_name}_link_3">
+        <link name="link_3">
             <inertial>
             <origin rpy="0 0 0" xyz="5.689213978259012e-08 0.03491265072974692 0.12310820658934007"/>
@@ -150,8 +150,8 @@
             </collision>
         </link>
-        <joint name="${robot_name}_joint_4" type="revolute">
+        <joint name="joint_4" type="revolute">
             <origin rpy="0 0 0" xyz="0.0 0.0105 0.192"/>
-            <parent link="${robot_name}_link_3"/>
-            <child link="${robot_name}_link_4"/>
+            <parent link="link_3"/>
+            <child link="link_4"/>
             <axis xyz="0.0 -0.01 0.0"/>
             <limit effort="${max_effort}" lower="${-120 * PI / 180}" upper="${120 * PI / 180}" velocity="${max_velocity}"/>
@@ -164,5 +164,5 @@
             <dynamics damping="${joint_damping}"/>
         </joint>
-        <link name="${robot_name}_link_4">
+        <link name="link_4">
             <inertial>
             <origin rpy="0 0 0" xyz="-3.025185496951432e-08 -0.03979329512420171 0.08694364647762443"/>
@@ -186,8 +186,8 @@
             </collision>
         </link>
-        <joint name="${robot_name}_joint_5" type="revolute">
+        <joint name="joint_5" type="revolute">
             <origin rpy="0 0 0" xyz="0.0 -0.0105 0.2075"/>
-            <parent link="${robot_name}_link_4"/>
-            <child link="${robot_name}_link_5"/>
+            <parent link="link_4"/>
+            <child link="link_5"/>
             <axis xyz="0.0 0.0 0.01"/>
             <limit effort="${max_effort}" lower="${-170 * PI / 180}" upper="${170 * PI / 180}" velocity="${max_velocity}"/>
@@ -200,5 +200,5 @@
             <dynamics damping="${joint_damping}"/>
         </joint>
-        <link name="${robot_name}_link_5">
+        <link name="link_5">
             <inertial>
             <origin rpy="0 0 0" xyz="3.8871741664391765e-08 -0.029824284088761824 0.07626701716135809"/>
@@ -222,8 +222,8 @@
             </collision>
         </link>
-        <joint name="${robot_name}_joint_6" type="revolute">
+        <joint name="joint_6" type="revolute">
             <origin rpy="0 0 0" xyz="0.0 -0.0707 0.1925"/>
-            <parent link="${robot_name}_link_5"/>
-            <child link="${robot_name}_link_6"/>
+            <parent link="link_5"/>
+            <child link="link_6"/>
             <axis xyz="0.0 0.01 0.0"/>
             <limit effort="${max_effort}" lower="${-120 * PI / 180}" upper="${120 * PI / 180}" velocity="${max_velocity}"/>
@@ -236,5 +236,5 @@
             <dynamics damping="${joint_damping}"/>
         </joint>
-        <link name="${robot_name}_link_6">
+        <link name="link_6">
             <inertial>
             <origin rpy="0 0 0" xyz="-7.073221484902805e-07 0.07101990943401978 0.004952526180380223"/>
@@ -258,8 +258,8 @@
             </collision>
         </link>
-        <joint name="${robot_name}_joint_7" type="revolute">
+        <joint name="joint_7" type="revolute">
             <origin rpy="0 0 0" xyz="0.0 0.0707 0.091"/>
-            <parent link="${robot_name}_link_6"/>
-            <child link="${robot_name}_link_7"/>
+            <parent link="link_6"/>
+            <child link="link_7"/>
             <axis xyz="0.0 0.0 0.01"/>
             <limit effort="${max_effort}" lower="${-175 * PI / 180}" upper="${175 * PI / 180}" velocity="${max_velocity}"/>
@@ -272,5 +272,5 @@
             <dynamics damping="${joint_damping}"/>
         </joint>
-        <link name="${robot_name}_link_7">
+        <link name="link_7">
             <inertial>
             <origin rpy="0 0 0" xyz="3.121827460016089e-06 -1.635815563460264e-06 0.0137822955218736"/>
@@ -295,5 +295,5 @@
         </link>
         <!-- extensions -->
-        <xacro:med_gazebo robot_name="${robot_name}"/>
+        <xacro:med_gazebo/>
         <xacro:lbr_transmission hardware_interface="${hardware_interface}" robot_name="${robot_name}"/>
     </xacro:macro>

File: lbr_description/urdf/med7.xacro (robot description, xacro)
@@ -18,7 +18,7 @@
             <xacro:insert_block name="origin"/>
             <parent link="${parent}"/>
-            <child link="${robot_name}_link_0"/>
-        </joint>
-        <link name="${robot_name}_link_0">
+            <child link="link_0"/>
+        </joint>
+        <link name="link_0">
             <inertial>
             <origin rpy="0 0 0" xyz="-0.0018958727522859222 -8.736009549202623e-09 0.07626305487275586"/>
@@ -42,8 +42,8 @@
             </collision>
         </link>
-        <joint name="${robot_name}_joint_1" type="revolute">
+        <joint name="joint_1" type="revolute">
             <origin rpy="0 0 0" xyz="0.0 0.0 0.1475"/>
-            <parent link="${robot_name}_link_0"/>
-            <child link="${robot_name}_link_1"/>
+            <parent link="link_0"/>
+            <child link="link_1"/>
             <axis xyz="0.0 0.0 0.01"/>
             <limit effort="${max_effort}" lower="${-170 * PI / 180}" upper="${170 * PI / 180}" velocity="${max_velocity}"/>
@@ -56,5 +56,5 @@
             <dynamics damping="${joint_damping}"/>
         </joint>
-        <link name="${robot_name}_link_1">
+        <link name="link_1">
             <inertial>
             <origin rpy="0 0 0" xyz="5.010328793588479e-08 -0.03481903813472808 0.12329857163085542"/>
@@ -78,8 +78,8 @@
             </collision>
         </link>
-        <joint name="${robot_name}_joint_2" type="revolute">
+        <joint name="joint_2" type="revolute">
             <origin rpy="0 0 0" xyz="-0.0 -0.0105 0.1925"/>
-            <parent link="${robot_name}_link_1"/>
-            <child link="${robot_name}_link_2"/>
+            <parent link="link_1"/>
+            <child link="link_2"/>
             <axis xyz="0.0 0.01 0.0"/>
             <limit effort="${max_effort}" lower="${-120 * PI / 180}" upper="${120 * PI / 180}" velocity="${max_velocity}"/>
@@ -92,5 +92,5 @@
             <dynamics damping="${joint_damping}"/>
         </joint>
-        <link name="${robot_name}_link_2">
+        <link name="link_2">
             <inertial>
             <origin rpy="0 0 0" xyz="2.958275959973659e-08 0.03979295468456965 0.08694361150855662"/>
@@ -114,8 +114,8 @@
             </collision>
         </link>
-        <joint name="${robot_name}_joint_3" type="revolute">
+        <joint name="joint_3" type="revolute">
             <origin rpy="0 0 0" xyz="0.0 0.0105 0.2075"/>
-            <parent link="${robot_name}_link_2"/>
-            <child link="${robot_name}_link_3"/>
+            <parent link="link_2"/>
+            <child link="link_3"/>
             <axis xyz="0.0 0.0 0.01"/>
             <limit effort="${max_effort}" lower="${-170 * PI / 180}" upper="${170 * PI / 180}" velocity="${max_velocity}"/>
@@ -128,5 +128,5 @@
             <dynamics damping="${joint_damping}"/>
         </joint>
-        <link name="${robot_name}_link_3">
+        <link name="link_3">
             <inertial>
             <origin rpy="0 0 0" xyz="-5.010330962930412e-08 0.03481903813473644 0.1232985716309013"/>
@@ -150,8 +150,8 @@
             </collision>
         </link>
-        <joint name="${robot_name}_joint_4" type="revolute">
+        <joint name="joint_4" type="revolute">
             <origin rpy="0 0 0" xyz="0.0 0.0105 0.1925"/>
-            <parent link="${robot_name}_link_3"/>
-            <child link="${robot_name}_link_4"/>
+            <parent link="link_3"/>
+            <child link="link_4"/>
             <axis xyz="0.0 -0.01 0.0"/>
             <limit effort="${max_effort}" lower="${-120 * PI / 180}" upper="${120 * PI / 180}" velocity="${max_velocity}"/>
@@ -164,5 +164,5 @@
             <dynamics damping="${joint_damping}"/>
         </joint>
-        <link name="${robot_name}_link_4">
+        <link name="link_4">
             <inertial>
             <origin rpy="0 0 0" xyz="-3.025230048709993e-08 -0.03979329512443697 0.08694363375610437"/>
@@ -186,8 +186,8 @@
             </collision>
         </link>
-        <joint name="${robot_name}_joint_5" type="revolute">
+        <joint name="joint_5" type="revolute">
             <origin rpy="0 0 0" xyz="-0.0 -0.0105 0.2075"/>
-            <parent link="${robot_name}_link_4"/>
-            <child link="${robot_name}_link_5"/>
+            <parent link="link_4"/>
+            <child link="link_5"/>
             <axis xyz="0.0 0.0 0.01"/>
             <limit effort="${max_effort}" lower="${-170 * PI / 180}" upper="${170 * PI / 180}" velocity="${max_velocity}"/>
@@ -200,5 +200,5 @@
             <dynamics damping="${joint_damping}"/>
         </joint>
-        <link name="${robot_name}_link_5">
+        <link name="link_5">
             <inertial>
             <origin rpy="0 0 0" xyz="3.887174133882675e-08 -0.02982428408876193 0.07626701716135398"/>
@@ -222,8 +222,8 @@
             </collision>
         </link>
-        <joint name="${robot_name}_joint_6" type="revolute">
+        <joint name="joint_6" type="revolute">
             <origin rpy="0 0 0" xyz="0.0 -0.0707 0.1925"/>
-            <parent link="${robot_name}_link_5"/>
-            <child link="${robot_name}_link_6"/>
+            <parent link="link_5"/>
+            <child link="link_6"/>
             <axis xyz="0.0 0.01 0.0"/>
             <limit effort="${max_effort}" lower="${-120 * PI / 180}" upper="${120 * PI / 180}" velocity="${max_velocity}"/>
@@ -236,5 +236,5 @@
             <dynamics damping="${joint_damping}"/>
         </joint>
-        <link name="${robot_name}_link_6">
+        <link name="link_6">
             <inertial>
             <origin rpy="0 0 0" xyz="-7.073221144775636e-07 0.07101990943401648 0.004952526180360017"/>
@@ -258,8 +258,8 @@
             </collision>
         </link>
-        <joint name="${robot_name}_joint_7" type="revolute">
+        <joint name="joint_7" type="revolute">
             <origin rpy="0 0 0" xyz="0.0 0.0707 0.091"/>
-            <parent link="${robot_name}_link_6"/>
-            <child link="${robot_name}_link_7"/>
+            <parent link="link_6"/>
+            <child link="link_7"/>
             <axis xyz="0.0 0.0 0.01"/>
             <limit effort="${max_effort}" lower="${-175 * PI / 180}" upper="${175 * PI / 180}" velocity="${max_velocity}"/>
@@ -272,5 +272,5 @@
             <dynamics damping="${joint_damping}"/>
         </joint>
-        <link name="${robot_name}_link_7">
+        <link name="link_7">
             <inertial>
             <origin rpy="0 0 0" xyz="3.1218274599808524e-06 -1.6358155634513969e-06 0.013782295521067356"/>
@@ -295,5 +295,5 @@
         </link>
         <!-- extensions -->
-        <xacro:med_gazebo robot_name="${robot_name}"/>
+        <xacro:med_gazebo/>
         <xacro:lbr_transmission hardware_interface="${hardware_interface}" robot_name="${robot_name}"/>
     </xacro:macro>

Commit message: added robot_name paramter

File: lbr_description/urdf/iiwa.gazebo.xacro (robot description, xacro)
@@ -1,5 +1,5 @@
 <?xml version="1.0"?>
 <robot xmlns:xacro="http://www.ros.org/wiki/xacro">
-    <xacro:macro name="iiwa_gazebo">
+    <xacro:macro name="iiwa_gazebo" params="robot_name">
         <!-- ros_control-plugin -->
         <gazebo>

File: lbr_description/urdf/iiwa14.xacro (robot description, xacro)
@@ -295,5 +295,5 @@
         </link>
         <!-- extensions -->
-        <xacro:iiwa_gazebo/>
+        <xacro:iiwa_gazebo robot_name="${robot_name}"/>
         <xacro:lbr_transmission hardware_interface="${hardware_interface}" robot_name="${robot_name}"/>
     </xacro:macro>

File: lbr_description/urdf/iiwa7.xacro (robot description, xacro)
@@ -295,5 +295,5 @@
         </link>
         <!-- extensions -->
-        <xacro:iiwa_gazebo/>
+        <xacro:iiwa_gazebo robot_name="${robot_name}"/>
         <xacro:lbr_transmission hardware_interface="${hardware_interface}" robot_name="${robot_name}"/>
     </xacro:macro>

File: lbr_description/urdf/med.gazebo.xacro (robot description, xacro)
@@ -1,5 +1,5 @@
 <?xml version="1.0"?>
 <robot xmlns:xacro="http://www.ros.org/wiki/xacro">
-    <xacro:macro name="med_gazebo">
+    <xacro:macro name="med_gazebo" params="robot_name">
         <!-- ros_control-plugin -->
         <gazebo>

File: lbr_description/urdf/med14.xacro (robot description, xacro)
@@ -295,5 +295,5 @@
         </link>
         <!-- extensions -->
-        <xacro:med_gazebo/>
+        <xacro:med_gazebo robot_name="${robot_name}"/>
         <xacro:lbr_transmission hardware_interface="${hardware_interface}" robot_name="${robot_name}"/>
     </xacro:macro>

File: lbr_description/urdf/med7.xacro (robot description, xacro)
@@ -295,5 +295,5 @@
         </link>
         <!-- extensions -->
-        <xacro:med_gazebo/>
+        <xacro:med_gazebo robot_name="${robot_name}"/>
         <xacro:lbr_transmission hardware_interface="${hardware_interface}" robot_name="${robot_name}"/>
     </xacro:macro>
