Commit message: added robot name prefix for multi robots

File: lbr_description/urdf/iiwa.gazebo.xacro (robot description, xacro)
@@ -9,5 +9,5 @@
         </gazebo>
         <!-- link 0 -->
-        <gazebo reference="link_0">
+        <gazebo reference="${robot_name}_link_0">
             <mu1>0.2</mu1>
             <mu2>0.2</mu2>
@@ -15,5 +15,5 @@
         </gazebo>
         <!-- link 1 -->
-        <gazebo reference="link_1">
+        <gazebo reference="${robot_name}_link_1">
             <mu1>0.2</mu1>
             <mu2>0.2</mu2>
@@ -21,5 +21,5 @@
         </gazebo>
         <!-- link 2 -->
-        <gazebo reference="link_2">
+        <gazebo reference="${robot_name}_link_2">
             <mu1>0.2</mu1>
             <mu2>0.2</mu2>
@@ -27,5 +27,5 @@
         </gazebo>
         <!-- link 3 -->
-        <gazebo reference="link_3">
+        <gazebo reference="${robot_name}_link_3">
             <mu1>0.2</mu1>
             <mu2>0.2</mu2>
@@ -33,5 +33,5 @@
         </gazebo>
         <!-- link 4 -->
-        <gazebo reference="link_4">
+        <gazebo reference="${robot_name}_link_4">
             <mu1>0.2</mu1>
             <mu2>0.2</mu2>
@@ -39,5 +39,5 @@
         </gazebo>
         <!-- link 5 -->
-        <gazebo reference="link_5">
+        <gazebo reference="${robot_name}_link_5">
             <mu1>0.2</mu1>
             <mu2>0.2</mu2>
@@ -45,5 +45,5 @@
         </gazebo>
         <!-- link 6 -->
-        <gazebo reference="link_6">
+        <gazebo reference="${robot_name}_link_6">
             <mu1>0.2</mu1>
             <mu2>0.2</mu2>
@@ -51,5 +51,5 @@
         </gazebo>
         <!-- link 7 -->
-        <gazebo reference="link_7">
+        <gazebo reference="${robot_name}_link_7">
             <mu1>0.2</mu1>
             <mu2>0.2</mu2>

File: lbr_description/urdf/iiwa14.xacro (robot description, xacro)
@@ -18,7 +18,7 @@
             <xacro:insert_block name="origin"/>
             <parent link="${parent}"/>
-            <child link="link_0"/>
-        </joint>
-        <link name="link_0">
+            <child link="${robot_name}_link_0"/>
+        </joint>
+        <link name="${robot_name}_link_0">
             <inertial>
             <origin rpy="0 0 0" xyz="-0.0128215344957798 -7.86364415362405e-08 0.07150661827888387"/>
@@ -42,8 +42,8 @@
             </collision>
         </link>
-        <joint name="joint_1" type="revolute">
+        <joint name="${robot_name}_joint_1" type="revolute">
             <origin rpy="0 0 0" xyz="0.0 0.0 0.1475"/>
-            <parent link="link_0"/>
-            <child link="link_1"/>
+            <parent link="${robot_name}_link_0"/>
+            <child link="${robot_name}_link_1"/>
             <axis xyz="0.0 0.0 0.01"/>
             <limit effort="${max_effort}" lower="${-170 * PI / 180}" upper="${170 * PI / 180}" velocity="${max_velocity}"/>
@@ -56,5 +56,5 @@
             <dynamics damping="${joint_damping}"/>
         </joint>
-        <link name="link_1">
+        <link name="${robot_name}_link_1">
             <inertial>
             <origin rpy="0 0 0" xyz="9.307232415315581e-08 -0.03379543155079102 0.13240370669453902"/>
@@ -78,8 +78,8 @@
             </collision>
         </link>
-        <joint name="joint_2" type="revolute">
+        <joint name="${robot_name}_joint_2" type="revolute">
             <origin rpy="0 0 0" xyz="0.0 -0.01 0.2125"/>
-            <parent link="link_1"/>
-            <child link="link_2"/>
+            <parent link="${robot_name}_link_1"/>
+            <child link="${robot_name}_link_2"/>
             <axis xyz="0.0 0.01 0.0"/>
             <limit effort="${max_effort}" lower="${-120 * PI / 180}" upper="${120 * PI / 180}" velocity="${max_velocity}"/>
@@ -92,5 +92,5 @@
             <dynamics damping="${joint_damping}"/>
         </joint>
-        <link name="link_2">
+        <link name="${robot_name}_link_2">
             <inertial>
             <origin rpy="0 0 0" xyz="0.00015188022518878674 0.051987109728758904 0.05880129877994178"/>
@@ -114,8 +114,8 @@
             </collision>
         </link>
-        <joint name="joint_3" type="revolute">
+        <joint name="${robot_name}_joint_3" type="revolute">
             <origin rpy="0 0 0" xyz="0.0 0.01 0.1945"/>
-            <parent link="link_2"/>
-            <child link="link_3"/>
+            <parent link="${robot_name}_link_2"/>
+            <child link="${robot_name}_link_3"/>
             <axis xyz="0.0 0.0 0.01"/>
             <limit effort="${max_effort}" lower="${-170 * PI / 180}" upper="${170 * PI / 180}" velocity="${max_velocity}"/>
@@ -128,5 +128,5 @@
             <dynamics damping="${joint_damping}"/>
         </joint>
-        <link name="link_3">
+        <link name="${robot_name}_link_3">
             <inertial>
             <origin rpy="0 0 0" xyz="-5.974614313346012e-09 0.029563618732667742 0.13650341869763982"/>
@@ -150,8 +150,8 @@
             </collision>
         </link>
-        <joint name="joint_4" type="revolute">
+        <joint name="${robot_name}_joint_4" type="revolute">
             <origin rpy="0 0 0" xyz="-0.0 0.0105 0.2255"/>
-            <parent link="link_3"/>
-            <child link="link_4"/>
+            <parent link="${robot_name}_link_3"/>
+            <child link="${robot_name}_link_4"/>
             <axis xyz="0.0 -0.01 0.0"/>
             <limit effort="${max_effort}" lower="${-120 * PI / 180}" upper="${120 * PI / 180}" velocity="${max_velocity}"/>
@@ -164,5 +164,5 @@
             <dynamics damping="${joint_damping}"/>
         </joint>
-        <link name="link_4">
+        <link name="${robot_name}_link_4">
             <inertial>
             <origin rpy="0 0 0" xyz="-2.09625967727708e-08 -0.04476439079596513 0.06741903952954653"/>
@@ -186,8 +186,8 @@
             </collision>
         </link>
-        <joint name="joint_5" type="revolute">
+        <joint name="${robot_name}_joint_5" type="revolute">
             <origin rpy="0 0 0" xyz="0.0 -0.0105 0.1745"/>
-            <parent link="link_4"/>
-            <child link="link_5"/>
+            <parent link="${robot_name}_link_4"/>
+            <child link="${robot_name}_link_5"/>
             <axis xyz="0.0 0.0 0.01"/>
             <limit effort="${max_effort}" lower="${-170 * PI / 180}" upper="${170 * PI / 180}" velocity="${max_velocity}"/>
@@ -200,5 +200,5 @@
             <dynamics damping="${joint_damping}"/>
         </joint>
-        <link name="link_5">
+        <link name="${robot_name}_link_5">
             <inertial>
             <origin rpy="0 0 0" xyz="-0.00012008657208039079 -0.021390023245727908 0.0854754261653966"/>
@@ -222,8 +222,8 @@
             </collision>
         </link>
-        <joint name="joint_6" type="revolute">
+        <joint name="${robot_name}_joint_6" type="revolute">
             <origin rpy="0 0 0" xyz="-0.0 -0.0707 0.2255"/>
-            <parent link="link_5"/>
-            <child link="link_6"/>
+            <parent link="${robot_name}_link_5"/>
+            <child link="${robot_name}_link_6"/>
             <axis xyz="0.0 0.01 0.0"/>
             <limit effort="${max_effort}" lower="${-120 * PI / 180}" upper="${120 * PI / 180}" velocity="${max_velocity}"/>
@@ -236,5 +236,5 @@
             <dynamics damping="${joint_damping}"/>
         </joint>
-        <link name="link_6">
+        <link name="${robot_name}_link_6">
             <inertial>
             <origin rpy="0 0 0" xyz="-6.000032555678588e-08 0.07103825551434698 0.000565530522845803"/>
@@ -258,8 +258,8 @@
             </collision>
         </link>
-        <joint name="joint_7" type="revolute">
+        <joint name="${robot_name}_joint_7" type="revolute">
             <origin rpy="0 0 0" xyz="0.0 0.0707 0.0711"/>
-            <parent link="link_6"/>
-            <child link="link_7"/>
+            <parent link="${robot_name}_link_6"/>
+            <child link="${robot_name}_link_7"/>
             <axis xyz="0.0 0.0 0.01"/>
             <limit effort="${max_effort}" lower="${-175 * PI / 180}" upper="${175 * PI / 180}" velocity="${max_velocity}"/>
@@ -272,5 +272,5 @@
             <dynamics damping="${joint_damping}"/>
         </joint>
-        <link name="link_7">
+        <link name="${robot_name}_link_7">
             <inertial>
             <origin rpy="0 0 0" xyz="3.963019849314055e-06 -1.5392768444664745e-08 0.027186686478491096"/>
@@ -294,10 +294,10 @@
             </collision>
         </link>
-        <joint name="joint_ee" type="fixed">
-            <parent link="$link_7"/>
-            <child link="$link_ee"/>
+        <joint name="${robot_name}_joint_ee" type="fixed">
+            <parent link="${robot_name}_link_7"/>
+            <child link="${robot_name}_link_ee"/>
             <origin xyz="0 0 0.045" rpy="0 0 0"/>
         </joint>
-        <link name="$link_ee">
+        <link name="${robot_name}_link_ee">
         </link>
         <!-- extensions -->

File: lbr_description/urdf/iiwa7.xacro (robot description, xacro)
@@ -18,7 +18,7 @@
             <xacro:insert_block name="origin"/>
             <parent link="${parent}"/>
-            <child link="link_0"/>
-        </joint>
-        <link name="link_0">
+            <child link="${robot_name}_link_0"/>
+        </joint>
+        <link name="${robot_name}_link_0">
             <inertial>
             <origin rpy="0 0 0" xyz="-0.01283618494463161 4.904567390585061e-08 0.07010682239932087"/>
@@ -42,8 +42,8 @@
             </collision>
         </link>
-        <joint name="joint_1" type="revolute">
+        <joint name="${robot_name}_joint_1" type="revolute">
             <origin rpy="0 0 0" xyz="0.0 0.0 0.1475"/>
-            <parent link="link_0"/>
-            <child link="link_1"/>
+            <parent link="${robot_name}_link_0"/>
+            <child link="${robot_name}_link_1"/>
             <axis xyz="0.0 0.0 0.01"/>
             <limit effort="${max_effort}" lower="${-170 * PI / 180}" upper="${170 * PI / 180}" velocity="${max_velocity}"/>
@@ -56,5 +56,5 @@
             <dynamics damping="${joint_damping}"/>
         </joint>
-        <link name="link_1">
+        <link name="${robot_name}_link_1">
             <inertial>
             <origin rpy="0 0 0" xyz="4.9980243666546455e-08 -0.0347335291089292 0.12351608478142942"/>
@@ -78,8 +78,8 @@
             </collision>
         </link>
-        <joint name="joint_2" type="revolute">
+        <joint name="${robot_name}_joint_2" type="revolute">
             <origin rpy="0 0 0" xyz="-0.0 -0.0105 0.193"/>
-            <parent link="link_1"/>
-            <child link="link_2"/>
+            <parent link="${robot_name}_link_1"/>
+            <child link="${robot_name}_link_2"/>
             <axis xyz="0.0 0.01 0.0"/>
             <limit effort="${max_effort}" lower="${-120 * PI / 180}" upper="${120 * PI / 180}" velocity="${max_velocity}"/>
@@ -92,5 +92,5 @@
             <dynamics damping="${joint_damping}"/>
         </joint>
-        <link name="link_2">
+        <link name="${robot_name}_link_2">
             <inertial>
             <origin rpy="0 0 0" xyz="4.0558428502019873e-08 0.04491581578298656 0.06732515284873997"/>
@@ -114,8 +114,8 @@
             </collision>
         </link>
-        <joint name="joint_3" type="revolute">
+        <joint name="${robot_name}_joint_3" type="revolute">
             <origin rpy="0 0 0" xyz="0.0 0.0105 0.1745"/>
-            <parent link="link_2"/>
-            <child link="link_3"/>
+            <parent link="${robot_name}_link_2"/>
+            <child link="${robot_name}_link_3"/>
             <axis xyz="0.0 0.0 0.01"/>
             <limit effort="${max_effort}" lower="${-170 * PI / 180}" upper="${170 * PI / 180}" velocity="${max_velocity}"/>
@@ -128,5 +128,5 @@
             <dynamics damping="${joint_damping}"/>
         </joint>
-        <link name="link_3">
+        <link name="${robot_name}_link_3">
             <inertial>
             <origin rpy="0 0 0" xyz="-5.881068064938613e-09 0.02956361869175564 0.1365034185434154"/>
@@ -150,8 +150,8 @@
             </collision>
         </link>
-        <joint name="joint_4" type="revolute">
+        <joint name="${robot_name}_joint_4" type="revolute">
             <origin rpy="0 0 0" xyz="0.0 0.0105 0.2255"/>
-            <parent link="link_3"/>
-            <child link="link_4"/>
+            <parent link="${robot_name}_link_3"/>
+            <child link="${robot_name}_link_4"/>
             <axis xyz="0.0 -0.01 0.0"/>
             <limit effort="${max_effort}" lower="${-120 * PI / 180}" upper="${120 * PI / 180}" velocity="${max_velocity}"/>
@@ -164,5 +164,5 @@
             <dynamics damping="${joint_damping}"/>
         </joint>
-        <link name="link_4">
+        <link name="${robot_name}_link_4">
             <inertial>
             <origin rpy="0 0 0" xyz="-4.1344813497116265e-08 -0.044916218629510306 0.06732501840381"/>
@@ -186,8 +186,8 @@
             </collision>
         </link>
-        <joint name="joint_5" type="revolute">
+        <joint name="${robot_name}_joint_5" type="revolute">
             <origin rpy="0 0 0" xyz="0.0 -0.0105 0.1745"/>
-            <parent link="link_4"/>
-            <child link="link_5"/>
+            <parent link="${robot_name}_link_4"/>
+            <child link="${robot_name}_link_5"/>
             <axis xyz="0.0 0.0 0.01"/>
             <limit effort="${max_effort}" lower="${-170 * PI / 180}" upper="${170 * PI / 180}" velocity="${max_velocity}"/>
@@ -200,5 +200,5 @@
             <dynamics damping="${joint_damping}"/>
         </joint>
-        <link name="link_5">
+        <link name="${robot_name}_link_5">
             <inertial>
             <origin rpy="0 0 0" xyz="2.416002990197734e-08 -0.021386601078580914 0.085468591256322"/>
@@ -222,8 +222,8 @@
             </collision>
         </link>
-        <joint name="joint_6" type="revolute">
+        <joint name="${robot_name}_joint_6" type="revolute">
             <origin rpy="0 0 0" xyz="0.0 -0.0707 0.2255"/>
-            <parent link="link_5"/>
-            <child link="link_6"/>
+            <parent link="${robot_name}_link_5"/>
+            <child link="${robot_name}_link_6"/>
             <axis xyz="0.0 0.01 0.0"/>
             <limit effort="${max_effort}" lower="${-120 * PI / 180}" upper="${120 * PI / 180}" velocity="${max_velocity}"/>
@@ -236,5 +236,5 @@
             <dynamics damping="${joint_damping}"/>
         </joint>
-        <link name="link_6">
+        <link name="${robot_name}_link_6">
             <inertial>
             <origin rpy="0 0 0" xyz="-9.07120004240837e-08 0.0709871260349443 0.002115721730276743"/>
@@ -258,8 +258,8 @@
             </collision>
         </link>
-        <joint name="joint_7" type="revolute">
+        <joint name="${robot_name}_joint_7" type="revolute">
             <origin rpy="0 0 0" xyz="0.0 0.0705 0.0909"/>
-            <parent link="link_6"/>
-            <child link="link_7"/>
+            <parent link="${robot_name}_link_6"/>
+            <child link="${robot_name}_link_7"/>
             <axis xyz="0.0 0.0 0.01"/>
             <limit effort="${max_effort}" lower="${-175 * PI / 180}" upper="${175 * PI / 180}" velocity="${max_velocity}"/>
@@ -272,5 +272,5 @@
             <dynamics damping="${joint_damping}"/>
         </joint>
-        <link name="link_7">
+        <link name="${robot_name}_link_7">
             <inertial>
             <origin rpy="0 0 0" xyz="4.535378460217862e-06 -1.7615872956281168e-08 0.009883270430701696"/>
@@ -294,10 +294,10 @@
             </collision>
         </link>
-        <joint name="joint_ee" type="fixed">
-            <parent link="$link_7"/>
-            <child link="$link_ee"/>
+        <joint name="${robot_name}_joint_ee" type="fixed">
+            <parent link="${robot_name}_link_7"/>
+            <child link="${robot_name}_link_ee"/>
             <origin xyz="0 0 0.045" rpy="0 0 0"/>
         </joint>
-        <link name="$link_ee">
+        <link name="${robot_name}_link_ee">
         </link>
         <!-- extensions -->

File: lbr_description/urdf/lbr.transmission.xacro (robot description, xacro)
@@ -3,11 +3,11 @@
     <xacro:macro name="lbr_transmission" params="hardware_interface robot_name">
     <!-- joint 1 -->
-    <transmission name="tran_1">
+    <transmission name="${robot_name}_tran_1">
         <robotNamespace>/${robot_name}</robotNamespace>
         <type>transmission_interface/SimpleTransmission</type>
-        <joint name="joint_1">
+        <joint name="${robot_name}_joint_1">
             <hardwareInterface>hardware_interface/${hardware_interface}</hardwareInterface>
         </joint>
-        <actuator name="motor_1">
+        <actuator name="${robot_name}_motor_1">
             <hardwareInterface>hardware_interface/${hardware_interface}</hardwareInterface>
             <mechanicalReduction>1</mechanicalReduction>
@@ -15,11 +15,11 @@
     </transmission>
     <!-- joint 2 -->
-    <transmission name="tran_2">
+    <transmission name="${robot_name}_tran_2">
         <robotNamespace>/${robot_name}</robotNamespace>
         <type>transmission_interface/SimpleTransmission</type>
-        <joint name="joint_2">
+        <joint name="${robot_name}_joint_2">
             <hardwareInterface>hardware_interface/${hardware_interface}</hardwareInterface>
         </joint>
-        <actuator name="motor_2">
+        <actuator name="${robot_name}_motor_2">
             <hardwareInterface>hardware_interface/${hardware_interface}</hardwareInterface>
             <mechanicalReduction>1</mechanicalReduction>
@@ -27,11 +27,11 @@
     </transmission>
     <!-- joint 3 -->
-    <transmission name="tran_3">
+    <transmission name="${robot_name}_tran_3">
         <robotNamespace>/${robot_name}</robotNamespace>
         <type>transmission_interface/SimpleTransmission</type>
-        <joint name="joint_3">
+        <joint name="${robot_name}_joint_3">
             <hardwareInterface>hardware_interface/${hardware_interface}</hardwareInterface>
         </joint>
-        <actuator name="motor_3">
+        <actuator name="${robot_name}_motor_3">
             <hardwareInterface>hardware_interface/${hardware_interface}</hardwareInterface>
             <mechanicalReduction>1</mechanicalReduction>
@@ -39,11 +39,11 @@
     </transmission>
     <!-- joint 4 -->
-    <transmission name="tran_4">
+    <transmission name="${robot_name}_tran_4">
         <robotNamespace>/${robot_name}</robotNamespace>
         <type>transmission_interface/SimpleTransmission</type>
-        <joint name="joint_4">
+        <joint name="${robot_name}_joint_4">
             <hardwareInterface>hardware_interface/${hardware_interface}</hardwareInterface>
         </joint>
-        <actuator name="motor_4">
+        <actuator name="${robot_name}_motor_4">
             <hardwareInterface>hardware_interface/${hardware_interface}</hardwareInterface>
             <mechanicalReduction>1</mechanicalReduction>
@@ -51,11 +51,11 @@
     </transmission>
     <!-- joint 5 -->
-    <transmission name="tran_5">
+    <transmission name="${robot_name}_tran_5">
         <robotNamespace>/${robot_name}</robotNamespace>
         <type>transmission_interface/SimpleTransmission</type>
-        <joint name="joint_5">
+        <joint name="${robot_name}_joint_5">
             <hardwareInterface>hardware_interface/${hardware_interface}</hardwareInterface>
         </joint>
-        <actuator name="motor_5">
+        <actuator name="${robot_name}_motor_5">
             <hardwareInterface>hardware_interface/${hardware_interface}</hardwareInterface>
             <mechanicalReduction>1</mechanicalReduction>
@@ -63,11 +63,11 @@
     </transmission>
     <!-- joint 6 -->
-    <transmission name="tran_6">
+    <transmission name="${robot_name}_tran_6">
         <robotNamespace>/${robot_name}</robotNamespace>
         <type>transmission_interface/SimpleTransmission</type>
-        <joint name="joint_6">
+        <joint name="${robot_name}_joint_6">
             <hardwareInterface>hardware_interface/${hardware_interface}</hardwareInterface>
         </joint>
-        <actuator name="motor_6">
+        <actuator name="${robot_name}_motor_6">
             <hardwareInterface>hardware_interface/${hardware_interface}</hardwareInterface>
             <mechanicalReduction>1</mechanicalReduction>
@@ -75,11 +75,11 @@
     </transmission>
     <!-- joint 7 -->
-    <transmission name="tran_7">
+    <transmission name="${robot_name}_tran_7">
         <robotNamespace>/${robot_name}</robotNamespace>
         <type>transmission_interface/SimpleTransmission</type>
-        <joint name="joint_7">
+        <joint name="${robot_name}_joint_7">
             <hardwareInterface>hardware_interface/${hardware_interface}</hardwareInterface>
         </joint>
-        <actuator name="motor_7">
+        <actuator name="${robot_name}_motor_7">
             <hardwareInterface>hardware_interface/${hardware_interface}</hardwareInterface>
             <mechanicalReduction>1</mechanicalReduction>

File: lbr_description/urdf/med.gazebo.xacro (robot description, xacro)
@@ -9,5 +9,5 @@
         </gazebo>
         <!-- link 0 -->
-        <gazebo reference="link_0">
+        <gazebo reference="${robot_name}_link_0">
             <mu1>0.2</mu1>
             <mu2>0.2</mu2>
@@ -15,5 +15,5 @@
         </gazebo>
         <!-- link 1 -->
-        <gazebo reference="link_1">
+        <gazebo reference="${robot_name}_link_1">
             <mu1>0.2</mu1>
             <mu2>0.2</mu2>
@@ -21,5 +21,5 @@
         </gazebo>
         <!-- link 2 -->
-        <gazebo reference="link_2">
+        <gazebo reference="${robot_name}_link_2">
             <mu1>0.2</mu1>
             <mu2>0.2</mu2>
@@ -27,5 +27,5 @@
         </gazebo>
         <!-- link 3 -->
-        <gazebo reference="link_3">
+        <gazebo reference="${robot_name}_link_3">
             <mu1>0.2</mu1>
             <mu2>0.2</mu2>
@@ -33,5 +33,5 @@
         </gazebo>
         <!-- link 4 -->
-        <gazebo reference="link_4">
+        <gazebo reference="${robot_name}_link_4">
             <mu1>0.2</mu1>
             <mu2>0.2</mu2>
@@ -39,5 +39,5 @@
         </gazebo>
         <!-- link 5 -->
-        <gazebo reference="link_5">
+        <gazebo reference="${robot_name}_link_5">
             <mu1>0.2</mu1>
             <mu2>0.2</mu2>
@@ -45,5 +45,5 @@
         </gazebo>
         <!-- link 6 -->
-        <gazebo reference="link_6">
+        <gazebo reference="${robot_name}_link_6">
             <mu1>0.2</mu1>
             <mu2>0.2</mu2>
@@ -51,5 +51,5 @@
         </gazebo>
         <!-- link 7 -->
-        <gazebo reference="link_7">
+        <gazebo reference="${robot_name}_link_7">
             <mu1>0.2</mu1>
             <mu2>0.2</mu2>
