Commit message: added robot name prefix for multi robots

File: lbr_description/urdf/med14.xacro (robot description, xacro)
@@ -18,7 +18,7 @@
             <xacro:insert_block name="origin"/>
             <parent link="${parent}"/>
-            <child link="link_0"/>
-        </joint>
-        <link name="link_0">
+            <child link="${robot_name}_link_0"/>
+        </joint>
+        <link name="${robot_name}_link_0">
             <inertial>
             <origin rpy="0 0 0" xyz="-0.0018642104260720833 -9.120393625716289e-09 0.07751683665104403"/>
@@ -42,8 +42,8 @@
             </collision>
         </link>
-        <joint name="joint_1" type="revolute">
+        <joint name="${robot_name}_joint_1" type="revolute">
             <origin rpy="0 0 0" xyz="0.0 0.0 0.147"/>
-            <parent link="link_0"/>
-            <child link="link_1"/>
+            <parent link="${robot_name}_link_0"/>
+            <child link="${robot_name}_link_1"/>
             <axis xyz="0.0 0.0 0.01"/>
             <limit effort="${max_effort}" lower="${-170 * PI / 180}" upper="${170 * PI / 180}" velocity="${max_velocity}"/>
@@ -56,5 +56,5 @@
             <dynamics damping="${joint_damping}"/>
         </joint>
-        <link name="link_1">
+        <link name="${robot_name}_link_1">
             <inertial>
             <origin rpy="0 0 0" xyz="9.307232415315581e-08 -0.033795431550791004 0.13240370669453896"/>
@@ -78,8 +78,8 @@
             </collision>
         </link>
-        <joint name="joint_2" type="revolute">
+        <joint name="${robot_name}_joint_2" type="revolute">
             <origin rpy="0 0 0" xyz="0.0 -0.01 0.2125"/>
-            <parent link="link_1"/>
-            <child link="link_2"/>
+            <parent link="${robot_name}_link_1"/>
+            <child link="${robot_name}_link_2"/>
             <axis xyz="0.0 0.01 0.0"/>
             <limit effort="${max_effort}" lower="${-120 * PI / 180}" upper="${120 * PI / 180}" velocity="${max_velocity}"/>
@@ -92,5 +92,5 @@
             <dynamics damping="${joint_damping}"/>
         </joint>
-        <link name="link_2">
+        <link name="${robot_name}_link_2">
             <inertial>
             <origin rpy="0 0 0" xyz="0.0001358226533474577 0.0475476440926152 0.07632205850106144"/>
@@ -114,8 +114,8 @@
             </collision>
         </link>
-        <joint name="joint_3" type="revolute">
+        <joint name="${robot_name}_joint_3" type="revolute">
             <origin rpy="0 0 0" xyz="-0.0 0.01 0.228"/>
-            <parent link="link_2"/>
-            <child link="link_3"/>
+            <parent link="${robot_name}_link_2"/>
+            <child link="${robot_name}_link_3"/>
             <axis xyz="0.0 0.0 0.01"/>
             <limit effort="${max_effort}" lower="${-170 * PI / 180}" upper="${170 * PI / 180}" velocity="${max_velocity}"/>
@@ -128,5 +128,5 @@
             <dynamics damping="${joint_damping}"/>
         </joint>
-        <link name="link_3">
+        <link name="${robot_name}_link_3">
             <inertial>
             <origin rpy="0 0 0" xyz="5.689213978259012e-08 0.03491265072974692 0.12310820658934007"/>
@@ -150,8 +150,8 @@
             </collision>
         </link>
-        <joint name="joint_4" type="revolute">
+        <joint name="${robot_name}_joint_4" type="revolute">
             <origin rpy="0 0 0" xyz="0.0 0.0105 0.192"/>
-            <parent link="link_3"/>
-            <child link="link_4"/>
+            <parent link="${robot_name}_link_3"/>
+            <child link="${robot_name}_link_4"/>
             <axis xyz="0.0 -0.01 0.0"/>
             <limit effort="${max_effort}" lower="${-120 * PI / 180}" upper="${120 * PI / 180}" velocity="${max_velocity}"/>
@@ -164,5 +164,5 @@
             <dynamics damping="${joint_damping}"/>
         </joint>
-        <link name="link_4">
+        <link name="${robot_name}_link_4">
             <inertial>
             <origin rpy="0 0 0" xyz="-3.025185496951432e-08 -0.03979329512420171 0.08694364647762443"/>
@@ -186,8 +186,8 @@
             </collision>
         </link>
-        <joint name="joint_5" type="revolute">
+        <joint name="${robot_name}_joint_5" type="revolute">
             <origin rpy="0 0 0" xyz="0.0 -0.0105 0.2075"/>
-            <parent link="link_4"/>
-            <child link="link_5"/>
+            <parent link="${robot_name}_link_4"/>
+            <child link="${robot_name}_link_5"/>
             <axis xyz="0.0 0.0 0.01"/>
             <limit effort="${max_effort}" lower="${-170 * PI / 180}" upper="${170 * PI / 180}" velocity="${max_velocity}"/>
@@ -200,5 +200,5 @@
             <dynamics damping="${joint_damping}"/>
         </joint>
-        <link name="link_5">
+        <link name="${robot_name}_link_5">
             <inertial>
             <origin rpy="0 0 0" xyz="3.8871741664391765e-08 -0.029824284088761824 0.07626701716135809"/>
@@ -222,8 +222,8 @@
             </collision>
         </link>
-        <joint name="joint_6" type="revolute">
+        <joint name="${robot_name}_joint_6" type="revolute">
             <origin rpy="0 0 0" xyz="0.0 -0.0707 0.1925"/>
-            <parent link="link_5"/>
-            <child link="link_6"/>
+            <parent link="${robot_name}_link_5"/>
+            <child link="${robot_name}_link_6"/>
             <axis xyz="0.0 0.01 0.0"/>
             <limit effort="${max_effort}" lower="${-120 * PI / 180}" upper="${120 * PI / 180}" velocity="${max_velocity}"/>
@@ -236,5 +236,5 @@
             <dynamics damping="${joint_damping}"/>
         </joint>
-        <link name="link_6">
+        <link name="${robot_name}_link_6">
             <inertial>
             <origin rpy="0 0 0" xyz="-7.073221484902805e-07 0.07101990943401978 0.004952526180380223"/>
@@ -258,8 +258,8 @@
             </collision>
         </link>
-        <joint name="joint_7" type="revolute">
+        <joint name="${robot_name}_joint_7" type="revolute">
             <origin rpy="0 0 0" xyz="0.0 0.0707 0.091"/>
-            <parent link="link_6"/>
-            <child link="link_7"/>
+            <parent link="${robot_name}_link_6"/>
+            <child link="${robot_name}_link_7"/>
             <axis xyz="0.0 0.0 0.01"/>
             <limit effort="${max_effort}" lower="${-175 * PI / 180}" upper="${175 * PI / 180}" velocity="${max_velocity}"/>
@@ -272,5 +272,5 @@
             <dynamics damping="${joint_damping}"/>
         </joint>
-        <link name="link_7">
+        <link name="${robot_name}_link_7">
             <inertial>
             <origin rpy="0 0 0" xyz="3.121827460016089e-06 -1.635815563460264e-06 0.0137822955218736"/>
@@ -294,10 +294,10 @@
             </collision>
         </link>
-        <joint name="joint_ee" type="fixed">
-            <parent link="$link_7"/>
-            <child link="$link_ee"/>
+        <joint name="${robot_name}_joint_ee" type="fixed">
+            <parent link="${robot_name}_link_7"/>
+            <child link="${robot_name}_link_ee"/>
             <origin xyz="0 0 0.045" rpy="0 0 0"/>
         </joint>
-        <link name="$link_ee">
+        <link name="${robot_name}_link_ee">
         </link>
         <!-- extensions -->

File: lbr_description/urdf/med7.xacro (robot description, xacro)
@@ -18,7 +18,7 @@
             <xacro:insert_block name="origin"/>
             <parent link="${parent}"/>
-            <child link="link_0"/>
-        </joint>
-        <link name="link_0">
+            <child link="${robot_name}_link_0"/>
+        </joint>
+        <link name="${robot_name}_link_0">
             <inertial>
             <origin rpy="0 0 0" xyz="-0.0018958727522859222 -8.736009549202623e-09 0.07626305487275586"/>
@@ -42,8 +42,8 @@
             </collision>
         </link>
-        <joint name="joint_1" type="revolute">
+        <joint name="${robot_name}_joint_1" type="revolute">
             <origin rpy="0 0 0" xyz="0.0 0.0 0.1475"/>
-            <parent link="link_0"/>
-            <child link="link_1"/>
+            <parent link="${robot_name}_link_0"/>
+            <child link="${robot_name}_link_1"/>
             <axis xyz="0.0 0.0 0.01"/>
             <limit effort="${max_effort}" lower="${-170 * PI / 180}" upper="${170 * PI / 180}" velocity="${max_velocity}"/>
@@ -56,5 +56,5 @@
             <dynamics damping="${joint_damping}"/>
         </joint>
-        <link name="link_1">
+        <link name="${robot_name}_link_1">
             <inertial>
             <origin rpy="0 0 0" xyz="5.010328793588479e-08 -0.03481903813472808 0.12329857163085542"/>
@@ -78,8 +78,8 @@
             </collision>
         </link>
-        <joint name="joint_2" type="revolute">
+        <joint name="${robot_name}_joint_2" type="revolute">
             <origin rpy="0 0 0" xyz="-0.0 -0.0105 0.1925"/>
-            <parent link="link_1"/>
-            <child link="link_2"/>
+            <parent link="${robot_name}_link_1"/>
+            <child link="${robot_name}_link_2"/>
             <axis xyz="0.0 0.01 0.0"/>
             <limit effort="${max_effort}" lower="${-120 * PI / 180}" upper="${120 * PI / 180}" velocity="${max_velocity}"/>
@@ -92,5 +92,5 @@
             <dynamics damping="${joint_damping}"/>
         </joint>
-        <link name="link_2">
+        <link name="${robot_name}_link_2">
             <inertial>
             <origin rpy="0 0 0" xyz="2.958275959973659e-08 0.03979295468456965 0.08694361150855662"/>
@@ -114,8 +114,8 @@
             </collision>
         </link>
-        <joint name="joint_3" type="revolute">
+        <joint name="${robot_name}_joint_3" type="revolute">
             <origin rpy="0 0 0" xyz="0.0 0.0105 0.2075"/>
-            <parent link="link_2"/>
-            <child link="link_3"/>
+            <parent link="${robot_name}_link_2"/>
+            <child link="${robot_name}_link_3"/>
             <axis xyz="0.0 0.0 0.01"/>
             <limit effort="${max_effort}" lower="${-170 * PI / 180}" upper="${170 * PI / 180}" velocity="${max_velocity}"/>
@@ -128,5 +128,5 @@
             <dynamics damping="${joint_damping}"/>
         </joint>
-        <link name="link_3">
+        <link name="${robot_name}_link_3">
             <inertial>
             <origin rpy="0 0 0" xyz="-5.010330962930412e-08 0.03481903813473644 0.1232985716309013"/>
@@ -150,8 +150,8 @@
             </collision>
         </link>
-        <joint name="joint_4" type="revolute">
+        <joint name="${robot_name}_joint_4" type="revolute">
             <origin rpy="0 0 0" xyz="0.0 0.0105 0.1925"/>
-            <parent link="link_3"/>
-            <child link="link_4"/>
+            <parent link="${robot_name}_link_3"/>
+            <child link="${robot_name}_link_4"/>
             <axis xyz="0.0 -0.01 0.0"/>
             <limit effort="${max_effort}" lower="${-120 * PI / 180}" upper="${120 * PI / 180}" velocity="${max_velocity}"/>
@@ -164,5 +164,5 @@
             <dynamics damping="${joint_damping}"/>
         </joint>
-        <link name="link_4">
+        <link name="${robot_name}_link_4">
             <inertial>
             <origin rpy="0 0 0" xyz="-3.025230048709993e-08 -0.03979329512443697 0.08694363375610437"/>
@@ -186,8 +186,8 @@
             </collision>
         </link>
-        <joint name="joint_5" type="revolute">
+        <joint name="${robot_name}_joint_5" type="revolute">
             <origin rpy="0 0 0" xyz="-0.0 -0.0105 0.2075"/>
-            <parent link="link_4"/>
-            <child link="link_5"/>
+            <parent link="${robot_name}_link_4"/>
+            <child link="${robot_name}_link_5"/>
             <axis xyz="0.0 0.0 0.01"/>
             <limit effort="${max_effort}" lower="${-170 * PI / 180}" upper="${170 * PI / 180}" velocity="${max_velocity}"/>
@@ -200,5 +200,5 @@
             <dynamics damping="${joint_damping}"/>
         </joint>
-        <link name="link_5">
+        <link name="${robot_name}_link_5">
             <inertial>
             <origin rpy="0 0 0" xyz="3.887174133882675e-08 -0.02982428408876193 0.07626701716135398"/>
@@ -222,8 +222,8 @@
             </collision>
         </link>
-        <joint name="joint_6" type="revolute">
+        <joint name="${robot_name}_joint_6" type="revolute">
             <origin rpy="0 0 0" xyz="0.0 -0.0707 0.1925"/>
-            <parent link="link_5"/>
-            <child link="link_6"/>
+            <parent link="${robot_name}_link_5"/>
+            <child link="${robot_name}_link_6"/>
             <axis xyz="0.0 0.01 0.0"/>
             <limit effort="${max_effort}" lower="${-120 * PI / 180}" upper="${120 * PI / 180}" velocity="${max_velocity}"/>
@@ -236,5 +236,5 @@
             <dynamics damping="${joint_damping}"/>
         </joint>
-        <link name="link_6">
+        <link name="${robot_name}_link_6">
             <inertial>
             <origin rpy="0 0 0" xyz="-7.073221144775636e-07 0.07101990943401648 0.004952526180360017"/>
@@ -258,8 +258,8 @@
             </collision>
         </link>
-        <joint name="joint_7" type="revolute">
+        <joint name="${robot_name}_joint_7" type="revolute">
             <origin rpy="0 0 0" xyz="0.0 0.0707 0.091"/>
-            <parent link="link_6"/>
-            <child link="link_7"/>
+            <parent link="${robot_name}_link_6"/>
+            <child link="${robot_name}_link_7"/>
             <axis xyz="0.0 0.0 0.01"/>
             <limit effort="${max_effort}" lower="${-175 * PI / 180}" upper="${175 * PI / 180}" velocity="${max_velocity}"/>
@@ -272,5 +272,5 @@
             <dynamics damping="${joint_damping}"/>
         </joint>
-        <link name="link_7">
+        <link name="${robot_name}_link_7">
             <inertial>
             <origin rpy="0 0 0" xyz="3.1218274599808524e-06 -1.6358155634513969e-06 0.013782295521067356"/>
@@ -294,10 +294,10 @@
             </collision>
         </link>
-        <joint name="joint_ee" type="fixed">
-            <parent link="$link_7"/>
-            <child link="$link_ee"/>
+        <joint name="${robot_name}_joint_ee" type="fixed">
+            <parent link="${robot_name}_link_7"/>
+            <child link="${robot_name}_link_ee"/>
             <origin xyz="0 0 0.045" rpy="0 0 0"/>
         </joint>
-        <link name="$link_ee">
+        <link name="${robot_name}_link_ee">
         </link>
         <!-- extensions -->

Commit message: removed materials and updated joints

File: lbr_description/urdf/iiwa.gazebo.xacro (robot description, xacro)
@@ -12,5 +12,4 @@
             <mu1>0.2</mu1>
             <mu2>0.2</mu2>
-            <material>Gazebo/Grey</material>
         </gazebo>
         <!-- link 1 -->
@@ -18,5 +17,4 @@
             <mu1>0.2</mu1>
             <mu2>0.2</mu2>
-            <material>Gazebo/Orange</material>
         </gazebo>
         <!-- link 2 -->
@@ -24,5 +22,4 @@
             <mu1>0.2</mu1>
             <mu2>0.2</mu2>
-            <material>Gazebo/Orange</material>
         </gazebo>
         <!-- link 3 -->
@@ -30,5 +27,4 @@
             <mu1>0.2</mu1>
             <mu2>0.2</mu2>
-            <material>Gazebo/Orange</material>
         </gazebo>
         <!-- link 4 -->
@@ -36,5 +32,4 @@
             <mu1>0.2</mu1>
             <mu2>0.2</mu2>
-            <material>Gazebo/Orange</material>
         </gazebo>
         <!-- link 5 -->
@@ -42,5 +37,4 @@
             <mu1>0.2</mu1>
             <mu2>0.2</mu2>
-            <material>Gazebo/Orange</material>
         </gazebo>
         <!-- link 6 -->
@@ -48,5 +42,4 @@
             <mu1>0.2</mu1>
             <mu2>0.2</mu2>
-            <material>Gazebo/Orange</material>
         </gazebo>
         <!-- link 7 -->
@@ -54,5 +47,4 @@
             <mu1>0.2</mu1>
             <mu2>0.2</mu2>
-            <material>Gazebo/Grey</material>
         </gazebo>
     </xacro:macro>

File: lbr_description/urdf/iiwa14.xacro (robot description, xacro)
@@ -5,6 +5,4 @@
     <!-- include transmission for ros_control -->
     <xacro:include filename="$(find lbr_description)/urdf/lbr.transmission.xacro" />
-    <!-- include materials -->
-    <xacro:include filename="$(find lbr_description)/urdf/lbr.materials.xacro" />
     <!-- some constants -->
     <xacro:property name="PI" value="3.1415926535897931" />
@@ -115,5 +113,5 @@
         </link>
         <joint name="${robot_name}_joint_3" type="revolute">
-            <origin rpy="0 0 0" xyz="0.0 0.01 0.1945" />
+            <origin rpy="0 0 0" xyz="0.0 0.01 0.228" />
             <parent link="${robot_name}_link_2" />
             <child link="${robot_name}_link_3" />
@@ -150,5 +148,5 @@
         </link>
         <joint name="${robot_name}_joint_4" type="revolute">
-            <origin rpy="0 0 0" xyz="-0.0 0.0105 0.2255" />
+            <origin rpy="0 0 0" xyz="0.0 0.0105 0.192" />
             <parent link="${robot_name}_link_3" />
             <child link="${robot_name}_link_4" />
@@ -185,5 +183,5 @@
         </link>
         <joint name="${robot_name}_joint_5" type="revolute">
-            <origin rpy="0 0 0" xyz="0.0 -0.0105 0.1745" />
+            <origin rpy="0 0 0" xyz="0.0 -0.0105 0.2075" />
             <parent link="${robot_name}_link_4" />
             <child link="${robot_name}_link_5" />
@@ -220,5 +218,5 @@
         </link>
         <joint name="${robot_name}_joint_6" type="revolute">
-            <origin rpy="0 0 0" xyz="-0.0 -0.0707 0.2255" />
+            <origin rpy="0 0 0" xyz="0.0 -0.0707 0.1925" />
             <parent link="${robot_name}_link_5" />
             <child link="${robot_name}_link_6" />
@@ -255,5 +253,5 @@
         </link>
         <joint name="${robot_name}_joint_7" type="revolute">
-            <origin rpy="0 0 0" xyz="0.0 0.0707 0.0711" />
+            <origin rpy="0 0 0" xyz="0.0 0.0707 0.091" />
             <parent link="${robot_name}_link_6" />
             <child link="${robot_name}_link_7" />

File: lbr_description/urdf/iiwa7.xacro (robot description, xacro)
@@ -5,6 +5,4 @@
     <!-- include transmission for ros_control -->
     <xacro:include filename="$(find lbr_description)/urdf/lbr.transmission.xacro" />
-    <!-- include materials -->
-    <xacro:include filename="$(find lbr_description)/urdf/lbr.materials.xacro" />
     <!-- some constants -->
     <xacro:property name="PI" value="3.1415926535897931" />
@@ -80,5 +78,5 @@
         </link>
         <joint name="${robot_name}_joint_2" type="revolute">
-            <origin rpy="0 0 0" xyz="-0.0 -0.0105 0.193" />
+            <origin rpy="0 0 0" xyz="0.0 -0.0105 0.1925" />
             <parent link="${robot_name}_link_1" />
             <child link="${robot_name}_link_2" />
@@ -115,5 +113,5 @@
         </link>
         <joint name="${robot_name}_joint_3" type="revolute">
-            <origin rpy="0 0 0" xyz="0.0 0.0105 0.1745" />
+            <origin rpy="0 0 0" xyz="0.0 0.0105 0.2075" />
             <parent link="${robot_name}_link_2" />
             <child link="${robot_name}_link_3" />
@@ -150,5 +148,5 @@
         </link>
         <joint name="${robot_name}_joint_4" type="revolute">
-            <origin rpy="0 0 0" xyz="0.0 0.0105 0.2255" />
+            <origin rpy="0 0 0" xyz="0.0 0.0105 0.1925" />
             <parent link="${robot_name}_link_3" />
             <child link="${robot_name}_link_4" />
@@ -185,5 +183,5 @@
         </link>
         <joint name="${robot_name}_joint_5" type="revolute">
-            <origin rpy="0 0 0" xyz="0.0 -0.0105 0.1745" />
+            <origin rpy="0 0 0" xyz="0.0 -0.0105 0.2075" />
             <parent link="${robot_name}_link_4" />
             <child link="${robot_name}_link_5" />
@@ -220,5 +218,5 @@
         </link>
         <joint name="${robot_name}_joint_6" type="revolute">
-            <origin rpy="0 0 0" xyz="0.0 -0.0707 0.2255" />
+            <origin rpy="0 0 0" xyz="0.0 -0.0707 0.1925" />
             <parent link="${robot_name}_link_5" />
             <child link="${robot_name}_link_6" />
@@ -255,5 +253,5 @@
         </link>
         <joint name="${robot_name}_joint_7" type="revolute">
-            <origin rpy="0 0 0" xyz="0.0 0.0705 0.0909" />
+            <origin rpy="0 0 0" xyz="0.0 0.0707 0.091" />
             <parent link="${robot_name}_link_6" />
             <child link="${robot_name}_link_7" />

File: lbr_description/urdf/med14.xacro (robot description, xacro)
@@ -5,6 +5,4 @@
     <!-- include transmission for ros_control -->
     <xacro:include filename="$(find lbr_description)/urdf/lbr.transmission.xacro" />
-    <!-- include materials -->
-    <xacro:include filename="$(find lbr_description)/urdf/lbr.materials.xacro" />
     <!-- some constants -->
     <xacro:property name="PI" value="3.1415926535897931" />

File: lbr_description/urdf/med7.xacro (robot description, xacro)
@@ -5,6 +5,4 @@
     <!-- include transmission for ros_control -->
     <xacro:include filename="$(find lbr_description)/urdf/lbr.transmission.xacro" />
-    <!-- include materials -->
-    <xacro:include filename="$(find lbr_description)/urdf/lbr.materials.xacro" />
     <!-- some constants -->
     <xacro:property name="PI" value="3.1415926535897931" />
