Commit message: removed legacy material

File: lbr_description/urdf/med.gazebo.xacro (robot description, xacro)
@@ -12,5 +12,4 @@
             <mu1>0.2</mu1>
             <mu2>0.2</mu2>
-            <material>Gazebo/White</material>
         </gazebo>
         <!-- link 1 -->
@@ -18,5 +17,4 @@
             <mu1>0.2</mu1>
             <mu2>0.2</mu2>
-            <material>Gazebo/White</material>
         </gazebo>
         <!-- link 2 -->
@@ -24,5 +22,4 @@
             <mu1>0.2</mu1>
             <mu2>0.2</mu2>
-            <material>Gazebo/White</material>
         </gazebo>
         <!-- link 3 -->
@@ -30,5 +27,4 @@
             <mu1>0.2</mu1>
             <mu2>0.2</mu2>
-            <material>Gazebo/White</material>
         </gazebo>
         <!-- link 4 -->
@@ -36,5 +32,4 @@
             <mu1>0.2</mu1>
             <mu2>0.2</mu2>
-            <material>Gazebo/White</material>
         </gazebo>
         <!-- link 5 -->
@@ -42,5 +37,4 @@
             <mu1>0.2</mu1>
             <mu2>0.2</mu2>
-            <material>Gazebo/White</material>
         </gazebo>
         <!-- link 6 -->
@@ -48,5 +42,4 @@
             <mu1>0.2</mu1>
             <mu2>0.2</mu2>
-            <material>Gazebo/White</material>
         </gazebo>
         <!-- link 7 -->
@@ -54,5 +47,4 @@
             <mu1>0.2</mu1>
             <mu2>0.2</mu2>
-            <material>Gazebo/Grey</material>
         </gazebo>
     </xacro:macro>
