Commit message: fixed typo

File: lbr_description/urdf/med7/med7_description.urdf.xacro (robot description, xacro)
@@ -16,5 +16,5 @@
         <joint name="${parent}_${robot_name}_joint" type="fixed">
             <parent link="${parent}"/>
-            <child link="${robot_name}_link_0"/>=
+            <child link="${robot_name}_link_0"/>
         </joint>
         <link name="${robot_name}_link_0">
