Commit message: fixed xacro tag gazebo xacro tag #10

File: lbr_description/gazebo/med.gazebo.xacro (robot description, xacro)
@@ -1,5 +1,5 @@
 <?xml version="1.0"?>
 <robot xmlns:xacro="http://www.ros.org/wiki/xacro">
-    <xacro:macro name="iiwa_gazebo" params="robot_name:=^|lbr">
+    <xacro:macro name="med_gazebo" params="robot_name:=^|lbr">
         <!-- ros_control-plugin -->
         <gazebo>

File: lbr_description/urdf/med14/med14_description.urdf.xacro (robot description, xacro)
@@ -241,5 +241,5 @@
         <link name="${robot_name}_link_ee">
         </link>
-        <xacro:iiwa_gazebo robot_name="${robot_name}"/>
+        <xacro:med_gazebo robot_name="${robot_name}"/>
         <!-- TODO: move modes to args, decouple urdf/gazebo/controls -->
         <xacro:lbr_hardware_interface sim="${sim}" remote_host="INADDR_ANY" port="30200" robot_name="${robot_name}"/>

File: lbr_description/urdf/med7/med7_description.urdf.xacro (robot description, xacro)
@@ -241,5 +241,5 @@
         <link name="${robot_name}_link_ee">
         </link>
-        <xacro:iiwa_gazebo robot_name="${robot_name}"/>
+        <xacro:med_gazebo robot_name="${robot_name}"/>
         <!-- TODO: move modes to args, decouple urdf/gazebo/controls -->
         <!-- add notice for remote host to set to kuka controller -->
