Commit message: removed robot name prefix from configs

File: lbr_description/gazebo/iiwa.gazebo.xacro (robot description, xacro)
@@ -10,5 +10,5 @@
         </gazebo>
         <!-- link 0 -->
-        <gazebo reference="${robot_name}_link_0">
+        <gazebo reference="link_0">
             <mu1>0.2</mu1>
             <mu2>0.2</mu2>
@@ -16,5 +16,5 @@
         </gazebo>
         <!-- link 1 -->
-        <gazebo reference="${robot_name}_link_1">
+        <gazebo reference="link_1">
             <mu1>0.2</mu1>
             <mu2>0.2</mu2>
@@ -22,5 +22,5 @@
         </gazebo>
         <!-- link 2 -->
-        <gazebo reference="${robot_name}_link_2">
+        <gazebo reference="link_2">
             <mu1>0.2</mu1>
             <mu2>0.2</mu2>
@@ -28,5 +28,5 @@
         </gazebo>
         <!-- link 3 -->
-        <gazebo reference="${robot_name}_link_3">
+        <gazebo reference="link_3">
             <mu1>0.2</mu1>
             <mu2>0.2</mu2>
@@ -34,5 +34,5 @@
         </gazebo>
         <!-- link 4 -->
-        <gazebo reference="${robot_name}_link_4">
+        <gazebo reference="link_4">
             <mu1>0.2</mu1>
             <mu2>0.2</mu2>
@@ -40,5 +40,5 @@
         </gazebo>
         <!-- link 5 -->
-        <gazebo reference="${robot_name}_link_5">
+        <gazebo reference="link_5">
             <mu1>0.2</mu1>
             <mu2>0.2</mu2>
@@ -46,5 +46,5 @@
         </gazebo>
         <!-- link 6 -->
-        <gazebo reference="${robot_name}_link_6">
+        <gazebo reference="link_6">
             <mu1>0.2</mu1>
             <mu2>0.2</mu2>
@@ -52,5 +52,5 @@
         </gazebo>
         <!-- link 7 -->
-        <gazebo reference="${robot_name}_link_7">
+        <gazebo reference="link_7">
             <mu1>0.2</mu1>
             <mu2>0.2</mu2>

File: lbr_description/gazebo/med.gazebo.xacro (robot description, xacro)
@@ -10,5 +10,5 @@
         </gazebo>
         <!-- link 0 -->
-        <gazebo reference="${robot_name}_link_0">
+        <gazebo reference="link_0">
             <mu1>0.2</mu1>
             <mu2>0.2</mu2>
@@ -16,5 +16,5 @@
         </gazebo>
         <!-- link 1 -->
-        <gazebo reference="${robot_name}_link_1">
+        <gazebo reference="link_1">
             <mu1>0.2</mu1>
             <mu2>0.2</mu2>
@@ -22,5 +22,5 @@
         </gazebo>
         <!-- link 2 -->
-        <gazebo reference="${robot_name}_link_2">
+        <gazebo reference="link_2">
             <mu1>0.2</mu1>
             <mu2>0.2</mu2>
@@ -28,5 +28,5 @@
         </gazebo>
         <!-- link 3 -->
-        <gazebo reference="${robot_name}_link_3">
+        <gazebo reference="link_3">
             <mu1>0.2</mu1>
             <mu2>0.2</mu2>
@@ -34,5 +34,5 @@
         </gazebo>
         <!-- link 4 -->
-        <gazebo reference="${robot_name}_link_4">
+        <gazebo reference="link_4">
             <mu1>0.2</mu1>
             <mu2>0.2</mu2>
@@ -40,5 +40,5 @@
         </gazebo>
         <!-- link 5 -->
-        <gazebo reference="${robot_name}_link_5">
+        <gazebo reference="link_5">
             <mu1>0.2</mu1>
             <mu2>0.2</mu2>
@@ -46,5 +46,5 @@
         </gazebo>
         <!-- link 6 -->
-        <gazebo reference="${robot_name}_link_6">
+        <gazebo reference="link_6">
             <mu1>0.2</mu1>
             <mu2>0.2</mu2>
@@ -52,5 +52,5 @@
         </gazebo>
         <!-- link 7 -->
-        <gazebo reference="${robot_name}_link_7">
+        <gazebo reference="link_7">
             <mu1>0.2</mu1>
             <mu2>0.2</mu2>

File: lbr_description/ros2_control/lbr.ros2_control.xacro (robot description, xacro)
@@ -32,5 +32,5 @@
             https://github.com/ros-controls/roadmap/blob/master/design_drafts/components_architecture_and_urdf_examples.md -->
             <xacro:unless value="${sim}">
-                <sensor name="${robot_name}_fri_sensor">
+                <sensor name="fri_sensor">
                     <!-- see KUKA::FRI::LBRState -->
                     <state_interface name="sample_time" />
@@ -49,5 +49,5 @@
             </xacro:unless>
             <!-- define joints and command/state interfaces for each joint -->
-            <joint name="${robot_name}_A1">
+            <joint name="A1">
                 <command_interface name="position">
                     <!-- better to use radians as min max first -->
@@ -69,5 +69,5 @@
                 </xacro:unless>
             </joint>
-            <joint name="${robot_name}_A2">
+            <joint name="A2">
                 <command_interface name="position">
                     <param name="min">-${joint_1_position_limit}</param>
@@ -88,5 +88,5 @@
                 </xacro:unless>
             </joint>
-            <joint name="${robot_name}_A3">
+            <joint name="A3">
                 <command_interface name="position">
                     <param name="min">-${joint_2_position_limit}</param>
@@ -107,5 +107,5 @@
                 </xacro:unless>
             </joint>
-            <joint name="${robot_name}_A4">
+            <joint name="A4">
                 <command_interface name="position">
                     <param name="min">-${joint_3_position_limit}</param>
@@ -126,5 +126,5 @@
                 </xacro:unless>
             </joint>
-            <joint name="${robot_name}_A5">
+            <joint name="A5">
                 <command_interface name="position">
                     <param name="min">-${joint_4_position_limit}</param>
@@ -145,5 +145,5 @@
                 </xacro:unless>
             </joint>
-            <joint name="${robot_name}_A6">
+            <joint name="A6">
                 <command_interface name="position">
                     <param name="min">-${joint_5_position_limit}</param>
@@ -164,5 +164,5 @@
                 </xacro:unless>
             </joint>
-            <joint name="${robot_name}_A7">
+            <joint name="A7">
                 <command_interface name="position">
                     <param name="min">-${joint_6_position_limit}</param>

File: lbr_description/urdf/iiwa14/iiwa14_description.urdf.xacro (robot description, xacro)
@@ -28,9 +28,9 @@
         <!--joint
         between {base_frame} and link_0-->
-        <joint name="${base_frame}_${robot_name}_joint" type="fixed">
+        <joint name="${base_frame}_joint" type="fixed">
             <parent link="${base_frame}" />
-            <child link="${robot_name}_link_0" />
-        </joint>
-        <link name="${robot_name}_link_0">
+            <child link="link_0" />
+        </joint>
+        <link name="link_0">
             <inertial>
                 <origin rpy="0 0 0"
@@ -54,8 +54,8 @@
             </collision>
         </link>
-        <joint name="${robot_name}_A1" type="revolute">
+        <joint name="A1" type="revolute">
             <origin rpy="0 0 0" xyz="0.0 0.0 0.1475" />
-            <parent link="${robot_name}_link_0" />
-            <child link="${robot_name}_link_1" />
+            <parent link="link_0" />
+            <child link="link_1" />
             <axis xyz="0.0 0.0 1.0" />
             <limit effort="${effort_limit}" lower="${-joint_0_position_limit * PI / 180}"
@@ -64,5 +64,5 @@
             <dynamics damping="${joint_damping}" friction="${joint_friction}" />
         </joint>
-        <link name="${robot_name}_link_1">
+        <link name="link_1">
             <inertial>
                 <origin rpy="0 0 0"
@@ -86,8 +86,8 @@
             </collision>
         </link>
-        <joint name="${robot_name}_A2" type="revolute">
+        <joint name="A2" type="revolute">
             <origin rpy="0 0 0" xyz="0.0 -0.01 0.2125" />
-            <parent link="${robot_name}_link_1" />
-            <child link="${robot_name}_link_2" />
+            <parent link="link_1" />
+            <child link="link_2" />
             <axis xyz="0.0 1.0 0.0" />
             <limit effort="${effort_limit}" lower="${-joint_1_position_limit * PI / 180}"
@@ -96,5 +96,5 @@
             <dynamics damping="${joint_damping}" friction="${joint_friction}" />
         </joint>
-        <link name="${robot_name}_link_2">
+        <link name="link_2">
             <inertial>
                 <origin rpy="0 0 0"
@@ -118,8 +118,8 @@
             </collision>
         </link>
-        <joint name="${robot_name}_A3" type="revolute">
+        <joint name="A3" type="revolute">
             <origin rpy="0 0 0" xyz="0.0 0.01 0.1945" />
-            <parent link="${robot_name}_link_2" />
-            <child link="${robot_name}_link_3" />
+            <parent link="link_2" />
+            <child link="link_3" />
             <axis xyz="0.0 0.0 1.0" />
             <limit effort="${effort_limit}" lower="${-joint_2_position_limit * PI / 180}"
@@ -128,5 +128,5 @@
             <dynamics damping="${joint_damping}" friction="${joint_friction}" />
         </joint>
-        <link name="${robot_name}_link_3">
+        <link name="link_3">
             <inertial>
                 <origin rpy="0 0 0"
@@ -150,8 +150,8 @@
             </collision>
         </link>
-        <joint name="${robot_name}_A4" type="revolute">
+        <joint name="A4" type="revolute">
             <origin rpy="0 0 0" xyz="-0.0 0.0105 0.2255" />
-            <parent link="${robot_name}_link_3" />
-            <child link="${robot_name}_link_4" />
+            <parent link="link_3" />
+            <child link="link_4" />
             <axis xyz="0.0 -1.0 0.0" />
             <limit effort="${effort_limit}" lower="${-joint_3_position_limit * PI / 180}"
@@ -160,5 +160,5 @@
             <dynamics damping="${joint_damping}" friction="${joint_friction}" />
         </joint>
-        <link name="${robot_name}_link_4">
+        <link name="link_4">
             <inertial>
                 <origin rpy="0 0 0"
@@ -182,8 +182,8 @@
             </collision>
         </link>
-        <joint name="${robot_name}_A5" type="revolute">
+        <joint name="A5" type="revolute">
             <origin rpy="0 0 0" xyz="0.0 -0.0105 0.1745" />
-            <parent link="${robot_name}_link_4" />
-            <child link="${robot_name}_link_5" />
+            <parent link="link_4" />
+            <child link="link_5" />
             <axis xyz="0.0 0.0 1.0" />
             <limit effort="${effort_limit}" lower="${-joint_4_position_limit * PI / 180}"
@@ -192,5 +192,5 @@
             <dynamics damping="${joint_damping}" friction="${joint_friction}" />
         </joint>
-        <link name="${robot_name}_link_5">
+        <link name="link_5">
             <inertial>
                 <origin rpy="0 0 0"
@@ -214,8 +214,8 @@
             </collision>
         </link>
-        <joint name="${robot_name}_A6" type="revolute">
+        <joint name="A6" type="revolute">
             <origin rpy="0 0 0" xyz="-0.0 -0.0707 0.2255" />
-            <parent link="${robot_name}_link_5" />
-            <child link="${robot_name}_link_6" />
+            <parent link="link_5" />
+            <child link="link_6" />
             <axis xyz="0.0 1.0 0.0" />
             <limit effort="${effort_limit}" lower="${-joint_5_position_limit * PI / 180}"
@@ -224,5 +224,5 @@
             <dynamics damping="${joint_damping}" friction="${joint_friction}" />
         </joint>
-        <link name="${robot_name}_link_6">
+        <link name="link_6">
             <inertial>
                 <origin rpy="0 0 0"
@@ -246,8 +246,8 @@
             </collision>
         </link>
-        <joint name="${robot_name}_A7" type="revolute">
+        <joint name="A7" type="revolute">
             <origin rpy="0 0 0" xyz="0.0 0.0707 0.0711" />
-            <parent link="${robot_name}_link_6" />
-            <child link="${robot_name}_link_7" />
+            <parent link="link_6" />
+            <child link="link_7" />
             <axis xyz="0.0 0.0 1.0" />
             <limit effort="${effort_limit}" lower="${-joint_6_position_limit * PI / 180}"
@@ -256,5 +256,5 @@
             <dynamics damping="${joint_damping}" friction="${joint_friction}" />
         </joint>
-        <link name="${robot_name}_link_7">
+        <link name="link_7">
             <inertial>
                 <origin rpy="0 0 0"
@@ -278,10 +278,10 @@
             </collision>
         </link>
-        <joint name="${robot_name}_joint_ee" type="fixed">
-            <parent link="${robot_name}_link_7" />
-            <child link="${robot_name}_link_ee" />
+        <joint name="joint_ee" type="fixed">
+            <parent link="link_7" />
+            <child link="link_ee" />
             <origin xyz="0 0 0.035" rpy="0 0 0" />
         </joint>
-        <link name="${robot_name}_link_ee">
+        <link name="link_ee">
         </link>
         <xacro:iiwa_gazebo robot_name="${robot_name}" />

File: lbr_description/urdf/iiwa7/iiwa7_description.urdf.xacro (robot description, xacro)
@@ -28,9 +28,9 @@
         <!--joint
         between {base_frame} and link_0-->
-        <joint name="${base_frame}_${robot_name}_joint" type="fixed">
+        <joint name="${base_frame}_joint" type="fixed">
             <parent link="${base_frame}" />
-            <child link="${robot_name}_link_0" />
-        </joint>
-        <link name="${robot_name}_link_0">
+            <child link="link_0" />
+        </joint>
+        <link name="link_0">
             <inertial>
                 <origin rpy="0 0 0"
@@ -54,8 +54,8 @@
             </collision>
         </link>
-        <joint name="${robot_name}_A1" type="revolute">
+        <joint name="A1" type="revolute">
             <origin rpy="0 0 0" xyz="0.0 0.0 0.1475" />
-            <parent link="${robot_name}_link_0" />
-            <child link="${robot_name}_link_1" />
+            <parent link="link_0" />
+            <child link="link_1" />
             <axis xyz="0.0 0.0 1.0" />
             <limit effort="${effort_limit}" lower="${-joint_0_position_limit * PI / 180}"
@@ -64,5 +64,5 @@
             <dynamics damping="${joint_damping}" friction="${joint_friction}" />
         </joint>
-        <link name="${robot_name}_link_1">
+        <link name="link_1">
             <inertial>
                 <origin rpy="0 0 0"
@@ -86,8 +86,8 @@
             </collision>
         </link>
-        <joint name="${robot_name}_A2" type="revolute">
+        <joint name="A2" type="revolute">
             <origin rpy="0 0 0" xyz="-0.0 -0.0105 0.193" />
-            <parent link="${robot_name}_link_1" />
-            <child link="${robot_name}_link_2" />
+            <parent link="link_1" />
+            <child link="link_2" />
             <axis xyz="0.0 1.0 0.0" />
             <limit effort="${effort_limit}" lower="${-joint_1_position_limit * PI / 180}"
@@ -96,5 +96,5 @@
             <dynamics damping="${joint_damping}" friction="${joint_friction}" />
         </joint>
-        <link name="${robot_name}_link_2">
+        <link name="link_2">
             <inertial>
                 <origin rpy="0 0 0"
@@ -118,8 +118,8 @@
             </collision>
         </link>
-        <joint name="${robot_name}_A3" type="revolute">
+        <joint name="A3" type="revolute">
             <origin rpy="0 0 0" xyz="0.0 0.0105 0.1745" />
-            <parent link="${robot_name}_link_2" />
-            <child link="${robot_name}_link_3" />
+            <parent link="link_2" />
+            <child link="link_3" />
             <axis xyz="0.0 0.0 1.0" />
             <limit effort="${effort_limit}" lower="${-joint_2_position_limit * PI / 180}"
@@ -128,5 +128,5 @@
             <dynamics damping="${joint_damping}" friction="${joint_friction}" />
         </joint>
-        <link name="${robot_name}_link_3">
+        <link name="link_3">
             <inertial>
                 <origin rpy="0 0 0"
@@ -150,8 +150,8 @@
             </collision>
         </link>
-        <joint name="${robot_name}_A4" type="revolute">
+        <joint name="A4" type="revolute">
             <origin rpy="0 0 0" xyz="0.0 0.0105 0.2255" />
-            <parent link="${robot_name}_link_3" />
-            <child link="${robot_name}_link_4" />
+            <parent link="link_3" />
+            <child link="link_4" />
             <axis xyz="0.0 -1.0 0.0" />
             <limit effort="${effort_limit}" lower="${-joint_3_position_limit * PI / 180}"
@@ -160,5 +160,5 @@
             <dynamics damping="${joint_damping}" friction="${joint_friction}" />
         </joint>
-        <link name="${robot_name}_link_4">
+        <link name="link_4">
             <inertial>
                 <origin rpy="0 0 0"
@@ -182,8 +182,8 @@
             </collision>
         </link>
-        <joint name="${robot_name}_A5" type="revolute">
+        <joint name="A5" type="revolute">
             <origin rpy="0 0 0" xyz="0.0 -0.0105 0.1745" />
-            <parent link="${robot_name}_link_4" />
-            <child link="${robot_name}_link_5" />
+            <parent link="link_4" />
+            <child link="link_5" />
             <axis xyz="0.0 0.0 1.0" />
             <limit effort="${effort_limit}" lower="${-joint_4_position_limit * PI / 180}"
@@ -192,5 +192,5 @@
             <dynamics damping="${joint_damping}" friction="${joint_friction}" />
         </joint>
-        <link name="${robot_name}_link_5">
+        <link name="link_5">
             <inertial>
                 <origin rpy="0 0 0"
@@ -214,8 +214,8 @@
             </collision>
         </link>
-        <joint name="${robot_name}_A6" type="revolute">
+        <joint name="A6" type="revolute">
             <origin rpy="0 0 0" xyz="0.0 -0.0707 0.2255" />
-            <parent link="${robot_name}_link_5" />
-            <child link="${robot_name}_link_6" />
+            <parent link="link_5" />
+            <child link="link_6" />
             <axis xyz="0.0 1.0 0.0" />
             <limit effort="${effort_limit}" lower="${-joint_5_position_limit * PI / 180}"
@@ -224,5 +224,5 @@
             <dynamics damping="${joint_damping}" friction="${joint_friction}" />
         </joint>
-        <link name="${robot_name}_link_6">
+        <link name="link_6">
             <inertial>
                 <origin rpy="0 0 0"
@@ -246,8 +246,8 @@
             </collision>
         </link>
-        <joint name="${robot_name}_A7" type="revolute">
+        <joint name="A7" type="revolute">
             <origin rpy="0 0 0" xyz="0.0 0.0705 0.0909" />
-            <parent link="${robot_name}_link_6" />
-            <child link="${robot_name}_link_7" />
+            <parent link="link_6" />
+            <child link="link_7" />
             <axis xyz="0.0 0.0 1.0" />
             <limit effort="${effort_limit}" lower="${-joint_6_position_limit * PI / 180}"
@@ -256,5 +256,5 @@
             <dynamics damping="${joint_damping}" friction="${joint_friction}" />
         </joint>
-        <link name="${robot_name}_link_7">
+        <link name="link_7">
             <inertial>
                 <origin rpy="0 0 0"
@@ -278,10 +278,10 @@
             </collision>
         </link>
-        <joint name="${robot_name}_joint_ee" type="fixed">
-            <parent link="${robot_name}_link_7" />
-            <child link="${robot_name}_link_ee" />
+        <joint name="joint_ee" type="fixed">
+            <parent link="link_7" />
+            <child link="link_ee" />
             <origin xyz="0 0 0.035" rpy="0 0 0" />
         </joint>
-        <link name="${robot_name}_link_ee">
+        <link name="link_ee">
         </link>
         <xacro:iiwa_gazebo robot_name="${robot_name}" />
