Commit message: removed robot name prefix from configs

File: lbr_description/urdf/med14/med14_description.urdf.xacro (robot description, xacro)
@@ -28,9 +28,9 @@
         <!--joint
         between {base_frame} and link_0-->
-        <joint name="${base_frame}_${robot_name}_joint" type="fixed">
+        <joint name="${base_frame}_joint" type="fixed">
             <parent link="${base_frame}" />
-            <child link="${robot_name}_link_0" />
-        </joint>
-        <link name="${robot_name}_link_0">
+            <child link="link_0" />
+        </joint>
+        <link name="link_0">
             <inertial>
                 <origin rpy="0 0 0"
@@ -54,8 +54,8 @@
             </collision>
         </link>
-        <joint name="${robot_name}_A1" type="revolute">
+        <joint name="A1" type="revolute">
             <origin rpy="0 0 0" xyz="0.0 0.0 0.147" />
-            <parent link="${robot_name}_link_0" />
-            <child link="${robot_name}_link_1" />
+            <parent link="link_0" />
+            <child link="link_1" />
             <axis xyz="0.0 0.0 1.0" />
             <limit effort="${effort_limit}" lower="${-joint_0_position_limit * PI / 180}"
@@ -64,5 +64,5 @@
             <dynamics damping="${joint_damping}" friction="${joint_friction}" />
         </joint>
-        <link name="${robot_name}_link_1">
+        <link name="link_1">
             <inertial>
                 <origin rpy="0 0 0"
@@ -86,8 +86,8 @@
             </collision>
         </link>
-        <joint name="${robot_name}_A2" type="revolute">
+        <joint name="A2" type="revolute">
             <origin rpy="0 0 0" xyz="0.0 -0.01 0.2125" />
-            <parent link="${robot_name}_link_1" />
-            <child link="${robot_name}_link_2" />
+            <parent link="link_1" />
+            <child link="link_2" />
             <axis xyz="0.0 1.0 0.0" />
             <limit effort="${effort_limit}" lower="${-joint_1_position_limit * PI / 180}"
@@ -96,5 +96,5 @@
             <dynamics damping="${joint_damping}" friction="${joint_friction}" />
         </joint>
-        <link name="${robot_name}_link_2">
+        <link name="link_2">
             <inertial>
                 <origin rpy="0 0 0"
@@ -118,8 +118,8 @@
             </collision>
         </link>
-        <joint name="${robot_name}_A3" type="revolute">
+        <joint name="A3" type="revolute">
             <origin rpy="0 0 0" xyz="-0.0 0.01 0.228" />
-            <parent link="${robot_name}_link_2" />
-            <child link="${robot_name}_link_3" />
+            <parent link="link_2" />
+            <child link="link_3" />
             <axis xyz="0.0 0.0 1.0" />
             <limit effort="${effort_limit}" lower="${-joint_2_position_limit * PI / 180}"
@@ -128,5 +128,5 @@
             <dynamics damping="${joint_damping}" friction="${joint_friction}" />
         </joint>
-        <link name="${robot_name}_link_3">
+        <link name="link_3">
             <inertial>
                 <origin rpy="0 0 0"
@@ -150,8 +150,8 @@
             </collision>
         </link>
-        <joint name="${robot_name}_A4" type="revolute">
+        <joint name="A4" type="revolute">
             <origin rpy="0 0 0" xyz="0.0 0.0105 0.192" />
-            <parent link="${robot_name}_link_3" />
-            <child link="${robot_name}_link_4" />
+            <parent link="link_3" />
+            <child link="link_4" />
             <axis xyz="0.0 -1.0 0.0" />
             <limit effort="${effort_limit}" lower="${-joint_3_position_limit * PI / 180}"
@@ -160,5 +160,5 @@
             <dynamics damping="${joint_damping}" friction="${joint_friction}" />
         </joint>
-        <link name="${robot_name}_link_4">
+        <link name="link_4">
             <inertial>
                 <origin rpy="0 0 0"
@@ -182,8 +182,8 @@
             </collision>
         </link>
-        <joint name="${robot_name}_A5" type="revolute">
+        <joint name="A5" type="revolute">
             <origin rpy="0 0 0" xyz="0.0 -0.0105 0.2075" />
-            <parent link="${robot_name}_link_4" />
-            <child link="${robot_name}_link_5" />
+            <parent link="link_4" />
+            <child link="link_5" />
             <axis xyz="0.0 0.0 1.0" />
             <limit effort="${effort_limit}" lower="${-joint_4_position_limit * PI / 180}"
@@ -192,5 +192,5 @@
             <dynamics damping="${joint_damping}" friction="${joint_friction}" />
         </joint>
-        <link name="${robot_name}_link_5">
+        <link name="link_5">
             <inertial>
                 <origin rpy="0 0 0"
@@ -214,8 +214,8 @@
             </collision>
         </link>
-        <joint name="${robot_name}_A6" type="revolute">
+        <joint name="A6" type="revolute">
             <origin rpy="0 0 0" xyz="0.0 -0.0707 0.1925" />
-            <parent link="${robot_name}_link_5" />
-            <child link="${robot_name}_link_6" />
+            <parent link="link_5" />
+            <child link="link_6" />
             <axis xyz="0.0 1.0 0.0" />
             <limit effort="${effort_limit}" lower="${-joint_5_position_limit * PI / 180}"
@@ -224,5 +224,5 @@
             <dynamics damping="${joint_damping}" friction="${joint_friction}" />
         </joint>
-        <link name="${robot_name}_link_6">
+        <link name="link_6">
             <inertial>
                 <origin rpy="0 0 0"
@@ -246,8 +246,8 @@
             </collision>
         </link>
-        <joint name="${robot_name}_A7" type="revolute">
+        <joint name="A7" type="revolute">
             <origin rpy="0 0 0" xyz="0.0 0.0707 0.091" />
-            <parent link="${robot_name}_link_6" />
-            <child link="${robot_name}_link_7" />
+            <parent link="link_6" />
+            <child link="link_7" />
             <axis xyz="0.0 0.0 1.0" />
             <limit effort="${effort_limit}" lower="${-joint_6_position_limit * PI / 180}"
@@ -256,5 +256,5 @@
             <dynamics damping="${joint_damping}" friction="${joint_friction}" />
         </joint>
-        <link name="${robot_name}_link_7">
+        <link name="link_7">
             <inertial>
                 <origin rpy="0 0 0"
@@ -278,10 +278,10 @@
             </collision>
         </link>
-        <joint name="${robot_name}_joint_ee" type="fixed">
-            <parent link="${robot_name}_link_7" />
-            <child link="${robot_name}_link_ee" />
+        <joint name="joint_ee" type="fixed">
+            <parent link="link_7" />
+            <child link="link_ee" />
             <origin xyz="0 0 0.035" rpy="0 0 0" />
         </joint>
-        <link name="${robot_name}_link_ee">
+        <link name="link_ee">
         </link>
         <xacro:med_gazebo robot_name="${robot_name}" />

File: lbr_description/urdf/med7/med7_description.urdf.xacro (robot description, xacro)
@@ -28,9 +28,9 @@
         <!--joint
         between {base_frame} and link_0-->
-        <joint name="${base_frame}_${robot_name}_joint" type="fixed">
+        <joint name="${base_frame}_joint" type="fixed">
             <parent link="${base_frame}" />
-            <child link="${robot_name}_link_0" />
-        </joint>
-        <link name="${robot_name}_link_0">
+            <child link="link_0" />
+        </joint>
+        <link name="link_0">
             <inertial>
                 <origin rpy="0 0 0"
@@ -54,8 +54,8 @@
             </collision>
         </link>
-        <joint name="${robot_name}_A1" type="revolute">
+        <joint name="A1" type="revolute">
             <origin rpy="0 0 0" xyz="0.0 0.0 0.1475" />
-            <parent link="${robot_name}_link_0" />
-            <child link="${robot_name}_link_1" />
+            <parent link="link_0" />
+            <child link="link_1" />
             <axis xyz="0.0 0.0 1.0" />
             <limit effort="${effort_limit}" lower="${-joint_0_position_limit * PI / 180}"
@@ -64,5 +64,5 @@
             <dynamics damping="${joint_damping}" friction="${joint_friction}" />
         </joint>
-        <link name="${robot_name}_link_1">
+        <link name="link_1">
             <inertial>
                 <origin rpy="0 0 0"
@@ -86,8 +86,8 @@
             </collision>
         </link>
-        <joint name="${robot_name}_A2" type="revolute">
+        <joint name="A2" type="revolute">
             <origin rpy="0 0 0" xyz="-0.0 -0.0105 0.1925" />
-            <parent link="${robot_name}_link_1" />
-            <child link="${robot_name}_link_2" />
+            <parent link="link_1" />
+            <child link="link_2" />
             <axis xyz="0.0 1.0 0.0" />
             <limit effort="${effort_limit}" lower="${-joint_1_position_limit * PI / 180}"
@@ -96,5 +96,5 @@
             <dynamics damping="${joint_damping}" friction="${joint_friction}" />
         </joint>
-        <link name="${robot_name}_link_2">
+        <link name="link_2">
             <inertial>
                 <origin rpy="0 0 0"
@@ -118,8 +118,8 @@
             </collision>
         </link>
-        <joint name="${robot_name}_A3" type="revolute">
+        <joint name="A3" type="revolute">
             <origin rpy="0 0 0" xyz="0.0 0.0105 0.2075" />
-            <parent link="${robot_name}_link_2" />
-            <child link="${robot_name}_link_3" />
+            <parent link="link_2" />
+            <child link="link_3" />
             <axis xyz="0.0 0.0 1.0" />
             <limit effort="${effort_limit}" lower="${-joint_2_position_limit * PI / 180}"
@@ -128,5 +128,5 @@
             <dynamics damping="${joint_damping}" friction="${joint_friction}" />
         </joint>
-        <link name="${robot_name}_link_3">
+        <link name="link_3">
             <inertial>
                 <origin rpy="0 0 0"
@@ -150,8 +150,8 @@
             </collision>
         </link>
-        <joint name="${robot_name}_A4" type="revolute">
+        <joint name="A4" type="revolute">
             <origin rpy="0 0 0" xyz="0.0 0.0105 0.1925" />
-            <parent link="${robot_name}_link_3" />
-            <child link="${robot_name}_link_4" />
+            <parent link="link_3" />
+            <child link="link_4" />
             <axis xyz="0.0 -1.0 0.0" />
             <limit effort="${effort_limit}" lower="${-joint_3_position_limit * PI / 180}"
@@ -160,5 +160,5 @@
             <dynamics damping="${joint_damping}" friction="${joint_friction}" />
         </joint>
-        <link name="${robot_name}_link_4">
+        <link name="link_4">
             <inertial>
                 <origin rpy="0 0 0"
@@ -182,8 +182,8 @@
             </collision>
         </link>
-        <joint name="${robot_name}_A5" type="revolute">
+        <joint name="A5" type="revolute">
             <origin rpy="0 0 0" xyz="-0.0 -0.0105 0.2075" />
-            <parent link="${robot_name}_link_4" />
-            <child link="${robot_name}_link_5" />
+            <parent link="link_4" />
+            <child link="link_5" />
             <axis xyz="0.0 0.0 1.0" />
             <limit effort="${effort_limit}" lower="${-joint_4_position_limit * PI / 180}"
@@ -192,5 +192,5 @@
             <dynamics damping="${joint_damping}" friction="${joint_friction}" />
         </joint>
-        <link name="${robot_name}_link_5">
+        <link name="link_5">
             <inertial>
                 <origin rpy="0 0 0"
@@ -214,8 +214,8 @@
             </collision>
         </link>
-        <joint name="${robot_name}_A6" type="revolute">
+        <joint name="A6" type="revolute">
             <origin rpy="0 0 0" xyz="0.0 -0.0707 0.1925" />
-            <parent link="${robot_name}_link_5" />
-            <child link="${robot_name}_link_6" />
+            <parent link="link_5" />
+            <child link="link_6" />
             <axis xyz="0.0 1.0 0.0" />
             <limit effort="${effort_limit}" lower="${-joint_5_position_limit * PI / 180}"
@@ -224,5 +224,5 @@
             <dynamics damping="${joint_damping}" friction="${joint_friction}" />
         </joint>
-        <link name="${robot_name}_link_6">
+        <link name="link_6">
             <inertial>
                 <origin rpy="0 0 0"
@@ -246,8 +246,8 @@
             </collision>
         </link>
-        <joint name="${robot_name}_A7" type="revolute">
+        <joint name="A7" type="revolute">
             <origin rpy="0 0 0" xyz="0.0 0.0707 0.091" />
-            <parent link="${robot_name}_link_6" />
-            <child link="${robot_name}_link_7" />
+            <parent link="link_6" />
+            <child link="link_7" />
             <axis xyz="0.0 0.0 1.0" />
             <limit effort="${effort_limit}" lower="${-joint_6_position_limit * PI / 180}"
@@ -256,5 +256,5 @@
             <dynamics damping="${joint_damping}" friction="${joint_friction}" />
         </joint>
-        <link name="${robot_name}_link_7">
+        <link name="link_7">
             <inertial>
                 <origin rpy="0 0 0"
@@ -278,10 +278,10 @@
             </collision>
         </link>
-        <joint name="${robot_name}_joint_ee" type="fixed">
-            <parent link="${robot_name}_link_7" />
-            <child link="${robot_name}_link_ee" />
+        <joint name="joint_ee" type="fixed">
+            <parent link="link_7" />
+            <child link="link_ee" />
             <origin xyz="0 0 0.035" rpy="0 0 0" />
         </joint>
-        <link name="${robot_name}_link_ee">
+        <link name="link_ee">
         </link>
         <xacro:med_gazebo robot_name="${robot_name}" />
