Commit message: stl -> dae

File: lbr_description/gazebo/iiwa.gazebo.xacro (robot description, xacro)
@@ -13,5 +13,4 @@
             <mu1>0.2</mu1>
             <mu2>0.2</mu2>
-            <material>Gazebo/Grey</material>
         </gazebo>
         <!-- link 1 -->
@@ -19,5 +18,4 @@
             <mu1>0.2</mu1>
             <mu2>0.2</mu2>
-            <material>Gazebo/Orange</material>
         </gazebo>
         <!-- link 2 -->
@@ -25,5 +23,4 @@
             <mu1>0.2</mu1>
             <mu2>0.2</mu2>
-            <material>Gazebo/Orange</material>
         </gazebo>
         <!-- link 3 -->
@@ -31,5 +28,4 @@
             <mu1>0.2</mu1>
             <mu2>0.2</mu2>
-            <material>Gazebo/Orange</material>
         </gazebo>
         <!-- link 4 -->
@@ -37,5 +33,4 @@
             <mu1>0.2</mu1>
             <mu2>0.2</mu2>
-            <material>Gazebo/Orange</material>
         </gazebo>
         <!-- link 5 -->
@@ -43,5 +38,4 @@
             <mu1>0.2</mu1>
             <mu2>0.2</mu2>
-            <material>Gazebo/Orange</material>
         </gazebo>
         <!-- link 6 -->
@@ -49,5 +43,4 @@
             <mu1>0.2</mu1>
             <mu2>0.2</mu2>
-            <material>Gazebo/Orange</material>
         </gazebo>
         <!-- link 7 -->
@@ -55,5 +48,4 @@
             <mu1>0.2</mu1>
             <mu2>0.2</mu2>
-            <material>Gazebo/Grey</material>
         </gazebo>
     </xacro:macro>

File: lbr_description/gazebo/med.gazebo.xacro (robot description, xacro)
@@ -13,5 +13,4 @@
             <mu1>0.2</mu1>
             <mu2>0.2</mu2>
-            <material>Gazebo/White</material>
         </gazebo>
         <!-- link 1 -->
@@ -19,5 +18,4 @@
             <mu1>0.2</mu1>
             <mu2>0.2</mu2>
-            <material>Gazebo/White</material>
         </gazebo>
         <!-- link 2 -->
@@ -25,5 +23,4 @@
             <mu1>0.2</mu1>
             <mu2>0.2</mu2>
-            <material>Gazebo/White</material>
         </gazebo>
         <!-- link 3 -->
@@ -31,5 +28,4 @@
             <mu1>0.2</mu1>
             <mu2>0.2</mu2>
-            <material>Gazebo/White</material>
         </gazebo>
         <!-- link 4 -->
@@ -37,5 +33,4 @@
             <mu1>0.2</mu1>
             <mu2>0.2</mu2>
-            <material>Gazebo/White</material>
         </gazebo>
         <!-- link 5 -->
@@ -43,5 +38,4 @@
             <mu1>0.2</mu1>
             <mu2>0.2</mu2>
-            <material>Gazebo/White</material>
         </gazebo>
         <!-- link 6 -->
@@ -49,5 +43,4 @@
             <mu1>0.2</mu1>
             <mu2>0.2</mu2>
-            <material>Gazebo/White</material>
         </gazebo>
         <!-- link 7 -->
@@ -55,5 +48,4 @@
             <mu1>0.2</mu1>
             <mu2>0.2</mu2>
-            <material>Gazebo/Grey</material>
         </gazebo>
     </xacro:macro>

File: lbr_description/urdf/iiwa14/iiwa14_description.urdf.xacro (robot description, xacro)
@@ -43,5 +43,5 @@
                 <origin rpy="0 0 0" xyz="0 0 0" />
                 <geometry>
-                    <mesh filename="package://lbr_description/meshes/iiwa14/visual/link_0.stl" />
+                    <mesh filename="package://lbr_description/meshes/iiwa14/visual/link_0.dae" />
                 </geometry>
                 <material name="silver" />
@@ -75,5 +75,5 @@
                 <origin rpy="0 0 0" xyz="-0.0 0.0 -0.1475" />
                 <geometry>
-                    <mesh filename="package://lbr_description/meshes/iiwa14/visual/link_1.stl" />
+                    <mesh filename="package://lbr_description/meshes/iiwa14/visual/link_1.dae" />
                 </geometry>
                 <material name="orange" />
@@ -107,5 +107,5 @@
                 <origin rpy="0 0 0" xyz="-0.0 0.01 -0.36" />
                 <geometry>
-                    <mesh filename="package://lbr_description/meshes/iiwa14/visual/link_2.stl" />
+                    <mesh filename="package://lbr_description/meshes/iiwa14/visual/link_2.dae" />
                 </geometry>
                 <material name="orange" />
@@ -139,5 +139,5 @@
                 <origin rpy="0 0 0" xyz="-0.0 0.0 -0.5545" />
                 <geometry>
-                    <mesh filename="package://lbr_description/meshes/iiwa14/visual/link_3.stl" />
+                    <mesh filename="package://lbr_description/meshes/iiwa14/visual/link_3.dae" />
                 </geometry>
                 <material name="orange" />
@@ -171,5 +171,5 @@
                 <origin rpy="0 0 0" xyz="0.0 -0.0105 -0.78" />
                 <geometry>
-                    <mesh filename="package://lbr_description/meshes/iiwa14/visual/link_4.stl" />
+                    <mesh filename="package://lbr_description/meshes/iiwa14/visual/link_4.dae" />
                 </geometry>
                 <material name="orange" />
@@ -203,5 +203,5 @@
                 <origin rpy="0 0 0" xyz="-0.0 0.0 -0.9545" />
                 <geometry>
-                    <mesh filename="package://lbr_description/meshes/iiwa14/visual/link_5.stl" />
+                    <mesh filename="package://lbr_description/meshes/iiwa14/visual/link_5.dae" />
                 </geometry>
                 <material name="orange" />
@@ -235,5 +235,5 @@
                 <origin rpy="0 0 0" xyz="0.0 0.0707 -1.18" />
                 <geometry>
-                    <mesh filename="package://lbr_description/meshes/iiwa14/visual/link_6.stl" />
+                    <mesh filename="package://lbr_description/meshes/iiwa14/visual/link_6.dae" />
                 </geometry>
                 <material name="orange" />
@@ -267,5 +267,5 @@
                 <origin rpy="0 0 0" xyz="0.0 0.0 -1.2511" />
                 <geometry>
-                    <mesh filename="package://lbr_description/meshes/iiwa14/visual/link_7.stl" />
+                    <mesh filename="package://lbr_description/meshes/iiwa14/visual/link_7.dae" />
                 </geometry>
                 <material name="silver" />

File: lbr_description/urdf/iiwa7/iiwa7_description.urdf.xacro (robot description, xacro)
@@ -43,5 +43,5 @@
                 <origin rpy="0 0 0" xyz="0 0 0" />
                 <geometry>
-                    <mesh filename="package://lbr_description/meshes/iiwa7/visual/link_0.stl" />
+                    <mesh filename="package://lbr_description/meshes/iiwa7/visual/link_0.dae" />
                 </geometry>
                 <material name="silver" />
@@ -75,5 +75,5 @@
                 <origin rpy="0 0 0" xyz="-0.0 0.0 -0.1475" />
                 <geometry>
-                    <mesh filename="package://lbr_description/meshes/iiwa7/visual/link_1.stl" />
+                    <mesh filename="package://lbr_description/meshes/iiwa7/visual/link_1.dae" />
                 </geometry>
                 <material name="orange" />
@@ -107,5 +107,5 @@
                 <origin rpy="0 0 0" xyz="0.0 0.0105 -0.3405" />
                 <geometry>
-                    <mesh filename="package://lbr_description/meshes/iiwa7/visual/link_2.stl" />
+                    <mesh filename="package://lbr_description/meshes/iiwa7/visual/link_2.dae" />
                 </geometry>
                 <material name="orange" />
@@ -139,5 +139,5 @@
                 <origin rpy="0 0 0" xyz="0.0 0.0 -0.515" />
                 <geometry>
-                    <mesh filename="package://lbr_description/meshes/iiwa7/visual/link_3.stl" />
+                    <mesh filename="package://lbr_description/meshes/iiwa7/visual/link_3.dae" />
                 </geometry>
                 <material name="orange" />
@@ -171,5 +171,5 @@
                 <origin rpy="0 0 0" xyz="0.0 -0.0105 -0.7405" />
                 <geometry>
-                    <mesh filename="package://lbr_description/meshes/iiwa7/visual/link_4.stl" />
+                    <mesh filename="package://lbr_description/meshes/iiwa7/visual/link_4.dae" />
                 </geometry>
                 <material name="orange" />
@@ -203,5 +203,5 @@
                 <origin rpy="0 0 0" xyz="0.0 0.0 -0.915" />
                 <geometry>
-                    <mesh filename="package://lbr_description/meshes/iiwa7/visual/link_5.stl" />
+                    <mesh filename="package://lbr_description/meshes/iiwa7/visual/link_5.dae" />
                 </geometry>
                 <material name="orange" />
@@ -235,5 +235,5 @@
                 <origin rpy="0 0 0" xyz="0.0 0.0707 -1.1405" />
                 <geometry>
-                    <mesh filename="package://lbr_description/meshes/iiwa7/visual/link_6.stl" />
+                    <mesh filename="package://lbr_description/meshes/iiwa7/visual/link_6.dae" />
                 </geometry>
                 <material name="orange" />
@@ -267,5 +267,5 @@
                 <origin rpy="0 0 0" xyz="0.0 0.0002 -1.2314" />
                 <geometry>
-                    <mesh filename="package://lbr_description/meshes/iiwa7/visual/link_7.stl" />
+                    <mesh filename="package://lbr_description/meshes/iiwa7/visual/link_7.dae" />
                 </geometry>
                 <material name="silver" />

File: lbr_description/urdf/med14/med14_description.urdf.xacro (robot description, xacro)
@@ -43,5 +43,5 @@
                 <origin rpy="0 0 0" xyz="0 0 0" />
                 <geometry>
-                    <mesh filename="package://lbr_description/meshes/med14/visual/link_0.stl" />
+                    <mesh filename="package://lbr_description/meshes/med14/visual/link_0.dae" />
                 </geometry>
                 <material name="white" />
@@ -75,5 +75,5 @@
                 <origin rpy="0 0 0" xyz="-0.0 -0.0 -0.147" />
                 <geometry>
-                    <mesh filename="package://lbr_description/meshes/med14/visual/link_1.stl" />
+                    <mesh filename="package://lbr_description/meshes/med14/visual/link_1.dae" />
                 </geometry>
                 <material name="white" />
@@ -107,5 +107,5 @@
                 <origin rpy="0 0 0" xyz="-0.0 0.01 -0.3595" />
                 <geometry>
-                    <mesh filename="package://lbr_description/meshes/med14/visual/link_2.stl" />
+                    <mesh filename="package://lbr_description/meshes/med14/visual/link_2.dae" />
                 </geometry>
                 <material name="white" />
@@ -139,5 +139,5 @@
                 <origin rpy="0 0 0" xyz="0.0 -0.0 -0.5875" />
                 <geometry>
-                    <mesh filename="package://lbr_description/meshes/med14/visual/link_3.stl" />
+                    <mesh filename="package://lbr_description/meshes/med14/visual/link_3.dae" />
                 </geometry>
                 <material name="white" />
@@ -171,5 +171,5 @@
                 <origin rpy="0 0 0" xyz="0.0 -0.0105 -0.7795" />
                 <geometry>
-                    <mesh filename="package://lbr_description/meshes/med14/visual/link_4.stl" />
+                    <mesh filename="package://lbr_description/meshes/med14/visual/link_4.dae" />
                 </geometry>
                 <material name="white" />
@@ -203,5 +203,5 @@
                 <origin rpy="0 0 0" xyz="-0.0 0.0 -0.987" />
                 <geometry>
-                    <mesh filename="package://lbr_description/meshes/med14/visual/link_5.stl" />
+                    <mesh filename="package://lbr_description/meshes/med14/visual/link_5.dae" />
                 </geometry>
                 <material name="white" />
@@ -235,5 +235,5 @@
                 <origin rpy="0 0 0" xyz="-0.0 0.0707 -1.1795" />
                 <geometry>
-                    <mesh filename="package://lbr_description/meshes/med14/visual/link_6.stl" />
+                    <mesh filename="package://lbr_description/meshes/med14/visual/link_6.dae" />
                 </geometry>
                 <material name="white" />
@@ -267,5 +267,5 @@
                 <origin rpy="0 0 0" xyz="-0.0 -0.0 -1.2705" />
                 <geometry>
-                    <mesh filename="package://lbr_description/meshes/med14/visual/link_7.stl" />
+                    <mesh filename="package://lbr_description/meshes/med14/visual/link_7.dae" />
                 </geometry>
                 <material name="silver" />

File: lbr_description/urdf/med7/med7_description.urdf.xacro (robot description, xacro)
@@ -43,5 +43,5 @@
                 <origin rpy="0 0 0" xyz="0 0 0" />
                 <geometry>
-                    <mesh filename="package://lbr_description/meshes/med7/visual/link_0.stl" />
+                    <mesh filename="package://lbr_description/meshes/med7/visual/link_0.dae" />
                 </geometry>
                 <material name="white" />
@@ -75,5 +75,5 @@
                 <origin rpy="0 0 0" xyz="-0.0 0.0 -0.1475" />
                 <geometry>
-                    <mesh filename="package://lbr_description/meshes/med7/visual/link_1.stl" />
+                    <mesh filename="package://lbr_description/meshes/med7/visual/link_1.dae" />
                 </geometry>
                 <material name="white" />
@@ -107,5 +107,5 @@
                 <origin rpy="0 0 0" xyz="0.0 0.0105 -0.34" />
                 <geometry>
-                    <mesh filename="package://lbr_description/meshes/med7/visual/link_2.stl" />
+                    <mesh filename="package://lbr_description/meshes/med7/visual/link_2.dae" />
                 </geometry>
                 <material name="white" />
@@ -139,5 +139,5 @@
                 <origin rpy="0 0 0" xyz="0.0 -0.0 -0.5475" />
                 <geometry>
-                    <mesh filename="package://lbr_description/meshes/med7/visual/link_3.stl" />
+                    <mesh filename="package://lbr_description/meshes/med7/visual/link_3.dae" />
                 </geometry>
                 <material name="white" />
@@ -171,5 +171,5 @@
                 <origin rpy="0 0 0" xyz="-0.0 -0.0105 -0.74" />
                 <geometry>
-                    <mesh filename="package://lbr_description/meshes/med7/visual/link_4.stl" />
+                    <mesh filename="package://lbr_description/meshes/med7/visual/link_4.dae" />
                 </geometry>
                 <material name="white" />
@@ -203,5 +203,5 @@
                 <origin rpy="0 0 0" xyz="0.0 0.0 -0.9475" />
                 <geometry>
-                    <mesh filename="package://lbr_description/meshes/med7/visual/link_5.stl" />
+                    <mesh filename="package://lbr_description/meshes/med7/visual/link_5.dae" />
                 </geometry>
                 <material name="white" />
@@ -235,5 +235,5 @@
                 <origin rpy="0 0 0" xyz="0.0 0.0707 -1.14" />
                 <geometry>
-                    <mesh filename="package://lbr_description/meshes/med7/visual/link_6.stl" />
+                    <mesh filename="package://lbr_description/meshes/med7/visual/link_6.dae" />
                 </geometry>
                 <material name="white" />
@@ -267,5 +267,5 @@
                 <origin rpy="0 0 0" xyz="-0.0 -0.0 -1.231" />
                 <geometry>
-                    <mesh filename="package://lbr_description/meshes/med7/visual/link_7.stl" />
+                    <mesh filename="package://lbr_description/meshes/med7/visual/link_7.dae" />
                 </geometry>
                 <material name="silver" />
