Commit message: merged gazebo

File: lbr_description/gazebo/lbr.gazebo.xacro (robot description, xacro)
@@ -1,5 +1,5 @@
 <?xml version="1.0"?>
 <robot xmlns:xacro="http://www.ros.org/wiki/xacro">
-    <xacro:macro name="iiwa_gazebo" params="robot_name:=^|lbr">
+    <xacro:macro name="lbr_gazebo" params="robot_name:=^|lbr">
         <!-- ros_control-plugin -->
         <gazebo>
@@ -14,8 +14,18 @@
             <mu2>0.2</mu2>
         </gazebo>
+        <!-- A1 -->
+        <gazebo reference="A1">
+            <implicitSpringDamper>true</implicitSpringDamper>
+            <provideFeedback>true</provideFeedback>
+        </gazebo>
         <!-- link 1 -->
         <gazebo reference="link_1">
             <mu1>0.2</mu1>
             <mu2>0.2</mu2>
+        </gazebo>
+        <!-- A2 -->
+        <gazebo reference="A2">
+            <implicitSpringDamper>true</implicitSpringDamper>
+            <provideFeedback>true</provideFeedback>
         </gazebo>
         <!-- link 2 -->
@@ -24,8 +34,18 @@
             <mu2>0.2</mu2>
         </gazebo>
+        <!-- A3 -->
+        <gazebo reference="A3">
+            <implicitSpringDamper>true</implicitSpringDamper>
+            <provideFeedback>true</provideFeedback>
+        </gazebo>
         <!-- link 3 -->
         <gazebo reference="link_3">
             <mu1>0.2</mu1>
             <mu2>0.2</mu2>
+        </gazebo>
+        <!-- A4 -->
+        <gazebo reference="A4">
+            <implicitSpringDamper>true</implicitSpringDamper>
+            <provideFeedback>true</provideFeedback>
         </gazebo>
         <!-- link 4 -->
@@ -34,4 +54,9 @@
             <mu2>0.2</mu2>
         </gazebo>
+        <!-- A5 -->
+        <gazebo reference="A5">
+            <implicitSpringDamper>true</implicitSpringDamper>
+            <provideFeedback>true</provideFeedback>
+        </gazebo>
         <!-- link 5 -->
         <gazebo reference="link_5">
@@ -39,8 +64,18 @@
             <mu2>0.2</mu2>
         </gazebo>
+        <!-- A6 -->
+        <gazebo reference="A6">
+            <implicitSpringDamper>true</implicitSpringDamper>
+            <provideFeedback>true</provideFeedback>
+        </gazebo>
         <!-- link 6 -->
         <gazebo reference="link_6">
             <mu1>0.2</mu1>
             <mu2>0.2</mu2>
+        </gazebo>
+        <!-- A7 -->
+        <gazebo reference="A7">
+            <implicitSpringDamper>true</implicitSpringDamper>
+            <provideFeedback>true</provideFeedback>
         </gazebo>
         <!-- link 7 -->

File: lbr_description/urdf/iiwa14/iiwa14_description.urdf.xacro (robot description, xacro)
@@ -285,5 +285,5 @@
         <link name="link_ee">
         </link>
-        <xacro:iiwa_gazebo robot_name="${robot_name}" />
+        <xacro:lbr_gazebo robot_name="${robot_name}" />
         <!-- TODO: move modes to args, decouple urdf/gazebo/controls -->
         <xacro:lbr_hardware_interface

File: lbr_description/urdf/iiwa7/iiwa7_description.urdf.xacro (robot description, xacro)
@@ -285,5 +285,5 @@
         <link name="link_ee">
         </link>
-        <xacro:iiwa_gazebo robot_name="${robot_name}" />
+        <xacro:lbr_gazebo robot_name="${robot_name}" />
         <!-- TODO: move modes to args, decouple urdf/gazebo/controls -->
         <xacro:lbr_hardware_interface

File: lbr_description/urdf/med14/med14_description.urdf.xacro (robot description, xacro)
@@ -285,5 +285,5 @@
         <link name="link_ee">
         </link>
-        <xacro:med_gazebo robot_name="${robot_name}" />
+        <xacro:lbr_gazebo robot_name="${robot_name}" />
         <!-- TODO: move modes to args, decouple urdf/gazebo/controls -->
         <xacro:lbr_hardware_interface

File: lbr_description/urdf/med7/med7_description.urdf.xacro (robot description, xacro)
@@ -285,5 +285,5 @@
         <link name="link_ee">
         </link>
-        <xacro:med_gazebo robot_name="${robot_name}" />
+        <xacro:lbr_gazebo robot_name="${robot_name}" />
         <!-- TODO: move modes to args, decouple urdf/gazebo/controls -->
         <xacro:lbr_hardware_interface

Commit message: merged gazebo

File: lbr_description/gazebo/lbr.gazebo.xacro (robot description, xacro)
@@ -1,5 +1,5 @@
 <?xml version="1.0"?>
 <robot xmlns:xacro="http://www.ros.org/wiki/xacro">
-    <xacro:macro name="med_gazebo" params="robot_name:=^|lbr">
+    <xacro:macro name="lbr_gazebo" params="robot_name:=^|lbr">
         <!-- ros_control-plugin -->
         <gazebo>
@@ -13,5 +13,9 @@
             <mu1>0.2</mu1>
             <mu2>0.2</mu2>
-            <material>Gazebo/White</material>
+        </gazebo>
+        <!-- A1 -->
+        <gazebo reference="A1">
+            <implicitSpringDamper>true</implicitSpringDamper>
+            <provideFeedback>true</provideFeedback>
         </gazebo>
         <!-- link 1 -->
@@ -19,5 +23,9 @@
             <mu1>0.2</mu1>
             <mu2>0.2</mu2>
-            <material>Gazebo/White</material>
+        </gazebo>
+        <!-- A2 -->
+        <gazebo reference="A2">
+            <implicitSpringDamper>true</implicitSpringDamper>
+            <provideFeedback>true</provideFeedback>
         </gazebo>
         <!-- link 2 -->
@@ -25,5 +33,9 @@
             <mu1>0.2</mu1>
             <mu2>0.2</mu2>
-            <material>Gazebo/White</material>
+        </gazebo>
+        <!-- A3 -->
+        <gazebo reference="A3">
+            <implicitSpringDamper>true</implicitSpringDamper>
+            <provideFeedback>true</provideFeedback>
         </gazebo>
         <!-- link 3 -->
@@ -31,5 +43,9 @@
             <mu1>0.2</mu1>
             <mu2>0.2</mu2>
-            <material>Gazebo/White</material>
+        </gazebo>
+        <!-- A4 -->
+        <gazebo reference="A4">
+            <implicitSpringDamper>true</implicitSpringDamper>
+            <provideFeedback>true</provideFeedback>
         </gazebo>
         <!-- link 4 -->
@@ -37,5 +53,9 @@
             <mu1>0.2</mu1>
             <mu2>0.2</mu2>
-            <material>Gazebo/White</material>
+        </gazebo>
+        <!-- A5 -->
+        <gazebo reference="A5">
+            <implicitSpringDamper>true</implicitSpringDamper>
+            <provideFeedback>true</provideFeedback>
         </gazebo>
         <!-- link 5 -->
@@ -43,5 +63,9 @@
             <mu1>0.2</mu1>
             <mu2>0.2</mu2>
-            <material>Gazebo/White</material>
+        </gazebo>
+        <!-- A6 -->
+        <gazebo reference="A6">
+            <implicitSpringDamper>true</implicitSpringDamper>
+            <provideFeedback>true</provideFeedback>
         </gazebo>
         <!-- link 6 -->
@@ -49,5 +73,9 @@
             <mu1>0.2</mu1>
             <mu2>0.2</mu2>
-            <material>Gazebo/White</material>
+        </gazebo>
+        <!-- A7 -->
+        <gazebo reference="A7">
+            <implicitSpringDamper>true</implicitSpringDamper>
+            <provideFeedback>true</provideFeedback>
         </gazebo>
         <!-- link 7 -->
@@ -55,5 +83,4 @@
             <mu1>0.2</mu1>
             <mu2>0.2</mu2>
-            <material>Gazebo/Grey</material>
         </gazebo>
     </xacro:macro>

File: lbr_description/urdf/iiwa14/iiwa14_description.urdf.xacro (robot description, xacro)
@@ -22,5 +22,5 @@
     <!-- includes -->
     <xacro:include filename="$(find lbr_description)/urdf/materials.urdf.xacro" />
-    <xacro:include filename="$(find lbr_description)/gazebo/iiwa.gazebo.xacro" />
+    <xacro:include filename="$(find lbr_description)/gazebo/lbr.gazebo.xacro" />
     <xacro:include filename="$(find lbr_description)/ros2_control/lbr.ros2_control.xacro" />
     <!-- robot as extracted via https://github.com/syuntoku14/fusion2urdf -->
@@ -285,5 +285,5 @@
         <link name="link_ee">
         </link>
-        <xacro:iiwa_gazebo robot_name="${robot_name}" />
+        <xacro:lbr_gazebo robot_name="${robot_name}" />
         <!-- TODO: move modes to args, decouple urdf/gazebo/controls -->
         <xacro:lbr_hardware_interface

File: lbr_description/urdf/iiwa7/iiwa7_description.urdf.xacro (robot description, xacro)
@@ -22,5 +22,5 @@
     <!-- includes -->
     <xacro:include filename="$(find lbr_description)/urdf/materials.urdf.xacro" />
-    <xacro:include filename="$(find lbr_description)/gazebo/iiwa.gazebo.xacro" />
+    <xacro:include filename="$(find lbr_description)/gazebo/lbr.gazebo.xacro" />
     <xacro:include filename="$(find lbr_description)/ros2_control/lbr.ros2_control.xacro" />
     <!-- robot as extracted via https://github.com/syuntoku14/fusion2urdf -->
@@ -285,5 +285,5 @@
         <link name="link_ee">
         </link>
-        <xacro:iiwa_gazebo robot_name="${robot_name}" />
+        <xacro:lbr_gazebo robot_name="${robot_name}" />
         <!-- TODO: move modes to args, decouple urdf/gazebo/controls -->
         <xacro:lbr_hardware_interface

File: lbr_description/urdf/med14/med14_description.urdf.xacro (robot description, xacro)
@@ -22,5 +22,5 @@
     <!-- includes -->
     <xacro:include filename="$(find lbr_description)/urdf/materials.urdf.xacro" />
-    <xacro:include filename="$(find lbr_description)/gazebo/med.gazebo.xacro" />
+    <xacro:include filename="$(find lbr_description)/gazebo/lbr.gazebo.xacro" />
     <xacro:include filename="$(find lbr_description)/ros2_control/lbr.ros2_control.xacro" />
     <!-- robot as extracted via https://github.com/syuntoku14/fusion2urdf -->
@@ -285,5 +285,5 @@
         <link name="link_ee">
         </link>
-        <xacro:med_gazebo robot_name="${robot_name}" />
+        <xacro:lbr_gazebo robot_name="${robot_name}" />
         <!-- TODO: move modes to args, decouple urdf/gazebo/controls -->
         <xacro:lbr_hardware_interface

File: lbr_description/urdf/med7/med7_description.urdf.xacro (robot description, xacro)
@@ -22,5 +22,5 @@
     <!-- includes -->
     <xacro:include filename="$(find lbr_description)/urdf/materials.urdf.xacro" />
-    <xacro:include filename="$(find lbr_description)/gazebo/med.gazebo.xacro" />
+    <xacro:include filename="$(find lbr_description)/gazebo/lbr.gazebo.xacro" />
     <xacro:include filename="$(find lbr_description)/ros2_control/lbr.ros2_control.xacro" />
     <!-- robot as extracted via https://github.com/syuntoku14/fusion2urdf -->
@@ -285,5 +285,5 @@
         <link name="link_ee">
         </link>
-        <xacro:med_gazebo robot_name="${robot_name}" />
+        <xacro:lbr_gazebo robot_name="${robot_name}" />
         <!-- TODO: move modes to args, decouple urdf/gazebo/controls -->
         <xacro:lbr_hardware_interface

Commit message: simplified gazebo xacro

File: lbr_description/gazebo/lbr.gazebo.xacro (robot description, xacro)
@@ -1,87 +1,41 @@
 <?xml version="1.0"?>
 <robot xmlns:xacro="http://www.ros.org/wiki/xacro">
-    <xacro:macro name="lbr_gazebo" params="robot_name:=^|lbr">
+    <xacro:macro name="lbr_gazebo">
         <!-- ros_control-plugin -->
         <gazebo>
-            <plugin name="ign_ros2_control::IgnitionROS2ControlPlugin" filename="ign_ros2_control-system">
+            <plugin name="ign_ros2_control::IgnitionROS2ControlPlugin"
+                filename="ign_ros2_control-system">
                 <parameters>$(find lbr_hardware_interface)/config/lbr_controllers.yml</parameters>
-                <robotNamespace>/${robot_name}</robotNamespace>
             </plugin>
         </gazebo>
-        <!-- link 0 -->
-        <gazebo reference="link_0">
-            <mu1>0.2</mu1>
-            <mu2>0.2</mu2>
-        </gazebo>
-        <!-- A1 -->
-        <gazebo reference="A1">
-            <implicitSpringDamper>true</implicitSpringDamper>
-            <provideFeedback>true</provideFeedback>
-        </gazebo>
-        <!-- link 1 -->
-        <gazebo reference="link_1">
-            <mu1>0.2</mu1>
-            <mu2>0.2</mu2>
-        </gazebo>
-        <!-- A2 -->
-        <gazebo reference="A2">
-            <implicitSpringDamper>true</implicitSpringDamper>
-            <provideFeedback>true</provideFeedback>
-        </gazebo>
-        <!-- link 2 -->
-        <gazebo reference="link_2">
-            <mu1>0.2</mu1>
-            <mu2>0.2</mu2>
-        </gazebo>
-        <!-- A3 -->
-        <gazebo reference="A3">
-            <implicitSpringDamper>true</implicitSpringDamper>
-            <provideFeedback>true</provideFeedback>
-        </gazebo>
-        <!-- link 3 -->
-        <gazebo reference="link_3">
-            <mu1>0.2</mu1>
-            <mu2>0.2</mu2>
-        </gazebo>
-        <!-- A4 -->
-        <gazebo reference="A4">
-            <implicitSpringDamper>true</implicitSpringDamper>
-            <provideFeedback>true</provideFeedback>
-        </gazebo>
-        <!-- link 4 -->
-        <gazebo reference="link_4">
-            <mu1>0.2</mu1>
-            <mu2>0.2</mu2>
-        </gazebo>
-        <!-- A5 -->
-        <gazebo reference="A5">
-            <implicitSpringDamper>true</implicitSpringDamper>
-            <provideFeedback>true</provideFeedback>
-        </gazebo>
-        <!-- link 5 -->
-        <gazebo reference="link_5">
-            <mu1>0.2</mu1>
-            <mu2>0.2</mu2>
-        </gazebo>
-        <!-- A6 -->
-        <gazebo reference="A6">
-            <implicitSpringDamper>true</implicitSpringDamper>
-            <provideFeedback>true</provideFeedback>
-        </gazebo>
-        <!-- link 6 -->
-        <gazebo reference="link_6">
-            <mu1>0.2</mu1>
-            <mu2>0.2</mu2>
-        </gazebo>
-        <!-- A7 -->
-        <gazebo reference="A7">
-            <implicitSpringDamper>true</implicitSpringDamper>
-            <provideFeedback>true</provideFeedback>
-        </gazebo>
-        <!-- link 7 -->
-        <gazebo reference="link_7">
-            <mu1>0.2</mu1>
-            <mu2>0.2</mu2>
-        </gazebo>
+        <!-- macros -->
+        <xacro:macro name="gazebo_link_reference" params="name">
+            <gazebo reference="${name}">
+                <mu1>0.2</mu1>
+                <mu2>0.2</mu2>
+            </gazebo>
+        </xacro:macro>
+        <xacro:macro name="gazebo_joint_reference" params="name">
+            <gazebo reference="${name}">
+                <implicitSpringDamper>true</implicitSpringDamper>
+                <provideFeedback>true</provideFeedback>
+            </gazebo>
+        </xacro:macro>
+        <!-- references -->
+        <xacro:gazebo_link_reference name="link_0" />
+        <xacro:gazebo_joint_reference name="A1" />
+        <xacro:gazebo_link_reference name="link_1" />
+        <xacro:gazebo_joint_reference name="A2" />
+        <xacro:gazebo_link_reference name="link_2" />
+        <xacro:gazebo_joint_reference name="A3" />
+        <xacro:gazebo_link_reference name="link_3" />
+        <xacro:gazebo_joint_reference name="A4" />
+        <xacro:gazebo_link_reference name="link_4" />
+        <xacro:gazebo_joint_reference name="A5" />
+        <xacro:gazebo_link_reference name="link_5" />
+        <xacro:gazebo_joint_reference name="A6" />
+        <xacro:gazebo_link_reference name="link_6" />
+        <xacro:gazebo_joint_reference name="A7" />
+        <xacro:gazebo_link_reference name="link_7" />
     </xacro:macro>
 </robot>
