Commit message: cleaned xacro files

File: lbr_description/gazebo/lbr.gazebo.xacro (robot description, xacro)
@@ -9,79 +9,33 @@
             </plugin>
         </gazebo>
-        <!-- link 0 -->
-        <gazebo reference="link_0">
-            <mu1>0.2</mu1>
-            <mu2>0.2</mu2>
-        </gazebo>
-        <!-- A1 -->
-        <gazebo reference="A1">
-            <implicitSpringDamper>true</implicitSpringDamper>
-            <provideFeedback>true</provideFeedback>
-        </gazebo>
-        <!-- link 1 -->
-        <gazebo reference="link_1">
-            <mu1>0.2</mu1>
-            <mu2>0.2</mu2>
-        </gazebo>
-        <!-- A2 -->
-        <gazebo reference="A2">
-            <implicitSpringDamper>true</implicitSpringDamper>
-            <provideFeedback>true</provideFeedback>
-        </gazebo>
-        <!-- link 2 -->
-        <gazebo reference="link_2">
-            <mu1>0.2</mu1>
-            <mu2>0.2</mu2>
-        </gazebo>
-        <!-- A3 -->
-        <gazebo reference="A3">
-            <implicitSpringDamper>true</implicitSpringDamper>
-            <provideFeedback>true</provideFeedback>
-        </gazebo>
-        <!-- link 3 -->
-        <gazebo reference="link_3">
-            <mu1>0.2</mu1>
-            <mu2>0.2</mu2>
-        </gazebo>
-        <!-- A4 -->
-        <gazebo reference="A4">
-            <implicitSpringDamper>true</implicitSpringDamper>
-            <provideFeedback>true</provideFeedback>
-        </gazebo>
-        <!-- link 4 -->
-        <gazebo reference="link_4">
-            <mu1>0.2</mu1>
-            <mu2>0.2</mu2>
-        </gazebo>
-        <!-- A5 -->
-        <gazebo reference="A5">
-            <implicitSpringDamper>true</implicitSpringDamper>
-            <provideFeedback>true</provideFeedback>
-        </gazebo>
-        <!-- link 5 -->
-        <gazebo reference="link_5">
-            <mu1>0.2</mu1>
-            <mu2>0.2</mu2>
-        </gazebo>
-        <!-- A6 -->
-        <gazebo reference="A6">
-            <implicitSpringDamper>true</implicitSpringDamper>
-            <provideFeedback>true</provideFeedback>
-        </gazebo>
-        <!-- link 6 -->
-        <gazebo reference="link_6">
-            <mu1>0.2</mu1>
-            <mu2>0.2</mu2>
-        </gazebo>
-        <!-- A7 -->
-        <gazebo reference="A7">
-            <implicitSpringDamper>true</implicitSpringDamper>
-            <provideFeedback>true</provideFeedback>
-        </gazebo>
-        <!-- link 7 -->
-        <gazebo reference="link_7">
-            <mu1>0.2</mu1>
-            <mu2>0.2</mu2>
-        </gazebo>
+        <!-- macros -->
+        <xacro:macro name="gazebo_link_reference" params="name">
+            <gazebo reference="${name}">
+                <mu1>0.2</mu1>
+                <mu2>0.2</mu2>
+            </gazebo>
+        </xacro:macro>
+        <xacro:macro name="gazebo_joint_reference" params="name">
+            <gazebo reference="${name}">
+                <implicitSpringDamper>true</implicitSpringDamper>
+                <provideFeedback>true</provideFeedback>
+            </gazebo>
+        </xacro:macro>
+        <!-- references -->
+        <xacro:gazebo_link_reference name="link_0" />
+        <xacro:gazebo_joint_reference name="A1" />
+        <xacro:gazebo_link_reference name="link_1" />
+        <xacro:gazebo_joint_reference name="A2" />
+        <xacro:gazebo_link_reference name="link_2" />
+        <xacro:gazebo_joint_reference name="A3" />
+        <xacro:gazebo_link_reference name="link_3" />
+        <xacro:gazebo_joint_reference name="A4" />
+        <xacro:gazebo_link_reference name="link_4" />
+        <xacro:gazebo_joint_reference name="A5" />
+        <xacro:gazebo_link_reference name="link_5" />
+        <xacro:gazebo_joint_reference name="A6" />
+        <xacro:gazebo_link_reference name="link_6" />
+        <xacro:gazebo_joint_reference name="A7" />
+        <xacro:gazebo_link_reference name="link_7" />
     </xacro:macro>
 </robot>

File: lbr_description/urdf/iiwa14/iiwa14_description.urdf.xacro (robot description, xacro)
@@ -5,11 +5,11 @@
     <xacro:property name="joint_damping" value="10.0" />
     <xacro:property name="joint_friction" value="0.1" />
-    <xacro:property name="joint_0_position_limit" value="170" />
-    <xacro:property name="joint_1_position_limit" value="120" />
-    <xacro:property name="joint_2_position_limit" value="170" />
-    <xacro:property name="joint_3_position_limit" value="120" />
-    <xacro:property name="joint_4_position_limit" value="170" />
-    <xacro:property name="joint_5_position_limit" value="120" />
-    <xacro:property name="joint_6_position_limit" value="175" />
+    <xacro:property name="A1_position_limit" value="170" />
+    <xacro:property name="A2_position_limit" value="120" />
+    <xacro:property name="A3_position_limit" value="170" />
+    <xacro:property name="A4_position_limit" value="120" />
+    <xacro:property name="A5_position_limit" value="170" />
+    <xacro:property name="A6_position_limit" value="120" />
+    <xacro:property name="A7_position_limit" value="175" />
     <xacro:property name="joint_0_velocity_limit" value="85" />
     <xacro:property name="joint_1_velocity_limit" value="85" />
@@ -51,6 +51,6 @@
             <child link="link_1" />
             <axis xyz="0.0 0.0 1.0" />
-            <limit effort="${effort_limit}" lower="${-joint_0_position_limit * PI / 180}"
-                upper="${joint_0_position_limit * PI / 180}"
+            <limit effort="${effort_limit}" lower="${-A1_position_limit * PI / 180}"
+                upper="${A1_position_limit * PI / 180}"
                 velocity="${joint_0_velocity_limit * PI / 180}" />
             <dynamics damping="${joint_damping}" friction="${joint_friction}" />
@@ -81,6 +81,6 @@
             <child link="link_2" />
             <axis xyz="0.0 1.0 0.0" />
-            <limit effort="${effort_limit}" lower="${-joint_1_position_limit * PI / 180}"
-                upper="${joint_1_position_limit * PI / 180}"
+            <limit effort="${effort_limit}" lower="${-A2_position_limit * PI / 180}"
+                upper="${A2_position_limit * PI / 180}"
                 velocity="${joint_1_velocity_limit * PI / 180}" />
             <dynamics damping="${joint_damping}" friction="${joint_friction}" />
@@ -111,6 +111,6 @@
             <child link="link_3" />
             <axis xyz="0.0 0.0 1.0" />
-            <limit effort="${effort_limit}" lower="${-joint_2_position_limit * PI / 180}"
-                upper="${joint_2_position_limit * PI / 180}"
+            <limit effort="${effort_limit}" lower="${-A3_position_limit * PI / 180}"
+                upper="${A3_position_limit * PI / 180}"
                 velocity="${joint_2_velocity_limit * PI / 180}" />
             <dynamics damping="${joint_damping}" friction="${joint_friction}" />
@@ -141,6 +141,6 @@
             <child link="link_4" />
             <axis xyz="0.0 -1.0 0.0" />
-            <limit effort="${effort_limit}" lower="${-joint_3_position_limit * PI / 180}"
-                upper="${joint_3_position_limit * PI / 180}"
+            <limit effort="${effort_limit}" lower="${-A4_position_limit * PI / 180}"
+                upper="${A4_position_limit * PI / 180}"
                 velocity="${joint_3_velocity_limit * PI / 180}" />
             <dynamics damping="${joint_damping}" friction="${joint_friction}" />
@@ -171,6 +171,6 @@
             <child link="link_5" />
             <axis xyz="0.0 0.0 1.0" />
-            <limit effort="${effort_limit}" lower="${-joint_4_position_limit * PI / 180}"
-                upper="${joint_4_position_limit * PI / 180}"
+            <limit effort="${effort_limit}" lower="${-A5_position_limit * PI / 180}"
+                upper="${A5_position_limit * PI / 180}"
                 velocity="${joint_4_velocity_limit * PI / 180}" />
             <dynamics damping="${joint_damping}" friction="${joint_friction}" />
@@ -201,6 +201,6 @@
             <child link="link_6" />
             <axis xyz="0.0 1.0 0.0" />
-            <limit effort="${effort_limit}" lower="${-joint_5_position_limit * PI / 180}"
-                upper="${joint_5_position_limit * PI / 180}"
+            <limit effort="${effort_limit}" lower="${-A6_position_limit * PI / 180}"
+                upper="${A6_position_limit * PI / 180}"
                 velocity="${joint_5_velocity_limit * PI / 180}" />
             <dynamics damping="${joint_damping}" friction="${joint_friction}" />
@@ -231,6 +231,6 @@
             <child link="link_7" />
             <axis xyz="0.0 0.0 1.0" />
-            <limit effort="${effort_limit}" lower="${-joint_6_position_limit * PI / 180}"
-                upper="${joint_6_position_limit * PI / 180}"
+            <limit effort="${effort_limit}" lower="${-A7_position_limit * PI / 180}"
+                upper="${A7_position_limit * PI / 180}"
                 velocity="${joint_6_velocity_limit * PI / 180}" />
             <dynamics damping="${joint_damping}" friction="${joint_friction}" />
@@ -265,11 +265,11 @@
         <!-- TODO: move modes to args, decouple urdf/gazebo/controls -->
         <xacro:lbr_system_interface
-            joint_0_position_limit="${joint_0_position_limit * PI / 180}"
-            joint_1_position_limit="${joint_1_position_limit * PI / 180}"
-            joint_2_position_limit="${joint_2_position_limit * PI / 180}"
-            joint_3_position_limit="${joint_3_position_limit * PI / 180}"
-            joint_4_position_limit="${joint_4_position_limit * PI / 180}"
-            joint_5_position_limit="${joint_5_position_limit * PI / 180}"
-            joint_6_position_limit="${joint_6_position_limit * PI / 180}"
+            A1_position_limit="${A1_position_limit * PI / 180}"
+            A2_position_limit="${A2_position_limit * PI / 180}"
+            A3_position_limit="${A3_position_limit * PI / 180}"
+            A4_position_limit="${A4_position_limit * PI / 180}"
+            A5_position_limit="${A5_position_limit * PI / 180}"
+            A6_position_limit="${A6_position_limit * PI / 180}"
+            A7_position_limit="${A7_position_limit * PI / 180}"
             effort_limit="${effort_limit}"
             sim="${sim}" remote_host="INADDR_ANY" port_id="${port_id}" />

File: lbr_description/urdf/iiwa7/iiwa7_description.urdf.xacro (robot description, xacro)
@@ -5,11 +5,11 @@
     <xacro:property name="joint_damping" value="10.0" />
     <xacro:property name="joint_friction" value="0.1" />
-    <xacro:property name="joint_0_position_limit" value="170" />
-    <xacro:property name="joint_1_position_limit" value="120" />
-    <xacro:property name="joint_2_position_limit" value="170" />
-    <xacro:property name="joint_3_position_limit" value="120" />
-    <xacro:property name="joint_4_position_limit" value="170" />
-    <xacro:property name="joint_5_position_limit" value="120" />
-    <xacro:property name="joint_6_position_limit" value="175" />
+    <xacro:property name="A1_position_limit" value="170" />
+    <xacro:property name="A2_position_limit" value="120" />
+    <xacro:property name="A3_position_limit" value="170" />
+    <xacro:property name="A4_position_limit" value="120" />
+    <xacro:property name="A5_position_limit" value="170" />
+    <xacro:property name="A6_position_limit" value="120" />
+    <xacro:property name="A7_position_limit" value="175" />
     <xacro:property name="joint_0_velocity_limit" value="98" />
     <xacro:property name="joint_1_velocity_limit" value="98" />
@@ -51,6 +51,6 @@
             <child link="link_1" />
             <axis xyz="0.0 0.0 1.0" />
-            <limit effort="${effort_limit}" lower="${-joint_0_position_limit * PI / 180}"
-                upper="${joint_0_position_limit * PI / 180}"
+            <limit effort="${effort_limit}" lower="${-A1_position_limit * PI / 180}"
+                upper="${A1_position_limit * PI / 180}"
                 velocity="${joint_0_velocity_limit * PI / 180}" />
             <dynamics damping="${joint_damping}" friction="${joint_friction}" />
@@ -81,6 +81,6 @@
             <child link="link_2" />
             <axis xyz="0.0 1.0 0.0" />
-            <limit effort="${effort_limit}" lower="${-joint_1_position_limit * PI / 180}"
-                upper="${joint_1_position_limit * PI / 180}"
+            <limit effort="${effort_limit}" lower="${-A2_position_limit * PI / 180}"
+                upper="${A2_position_limit * PI / 180}"
                 velocity="${joint_1_velocity_limit * PI / 180}" />
             <dynamics damping="${joint_damping}" friction="${joint_friction}" />
@@ -111,6 +111,6 @@
             <child link="link_3" />
             <axis xyz="0.0 0.0 1.0" />
-            <limit effort="${effort_limit}" lower="${-joint_2_position_limit * PI / 180}"
-                upper="${joint_2_position_limit * PI / 180}"
+            <limit effort="${effort_limit}" lower="${-A3_position_limit * PI / 180}"
+                upper="${A3_position_limit * PI / 180}"
                 velocity="${joint_2_velocity_limit * PI / 180}" />
             <dynamics damping="${joint_damping}" friction="${joint_friction}" />
@@ -141,6 +141,6 @@
             <child link="link_4" />
             <axis xyz="0.0 -1.0 0.0" />
-            <limit effort="${effort_limit}" lower="${-joint_3_position_limit * PI / 180}"
-                upper="${joint_3_position_limit * PI / 180}"
+            <limit effort="${effort_limit}" lower="${-A4_position_limit * PI / 180}"
+                upper="${A4_position_limit * PI / 180}"
                 velocity="${joint_3_velocity_limit * PI / 180}" />
             <dynamics damping="${joint_damping}" friction="${joint_friction}" />
@@ -171,6 +171,6 @@
             <child link="link_5" />
             <axis xyz="0.0 0.0 1.0" />
-            <limit effort="${effort_limit}" lower="${-joint_4_position_limit * PI / 180}"
-                upper="${joint_4_position_limit * PI / 180}"
+            <limit effort="${effort_limit}" lower="${-A5_position_limit * PI / 180}"
+                upper="${A5_position_limit * PI / 180}"
                 velocity="${joint_4_velocity_limit * PI / 180}" />
             <dynamics damping="${joint_damping}" friction="${joint_friction}" />
@@ -201,6 +201,6 @@
             <child link="link_6" />
             <axis xyz="0.0 1.0 0.0" />
-            <limit effort="${effort_limit}" lower="${-joint_5_position_limit * PI / 180}"
-                upper="${joint_5_position_limit * PI / 180}"
+            <limit effort="${effort_limit}" lower="${-A6_position_limit * PI / 180}"
+                upper="${A6_position_limit * PI / 180}"
                 velocity="${joint_5_velocity_limit * PI / 180}" />
             <dynamics damping="${joint_damping}" friction="${joint_friction}" />
@@ -231,6 +231,6 @@
             <child link="link_7" />
             <axis xyz="0.0 0.0 1.0" />
-            <limit effort="${effort_limit}" lower="${-joint_6_position_limit * PI / 180}"
-                upper="${joint_6_position_limit * PI / 180}"
+            <limit effort="${effort_limit}" lower="${-A7_position_limit * PI / 180}"
+                upper="${A7_position_limit * PI / 180}"
                 velocity="${joint_6_velocity_limit * PI / 180}" />
             <dynamics damping="${joint_damping}" friction="${joint_friction}" />
@@ -265,11 +265,11 @@
         <!-- TODO: move modes to args, decouple urdf/gazebo/controls -->
         <xacro:lbr_system_interface
-            joint_0_position_limit="${joint_0_position_limit * PI / 180}"
-            joint_1_position_limit="${joint_1_position_limit * PI / 180}"
-            joint_2_position_limit="${joint_2_position_limit * PI / 180}"
-            joint_3_position_limit="${joint_3_position_limit * PI / 180}"
-            joint_4_position_limit="${joint_4_position_limit * PI / 180}"
-            joint_5_position_limit="${joint_5_position_limit * PI / 180}"
-            joint_6_position_limit="${joint_6_position_limit * PI / 180}"
+            A1_position_limit="${A1_position_limit * PI / 180}"
+            A2_position_limit="${A2_position_limit * PI / 180}"
+            A3_position_limit="${A3_position_limit * PI / 180}"
+            A4_position_limit="${A4_position_limit * PI / 180}"
+            A5_position_limit="${A5_position_limit * PI / 180}"
+            A6_position_limit="${A6_position_limit * PI / 180}"
+            A7_position_limit="${A7_position_limit * PI / 180}"
             effort_limit="${effort_limit}"
             sim="${sim}" remote_host="INADDR_ANY" port_id="${port_id}" />

File: lbr_description/urdf/med14/med14_description.urdf.xacro (robot description, xacro)
@@ -5,11 +5,11 @@
     <xacro:property name="joint_damping" value="10.0" />
     <xacro:property name="joint_friction" value="0.1" />
-    <xacro:property name="joint_0_position_limit" value="170" />
-    <xacro:property name="joint_1_position_limit" value="120" />
-    <xacro:property name="joint_2_position_limit" value="170" />
-    <xacro:property name="joint_3_position_limit" value="120" />
-    <xacro:property name="joint_4_position_limit" value="170" />
-    <xacro:property name="joint_5_position_limit" value="120" />
-    <xacro:property name="joint_6_position_limit" value="175" />
+    <xacro:property name="A1_position_limit" value="170" />
+    <xacro:property name="A2_position_limit" value="120" />
+    <xacro:property name="A3_position_limit" value="170" />
+    <xacro:property name="A4_position_limit" value="120" />
+    <xacro:property name="A5_position_limit" value="170" />
+    <xacro:property name="A6_position_limit" value="120" />
+    <xacro:property name="A7_position_limit" value="175" />
     <xacro:property name="joint_0_velocity_limit" value="85" />
     <xacro:property name="joint_1_velocity_limit" value="85" />
@@ -51,6 +51,6 @@
             <child link="link_1" />
             <axis xyz="0.0 0.0 1.0" />
-            <limit effort="${effort_limit}" lower="${-joint_0_position_limit * PI / 180}"
-                upper="${joint_0_position_limit * PI / 180}"
+            <limit effort="${effort_limit}" lower="${-A1_position_limit * PI / 180}"
+                upper="${A1_position_limit * PI / 180}"
                 velocity="${joint_0_velocity_limit * PI / 180}" />
             <dynamics damping="${joint_damping}" friction="${joint_friction}" />
@@ -81,6 +81,6 @@
             <child link="link_2" />
             <axis xyz="0.0 1.0 0.0" />
-            <limit effort="${effort_limit}" lower="${-joint_1_position_limit * PI / 180}"
-                upper="${joint_1_position_limit * PI / 180}"
+            <limit effort="${effort_limit}" lower="${-A2_position_limit * PI / 180}"
+                upper="${A2_position_limit * PI / 180}"
                 velocity="${joint_1_velocity_limit * PI / 180}" />
             <dynamics damping="${joint_damping}" friction="${joint_friction}" />
@@ -111,6 +111,6 @@
             <child link="link_3" />
             <axis xyz="0.0 0.0 1.0" />
-            <limit effort="${effort_limit}" lower="${-joint_2_position_limit * PI / 180}"
-                upper="${joint_2_position_limit * PI / 180}"
+            <limit effort="${effort_limit}" lower="${-A3_position_limit * PI / 180}"
+                upper="${A3_position_limit * PI / 180}"
                 velocity="${joint_2_velocity_limit * PI / 180}" />
             <dynamics damping="${joint_damping}" friction="${joint_friction}" />
@@ -141,6 +141,6 @@
             <child link="link_4" />
             <axis xyz="0.0 -1.0 0.0" />
-            <limit effort="${effort_limit}" lower="${-joint_3_position_limit * PI / 180}"
-                upper="${joint_3_position_limit * PI / 180}"
+            <limit effort="${effort_limit}" lower="${-A4_position_limit * PI / 180}"
+                upper="${A4_position_limit * PI / 180}"
                 velocity="${joint_3_velocity_limit * PI / 180}" />
             <dynamics damping="${joint_damping}" friction="${joint_friction}" />
@@ -171,6 +171,6 @@
             <child link="link_5" />
             <axis xyz="0.0 0.0 1.0" />
-            <limit effort="${effort_limit}" lower="${-joint_4_position_limit * PI / 180}"
-                upper="${joint_4_position_limit * PI / 180}"
+            <limit effort="${effort_limit}" lower="${-A5_position_limit * PI / 180}"
+                upper="${A5_position_limit * PI / 180}"
                 velocity="${joint_4_velocity_limit * PI / 180}" />
             <dynamics damping="${joint_damping}" friction="${joint_friction}" />
@@ -201,6 +201,6 @@
             <child link="link_6" />
             <axis xyz="0.0 1.0 0.0" />
-            <limit effort="${effort_limit}" lower="${-joint_5_position_limit * PI / 180}"
-                upper="${joint_5_position_limit * PI / 180}"
+            <limit effort="${effort_limit}" lower="${-A6_position_limit * PI / 180}"
+                upper="${A6_position_limit * PI / 180}"
                 velocity="${joint_5_velocity_limit * PI / 180}" />
             <dynamics damping="${joint_damping}" friction="${joint_friction}" />
@@ -231,6 +231,6 @@
             <child link="link_7" />
             <axis xyz="0.0 0.0 1.0" />
-            <limit effort="${effort_limit}" lower="${-joint_6_position_limit * PI / 180}"
-                upper="${joint_6_position_limit * PI / 180}"
+            <limit effort="${effort_limit}" lower="${-A7_position_limit * PI / 180}"
+                upper="${A7_position_limit * PI / 180}"
                 velocity="${joint_6_velocity_limit * PI / 180}" />
             <dynamics damping="${joint_damping}" friction="${joint_friction}" />
@@ -265,11 +265,11 @@
         <!-- TODO: move modes to args, decouple urdf/gazebo/controls -->
         <xacro:lbr_system_interface
-            joint_0_position_limit="${joint_0_position_limit * PI / 180}"
-            joint_1_position_limit="${joint_1_position_limit * PI / 180}"
-            joint_2_position_limit="${joint_2_position_limit * PI / 180}"
-            joint_3_position_limit="${joint_3_position_limit * PI / 180}"
-            joint_4_position_limit="${joint_4_position_limit * PI / 180}"
-            joint_5_position_limit="${joint_5_position_limit * PI / 180}"
-            joint_6_position_limit="${joint_6_position_limit * PI / 180}"
+            A1_position_limit="${A1_position_limit * PI / 180}"
+            A2_position_limit="${A2_position_limit * PI / 180}"
+            A3_position_limit="${A3_position_limit * PI / 180}"
+            A4_position_limit="${A4_position_limit * PI / 180}"
+            A5_position_limit="${A5_position_limit * PI / 180}"
+            A6_position_limit="${A6_position_limit * PI / 180}"
+            A7_position_limit="${A7_position_limit * PI / 180}"
             effort_limit="${effort_limit}"
             sim="${sim}" remote_host="INADDR_ANY" port_id="${port_id}" />
