Commit message: robot name prefix in config files (#189)

File: lbr_description/gazebo/lbr_gazebo.xacro (robot description, xacro)
@@ -26,19 +26,19 @@
         </xacro:macro>
         <!-- references -->
-        <xacro:gazebo_link_reference name="link_0" />
-        <xacro:gazebo_joint_reference name="A1" />
-        <xacro:gazebo_link_reference name="link_1" />
-        <xacro:gazebo_joint_reference name="A2" />
-        <xacro:gazebo_link_reference name="link_2" />
-        <xacro:gazebo_joint_reference name="A3" />
-        <xacro:gazebo_link_reference name="link_3" />
-        <xacro:gazebo_joint_reference name="A4" />
-        <xacro:gazebo_link_reference name="link_4" />
-        <xacro:gazebo_joint_reference name="A5" />
-        <xacro:gazebo_link_reference name="link_5" />
-        <xacro:gazebo_joint_reference name="A6" />
-        <xacro:gazebo_link_reference name="link_6" />
-        <xacro:gazebo_joint_reference name="A7" />
-        <xacro:gazebo_link_reference name="link_7" />
+        <xacro:gazebo_link_reference name="${robot_name}_link_0" />
+        <xacro:gazebo_joint_reference name="${robot_name}_A1" />
+        <xacro:gazebo_link_reference name="${robot_name}_link_1" />
+        <xacro:gazebo_joint_reference name="${robot_name}_A2" />
+        <xacro:gazebo_link_reference name="${robot_name}_link_2" />
+        <xacro:gazebo_joint_reference name="${robot_name}_A3" />
+        <xacro:gazebo_link_reference name="${robot_name}_link_3" />
+        <xacro:gazebo_joint_reference name="${robot_name}_A4" />
+        <xacro:gazebo_link_reference name="${robot_name}_link_4" />
+        <xacro:gazebo_joint_reference name="${robot_name}_A5" />
+        <xacro:gazebo_link_reference name="${robot_name}_link_5" />
+        <xacro:gazebo_joint_reference name="${robot_name}_A6" />
+        <xacro:gazebo_link_reference name="${robot_name}_link_6" />
+        <xacro:gazebo_joint_reference name="${robot_name}_A7" />
+        <xacro:gazebo_link_reference name="${robot_name}_link_7" />
     </xacro:macro>
 </robot>

File: lbr_description/ros2_control/lbr_system_interface.xacro (robot description, xacro)
@@ -119,5 +119,5 @@
                 </joint>
             </xacro:macro>
-            <xacro:joint_interface name="A1"
+            <xacro:joint_interface name="${robot_name}_A1"
                 min_position="${joint_limits['A1']['lower'] * PI / 180}"
                 max_position="${joint_limits['A1']['upper'] * PI / 180}"
@@ -125,5 +125,5 @@
                 max_torque="${joint_limits['A1']['effort']}"
                 mode="${mode}" />
-            <xacro:joint_interface name="A2"
+            <xacro:joint_interface name="${robot_name}_A2"
                 min_position="${joint_limits['A2']['lower'] * PI / 180}"
                 max_position="${joint_limits['A2']['upper'] * PI / 180}"
@@ -131,5 +131,5 @@
                 max_torque="${joint_limits['A2']['effort']}"
                 mode="${mode}" />
-            <xacro:joint_interface name="A3"
+            <xacro:joint_interface name="${robot_name}_A3"
                 min_position="${joint_limits['A3']['lower'] * PI / 180}"
                 max_position="${joint_limits['A3']['upper'] * PI / 180}"
@@ -137,5 +137,5 @@
                 max_torque="${joint_limits['A3']['effort']}"
                 mode="${mode}" />
-            <xacro:joint_interface name="A4"
+            <xacro:joint_interface name="${robot_name}_A4"
                 min_position="${joint_limits['A4']['lower'] * PI / 180}"
                 max_position="${joint_limits['A4']['upper'] * PI / 180}"
@@ -143,5 +143,5 @@
                 max_torque="${joint_limits['A4']['effort']}"
                 mode="${mode}" />
-            <xacro:joint_interface name="A5"
+            <xacro:joint_interface name="${robot_name}_A5"
                 min_position="${joint_limits['A5']['lower'] * PI / 180}"
                 max_position="${joint_limits['A5']['upper'] * PI / 180}"
@@ -149,5 +149,5 @@
                 max_torque="${joint_limits['A5']['effort']}"
                 mode="${mode}" />
-            <xacro:joint_interface name="A6"
+            <xacro:joint_interface name="${robot_name}_A6"
                 min_position="${joint_limits['A6']['lower'] * PI / 180}"
                 max_position="${joint_limits['A6']['upper'] * PI / 180}"
@@ -155,5 +155,5 @@
                 max_torque="${joint_limits['A6']['effort']}"
                 mode="${mode}" />
-            <xacro:joint_interface name="A7"
+            <xacro:joint_interface name="${robot_name}_A7"
                 min_position="${joint_limits['A7']['lower'] * PI / 180}"
                 max_position="${joint_limits['A7']['upper'] * PI / 180}"

File: lbr_description/urdf/iiwa14/iiwa14.xacro (robot description, xacro)
@@ -15,5 +15,5 @@
     <joint name="world_joint" type="fixed">
         <parent link="world" />
-        <child link="link_0" />
+        <child link="$(arg robot_name)_link_0" />
     </joint>
     <!-- iiwa -->

File: lbr_description/urdf/iiwa14/iiwa14_description.xacro (robot description, xacro)
@@ -21,5 +21,5 @@
             joint_limits="${joint_limits}"
             system_parameters_path="${system_parameters_path}" />
-        <link name="link_0">
+        <link name="${robot_name}_link_0">
             <inertial>
                 <origin rpy="0 0 0" xyz="-0.012822 0.0 0.071507" />
@@ -41,8 +41,8 @@
             </collision>
         </link>
-        <joint name="A1" type="revolute">
+        <joint name="${robot_name}_A1" type="revolute">
             <origin rpy="0 0 0" xyz="0.0 0.0 0.1475" />
-            <parent link="link_0" />
-            <child link="link_1" />
+            <parent link="${robot_name}_link_0" />
+            <child link="${robot_name}_link_1" />
             <axis xyz="0.0 0.0 1.0" />
             <limit
@@ -53,5 +53,5 @@
             <dynamics damping="${joint_damping}" friction="${joint_friction}" />
         </joint>
-        <link name="link_1">
+        <link name="${robot_name}_link_1">
             <inertial>
                 <origin rpy="0 0 0" xyz="0.0 -0.033795 0.132404" />
@@ -73,8 +73,8 @@
             </collision>
         </link>
-        <joint name="A2" type="revolute">
+        <joint name="${robot_name}_A2" type="revolute">
             <origin rpy="0 0 0" xyz="0.0 -0.01 0.2125" />
-            <parent link="link_1" />
-            <child link="link_2" />
+            <parent link="${robot_name}_link_1" />
+            <child link="${robot_name}_link_2" />
             <axis xyz="0.0 1.0 0.0" />
             <limit
@@ -85,5 +85,5 @@
             <dynamics damping="${joint_damping}" friction="${joint_friction}" />
         </joint>
-        <link name="link_2">
+        <link name="${robot_name}_link_2">
             <inertial>
                 <origin rpy="0 0 0" xyz="0.000136 0.047548 0.076322" />
@@ -105,8 +105,8 @@
             </collision>
         </link>
-        <joint name="A3" type="revolute">
+        <joint name="${robot_name}_A3" type="revolute">
             <origin rpy="0 0 0" xyz="0.0 0.01 0.228" />
-            <parent link="link_2" />
-            <child link="link_3" />
+            <parent link="${robot_name}_link_2" />
+            <child link="${robot_name}_link_3" />
             <axis xyz="0.0 0.0 1.0" />
             <limit
@@ -117,5 +117,5 @@
             <dynamics damping="${joint_damping}" friction="${joint_friction}" />
         </joint>
-        <link name="link_3">
+        <link name="${robot_name}_link_3">
             <inertial>
                 <origin rpy="0 0 0" xyz="0.0 0.034913 0.123108" />
@@ -137,8 +137,8 @@
             </collision>
         </link>
-        <joint name="A4" type="revolute">
+        <joint name="${robot_name}_A4" type="revolute">
             <origin rpy="0 0 0" xyz="0.0 0.0105 0.192" />
-            <parent link="link_3" />
-            <child link="link_4" />
+            <parent link="${robot_name}_link_3" />
+            <child link="${robot_name}_link_4" />
             <axis xyz="0.0 -1.0 0.0" />
             <limit
@@ -149,5 +149,5 @@
             <dynamics damping="${joint_damping}" friction="${joint_friction}" />
         </joint>
-        <link name="link_4">
+        <link name="${robot_name}_link_4">
             <inertial>
                 <origin rpy="0 0 0" xyz="0.0 -0.039793 0.086944" />
@@ -169,8 +169,8 @@
             </collision>
         </link>
-        <joint name="A5" type="revolute">
+        <joint name="${robot_name}_A5" type="revolute">
             <origin rpy="0 0 0" xyz="0.0 -0.0105 0.2075" />
-            <parent link="link_4" />
-            <child link="link_5" />
+            <parent link="${robot_name}_link_4" />
+            <child link="${robot_name}_link_5" />
             <axis xyz="0.0 0.0 1.0" />
             <limit
@@ -181,5 +181,5 @@
             <dynamics damping="${joint_damping}" friction="${joint_friction}" />
         </joint>
-        <link name="link_5">
+        <link name="${robot_name}_link_5">
             <inertial>
                 <origin rpy="0 0 0" xyz="0.0 -0.029824 0.076267" />
@@ -201,8 +201,8 @@
             </collision>
         </link>
-        <joint name="A6" type="revolute">
+        <joint name="${robot_name}_A6" type="revolute">
             <origin rpy="0 0 0" xyz="0.0 -0.0707 0.1925" />
-            <parent link="link_5" />
-            <child link="link_6" />
+            <parent link="${robot_name}_link_5" />
+            <child link="${robot_name}_link_6" />
             <axis xyz="0.0 1.0 0.0" />
             <limit
@@ -213,5 +213,5 @@
             <dynamics damping="${joint_damping}" friction="${joint_friction}" />
         </joint>
-        <link name="link_6">
+        <link name="${robot_name}_link_6">
             <inertial>
                 <origin rpy="0 0 0" xyz="0.0 0.07102 0.00495" />
@@ -233,8 +233,8 @@
             </collision>
         </link>
-        <joint name="A7" type="revolute">
+        <joint name="${robot_name}_A7" type="revolute">
             <origin rpy="0 0 0" xyz="0.0 0.0707 0.091" />
-            <parent link="link_6" />
-            <child link="link_7" />
+            <parent link="${robot_name}_link_6" />
+            <child link="${robot_name}_link_7" />
             <axis xyz="0.0 0.0 1.0" />
             <limit
@@ -245,5 +245,5 @@
             <dynamics damping="${joint_damping}" friction="${joint_friction}" />
         </joint>
-        <link name="link_7">
+        <link name="${robot_name}_link_7">
             <inertial>
                 <origin rpy="0 0 0" xyz="3.0000e-06 -2.0000e-06 1.3782e-02" />
@@ -265,9 +265,9 @@
         </link>
         <joint name="joint_ee" type="fixed">
-            <parent link="link_7" />
-            <child link="link_ee" />
+            <parent link="${robot_name}_link_7" />
+            <child link="${robot_name}_link_ee" />
             <origin xyz="0 0 0.035" rpy="0 0 0" />
         </joint>
-        <link name="link_ee">
+        <link name="${robot_name}_link_ee">
         </link>
     </xacro:macro>

File: lbr_description/urdf/iiwa7/iiwa7.xacro (robot description, xacro)
@@ -15,5 +15,5 @@
     <joint name="world_joint" type="fixed">
         <parent link="world" />
-        <child link="link_0" />
+        <child link="$(arg robot_name)_link_0" />
     </joint>
     <!-- iiwa -->

File: lbr_description/urdf/iiwa7/iiwa7_description.xacro (robot description, xacro)
@@ -21,5 +21,5 @@
             joint_limits="${joint_limits}"
             system_parameters_path="${system_parameters_path}" />
-        <link name="link_0">
+        <link name="${robot_name}_link_0">
             <inertial>
                 <origin rpy="0 0 0" xyz="-0.012857 0.0 0.069964" />
@@ -41,8 +41,8 @@
             </collision>
         </link>
-        <joint name="A1" type="revolute">
+        <joint name="${robot_name}_A1" type="revolute">
             <origin rpy="0 0 0" xyz="0.0 0.0 0.1475" />
-            <parent link="link_0" />
-            <child link="link_1" />
+            <parent link="${robot_name}_link_0" />
+            <child link="${robot_name}_link_1" />
             <axis xyz="0.0 0.0 1.0" />
             <limit
@@ -53,5 +53,5 @@
             <dynamics damping="${joint_damping}" friction="${joint_friction}" />
         </joint>
-        <link name="link_1">
+        <link name="${robot_name}_link_1">
             <inertial>
                 <origin rpy="0 0 0" xyz="0.0 -0.034819 0.123299" />
@@ -73,8 +73,8 @@
             </collision>
         </link>
-        <joint name="A2" type="revolute">
+        <joint name="${robot_name}_A2" type="revolute">
             <origin rpy="0 0 0" xyz="0.0 -0.0105 0.1925" />
-            <parent link="link_1" />
-            <child link="link_2" />
+            <parent link="${robot_name}_link_1" />
+            <child link="${robot_name}_link_2" />
             <axis xyz="0.0 1.0 0.0" />
             <limit
@@ -85,5 +85,5 @@
             <dynamics damping="${joint_damping}" friction="${joint_friction}" />
         </joint>
-        <link name="link_2">
+        <link name="${robot_name}_link_2">
             <inertial>
                 <origin rpy="0 0 0" xyz="0.0 0.039793 0.086944" />
@@ -105,8 +105,8 @@
             </collision>
         </link>
-        <joint name="A3" type="revolute">
+        <joint name="${robot_name}_A3" type="revolute">
             <origin rpy="0 0 0" xyz="0.0 0.0105 0.2075" />
-            <parent link="link_2" />
-            <child link="link_3" />
+            <parent link="${robot_name}_link_2" />
+            <child link="${robot_name}_link_3" />
             <axis xyz="0.0 0.0 1.0" />
             <limit
@@ -117,5 +117,5 @@
             <dynamics damping="${joint_damping}" friction="${joint_friction}" />
         </joint>
-        <link name="link_3">
+        <link name="${robot_name}_link_3">
             <inertial>
                 <origin rpy="0 0 0" xyz="0.0 0.034819 0.123299" />
@@ -137,8 +137,8 @@
             </collision>
         </link>
-        <joint name="A4" type="revolute">
+        <joint name="${robot_name}_A4" type="revolute">
             <origin rpy="0 0 0" xyz="0.0 0.0105 0.1925" />
-            <parent link="link_3" />
-            <child link="link_4" />
+            <parent link="${robot_name}_link_3" />
+            <child link="${robot_name}_link_4" />
             <axis xyz="0.0 -1.0 0.0" />
             <limit
@@ -149,5 +149,5 @@
             <dynamics damping="${joint_damping}" friction="${joint_friction}" />
         </joint>
-        <link name="link_4">
+        <link name="${robot_name}_link_4">
             <inertial>
                 <origin rpy="0 0 0" xyz="0.0 -0.039793 0.086944" />
@@ -169,8 +169,8 @@
             </collision>
         </link>
-        <joint name="A5" type="revolute">
+        <joint name="${robot_name}_A5" type="revolute">
             <origin rpy="0 0 0" xyz="0.0 -0.0105 0.2075" />
-            <parent link="link_4" />
-            <child link="link_5" />
+            <parent link="${robot_name}_link_4" />
+            <child link="${robot_name}_link_5" />
             <axis xyz="0.0 0.0 1.0" />
             <limit
@@ -181,5 +181,5 @@
             <dynamics damping="${joint_damping}" friction="${joint_friction}" />
         </joint>
-        <link name="link_5">
+        <link name="${robot_name}_link_5">
             <inertial>
                 <origin rpy="0 0 0" xyz="0.0 -0.029824 0.076267" />
@@ -201,8 +201,8 @@
             </collision>
         </link>
-        <joint name="A6" type="revolute">
+        <joint name="${robot_name}_A6" type="revolute">
             <origin rpy="0 0 0" xyz="0.0 -0.0707 0.1925" />
-            <parent link="link_5" />
-            <child link="link_6" />
+            <parent link="${robot_name}_link_5" />
+            <child link="${robot_name}_link_6" />
             <axis xyz="0.0 1.0 0.0" />
             <limit
@@ -213,5 +213,5 @@
             <dynamics damping="${joint_damping}" friction="${joint_friction}" />
         </joint>
-        <link name="link_6">
+        <link name="${robot_name}_link_6">
             <inertial>
                 <origin rpy="0 0 0" xyz="0.0 0.07102 0.00495" />
@@ -233,8 +233,8 @@
             </collision>
         </link>
-        <joint name="A7" type="revolute">
+        <joint name="${robot_name}_A7" type="revolute">
             <origin rpy="0 0 0" xyz="0.0 0.0707 0.091" />
-            <parent link="link_6" />
-            <child link="link_7" />
+            <parent link="${robot_name}_link_6" />
+            <child link="${robot_name}_link_7" />
             <axis xyz="0.0 0.0 1.0" />
             <limit
@@ -245,5 +245,5 @@
             <dynamics damping="${joint_damping}" friction="${joint_friction}" />
         </joint>
-        <link name="link_7">
+        <link name="${robot_name}_link_7">
             <inertial>
                 <origin rpy="0 0 0" xyz="3.0000e-06 -2.0000e-06 1.3782e-02" />
@@ -265,9 +265,9 @@
         </link>
         <joint name="joint_ee" type="fixed">
-            <parent link="link_7" />
-            <child link="link_ee" />
+            <parent link="${robot_name}_link_7" />
+            <child link="${robot_name}_link_ee" />
             <origin xyz="0 0 0.035" rpy="0 0 0" />
         </joint>
-        <link name="link_ee">
+        <link name="${robot_name}_link_ee">
         </link>
     </xacro:macro>

File: lbr_description/urdf/med14/med14.xacro (robot description, xacro)
@@ -15,5 +15,5 @@
     <joint name="world_joint" type="fixed">
         <parent link="world" />
-        <child link="link_0" />
+        <child link="$(arg robot_name)_link_0" />
     </joint>
     <!-- med -->
