Commit message: robot name prefix in config files (#189)

File: lbr_description/urdf/med14/med14_description.xacro (robot description, xacro)
@@ -21,5 +21,5 @@
             joint_limits="${joint_limits}"
             system_parameters_path="${system_parameters_path}" />
-        <link name="link_0">
+        <link name="${robot_name}_link_0">
             <inertial>
                 <origin rpy="0 0 0" xyz="-0.001864 0.0 0.077517" />
@@ -41,8 +41,8 @@
             </collision>
         </link>
-        <joint name="A1" type="revolute">
+        <joint name="${robot_name}_A1" type="revolute">
             <origin rpy="0 0 0" xyz="0.0 0.0 0.147" />
-            <parent link="link_0" />
-            <child link="link_1" />
+            <parent link="${robot_name}_link_0" />
+            <child link="${robot_name}_link_1" />
             <axis xyz="0.0 0.0 1.0" />
             <limit
@@ -53,5 +53,5 @@
             <dynamics damping="${joint_damping}" friction="${joint_friction}" />
         </joint>
-        <link name="link_1">
+        <link name="${robot_name}_link_1">
             <inertial>
                 <origin rpy="0 0 0" xyz="0.0 -0.033795  0.132404" />
@@ -73,8 +73,8 @@
             </collision>
         </link>
-        <joint name="A2" type="revolute">
+        <joint name="${robot_name}_A2" type="revolute">
             <origin rpy="0 0 0" xyz="0.0 -0.01 0.2125" />
-            <parent link="link_1" />
-            <child link="link_2" />
+            <parent link="${robot_name}_link_1" />
+            <child link="${robot_name}_link_2" />
             <axis xyz="0.0 1.0 0.0" />
             <limit
@@ -85,5 +85,5 @@
             <dynamics damping="${joint_damping}" friction="${joint_friction}" />
         </joint>
-        <link name="link_2">
+        <link name="${robot_name}_link_2">
             <inertial>
                 <origin rpy="0 0 0" xyz="0.000136 0.047546 0.076324" />
@@ -105,8 +105,8 @@
             </collision>
         </link>
-        <joint name="A3" type="revolute">
+        <joint name="${robot_name}_A3" type="revolute">
             <origin rpy="0 0 0" xyz="0.0 0.01 0.228" />
-            <parent link="link_2" />
-            <child link="link_3" />
+            <parent link="${robot_name}_link_2" />
+            <child link="${robot_name}_link_3" />
             <axis xyz="0.0 0.0 1.0" />
             <limit
@@ -117,5 +117,5 @@
             <dynamics damping="${joint_damping}" friction="${joint_friction}" />
         </joint>
-        <link name="link_3">
+        <link name="${robot_name}_link_3">
             <inertial>
                 <origin rpy="0 0 0" xyz="0.0 0.034913 0.123108" />
@@ -137,8 +137,8 @@
             </collision>
         </link>
-        <joint name="A4" type="revolute">
+        <joint name="${robot_name}_A4" type="revolute">
             <origin rpy="0 0 0" xyz="0.0 0.0105 0.192" />
-            <parent link="link_3" />
-            <child link="link_4" />
+            <parent link="${robot_name}_link_3" />
+            <child link="${robot_name}_link_4" />
             <axis xyz="0.0 -1.0 0.0" />
             <limit
@@ -149,5 +149,5 @@
             <dynamics damping="${joint_damping}" friction="${joint_friction}" />
         </joint>
-        <link name="link_4">
+        <link name="${robot_name}_link_4">
             <inertial>
                 <origin rpy="0 0 0" xyz="0.0 -0.039793  0.086944" />
@@ -169,8 +169,8 @@
             </collision>
         </link>
-        <joint name="A5" type="revolute">
+        <joint name="${robot_name}_A5" type="revolute">
             <origin rpy="0 0 0" xyz="0.0 -0.0105 0.2075" />
-            <parent link="link_4" />
-            <child link="link_5" />
+            <parent link="${robot_name}_link_4" />
+            <child link="${robot_name}_link_5" />
             <axis xyz="0.0 0.0 1.0" />
             <limit
@@ -181,5 +181,5 @@
             <dynamics damping="${joint_damping}" friction="${joint_friction}" />
         </joint>
-        <link name="link_5">
+        <link name="${robot_name}_link_5">
             <inertial>
                 <origin rpy="0 0 0" xyz="0.0 -0.029824  0.076267" />
@@ -201,8 +201,8 @@
             </collision>
         </link>
-        <joint name="A6" type="revolute">
+        <joint name="${robot_name}_A6" type="revolute">
             <origin rpy="0 0 0" xyz="0.0 -0.0707 0.1925" />
-            <parent link="link_5" />
-            <child link="link_6" />
+            <parent link="${robot_name}_link_5" />
+            <child link="${robot_name}_link_6" />
             <axis xyz="0.0 1.0 0.0" />
             <limit
@@ -213,5 +213,5 @@
             <dynamics damping="${joint_damping}" friction="${joint_friction}" />
         </joint>
-        <link name="link_6">
+        <link name="${robot_name}_link_6">
             <inertial>
                 <origin rpy="0 0 0" xyz="-1.000e-06 7.102e-02 4.953e-03" />
@@ -233,8 +233,8 @@
             </collision>
         </link>
-        <joint name="A7" type="revolute">
+        <joint name="${robot_name}_A7" type="revolute">
             <origin rpy="0 0 0" xyz="0.0 0.0707 0.091" />
-            <parent link="link_6" />
-            <child link="link_7" />
+            <parent link="${robot_name}_link_6" />
+            <child link="${robot_name}_link_7" />
             <axis xyz="0.0 0.0 1.0" />
             <limit
@@ -245,5 +245,5 @@
             <dynamics damping="${joint_damping}" friction="${joint_friction}" />
         </joint>
-        <link name="link_7">
+        <link name="${robot_name}_link_7">
             <inertial>
                 <origin rpy="0 0 0" xyz="3.0000e-06 -2.0000e-06 1.3782e-02" />
@@ -265,9 +265,9 @@
         </link>
         <joint name="joint_ee" type="fixed">
-            <parent link="link_7" />
-            <child link="link_ee" />
+            <parent link="${robot_name}_link_7" />
+            <child link="${robot_name}_link_ee" />
             <origin xyz="0 0 0.035" rpy="0 0 0" />
         </joint>
-        <link name="link_ee">
+        <link name="${robot_name}_link_ee">
         </link>
     </xacro:macro>

File: lbr_description/urdf/med7/med7.xacro (robot description, xacro)
@@ -15,5 +15,5 @@
     <joint name="world_joint" type="fixed">
         <parent link="world" />
-        <child link="link_0" />
+        <child link="$(arg robot_name)_link_0" />
     </joint>
     <!-- med -->

File: lbr_description/urdf/med7/med7_description.xacro (robot description, xacro)
@@ -22,5 +22,5 @@
             system_parameters_path="${system_parameters_path}" />
         <!-- properties -->
-        <link name="link_0">
+        <link name="${robot_name}_link_0">
             <inertial>
                 <origin rpy="0 0 0" xyz="-0.001896 0.0 0.076263" />
@@ -42,8 +42,8 @@
             </collision>
         </link>
-        <joint name="A1" type="revolute">
+        <joint name="${robot_name}_A1" type="revolute">
             <origin rpy="0 0 0" xyz="0.0 0.0 0.1475" />
-            <parent link="link_0" />
-            <child link="link_1" />
+            <parent link="${robot_name}_link_0" />
+            <child link="${robot_name}_link_1" />
             <axis xyz="0.0 0.0 1.0" />
             <limit
@@ -54,5 +54,5 @@
             <dynamics damping="${joint_damping}" friction="${joint_friction}" />
         </joint>
-        <link name="link_1">
+        <link name="${robot_name}_link_1">
             <inertial>
                 <origin rpy="0 0 0" xyz="0.0 -0.034819  0.123299" />
@@ -74,8 +74,8 @@
             </collision>
         </link>
-        <joint name="A2" type="revolute">
+        <joint name="${robot_name}_A2" type="revolute">
             <origin rpy="0 0 0" xyz="0.0 -0.0105 0.1925" />
-            <parent link="link_1" />
-            <child link="link_2" />
+            <parent link="${robot_name}_link_1" />
+            <child link="${robot_name}_link_2" />
             <axis xyz="0.0 1.0 0.0" />
             <limit
@@ -86,5 +86,5 @@
             <dynamics damping="${joint_damping}" friction="${joint_friction}" />
         </joint>
-        <link name="link_2">
+        <link name="${robot_name}_link_2">
             <inertial>
                 <origin rpy="0 0 0" xyz="0.0 0.039793 0.086944" />
@@ -106,8 +106,8 @@
             </collision>
         </link>
-        <joint name="A3" type="revolute">
+        <joint name="${robot_name}_A3" type="revolute">
             <origin rpy="0 0 0" xyz="0.0 0.0105 0.2075" />
-            <parent link="link_2" />
-            <child link="link_3" />
+            <parent link="${robot_name}_link_2" />
+            <child link="${robot_name}_link_3" />
             <axis xyz="0.0 0.0 1.0" />
             <limit
@@ -118,5 +118,5 @@
             <dynamics damping="${joint_damping}" friction="${joint_friction}" />
         </joint>
-        <link name="link_3">
+        <link name="${robot_name}_link_3">
             <inertial>
                 <origin rpy="0 0 0" xyz="0.0 0.034819  0.123299" />
@@ -138,8 +138,8 @@
             </collision>
         </link>
-        <joint name="A4" type="revolute">
+        <joint name="${robot_name}_A4" type="revolute">
             <origin rpy="0 0 0" xyz="0.0 0.0105 0.1925" />
-            <parent link="link_3" />
-            <child link="link_4" />
+            <parent link="${robot_name}_link_3" />
+            <child link="${robot_name}_link_4" />
             <axis xyz="0.0 -1.0 0.0" />
             <limit
@@ -150,5 +150,5 @@
             <dynamics damping="${joint_damping}" friction="${joint_friction}" />
         </joint>
-        <link name="link_4">
+        <link name="${robot_name}_link_4">
             <inertial>
                 <origin rpy="0 0 0" xyz="0.0 -0.039793  0.086944" />
@@ -170,8 +170,8 @@
             </collision>
         </link>
-        <joint name="A5" type="revolute">
+        <joint name="${robot_name}_A5" type="revolute">
             <origin rpy="0 0 0" xyz="0.0 -0.0105 0.2075" />
-            <parent link="link_4" />
-            <child link="link_5" />
+            <parent link="${robot_name}_link_4" />
+            <child link="${robot_name}_link_5" />
             <axis xyz="0.0 0.0 1.0" />
             <limit
@@ -182,5 +182,5 @@
             <dynamics damping="${joint_damping}" friction="${joint_friction}" />
         </joint>
-        <link name="link_5">
+        <link name="${robot_name}_link_5">
             <inertial>
                 <origin rpy="0 0 0" xyz="0.0 -0.029824 0.076267" />
@@ -202,8 +202,8 @@
             </collision>
         </link>
-        <joint name="A6" type="revolute">
+        <joint name="${robot_name}_A6" type="revolute">
             <origin rpy="0 0 0" xyz="0.0 -0.0707 0.1925" />
-            <parent link="link_5" />
-            <child link="link_6" />
+            <parent link="${robot_name}_link_5" />
+            <child link="${robot_name}_link_6" />
             <axis xyz="0.0 1.0 0.0" />
             <limit
@@ -214,5 +214,5 @@
             <dynamics damping="${joint_damping}" friction="${joint_friction}" />
         </joint>
-        <link name="link_6">
+        <link name="${robot_name}_link_6">
             <inertial>
                 <origin rpy="0 0 0" xyz="-1.000e-06 7.102e-02 4.953e-03" />
@@ -234,8 +234,8 @@
             </collision>
         </link>
-        <joint name="A7" type="revolute">
+        <joint name="${robot_name}_A7" type="revolute">
             <origin rpy="0 0 0" xyz="0.0 0.0707 0.091" />
-            <parent link="link_6" />
-            <child link="link_7" />
+            <parent link="${robot_name}_link_6" />
+            <child link="${robot_name}_link_7" />
             <axis xyz="0.0 0.0 1.0" />
             <limit
@@ -246,5 +246,5 @@
             <dynamics damping="${joint_damping}" friction="${joint_friction}" />
         </joint>
-        <link name="link_7">
+        <link name="${robot_name}_link_7">
             <inertial>
                 <origin rpy="0 0 0" xyz="3.0000e-06 -2.0000e-06 1.3782e-02" />
@@ -266,9 +266,9 @@
         </link>
         <joint name="joint_ee" type="fixed">
-            <parent link="link_7" />
-            <child link="link_ee" />
+            <parent link="${robot_name}_link_7" />
+            <child link="${robot_name}_link_ee" />
             <origin xyz="0 0 0.035" rpy="0 0 0" />
         </joint>
-        <link name="link_ee">
+        <link name="${robot_name}_link_ee">
         </link>
     </xacro:macro>
