Commit message: set default remote to INADDR_ANY

File: lbr_description/ros2_control/lbr.ros2_control.xacro (robot description, xacro)
@@ -1,5 +1,5 @@
 <?xml version="1.0"?>
 <robot xmlns:xacro="http://www.ros.org/wiki/xacro">
-    <xacro:macro name="lbr_hardware_interface" params="sim:=^|true operation_mode:=^|TEST_MODE_1 remote_host:=^|172.31.1.147 port:=^|-1 robot_name:=^|lbr">
+    <xacro:macro name="lbr_hardware_interface" params="sim:=^|true operation_mode:=^|TEST_MODE_1 remote_host:=^|INADDR_ANY port:=^|30200 robot_name:=^|lbr">
         <!-- arg for control mode -->
         <ros2_control name="lbr_hardware_interface" type="system">

File: lbr_description/urdf/iiwa14/iiwa14_description.urdf.xacro (robot description, xacro)
@@ -287,5 +287,5 @@
         <xacro:iiwa_gazebo robot_name="${robot_name}"/>
         <!-- TODO: move modes to args, decouple urdf/gazebo/controls -->
-        <xacro:lbr_hardware_interface sim="${sim}" operation_mode="TEST_MODE_1" remote_host="-1" port="30200" robot_name="${robot_name}"/>
+        <xacro:lbr_hardware_interface sim="${sim}" operation_mode="TEST_MODE_1" remote_host="INADDR_ANY" port="30200" robot_name="${robot_name}"/>
     </xacro:macro>
 </robot>

File: lbr_description/urdf/iiwa7/iiwa7_description.urdf.xacro (robot description, xacro)
@@ -287,5 +287,5 @@
         <xacro:iiwa_gazebo robot_name="${robot_name}"/>
         <!-- TODO: move modes to args, decouple urdf/gazebo/controls -->
-        <xacro:lbr_hardware_interface sim="${sim}" operation_mode="TEST_MODE_1" remote_host="-1" port="30200" robot_name="${robot_name}"/>
+        <xacro:lbr_hardware_interface sim="${sim}" operation_mode="TEST_MODE_1" remote_host="INADDR_ANY" port="30200" robot_name="${robot_name}"/>
     </xacro:macro>
 </robot>

File: lbr_description/urdf/med14/med14_description.urdf.xacro (robot description, xacro)
@@ -287,5 +287,5 @@
         <xacro:iiwa_gazebo robot_name="${robot_name}"/>
         <!-- TODO: move modes to args, decouple urdf/gazebo/controls -->
-        <xacro:lbr_hardware_interface sim="${sim}" operation_mode="TEST_MODE_1" remote_host="-1" port="30200" robot_name="${robot_name}"/>
+        <xacro:lbr_hardware_interface sim="${sim}" operation_mode="TEST_MODE_1" remote_host="INADDR_ANY" port="30200" robot_name="${robot_name}"/>
     </xacro:macro>
 </robot>

File: lbr_description/urdf/med7/med7_description.urdf.xacro (robot description, xacro)
@@ -287,5 +287,6 @@
         <xacro:iiwa_gazebo robot_name="${robot_name}"/>
         <!-- TODO: move modes to args, decouple urdf/gazebo/controls -->
-        <xacro:lbr_hardware_interface sim="${sim}" operation_mode="TEST_MODE_1" remote_host="-1" port="30200" robot_name="${robot_name}"/>
+        <!-- add notice for remote host to set to kuka controller -->
+        <xacro:lbr_hardware_interface sim="${sim}" operation_mode="TEST_MODE_1" remote_host="INADDR_ANY" port="30200" robot_name="${robot_name}"/>
     </xacro:macro>
 </robot>

Commit message: fixed threading

File: lbr_description/ros2_control/lbr.ros2_control.xacro (robot description, xacro)
@@ -1,5 +1,5 @@
 <?xml version="1.0"?>
 <robot xmlns:xacro="http://www.ros.org/wiki/xacro">
-    <xacro:macro name="lbr_hardware_interface" params="sim:=^|true operation_mode:=^|TEST_MODE_1 remote_host:=^|INADDR_ANY port:=^|30200 robot_name:=^|lbr">
+    <xacro:macro name="lbr_hardware_interface" params="sim:=^|true remote_host:=^|INADDR_ANY port:=^|30200 robot_name:=^|lbr">
         <!-- arg for control mode -->
         <ros2_control name="lbr_hardware_interface" type="system">
@@ -13,5 +13,4 @@
                 <hardware>
                     <plugin>LBR::FRIHardwareInterface</plugin>
-                    <param name="operation_mode">${operation_mode}</param>
                     <param name="remote_host">${remote_host}</param>
                     <param name="port">${port}</param>

File: lbr_description/urdf/iiwa14/iiwa14_description.urdf.xacro (robot description, xacro)
@@ -286,5 +286,5 @@
         <xacro:iiwa_gazebo robot_name="${robot_name}"/>
         <!-- TODO: move modes to args, decouple urdf/gazebo/controls -->
-        <xacro:lbr_hardware_interface sim="${sim}" operation_mode="TEST_MODE_1" remote_host="INADDR_ANY" port="30200" robot_name="${robot_name}"/>
+        <xacro:lbr_hardware_interface sim="${sim}" remote_host="INADDR_ANY" port="30200" robot_name="${robot_name}"/>
     </xacro:macro>
 </robot>

File: lbr_description/urdf/iiwa7/iiwa7_description.urdf.xacro (robot description, xacro)
@@ -286,5 +286,5 @@
         <xacro:iiwa_gazebo robot_name="${robot_name}"/>
         <!-- TODO: move modes to args, decouple urdf/gazebo/controls -->
-        <xacro:lbr_hardware_interface sim="${sim}" operation_mode="TEST_MODE_1" remote_host="INADDR_ANY" port="30200" robot_name="${robot_name}"/>
+        <xacro:lbr_hardware_interface sim="${sim}" remote_host="INADDR_ANY" port="30200" robot_name="${robot_name}"/>
     </xacro:macro>
 </robot>

File: lbr_description/urdf/med14/med14_description.urdf.xacro (robot description, xacro)
@@ -286,5 +286,5 @@
         <xacro:iiwa_gazebo robot_name="${robot_name}"/>
         <!-- TODO: move modes to args, decouple urdf/gazebo/controls -->
-        <xacro:lbr_hardware_interface sim="${sim}" operation_mode="TEST_MODE_1" remote_host="INADDR_ANY" port="30200" robot_name="${robot_name}"/>
+        <xacro:lbr_hardware_interface sim="${sim}" remote_host="INADDR_ANY" port="30200" robot_name="${robot_name}"/>
     </xacro:macro>
 </robot>

File: lbr_description/urdf/med7/med7_description.urdf.xacro (robot description, xacro)
@@ -287,5 +287,5 @@
         <!-- TODO: move modes to args, decouple urdf/gazebo/controls -->
         <!-- add notice for remote host to set to kuka controller -->
-        <xacro:lbr_hardware_interface sim="${sim}" operation_mode="TEST_MODE_1" remote_host="INADDR_ANY" port="30200" robot_name="${robot_name}"/>
+        <xacro:lbr_hardware_interface sim="${sim}" remote_host="INADDR_ANY" port="30200" robot_name="${robot_name}"/>
     </xacro:macro>
 </robot>

Commit message: added hw if logic

File: lbr_description/ros2_control/lbr.ros2_control.xacro (robot description, xacro)
@@ -1,5 +1,5 @@
 <?xml version="1.0"?>
 <robot xmlns:xacro="http://www.ros.org/wiki/xacro">
-    <xacro:macro name="lbr_hardware_interface" params="sim:=^|true remote_host:=^|INADDR_ANY port:=^|30200 robot_name:=^|lbr">
+    <xacro:macro name="lbr_hardware_interface" params="sim:=^|true remote_host:=^|INADDR_ANY port_id:=^|30200 robot_name:=^|lbr">
         <!-- arg for control mode -->
         <ros2_control name="lbr_hardware_interface" type="system">
@@ -14,14 +14,23 @@
                     <plugin>lbr_hardware::LBRHardwareInterface</plugin>
                     <param name="remote_host">${remote_host}</param>
-                    <param name="port">${port}</param>
+                    <param name="port_id">${port_id}</param>
                 </hardware>
             </xacro:unless>
             <!-- define lbr specific state interfaces as sensor, see https://github.com/ros-controls/roadmap/blob/master/design_drafts/components_architecture_and_urdf_examples.md -->
             <xacro:unless value="${sim}">
-                <sensor name="${robot_name}_state">
+                <sensor name="${robot_name}_fri_sensor">
                     <!-- see KUKA::FRI::LBRState -->
                     <state_interface name="sample_time"/>
+                    <state_interface name="session_state"/>
+                    <state_interface name="connection_quality"/>
+                    <state_interface name="safety_state"/>
+                    <state_interface name="operation_mode"/>
+                    <state_interface name="drive_state"/>
+                    <state_interface name="client_command_mode"/>
+                    <state_interface name="overlay_type"/>
+                    <state_interface name="control_mode"/>
                     <state_interface name="time_stamp_sec"/>
                     <state_interface name="time_stamp_nano_sec"/>
+                    <state_interface name="tracking_performance"/>
                 </sensor>
             </xacro:unless>
@@ -37,8 +46,15 @@
                     <param name="max"> 1</param>
                 </command_interface>
+                <command_interface name="wrench">
+                    <param name="min">-1</param>
+                    <param name="max"> 1</param>
+                </command_interface>
                 <state_interface name="position"/>
                 <state_interface name="effort"/>
                 <xacro:unless value="${sim}">
+                    <state_interface name="commanded_joint_position"/>
+                    <state_interface name="commanded_torque"/>
                     <state_interface name="external_torque"/>
+                    <state_interface name="ipo_joint_position"/>
                 </xacro:unless>
             </joint>
@@ -52,8 +68,15 @@
                     <param name="max"> 1</param>
                 </command_interface>
+                <command_interface name="wrench">
+                    <param name="min">-1</param>
+                    <param name="max"> 1</param>
+                </command_interface>
                 <state_interface name="position"/>
                 <state_interface name="effort"/>
                 <xacro:unless value="${sim}">
+                    <state_interface name="commanded_joint_position"/>
+                    <state_interface name="commanded_torque"/>
                     <state_interface name="external_torque"/>
+                    <state_interface name="ipo_joint_position"/>
                 </xacro:unless>
             </joint>
@@ -67,8 +90,15 @@
                     <param name="max"> 1</param>
                 </command_interface>
+                <command_interface name="wrench">
+                    <param name="min">-1</param>
+                    <param name="max"> 1</param>
+                </command_interface>
                 <state_interface name="position"/>
                 <state_interface name="effort"/>
                 <xacro:unless value="${sim}">
+                    <state_interface name="commanded_joint_position"/>
+                    <state_interface name="commanded_torque"/>
                     <state_interface name="external_torque"/>
+                    <state_interface name="ipo_joint_position"/>
                 </xacro:unless>
             </joint>
@@ -82,8 +112,15 @@
                     <param name="max"> 1</param>
                 </command_interface>
+                <command_interface name="wrench">
+                    <param name="min">-1</param>
+                    <param name="max"> 1</param>
+                </command_interface>
                 <state_interface name="position"/>
                 <state_interface name="effort"/>
                 <xacro:unless value="${sim}">
+                    <state_interface name="commanded_joint_position"/>
+                    <state_interface name="commanded_torque"/>
                     <state_interface name="external_torque"/>
+                    <state_interface name="ipo_joint_position"/>
                 </xacro:unless>
             </joint>
@@ -97,8 +134,15 @@
                     <param name="max"> 1</param>
                 </command_interface>
+                <command_interface name="wrench">
+                    <param name="min">-1</param>
+                    <param name="max"> 1</param>
+                </command_interface>
                 <state_interface name="position"/>
                 <state_interface name="effort"/>
                 <xacro:unless value="${sim}">
+                    <state_interface name="commanded_joint_position"/>
+                    <state_interface name="commanded_torque"/>
                     <state_interface name="external_torque"/>
+                    <state_interface name="ipo_joint_position"/>
                 </xacro:unless>
             </joint>
@@ -112,8 +156,15 @@
                     <param name="max"> 1</param>
                 </command_interface>
+                <command_interface name="wrench">
+                    <param name="min">-1</param>
+                    <param name="max"> 1</param>
+                </command_interface>
                 <state_interface name="position"/>
                 <state_interface name="effort"/>
                 <xacro:unless value="${sim}">
+                    <state_interface name="commanded_joint_position"/>
+                    <state_interface name="commanded_torque"/>
                     <state_interface name="external_torque"/>
+                    <state_interface name="ipo_joint_position"/>
                 </xacro:unless>
             </joint>
@@ -127,8 +178,15 @@
                     <param name="max"> 1</param>
                 </command_interface>
+                <command_interface name="wrench">
+                    <param name="min">-1</param>
+                    <param name="max"> 1</param>
+                </command_interface>
                 <state_interface name="position"/>
                 <state_interface name="effort"/>
                 <xacro:unless value="${sim}">
+                    <state_interface name="commanded_joint_position"/>
+                    <state_interface name="commanded_torque"/>
                     <state_interface name="external_torque"/>
+                    <state_interface name="ipo_joint_position"/>
                 </xacro:unless>
             </joint>
