Commit message: updated joint names to follow KUKA convention

File: lbr_description/ros2_control/lbr.ros2_control.xacro (robot description, xacro)
@@ -49,5 +49,5 @@
             </xacro:unless>
             <!-- define joints and command/state interfaces for each joint -->
-            <joint name="${robot_name}_joint_0">
+            <joint name="${robot_name}_A1">
                 <command_interface name="position">
                     <!-- better to use radians as min max first -->
@@ -69,5 +69,5 @@
                 </xacro:unless>
             </joint>
-            <joint name="${robot_name}_joint_1">
+            <joint name="${robot_name}_A2">
                 <command_interface name="position">
                     <param name="min">-${joint_1_position_limit}</param>
@@ -88,5 +88,5 @@
                 </xacro:unless>
             </joint>
-            <joint name="${robot_name}_joint_2">
+            <joint name="${robot_name}_A3">
                 <command_interface name="position">
                     <param name="min">-${joint_2_position_limit}</param>
@@ -107,5 +107,5 @@
                 </xacro:unless>
             </joint>
-            <joint name="${robot_name}_joint_3">
+            <joint name="${robot_name}_A4">
                 <command_interface name="position">
                     <param name="min">-${joint_3_position_limit}</param>
@@ -126,5 +126,5 @@
                 </xacro:unless>
             </joint>
-            <joint name="${robot_name}_joint_4">
+            <joint name="${robot_name}_A5">
                 <command_interface name="position">
                     <param name="min">-${joint_4_position_limit}</param>
@@ -145,5 +145,5 @@
                 </xacro:unless>
             </joint>
-            <joint name="${robot_name}_joint_5">
+            <joint name="${robot_name}_A6">
                 <command_interface name="position">
                     <param name="min">-${joint_5_position_limit}</param>
@@ -164,5 +164,5 @@
                 </xacro:unless>
             </joint>
-            <joint name="${robot_name}_joint_6">
+            <joint name="${robot_name}_A7">
                 <command_interface name="position">
                     <param name="min">-${joint_6_position_limit}</param>

File: lbr_description/urdf/iiwa14/iiwa14_description.urdf.xacro (robot description, xacro)
@@ -54,5 +54,5 @@
             </collision>
         </link>
-        <joint name="${robot_name}_joint_0" type="revolute">
+        <joint name="${robot_name}_A1" type="revolute">
             <origin rpy="0 0 0" xyz="0.0 0.0 0.1475" />
             <parent link="${robot_name}_link_0" />
@@ -86,5 +86,5 @@
             </collision>
         </link>
-        <joint name="${robot_name}_joint_1" type="revolute">
+        <joint name="${robot_name}_A2" type="revolute">
             <origin rpy="0 0 0" xyz="0.0 -0.01 0.2125" />
             <parent link="${robot_name}_link_1" />
@@ -118,5 +118,5 @@
             </collision>
         </link>
-        <joint name="${robot_name}_joint_2" type="revolute">
+        <joint name="${robot_name}_A3" type="revolute">
             <origin rpy="0 0 0" xyz="0.0 0.01 0.1945" />
             <parent link="${robot_name}_link_2" />
@@ -150,5 +150,5 @@
             </collision>
         </link>
-        <joint name="${robot_name}_joint_3" type="revolute">
+        <joint name="${robot_name}_A4" type="revolute">
             <origin rpy="0 0 0" xyz="-0.0 0.0105 0.2255" />
             <parent link="${robot_name}_link_3" />
@@ -182,5 +182,5 @@
             </collision>
         </link>
-        <joint name="${robot_name}_joint_4" type="revolute">
+        <joint name="${robot_name}_A5" type="revolute">
             <origin rpy="0 0 0" xyz="0.0 -0.0105 0.1745" />
             <parent link="${robot_name}_link_4" />
@@ -214,5 +214,5 @@
             </collision>
         </link>
-        <joint name="${robot_name}_joint_5" type="revolute">
+        <joint name="${robot_name}_A6" type="revolute">
             <origin rpy="0 0 0" xyz="-0.0 -0.0707 0.2255" />
             <parent link="${robot_name}_link_5" />
@@ -246,5 +246,5 @@
             </collision>
         </link>
-        <joint name="${robot_name}_joint_6" type="revolute">
+        <joint name="${robot_name}_A7" type="revolute">
             <origin rpy="0 0 0" xyz="0.0 0.0707 0.0711" />
             <parent link="${robot_name}_link_6" />

File: lbr_description/urdf/iiwa7/iiwa7_description.urdf.xacro (robot description, xacro)
@@ -54,5 +54,5 @@
             </collision>
         </link>
-        <joint name="${robot_name}_joint_0" type="revolute">
+        <joint name="${robot_name}_A1" type="revolute">
             <origin rpy="0 0 0" xyz="0.0 0.0 0.1475" />
             <parent link="${robot_name}_link_0" />
@@ -86,5 +86,5 @@
             </collision>
         </link>
-        <joint name="${robot_name}_joint_1" type="revolute">
+        <joint name="${robot_name}_A2" type="revolute">
             <origin rpy="0 0 0" xyz="-0.0 -0.0105 0.193" />
             <parent link="${robot_name}_link_1" />
@@ -118,5 +118,5 @@
             </collision>
         </link>
-        <joint name="${robot_name}_joint_2" type="revolute">
+        <joint name="${robot_name}_A3" type="revolute">
             <origin rpy="0 0 0" xyz="0.0 0.0105 0.1745" />
             <parent link="${robot_name}_link_2" />
@@ -150,5 +150,5 @@
             </collision>
         </link>
-        <joint name="${robot_name}_joint_3" type="revolute">
+        <joint name="${robot_name}_A4" type="revolute">
             <origin rpy="0 0 0" xyz="0.0 0.0105 0.2255" />
             <parent link="${robot_name}_link_3" />
@@ -182,5 +182,5 @@
             </collision>
         </link>
-        <joint name="${robot_name}_joint_4" type="revolute">
+        <joint name="${robot_name}_A5" type="revolute">
             <origin rpy="0 0 0" xyz="0.0 -0.0105 0.1745" />
             <parent link="${robot_name}_link_4" />
@@ -214,5 +214,5 @@
             </collision>
         </link>
-        <joint name="${robot_name}_joint_5" type="revolute">
+        <joint name="${robot_name}_A6" type="revolute">
             <origin rpy="0 0 0" xyz="0.0 -0.0707 0.2255" />
             <parent link="${robot_name}_link_5" />
@@ -246,5 +246,5 @@
             </collision>
         </link>
-        <joint name="${robot_name}_joint_6" type="revolute">
+        <joint name="${robot_name}_A7" type="revolute">
             <origin rpy="0 0 0" xyz="0.0 0.0705 0.0909" />
             <parent link="${robot_name}_link_6" />

File: lbr_description/urdf/med14/med14_description.urdf.xacro (robot description, xacro)
@@ -54,5 +54,5 @@
             </collision>
         </link>
-        <joint name="${robot_name}_joint_0" type="revolute">
+        <joint name="${robot_name}_A1" type="revolute">
             <origin rpy="0 0 0" xyz="0.0 0.0 0.147" />
             <parent link="${robot_name}_link_0" />
@@ -86,5 +86,5 @@
             </collision>
         </link>
-        <joint name="${robot_name}_joint_1" type="revolute">
+        <joint name="${robot_name}_A2" type="revolute">
             <origin rpy="0 0 0" xyz="0.0 -0.01 0.2125" />
             <parent link="${robot_name}_link_1" />
@@ -118,5 +118,5 @@
             </collision>
         </link>
-        <joint name="${robot_name}_joint_2" type="revolute">
+        <joint name="${robot_name}_A3" type="revolute">
             <origin rpy="0 0 0" xyz="-0.0 0.01 0.228" />
             <parent link="${robot_name}_link_2" />
@@ -150,5 +150,5 @@
             </collision>
         </link>
-        <joint name="${robot_name}_joint_3" type="revolute">
+        <joint name="${robot_name}_A4" type="revolute">
             <origin rpy="0 0 0" xyz="0.0 0.0105 0.192" />
             <parent link="${robot_name}_link_3" />
@@ -182,5 +182,5 @@
             </collision>
         </link>
-        <joint name="${robot_name}_joint_4" type="revolute">
+        <joint name="${robot_name}_A5" type="revolute">
             <origin rpy="0 0 0" xyz="0.0 -0.0105 0.2075" />
             <parent link="${robot_name}_link_4" />
@@ -214,5 +214,5 @@
             </collision>
         </link>
-        <joint name="${robot_name}_joint_5" type="revolute">
+        <joint name="${robot_name}_A6" type="revolute">
             <origin rpy="0 0 0" xyz="0.0 -0.0707 0.1925" />
             <parent link="${robot_name}_link_5" />
@@ -246,5 +246,5 @@
             </collision>
         </link>
-        <joint name="${robot_name}_joint_6" type="revolute">
+        <joint name="${robot_name}_A7" type="revolute">
             <origin rpy="0 0 0" xyz="0.0 0.0707 0.091" />
             <parent link="${robot_name}_link_6" />

File: lbr_description/urdf/med7/med7_description.urdf.xacro (robot description, xacro)
@@ -54,5 +54,5 @@
             </collision>
         </link>
-        <joint name="${robot_name}_joint_0" type="revolute">
+        <joint name="${robot_name}_A1" type="revolute">
             <origin rpy="0 0 0" xyz="0.0 0.0 0.1475" />
             <parent link="${robot_name}_link_0" />
@@ -86,5 +86,5 @@
             </collision>
         </link>
-        <joint name="${robot_name}_joint_1" type="revolute">
+        <joint name="${robot_name}_A2" type="revolute">
             <origin rpy="0 0 0" xyz="-0.0 -0.0105 0.1925" />
             <parent link="${robot_name}_link_1" />
@@ -118,5 +118,5 @@
             </collision>
         </link>
-        <joint name="${robot_name}_joint_2" type="revolute">
+        <joint name="${robot_name}_A3" type="revolute">
             <origin rpy="0 0 0" xyz="0.0 0.0105 0.2075" />
             <parent link="${robot_name}_link_2" />
@@ -150,5 +150,5 @@
             </collision>
         </link>
-        <joint name="${robot_name}_joint_3" type="revolute">
+        <joint name="${robot_name}_A4" type="revolute">
             <origin rpy="0 0 0" xyz="0.0 0.0105 0.1925" />
             <parent link="${robot_name}_link_3" />
@@ -182,5 +182,5 @@
             </collision>
         </link>
-        <joint name="${robot_name}_joint_4" type="revolute">
+        <joint name="${robot_name}_A5" type="revolute">
             <origin rpy="0 0 0" xyz="-0.0 -0.0105 0.2075" />
             <parent link="${robot_name}_link_4" />
@@ -214,5 +214,5 @@
             </collision>
         </link>
-        <joint name="${robot_name}_joint_5" type="revolute">
+        <joint name="${robot_name}_A6" type="revolute">
             <origin rpy="0 0 0" xyz="0.0 -0.0707 0.1925" />
             <parent link="${robot_name}_link_5" />
@@ -246,5 +246,5 @@
             </collision>
         </link>
-        <joint name="${robot_name}_joint_6" type="revolute">
+        <joint name="${robot_name}_A7" type="revolute">
             <origin rpy="0 0 0" xyz="0.0 0.0707 0.091" />
             <parent link="${robot_name}_link_6" />

Commit message: hardware interface -> system interface

File: lbr_description/ros2_control/lbr.ros2_control.xacro (robot description, xacro)
@@ -1,5 +1,5 @@
 <?xml version="1.0"?>
 <robot xmlns:xacro="http://www.ros.org/wiki/xacro">
-    <xacro:macro name="lbr_hardware_interface"
+    <xacro:macro name="lbr_system_interface"
         params="
         joint_0_position_limit
@@ -13,5 +13,5 @@
         sim:=^|true port_id:=^|30200 remote_host:=^|INADDR_ANY rt_prio:=^|80">
         <!-- arg for control mode -->
-        <ros2_control name="lbr_hardware_interface" type="system">
+        <ros2_control name="lbr_system_interface" type="system">
             <!-- define hardware including parameters, also gazebo -->
             <xacro:if value="${sim}">
@@ -22,5 +22,5 @@
             <xacro:unless value="${sim}">
                 <hardware>
-                    <plugin>lbr_ros2_control::SystemInterface</plugin>
+                    <plugin>lbr_ros2_control::LBRSystemInterface</plugin>
                     <param name="port_id">${port_id}</param>
                     <param name="remote_host">${remote_host}</param>

File: lbr_description/urdf/iiwa14/iiwa14_description.urdf.xacro (robot description, xacro)
@@ -278,5 +278,5 @@
         <xacro:lbr_gazebo robot_name="${robot_name}" />
         <!-- TODO: move modes to args, decouple urdf/gazebo/controls -->
-        <xacro:lbr_hardware_interface
+        <xacro:lbr_system_interface
             joint_0_position_limit="${joint_0_position_limit * PI / 180}"
             joint_1_position_limit="${joint_1_position_limit * PI / 180}"

File: lbr_description/urdf/iiwa7/iiwa7_description.urdf.xacro (robot description, xacro)
@@ -278,5 +278,5 @@
         <xacro:lbr_gazebo robot_name="${robot_name}" />
         <!-- TODO: move modes to args, decouple urdf/gazebo/controls -->
-        <xacro:lbr_hardware_interface
+        <xacro:lbr_system_interface
             joint_0_position_limit="${joint_0_position_limit * PI / 180}"
             joint_1_position_limit="${joint_1_position_limit * PI / 180}"

File: lbr_description/urdf/med14/med14_description.urdf.xacro (robot description, xacro)
@@ -278,5 +278,5 @@
         <xacro:lbr_gazebo robot_name="${robot_name}" />
         <!-- TODO: move modes to args, decouple urdf/gazebo/controls -->
-        <xacro:lbr_hardware_interface
+        <xacro:lbr_system_interface
             joint_0_position_limit="${joint_0_position_limit * PI / 180}"
             joint_1_position_limit="${joint_1_position_limit * PI / 180}"

File: lbr_description/urdf/med7/med7_description.urdf.xacro (robot description, xacro)
@@ -278,5 +278,5 @@
         <xacro:lbr_gazebo robot_name="${robot_name}" />
         <!-- TODO: move modes to args, decouple urdf/gazebo/controls -->
-        <xacro:lbr_hardware_interface
+        <xacro:lbr_system_interface
             joint_0_position_limit="${joint_0_position_limit * PI / 180}"
             joint_1_position_limit="${joint_1_position_limit * PI / 180}"
