Commit message: added system config to launch arguments

File: lbr_description/ros2_control/lbr_system_interface.xacro (robot description, xacro)
@@ -2,8 +2,8 @@
 <robot xmlns:xacro="http://www.ros.org/wiki/xacro">
     <xacro:macro name="lbr_system_interface"
-        params="robot_name mode joint_limits system_parameters_path">
+        params="robot_name mode joint_limits system_config_path">
         <!-- load system parameters via yaml -->
-        <xacro:property name="system_parameters"
-            value="${xacro.load_yaml(system_parameters_path)}" />
+        <xacro:property name="system_config"
+            value="${xacro.load_yaml(system_config_path)}" />
         <ros2_control name="lbr_system_interface" type="system">
             <!-- load plugin depending on mode -->
@@ -21,20 +21,20 @@
                 <hardware>
                     <plugin>lbr_ros2_control::SystemInterface</plugin>
-                    <param name="fri_client_sdk_major_version">${system_parameters['hardware']['fri_client_sdk']['major_version']}</param>
-                    <param name="fri_client_sdk_minor_version">${system_parameters['hardware']['fri_client_sdk']['minor_version']}</param>
-                    <param name="client_command_mode">${system_parameters['hardware']['client_command_mode']}</param>
-                    <param name="port_id">${system_parameters['hardware']['port_id']}</param>
-                    <param name="remote_host">${system_parameters['hardware']['remote_host']}</param>
-                    <param name="rt_prio">${system_parameters['hardware']['rt_prio']}</param>
-                    <param name="pid_p">${system_parameters['hardware']['pid_p']}</param>
-                    <param name="pid_i">${system_parameters['hardware']['pid_i']}</param>
-                    <param name="pid_d">${system_parameters['hardware']['pid_d']}</param>
-                    <param name="pid_i_max">${system_parameters['hardware']['pid_i_max']}</param>
-                    <param name="pid_i_min">${system_parameters['hardware']['pid_i_min']}</param>
-                    <param name="pid_antiwindup">${system_parameters['hardware']['pid_antiwindup']}</param>
-                    <param name="command_guard_variant">${system_parameters['hardware']['command_guard_variant']}</param>
-                    <param name="external_torque_cutoff_frequency">${system_parameters['hardware']['external_torque_cutoff_frequency']}</param>
-                    <param name="measured_torque_cutoff_frequency">${system_parameters['hardware']['measured_torque_cutoff_frequency']}</param>
-                    <param name="open_loop">${system_parameters['hardware']['open_loop']}</param>
+                    <param name="fri_client_sdk_major_version">${system_config['hardware']['fri_client_sdk']['major_version']}</param>
+                    <param name="fri_client_sdk_minor_version">${system_config['hardware']['fri_client_sdk']['minor_version']}</param>
+                    <param name="client_command_mode">${system_config['hardware']['client_command_mode']}</param>
+                    <param name="port_id">${system_config['hardware']['port_id']}</param>
+                    <param name="remote_host">${system_config['hardware']['remote_host']}</param>
+                    <param name="rt_prio">${system_config['hardware']['rt_prio']}</param>
+                    <param name="pid_p">${system_config['hardware']['pid_p']}</param>
+                    <param name="pid_i">${system_config['hardware']['pid_i']}</param>
+                    <param name="pid_d">${system_config['hardware']['pid_d']}</param>
+                    <param name="pid_i_max">${system_config['hardware']['pid_i_max']}</param>
+                    <param name="pid_i_min">${system_config['hardware']['pid_i_min']}</param>
+                    <param name="pid_antiwindup">${system_config['hardware']['pid_antiwindup']}</param>
+                    <param name="command_guard_variant">${system_config['hardware']['command_guard_variant']}</param>
+                    <param name="external_torque_cutoff_frequency">${system_config['hardware']['external_torque_cutoff_frequency']}</param>
+                    <param name="measured_torque_cutoff_frequency">${system_config['hardware']['measured_torque_cutoff_frequency']}</param>
+                    <param name="open_loop">${system_config['hardware']['open_loop']}</param>
                 </hardware>
             </xacro:if>
@@ -59,13 +59,13 @@
                 <sensor
                     name="estimated_ft_sensor">
-                    <param name="chain_root">${system_parameters['estimated_ft_sensor']['chain_root']}</param>
-                    <param name="chain_tip">${system_parameters['estimated_ft_sensor']['chain_tip']}</param>
-                    <param name="damping">${system_parameters['estimated_ft_sensor']['damping']}</param>
-                    <param name="force_x_th">${system_parameters['estimated_ft_sensor']['force_x_th']}</param>
-                    <param name="force_y_th">${system_parameters['estimated_ft_sensor']['force_y_th']}</param>
-                    <param name="force_z_th">${system_parameters['estimated_ft_sensor']['force_z_th']}</param>
-                    <param name="torque_x_th">${system_parameters['estimated_ft_sensor']['torque_x_th']}</param>
-                    <param name="torque_y_th">${system_parameters['estimated_ft_sensor']['torque_y_th']}</param>
-                    <param name="torque_z_th">${system_parameters['estimated_ft_sensor']['torque_z_th']}</param>
+                    <param name="chain_root">${system_config['estimated_ft_sensor']['chain_root']}</param>
+                    <param name="chain_tip">${system_config['estimated_ft_sensor']['chain_tip']}</param>
+                    <param name="damping">${system_config['estimated_ft_sensor']['damping']}</param>
+                    <param name="force_x_th">${system_config['estimated_ft_sensor']['force_x_th']}</param>
+                    <param name="force_y_th">${system_config['estimated_ft_sensor']['force_y_th']}</param>
+                    <param name="force_z_th">${system_config['estimated_ft_sensor']['force_z_th']}</param>
+                    <param name="torque_x_th">${system_config['estimated_ft_sensor']['torque_x_th']}</param>
+                    <param name="torque_y_th">${system_config['estimated_ft_sensor']['torque_y_th']}</param>
+                    <param name="torque_z_th">${system_config['estimated_ft_sensor']['torque_z_th']}</param>
                     <state_interface name="force.x" />
                     <state_interface name="force.y" />
@@ -110,5 +110,5 @@
                         <param name="max_velocity">${max_velocity}</param>
                         <param name="max_torque">${max_torque}</param>
-                        <xacro:if value="${system_parameters['hardware']['fri_client_sdk']['major_version'] == 1}">
+                        <xacro:if value="${system_config['hardware']['fri_client_sdk']['major_version'] == 1}">
                             <state_interface name="commanded_joint_position" />
                         </xacro:if>

File: lbr_description/urdf/iiwa14/iiwa14.xacro (robot description, xacro)
@@ -7,6 +7,6 @@
     <xacro:arg name="mode" default="true" />
     <xacro:arg
-        name="system_parameters_path"
-        default="$(find lbr_description)/ros2_control/lbr_system_parameters.yaml" />
+        name="system_config_path"
+        default="$(find lbr_description)/ros2_control/lbr_system_config.yaml" />
     <!-- fixed to world, see http://classic.gazebosim.org/tutorials?tut=ros_urdf&cat=connect_ros -->
     <link name="world" />
@@ -21,4 +21,4 @@
         robot_name="$(arg robot_name)"
         mode="$(arg mode)"
-        system_parameters_path="$(arg system_parameters_path)" />
+        system_config_path="$(arg system_config_path)" />
 </robot>

File: lbr_description/urdf/iiwa14/iiwa14_description.xacro (robot description, xacro)
@@ -3,5 +3,5 @@
     <!-- robot as extracted via https://github.com/syuntoku14/fusion2urdf -->
     <xacro:macro name="iiwa14"
-        params="robot_name:=^|lbr mode:=^|mock system_parameters_path:=^|'$(find lbr_description)/ros2_control/lbr_system_parameters.yaml'">
+        params="robot_name:=^|lbr mode:=^|mock system_config_path:=^|'$(find lbr_description)/ros2_control/lbr_system_config.yaml'">
         <!-- includes -->
         <xacro:include filename="$(find lbr_description)/gazebo/lbr_gazebo.xacro" />
@@ -21,5 +21,5 @@
             mode="${mode}"
             joint_limits="${joint_limits}"
-            system_parameters_path="${system_parameters_path}" />
+            system_config_path="${system_config_path}" />
         <link name="${robot_name}_link_0">
             <inertial>

File: lbr_description/urdf/iiwa7/iiwa7.xacro (robot description, xacro)
@@ -7,6 +7,6 @@
     <xacro:arg name="mode" default="mock" />
     <xacro:arg
-        name="system_parameters_path"
-        default="$(find lbr_description)/ros2_control/lbr_system_parameters.yaml" />
+        name="system_config_path"
+        default="$(find lbr_description)/ros2_control/lbr_system_config.yaml" />
     <!-- fixed to world, see http://classic.gazebosim.org/tutorials?tut=ros_urdf&cat=connect_ros -->
     <link name="world" />
@@ -21,4 +21,4 @@
         robot_name="$(arg robot_name)"
         mode="$(arg mode)"
-        system_parameters_path="$(arg system_parameters_path)" />
+        system_config_path="$(arg system_config_path)" />
 </robot>

File: lbr_description/urdf/iiwa7/iiwa7_description.xacro (robot description, xacro)
@@ -3,5 +3,5 @@
     <!-- robot as extracted via https://github.com/syuntoku14/fusion2urdf -->
     <xacro:macro name="iiwa7"
-        params="robot_name:=^|lbr mode:=^|mock system_parameters_path:=^|'$(find lbr_description)/ros2_control/lbr_system_parameters.yaml'">
+        params="robot_name:=^|lbr mode:=^|mock system_config_path:=^|'$(find lbr_description)/ros2_control/lbr_system_config.yaml'">
         <!-- includes -->
         <xacro:include filename="$(find lbr_description)/gazebo/lbr_gazebo.xacro" />
@@ -21,5 +21,5 @@
             mode="${mode}"
             joint_limits="${joint_limits}"
-            system_parameters_path="${system_parameters_path}" />
+            system_config_path="${system_config_path}" />
         <link name="${robot_name}_link_0">
             <inertial>

File: lbr_description/urdf/med14/med14.xacro (robot description, xacro)
@@ -7,6 +7,6 @@
     <xacro:arg name="mode" default="true" />
     <xacro:arg
-        name="system_parameters_path"
-        default="$(find lbr_description)/ros2_control/lbr_system_parameters.yaml" />
+        name="system_config_path"
+        default="$(find lbr_description)/ros2_control/lbr_system_config.yaml" />
     <!-- fixed to world, see http://classic.gazebosim.org/tutorials?tut=ros_urdf&cat=connect_ros -->
     <link name="world" />
@@ -21,4 +21,4 @@
         robot_name="$(arg robot_name)"
         mode="$(arg mode)"
-        system_parameters_path="$(arg system_parameters_path)" />
+        system_config_path="$(arg system_config_path)" />
 </robot>

File: lbr_description/urdf/med14/med14_description.xacro (robot description, xacro)
@@ -3,5 +3,5 @@
     <!-- robot as extracted via https://github.com/syuntoku14/fusion2urdf -->
     <xacro:macro name="med14"
-        params="robot_name:=^|lbr mode:=^|mock system_parameters_path:=^|'$(find lbr_description)/ros2_control/lbr_system_parameters.yaml'">
+        params="robot_name:=^|lbr mode:=^|mock system_config_path:=^|'$(find lbr_description)/ros2_control/lbr_system_config.yaml'">
         <!-- includes -->
         <xacro:include filename="$(find lbr_description)/gazebo/lbr_gazebo.xacro" />
@@ -21,5 +21,5 @@
             mode="${mode}"
             joint_limits="${joint_limits}"
-            system_parameters_path="${system_parameters_path}" />
+            system_config_path="${system_config_path}" />
         <link name="${robot_name}_link_0">
             <inertial>

File: lbr_description/urdf/med7/med7.xacro (robot description, xacro)
@@ -7,6 +7,6 @@
     <xacro:arg name="mode" default="true" />
     <xacro:arg
-        name="system_parameters_path"
-        default="$(find lbr_description)/ros2_control/lbr_system_parameters.yaml" />
+        name="system_config_path"
+        default="$(find lbr_description)/ros2_control/lbr_system_config.yaml" />
     <!-- fixed to world, see http://classic.gazebosim.org/tutorials?tut=ros_urdf&cat=connect_ros -->
     <link name="world" />
@@ -21,4 +21,4 @@
         robot_name="$(arg robot_name)"
         mode="$(arg mode)"
-        system_parameters_path="$(arg system_parameters_path)" />
+        system_config_path="$(arg system_config_path)" />
 </robot>

File: lbr_description/urdf/med7/med7_description.xacro (robot description, xacro)
@@ -3,5 +3,5 @@
     <!-- robot as extracted via https://github.com/syuntoku14/fusion2urdf -->
     <xacro:macro name="med7"
-        params="robot_name:=^|lbr mode:=^|mock system_parameters_path:=^|'$(find lbr_description)/ros2_control/lbr_system_parameters.yaml'">
+        params="robot_name:=^|lbr mode:=^|mock system_config_path:=^|'$(find lbr_description)/ros2_control/lbr_system_config.yaml'">
         <!-- includes -->
         <xacro:include filename="$(find lbr_description)/gazebo/lbr_gazebo.xacro" />
@@ -21,5 +21,5 @@
             mode="${mode}"
             joint_limits="${joint_limits}"
-            system_parameters_path="${system_parameters_path}" />
+            system_config_path="${system_config_path}" />
         <!-- properties -->
         <link name="${robot_name}_link_0">
