Commit message: de-couple URDF (#349)

File: lbr_description/ros2_control/lbr_system_interface.xacro (robot description, xacro)
@@ -2,5 +2,5 @@
 <robot xmlns:xacro="http://www.ros.org/wiki/xacro">
     <xacro:macro name="lbr_system_interface"
-        params="robot_name mode joint_limits system_config_path initial_joint_positions_path">
+        params="robot_name mode system_config_path initial_joint_positions_path">
         <!-- load system parameters via yaml -->
         <xacro:property name="system_config"
@@ -9,4 +9,6 @@
         <xacro:property name="initial_joint_positions"
             value="${xacro.load_yaml(initial_joint_positions_path)}" />
+        <!-- constants -->
+        <xacro:property name="PI" value="3.1415926535897931" />
         <ros2_control name="${robot_name}_system_interface" type="system">
             <!-- load plugin depending on mode -->
@@ -70,17 +72,11 @@
             <!-- define joints and command/state interfaces for each joint -->
             <xacro:macro name="joint_interface"
-                params="name min_position max_position max_velocity max_torque mode initial_position">
+                params="name mode initial_position">
                 <joint name="${name}">
-                    <command_interface name="position">
-                        <param name="min">${min_position}</param>
-                        <param name="max">${max_position}</param>
-                    </command_interface>
+                    <command_interface name="position"/>
                     <!-- only single command interface, refer
                     https://github.com/ros-controls/gz_ros2_control/issues/182 -->
                     <xacro:unless value="${mode == 'gazebo'}">
-                        <command_interface name="effort">
-                            <param name="min">-${max_torque}</param>
-                            <param name="max"> ${max_torque}</param>
-                        </command_interface>
+                        <command_interface name="effort"/>
                     </xacro:unless>
                     <state_interface name="position">
@@ -90,8 +86,4 @@
                     <state_interface name="effort" />
                     <xacro:if value="${mode == 'hardware'}">
-                        <param name="min_position">${min_position}</param>
-                        <param name="max_position">${max_position}</param>
-                        <param name="max_velocity">${max_velocity}</param>
-                        <param name="max_torque">${max_torque}</param>
                         <xacro:if
                             value="${system_config['fri_client_sdk']['major_version'] == 1}">
@@ -105,50 +97,22 @@
             </xacro:macro>
             <xacro:joint_interface name="${robot_name}_A1"
-                min_position="${joint_limits['A1']['lower'] * PI / 180}"
-                max_position="${joint_limits['A1']['upper'] * PI / 180}"
-                max_velocity="${joint_limits['A1']['velocity'] * PI / 180}"
-                max_torque="${joint_limits['A1']['effort']}"
                 mode="${mode}"
                 initial_position="${initial_joint_positions['A1'] * PI / 180}" />
             <xacro:joint_interface name="${robot_name}_A2"
-                min_position="${joint_limits['A2']['lower'] * PI / 180}"
-                max_position="${joint_limits['A2']['upper'] * PI / 180}"
-                max_velocity="${joint_limits['A2']['velocity'] * PI / 180}"
-                max_torque="${joint_limits['A2']['effort']}"
                 mode="${mode}"
                 initial_position="${initial_joint_positions['A2'] * PI / 180}" />
             <xacro:joint_interface name="${robot_name}_A3"
-                min_position="${joint_limits['A3']['lower'] * PI / 180}"
-                max_position="${joint_limits['A3']['upper'] * PI / 180}"
-                max_velocity="${joint_limits['A3']['velocity'] * PI / 180}"
-                max_torque="${joint_limits['A3']['effort']}"
                 mode="${mode}"
                 initial_position="${initial_joint_positions['A3'] * PI / 180}" />
             <xacro:joint_interface name="${robot_name}_A4"
-                min_position="${joint_limits['A4']['lower'] * PI / 180}"
-                max_position="${joint_limits['A4']['upper'] * PI / 180}"
-                max_velocity="${joint_limits['A4']['velocity'] * PI / 180}"
-                max_torque="${joint_limits['A4']['effort']}"
                 mode="${mode}"
                 initial_position="${initial_joint_positions['A4'] * PI / 180}"/>
             <xacro:joint_interface name="${robot_name}_A5"
-                min_position="${joint_limits['A5']['lower'] * PI / 180}"
-                max_position="${joint_limits['A5']['upper'] * PI / 180}"
-                max_velocity="${joint_limits['A5']['velocity'] * PI / 180}"
-                max_torque="${joint_limits['A5']['effort']}"
                 mode="${mode}"
                 initial_position="${initial_joint_positions['A5'] * PI / 180}"/>
             <xacro:joint_interface name="${robot_name}_A6"
-                min_position="${joint_limits['A6']['lower'] * PI / 180}"
-                max_position="${joint_limits['A6']['upper'] * PI / 180}"
-                max_velocity="${joint_limits['A6']['velocity'] * PI / 180}"
-                max_torque="${joint_limits['A6']['effort']}"
                 mode="${mode}"
                 initial_position="${initial_joint_positions['A6'] * PI / 180}" />
             <xacro:joint_interface name="${robot_name}_A7"
-                min_position="${joint_limits['A7']['lower'] * PI / 180}"
-                max_position="${joint_limits['A7']['upper'] * PI / 180}"
-                max_velocity="${joint_limits['A7']['velocity'] * PI / 180}"
-                max_torque="${joint_limits['A7']['effort']}"
                 mode="${mode}"
                 initial_position="${initial_joint_positions['A7'] * PI / 180}" />

File: lbr_description/urdf/iiwa14/iiwa14.urdf.xacro (robot description, xacro)
@@ -3,9 +3,6 @@
     <!-- robot as extracted via https://github.com/syuntoku14/fusion2urdf -->
     <xacro:macro name="iiwa14"
-        params="robot_name:=^|lbr mode:=^|mock system_config_path:=^|'$(find lbr_description)/ros2_control/lbr_system_config.yaml' joint_limits_path:=^|'$(find lbr_description)/urdf/iiwa14/joint_limits.yaml' initial_joint_positions_path:=^|'$(find lbr_description)/ros2_control/initial_joint_positions.yaml'">
-        <!-- includes -->
-        <xacro:include filename="$(find lbr_description)/gazebo/lbr_gazebo.xacro" />
-        <xacro:include filename="$(find lbr_description)/ros2_control/lbr_system_interface.xacro" />
-        <!-- joint limits via yaml -->
+        params="robot_name:=^|lbr joint_limits_path:=^|'$(find lbr_description)/urdf/iiwa14/joint_limits.yaml'">
+        <!-- load joint limits via yaml -->
         <xacro:property name="joint_limits" value="${xacro.load_yaml(joint_limits_path)}" />
         <!-- constants -->
@@ -13,12 +10,5 @@
         <xacro:property name="joint_damping" value="10.0" />
         <xacro:property name="joint_friction" value="0.1" />
-        <!-- macros for gazebo / mock / hardware -->
-        <xacro:lbr_gazebo robot_name="${robot_name}" />
-        <xacro:lbr_system_interface
-            robot_name="${robot_name}"
-            mode="${mode}"
-            joint_limits="${joint_limits}"
-            system_config_path="${system_config_path}"
-            initial_joint_positions_path="${initial_joint_positions_path}" />
+        <!-- links and joints -->
         <link name="${robot_name}_link_0">
             <inertial>

File: lbr_description/urdf/iiwa14/iiwa14.xacro (robot description, xacro)
@@ -2,14 +2,17 @@
 <!-- top level -->
 <robot name="iiwa14" xmlns:xacro="http://www.ros.org/wiki/xacro">
-    <!-- include the lbr iiwa macro -->
-    <xacro:include filename="$(find lbr_description)/urdf/iiwa14/iiwa14_description.xacro" />
+    <!-- include the iiwa macro and controller -->
+    <xacro:include filename="$(find lbr_description)/urdf/iiwa14/iiwa14.urdf.xacro" />
+    <xacro:include filename="$(find lbr_description)/gazebo/lbr_gazebo.xacro" />
+    <xacro:include filename="$(find lbr_description)/ros2_control/lbr_system_interface.xacro" />
+    <!-- arguments -->
     <xacro:arg name="robot_name" default="lbr" />
     <xacro:arg name="mode" default="true" />
     <xacro:arg
+        name="joint_limits_path"
+        default="$(find lbr_description)/urdf/iiwa14/joint_limits.yaml" />
+    <xacro:arg
         name="system_config_path"
         default="$(find lbr_description)/ros2_control/lbr_system_config.yaml" />
-    <xacro:arg
-        name="joint_limits_path"
-        default="$(find lbr_description)/urdf/iiwa14/joint_limits.yaml" />
     <xacro:arg
         name="initial_joint_positions_path"
@@ -24,10 +27,14 @@
         <child link="$(arg robot_name)_link_0" />
     </joint>
-    <!-- iiwa -->
-    <xacro:iiwa14
+    <!-- macros for gazebo / mock / hardware -->
+    <xacro:lbr_gazebo robot_name="$(arg robot_name)" />
+    <xacro:lbr_system_interface
         robot_name="$(arg robot_name)"
         mode="$(arg mode)"
         system_config_path="$(arg system_config_path)"
-        joint_limits_path="$(arg joint_limits_path)"
         initial_joint_positions_path="$(arg initial_joint_positions_path)" />
+    <!-- iiwa description -->
+    <xacro:iiwa14
+        robot_name="$(arg robot_name)"
+        joint_limits_path="$(arg joint_limits_path)" />
 </robot>

File: lbr_description/urdf/iiwa7/iiwa7.urdf.xacro (robot description, xacro)
@@ -3,9 +3,6 @@
     <!-- robot as extracted via https://github.com/syuntoku14/fusion2urdf -->
     <xacro:macro name="iiwa7"
-        params="robot_name:=^|lbr mode:=^|mock system_config_path:=^|'$(find lbr_description)/ros2_control/lbr_system_config.yaml' joint_limits_path:=^|'$(find lbr_description)/urdf/iiwa7/joint_limits.yaml' initial_joint_positions_path:=^|'$(find lbr_description)/ros2_control/initial_joint_positions.yaml'">
-        <!-- includes -->
-        <xacro:include filename="$(find lbr_description)/gazebo/lbr_gazebo.xacro" />
-        <xacro:include filename="$(find lbr_description)/ros2_control/lbr_system_interface.xacro" />
-        <!-- joint limits via yaml -->
+        params="robot_name:=^|lbr joint_limits_path:=^|'$(find lbr_description)/urdf/iiwa7/joint_limits.yaml'">
+        <!-- load joint limits via yaml -->
         <xacro:property name="joint_limits" value="${xacro.load_yaml(joint_limits_path)}" />
         <!-- constants -->
@@ -13,12 +10,5 @@
         <xacro:property name="joint_damping" value="10.0" />
         <xacro:property name="joint_friction" value="0.1" />
-        <!-- macros for gazebo / mock / hardware -->
-        <xacro:lbr_gazebo robot_name="${robot_name}" />
-        <xacro:lbr_system_interface
-            robot_name="${robot_name}"
-            mode="${mode}"
-            joint_limits="${joint_limits}"
-            system_config_path="${system_config_path}"
-            initial_joint_positions_path="${initial_joint_positions_path}" />
+        <!-- links and joints -->
         <link name="${robot_name}_link_0">
             <inertial>

File: lbr_description/urdf/iiwa7/iiwa7.xacro (robot description, xacro)
@@ -2,14 +2,17 @@
 <!-- top level -->
 <robot name="iiwa7" xmlns:xacro="http://www.ros.org/wiki/xacro">
-    <!-- include the lbr iiwa macro -->
-    <xacro:include filename="$(find lbr_description)/urdf/iiwa7/iiwa7_description.xacro" />
+    <!-- include the iiwa macro and controller -->
+    <xacro:include filename="$(find lbr_description)/urdf/iiwa7/iiwa7.urdf.xacro" />
+    <xacro:include filename="$(find lbr_description)/gazebo/lbr_gazebo.xacro" />
+    <xacro:include filename="$(find lbr_description)/ros2_control/lbr_system_interface.xacro" />
+    <!-- arguments -->
     <xacro:arg name="robot_name" default="lbr" />
     <xacro:arg name="mode" default="mock" />
     <xacro:arg
+        name="joint_limits_path"
+        default="$(find lbr_description)/urdf/iiwa7/joint_limits.yaml" />
+    <xacro:arg
         name="system_config_path"
         default="$(find lbr_description)/ros2_control/lbr_system_config.yaml" />
-    <xacro:arg
-        name="joint_limits_path"
-        default="$(find lbr_description)/urdf/iiwa7/joint_limits.yaml" />
     <xacro:arg
         name="initial_joint_positions_path"
@@ -24,10 +27,14 @@
         <child link="$(arg robot_name)_link_0" />
     </joint>
-    <!-- iiwa -->
-    <xacro:iiwa7
+    <!-- macros for gazebo / mock / hardware -->
+    <xacro:lbr_gazebo robot_name="$(arg robot_name)" />
+    <xacro:lbr_system_interface
         robot_name="$(arg robot_name)"
         mode="$(arg mode)"
         system_config_path="$(arg system_config_path)"
-        joint_limits_path="$(arg joint_limits_path)"
         initial_joint_positions_path="$(arg initial_joint_positions_path)" />
+    <!-- iiwa description -->
+    <xacro:iiwa7
+        robot_name="$(arg robot_name)"
+        joint_limits_path="$(arg joint_limits_path)" />
 </robot>

File: lbr_description/urdf/med14/med14.urdf.xacro (robot description, xacro)
@@ -3,9 +3,6 @@
     <!-- robot as extracted via https://github.com/syuntoku14/fusion2urdf -->
     <xacro:macro name="med14"
-        params="robot_name:=^|lbr mode:=^|mock system_config_path:=^|'$(find lbr_description)/ros2_control/lbr_system_config.yaml' joint_limits_path:=^|'$(find lbr_description)/urdf/med14/joint_limits.yaml' initial_joint_positions_path:=^|'$(find lbr_description)/ros2_control/initial_joint_positions.yaml'">
-        <!-- includes -->
-        <xacro:include filename="$(find lbr_description)/gazebo/lbr_gazebo.xacro" />
-        <xacro:include filename="$(find lbr_description)/ros2_control/lbr_system_interface.xacro" />
-        <!-- joint limits via yaml -->
+        params="robot_name:=^|lbr joint_limits_path:=^|'$(find lbr_description)/urdf/med14/joint_limits.yaml'">
+        <!-- load joint limits via yaml -->
         <xacro:property name="joint_limits" value="${xacro.load_yaml(joint_limits_path)}" />
         <!-- constants -->
@@ -13,12 +10,5 @@
         <xacro:property name="joint_damping" value="10.0" />
         <xacro:property name="joint_friction" value="0.1" />
-        <!-- macros for gazebo / mock / hardware -->
-        <xacro:lbr_gazebo robot_name="${robot_name}" />
-        <xacro:lbr_system_interface
-            robot_name="${robot_name}"
-            mode="${mode}"
-            joint_limits="${joint_limits}"
-            system_config_path="${system_config_path}"
-            initial_joint_positions_path="${initial_joint_positions_path}" />
+        <!-- links and joints -->
         <link name="${robot_name}_link_0">
             <inertial>

File: lbr_description/urdf/med14/med14.xacro (robot description, xacro)
@@ -2,14 +2,17 @@
 <!-- top level -->
 <robot name="med14" xmlns:xacro="http://www.ros.org/wiki/xacro">
-    <!-- include the lbr med macro -->
-    <xacro:include filename="$(find lbr_description)/urdf/med14/med14_description.xacro" />
+    <!-- include the med macro and controller -->
+    <xacro:include filename="$(find lbr_description)/urdf/med14/med14.urdf.xacro" />
+    <xacro:include filename="$(find lbr_description)/gazebo/lbr_gazebo.xacro" />
+    <xacro:include filename="$(find lbr_description)/ros2_control/lbr_system_interface.xacro" />
+    <!-- arguments -->
     <xacro:arg name="robot_name" default="lbr" />
     <xacro:arg name="mode" default="true" />
     <xacro:arg
+        name="joint_limits_path"
+        default="$(find lbr_description)/urdf/med14/joint_limits.yaml" />
+    <xacro:arg
         name="system_config_path"
         default="$(find lbr_description)/ros2_control/lbr_system_config.yaml" />
-    <xacro:arg
-        name="joint_limits_path"
-        default="$(find lbr_description)/urdf/med14/joint_limits.yaml" />
     <xacro:arg
         name="initial_joint_positions_path"
@@ -24,10 +27,14 @@
         <child link="$(arg robot_name)_link_0" />
     </joint>
-    <!-- med -->
-    <xacro:med14
+    <!-- macros for gazebo / mock / hardware -->
+    <xacro:lbr_gazebo robot_name="$(arg robot_name)" />
+    <xacro:lbr_system_interface
         robot_name="$(arg robot_name)"
         mode="$(arg mode)"
         system_config_path="$(arg system_config_path)"
-        joint_limits_path="$(arg joint_limits_path)"
         initial_joint_positions_path="$(arg initial_joint_positions_path)" />
+    <!-- med description -->
+    <xacro:med14
+        robot_name="$(arg robot_name)"
+        joint_limits_path="$(arg joint_limits_path)" />
 </robot>

File: lbr_description/urdf/med7/med7.urdf.xacro (robot description, xacro)
@@ -3,9 +3,6 @@
     <!-- robot as extracted via https://github.com/syuntoku14/fusion2urdf -->
     <xacro:macro name="med7"
-        params="robot_name:=^|lbr mode:=^|mock system_config_path:=^|'$(find lbr_description)/ros2_control/lbr_system_config.yaml' joint_limits_path:=^|'$(find lbr_description)/urdf/med7/joint_limits.yaml' initial_joint_positions_path:=^|'$(find lbr_description)/ros2_control/initial_joint_positions.yaml'">
-        <!-- includes -->
-        <xacro:include filename="$(find lbr_description)/gazebo/lbr_gazebo.xacro" />
-        <xacro:include filename="$(find lbr_description)/ros2_control/lbr_system_interface.xacro" />
-        <!-- joint limits via yaml -->
+        params="robot_name:=^|lbr joint_limits_path:=^|'$(find lbr_description)/urdf/med7/joint_limits.yaml'">
+        <!-- load joint limits via yaml -->
         <xacro:property name="joint_limits" value="${xacro.load_yaml(joint_limits_path)}" />
         <!-- constants -->
@@ -13,13 +10,5 @@
         <xacro:property name="joint_damping" value="10.0" />
         <xacro:property name="joint_friction" value="0.1" />
-        <!-- macros for gazebo / mock / hardware -->
-        <xacro:lbr_gazebo robot_name="${robot_name}" />
-        <xacro:lbr_system_interface
-            robot_name="${robot_name}"
-            mode="${mode}"
-            joint_limits="${joint_limits}"
-            system_config_path="${system_config_path}"
-            initial_joint_positions_path="${initial_joint_positions_path}" />
-        <!-- properties -->
+        <!-- links and joints -->
         <link name="${robot_name}_link_0">
             <inertial>

File: lbr_description/urdf/med7/med7.xacro (robot description, xacro)
@@ -2,14 +2,17 @@
 <!-- top level -->
 <robot name="med7" xmlns:xacro="http://www.ros.org/wiki/xacro">
-    <!-- include the lbr med macro -->
-    <xacro:include filename="$(find lbr_description)/urdf/med7/med7_description.xacro" />
+    <!-- include the med macro and controller -->
+    <xacro:include filename="$(find lbr_description)/urdf/med7/med7.urdf.xacro" />
+    <xacro:include filename="$(find lbr_description)/gazebo/lbr_gazebo.xacro" />
+    <xacro:include filename="$(find lbr_description)/ros2_control/lbr_system_interface.xacro" />
+    <!-- arguments -->
     <xacro:arg name="robot_name" default="lbr" />
     <xacro:arg name="mode" default="true" />
     <xacro:arg
+        name="joint_limits_path"
+        default="$(find lbr_description)/urdf/med7/joint_limits.yaml" />
+    <xacro:arg
         name="system_config_path"
         default="$(find lbr_description)/ros2_control/lbr_system_config.yaml" />
-    <xacro:arg
-        name="joint_limits_path"
-        default="$(find lbr_description)/urdf/med7/joint_limits.yaml" />
     <xacro:arg
         name="initial_joint_positions_path"
@@ -24,10 +27,14 @@
         <child link="$(arg robot_name)_link_0" />
     </joint>
-    <!-- med -->
-    <xacro:med7
+    <!-- macros for gazebo / mock / hardware -->
+    <xacro:lbr_gazebo robot_name="$(arg robot_name)" />
+    <xacro:lbr_system_interface
         robot_name="$(arg robot_name)"
         mode="$(arg mode)"
         system_config_path="$(arg system_config_path)"
-        joint_limits_path="$(arg joint_limits_path)"
         initial_joint_positions_path="$(arg initial_joint_positions_path)" />
+    <!-- med description -->
+    <xacro:med7
+        robot_name="$(arg robot_name)"
+        joint_limits_path="$(arg joint_limits_path)" />
 </robot>
