Commit message: removed redundancy

File: lbr_ros2_control/config/lbr_system_interface.xacro (robot description, xacro)
@@ -3,11 +3,11 @@
     <xacro:macro name="lbr_system_interface"
         params="
-        joint_0_position_limit
-        joint_1_position_limit
-        joint_2_position_limit
-        joint_3_position_limit
-        joint_4_position_limit
-        joint_5_position_limit
-        joint_6_position_limit
+        A1_position_limit
+        A2_position_limit
+        A3_position_limit
+        A4_position_limit
+        A5_position_limit
+        A6_position_limit
+        A7_position_limit
         effort_limit
         sim:=^|true port_id:=^|30200 remote_host:=^|INADDR_ANY rt_prio:=^|80 open_loop:=^|true">
@@ -49,138 +49,40 @@
             </xacro:unless>
             <!-- define joints and command/state interfaces for each joint -->
-            <joint name="A1">
-                <command_interface name="position">
-                    <!-- better to use radians as min max first -->
-                    <param name="min">-${joint_0_position_limit}</param>
-                    <param name="max"> ${joint_0_position_limit}</param>
-                </command_interface>
-                <command_interface name="effort">
-                    <param name="min">-${effort_limit}</param>
-                    <param name="max"> ${effort_limit}</param>
-                </command_interface>
-                <state_interface name="position" />
-                <state_interface name="velocity" />
-                <state_interface name="effort" />
-                <xacro:unless value="${sim}">
-                    <state_interface name="commanded_joint_position" />
-                    <state_interface name="commanded_torque" />
-                    <state_interface name="external_torque" />
-                    <state_interface name="ipo_joint_position" />
-                </xacro:unless>
-            </joint>
-            <joint name="A2">
-                <command_interface name="position">
-                    <param name="min">-${joint_1_position_limit}</param>
-                    <param name="max"> ${joint_1_position_limit}</param>
-                </command_interface>
-                <command_interface name="effort">
-                    <param name="min">-${effort_limit}</param>
-                    <param name="max"> ${effort_limit}</param>
-                </command_interface>
-                <state_interface name="position" />
-                <state_interface name="velocity" />
-                <state_interface name="effort" />
-                <xacro:unless value="${sim}">
-                    <state_interface name="commanded_joint_position" />
-                    <state_interface name="commanded_torque" />
-                    <state_interface name="external_torque" />
-                    <state_interface name="ipo_joint_position" />
-                </xacro:unless>
-            </joint>
-            <joint name="A3">
-                <command_interface name="position">
-                    <param name="min">-${joint_2_position_limit}</param>
-                    <param name="max"> ${joint_2_position_limit}</param>
-                </command_interface>
-                <command_interface name="effort">
-                    <param name="min">-${effort_limit}</param>
-                    <param name="max"> ${effort_limit}</param>
-                </command_interface>
-                <state_interface name="position" />
-                <state_interface name="velocity" />
-                <state_interface name="effort" />
-                <xacro:unless value="${sim}">
-                    <state_interface name="commanded_joint_position" />
-                    <state_interface name="commanded_torque" />
-                    <state_interface name="external_torque" />
-                    <state_interface name="ipo_joint_position" />
-                </xacro:unless>
-            </joint>
-            <joint name="A4">
-                <command_interface name="position">
-                    <param name="min">-${joint_3_position_limit}</param>
-                    <param name="max"> ${joint_3_position_limit}</param>
-                </command_interface>
-                <command_interface name="effort">
-                    <param name="min">-${effort_limit}</param>
-                    <param name="max"> ${effort_limit}</param>
-                </command_interface>
-                <state_interface name="position" />
-                <state_interface name="velocity" />
-                <state_interface name="effort" />
-                <xacro:unless value="${sim}">
-                    <state_interface name="commanded_joint_position" />
-                    <state_interface name="commanded_torque" />
-                    <state_interface name="external_torque" />
-                    <state_interface name="ipo_joint_position" />
-                </xacro:unless>
-            </joint>
-            <joint name="A5">
-                <command_interface name="position">
-                    <param name="min">-${joint_4_position_limit}</param>
-                    <param name="max"> ${joint_4_position_limit}</param>
-                </command_interface>
-                <command_interface name="effort">
-                    <param name="min">-${effort_limit}</param>
-                    <param name="max"> ${effort_limit}</param>
-                </command_interface>
-                <state_interface name="position" />
-                <state_interface name="velocity" />
-                <state_interface name="effort" />
-                <xacro:unless value="${sim}">
-                    <state_interface name="commanded_joint_position" />
-                    <state_interface name="commanded_torque" />
-                    <state_interface name="external_torque" />
-                    <state_interface name="ipo_joint_position" />
-                </xacro:unless>
-            </joint>
-            <joint name="A6">
-                <command_interface name="position">
-                    <param name="min">-${joint_5_position_limit}</param>
-                    <param name="max"> ${joint_5_position_limit}</param>
-                </command_interface>
-                <command_interface name="effort">
-                    <param name="min">-${effort_limit}</param>
-                    <param name="max"> ${effort_limit}</param>
-                </command_interface>
-                <state_interface name="position" />
-                <state_interface name="velocity" />
-                <state_interface name="effort" />
-                <xacro:unless value="${sim}">
-                    <state_interface name="commanded_joint_position" />
-                    <state_interface name="commanded_torque" />
-                    <state_interface name="external_torque" />
-                    <state_interface name="ipo_joint_position" />
-                </xacro:unless>
-            </joint>
-            <joint name="A7">
-                <command_interface name="position">
-                    <param name="min">-${joint_6_position_limit}</param>
-                    <param name="max"> ${joint_6_position_limit}</param>
-                </command_interface>
-                <command_interface name="effort">
-                    <param name="min">-${effort_limit}</param>
-                    <param name="max"> ${effort_limit}</param>
-                </command_interface>
-                <state_interface name="position" />
-                <state_interface name="velocity" />
-                <state_interface name="effort" />
-                <xacro:unless value="${sim}">
-                    <state_interface name="commanded_joint_position" />
-                    <state_interface name="commanded_torque" />
-                    <state_interface name="external_torque" />
-                    <state_interface name="ipo_joint_position" />
-                </xacro:unless>
-            </joint>
+            <xacro:macro name="joint_interface"
+                params="name min_position max_position effort_limit sim">
+                <joint name="${name}">
+                    <command_interface name="position">
+                        <param name="min">${min_position}</param>
+                        <param name="max">${max_position}</param>
+                    </command_interface>
+                    <command_interface name="effort">
+                        <param name="min">-${effort_limit}</param>
+                        <param name="max"> ${effort_limit}</param>
+                    </command_interface>
+                    <state_interface name="position" />
+                    <state_interface name="velocity" />
+                    <state_interface name="effort" />
+                    <xacro:unless value="${sim}">
+                        <state_interface name="commanded_joint_position" />
+                        <state_interface name="commanded_torque" />
+                        <state_interface name="external_torque" />
+                        <state_interface name="ipo_joint_position" />
+                    </xacro:unless>
+                </joint>
+            </xacro:macro>
+            <xacro:joint_interface name="A1" min_position="-${A1_position_limit}"
+                max_position="${A1_position_limit}" effort_limit="${effort_limit}" sim="${sim}" />
+            <xacro:joint_interface name="A2" min_position="-${A2_position_limit}"
+                max_position="${A2_position_limit}" effort_limit="${effort_limit}" sim="${sim}" />
+            <xacro:joint_interface name="A3" min_position="-${A3_position_limit}"
+                max_position="${A3_position_limit}" effort_limit="${effort_limit}" sim="${sim}" />
+            <xacro:joint_interface name="A4" min_position="-${A4_position_limit}"
+                max_position="${A4_position_limit}" effort_limit="${effort_limit}" sim="${sim}" />
+            <xacro:joint_interface name="A5" min_position="-${A5_position_limit}"
+                max_position="${A5_position_limit}" effort_limit="${effort_limit}" sim="${sim}" />
+            <xacro:joint_interface name="A6" min_position="-${A6_position_limit}"
+                max_position="${A6_position_limit}" effort_limit="${effort_limit}" sim="${sim}" />
+            <xacro:joint_interface name="A7" min_position="-${A7_position_limit}"
+                max_position="${A7_position_limit}" effort_limit="${effort_limit}" sim="${sim}" />
         </ros2_control>
     </xacro:macro>
