Commit message: removed unused params

File: lbr_description/urdf/iiwa14/iiwa14_description.urdf.xacro (robot description, xacro)
@@ -3,6 +3,4 @@
     <!-- some constants -->
     <xacro:property name="PI" value="3.1415926535897931"/>
-    <xacro:property name="safety_controller_k_pos" value="100"/>
-    <xacro:property name="safety_controller_k_vel" value="2"/>
     <xacro:property name="joint_damping" value="10.0"/>
     <xacro:property name="joint_friction" value="0.1"/>
@@ -43,12 +41,6 @@
             <parent link="${robot_name}_link_0"/>
             <child link="${robot_name}_link_1"/>
-            <axis xyz="0.0 0.0 0.01"/>
+            <axis xyz="0.0 0.0 1.0"/>
             <limit effort="${max_effort}" lower="${-170 * PI / 180}" upper="${170 * PI / 180}" velocity="${max_velocity}"/>
-            <safety_controller
-                soft_lower_limit="${-168 * PI / 180}"
-                soft_upper_limit="${168 * PI / 180}"
-                k_position="${safety_controller_k_pos}"
-                k_velocity="${safety_controller_k_vel}"
-            />
             <dynamics damping="${joint_damping}" friction="${joint_friction}"/>
         </joint>
@@ -77,12 +69,6 @@
             <parent link="${robot_name}_link_1"/>
             <child link="${robot_name}_link_2"/>
-            <axis xyz="0.0 0.01 0.0"/>
+            <axis xyz="0.0 1.0 0.0"/>
             <limit effort="${max_effort}" lower="${-120 * PI / 180}" upper="${120 * PI / 180}" velocity="${max_velocity}"/>
-            <safety_controller
-                soft_lower_limit="${-118 * PI / 180}"
-                soft_upper_limit="${118 * PI / 180}"
-                k_position="${safety_controller_k_pos}"
-                k_velocity="${safety_controller_k_vel}"
-            />
             <dynamics damping="${joint_damping}" friction="${joint_friction}"/>
         </joint>
@@ -111,12 +97,6 @@
             <parent link="${robot_name}_link_2"/>
             <child link="${robot_name}_link_3"/>
-            <axis xyz="0.0 0.0 0.01"/>
+            <axis xyz="0.0 0.0 1.0"/>
             <limit effort="${max_effort}" lower="${-170 * PI / 180}" upper="${170 * PI / 180}" velocity="${max_velocity}"/>
-            <safety_controller
-                soft_lower_limit="${-168 * PI / 180}"
-                soft_upper_limit="${168 * PI / 180}"
-                k_position="${safety_controller_k_pos}"
-                k_velocity="${safety_controller_k_vel}"
-            />
             <dynamics damping="${joint_damping}" friction="${joint_friction}"/>
         </joint>
@@ -145,12 +125,6 @@
             <parent link="${robot_name}_link_3"/>
             <child link="${robot_name}_link_4"/>
-            <axis xyz="0.0 -0.01 0.0"/>
+            <axis xyz="0.0 -1.0 0.0"/>
             <limit effort="${max_effort}" lower="${-120 * PI / 180}" upper="${120 * PI / 180}" velocity="${max_velocity}"/>
-            <safety_controller
-                soft_lower_limit="${-118 * PI / 180}"
-                soft_upper_limit="${118 * PI / 180}"
-                k_position="${safety_controller_k_pos}"
-                k_velocity="${safety_controller_k_vel}"
-            />
             <dynamics damping="${joint_damping}" friction="${joint_friction}"/>
         </joint>
@@ -179,12 +153,6 @@
             <parent link="${robot_name}_link_4"/>
             <child link="${robot_name}_link_5"/>
-            <axis xyz="0.0 0.0 0.01"/>
+            <axis xyz="0.0 0.0 1.0"/>
             <limit effort="${max_effort}" lower="${-170 * PI / 180}" upper="${170 * PI / 180}" velocity="${max_velocity}"/>
-            <safety_controller
-                soft_lower_limit="${-168 * PI / 180}"
-                soft_upper_limit="${168 * PI / 180}"
-                k_position="${safety_controller_k_pos}"
-                k_velocity="${safety_controller_k_vel}"
-            />
             <dynamics damping="${joint_damping}" friction="${joint_friction}"/>
         </joint>
@@ -213,12 +181,6 @@
             <parent link="${robot_name}_link_5"/>
             <child link="${robot_name}_link_6"/>
-            <axis xyz="0.0 0.01 0.0"/>
+            <axis xyz="0.0 1.0 0.0"/>
             <limit effort="${max_effort}" lower="${-120 * PI / 180}" upper="${120 * PI / 180}" velocity="${max_velocity}"/>
-            <safety_controller
-                soft_lower_limit="${-118 * PI / 180}"
-                soft_upper_limit="${118 * PI / 180}"
-                k_position="${safety_controller_k_pos}"
-                k_velocity="${safety_controller_k_vel}"
-            />
             <dynamics damping="${joint_damping}" friction="${joint_friction}"/>
         </joint>
@@ -247,12 +209,6 @@
             <parent link="${robot_name}_link_6"/>
             <child link="${robot_name}_link_7"/>
-            <axis xyz="0.0 0.0 0.01"/>
+            <axis xyz="0.0 0.0 1.0"/>
             <limit effort="${max_effort}" lower="${-175 * PI / 180}" upper="${175 * PI / 180}" velocity="${max_velocity}"/>
-            <safety_controller
-                soft_lower_limit="${-173 * PI / 180}"
-                soft_upper_limit="${173 * PI / 180}"
-                k_position="${safety_controller_k_pos}"
-                k_velocity="${safety_controller_k_vel}"
-            />
             <dynamics damping="${joint_damping}" friction="${joint_friction}"/>
         </joint>

File: lbr_description/urdf/iiwa7/iiwa7_description.urdf.xacro (robot description, xacro)
@@ -3,6 +3,4 @@
     <!-- some constants -->
     <xacro:property name="PI" value="3.1415926535897931"/>
-    <xacro:property name="safety_controller_k_pos" value="100"/>
-    <xacro:property name="safety_controller_k_vel" value="2"/>
     <xacro:property name="joint_damping" value="10.0"/>
     <xacro:property name="joint_friction" value="0.1"/>
@@ -43,12 +41,6 @@
             <parent link="${robot_name}_link_0"/>
             <child link="${robot_name}_link_1"/>
-            <axis xyz="0.0 0.0 0.01"/>
+            <axis xyz="0.0 0.0 1.0"/>
             <limit effort="${max_effort}" lower="${-170 * PI / 180}" upper="${170 * PI / 180}" velocity="${max_velocity}"/>
-            <safety_controller
-                soft_lower_limit="${-168 * PI / 180}"
-                soft_upper_limit="${168 * PI / 180}"
-                k_position="${safety_controller_k_pos}"
-                k_velocity="${safety_controller_k_vel}"
-            />
             <dynamics damping="${joint_damping}" friction="${joint_friction}"/>
         </joint>
@@ -77,12 +69,6 @@
             <parent link="${robot_name}_link_1"/>
             <child link="${robot_name}_link_2"/>
-            <axis xyz="0.0 0.01 0.0"/>
+            <axis xyz="0.0 1.0 0.0"/>
             <limit effort="${max_effort}" lower="${-120 * PI / 180}" upper="${120 * PI / 180}" velocity="${max_velocity}"/>
-            <safety_controller
-                soft_lower_limit="${-118 * PI / 180}"
-                soft_upper_limit="${118 * PI / 180}"
-                k_position="${safety_controller_k_pos}"
-                k_velocity="${safety_controller_k_vel}"
-            />
             <dynamics damping="${joint_damping}" friction="${joint_friction}"/>
         </joint>
@@ -111,12 +97,6 @@
             <parent link="${robot_name}_link_2"/>
             <child link="${robot_name}_link_3"/>
-            <axis xyz="0.0 0.0 0.01"/>
+            <axis xyz="0.0 0.0 1.0"/>
             <limit effort="${max_effort}" lower="${-170 * PI / 180}" upper="${170 * PI / 180}" velocity="${max_velocity}"/>
-            <safety_controller
-                soft_lower_limit="${-168 * PI / 180}"
-                soft_upper_limit="${168 * PI / 180}"
-                k_position="${safety_controller_k_pos}"
-                k_velocity="${safety_controller_k_vel}"
-            />
             <dynamics damping="${joint_damping}" friction="${joint_friction}"/>
         </joint>
@@ -145,12 +125,6 @@
             <parent link="${robot_name}_link_3"/>
             <child link="${robot_name}_link_4"/>
-            <axis xyz="0.0 -0.01 0.0"/>
+            <axis xyz="0.0 -1.0 0.0"/>
             <limit effort="${max_effort}" lower="${-120 * PI / 180}" upper="${120 * PI / 180}" velocity="${max_velocity}"/>
-            <safety_controller
-                soft_lower_limit="${-118 * PI / 180}"
-                soft_upper_limit="${118 * PI / 180}"
-                k_position="${safety_controller_k_pos}"
-                k_velocity="${safety_controller_k_vel}"
-            />
             <dynamics damping="${joint_damping}" friction="${joint_friction}"/>
         </joint>
@@ -179,12 +153,6 @@
             <parent link="${robot_name}_link_4"/>
             <child link="${robot_name}_link_5"/>
-            <axis xyz="0.0 0.0 0.01"/>
+            <axis xyz="0.0 0.0 1.0"/>
             <limit effort="${max_effort}" lower="${-170 * PI / 180}" upper="${170 * PI / 180}" velocity="${max_velocity}"/>
-            <safety_controller
-                soft_lower_limit="${-168 * PI / 180}"
-                soft_upper_limit="${168 * PI / 180}"
-                k_position="${safety_controller_k_pos}"
-                k_velocity="${safety_controller_k_vel}"
-            />
             <dynamics damping="${joint_damping}" friction="${joint_friction}"/>
         </joint>
@@ -213,12 +181,6 @@
             <parent link="${robot_name}_link_5"/>
             <child link="${robot_name}_link_6"/>
-            <axis xyz="0.0 0.01 0.0"/>
+            <axis xyz="0.0 1.0 0.0"/>
             <limit effort="${max_effort}" lower="${-120 * PI / 180}" upper="${120 * PI / 180}" velocity="${max_velocity}"/>
-            <safety_controller
-                soft_lower_limit="${-118 * PI / 180}"
-                soft_upper_limit="${118 * PI / 180}"
-                k_position="${safety_controller_k_pos}"
-                k_velocity="${safety_controller_k_vel}"
-            />
             <dynamics damping="${joint_damping}" friction="${joint_friction}"/>
         </joint>
@@ -247,12 +209,6 @@
             <parent link="${robot_name}_link_6"/>
             <child link="${robot_name}_link_7"/>
-            <axis xyz="0.0 0.0 0.01"/>
+            <axis xyz="0.0 0.0 1.0"/>
             <limit effort="${max_effort}" lower="${-175 * PI / 180}" upper="${175 * PI / 180}" velocity="${max_velocity}"/>
-            <safety_controller
-                soft_lower_limit="${-173 * PI / 180}"
-                soft_upper_limit="${173 * PI / 180}"
-                k_position="${safety_controller_k_pos}"
-                k_velocity="${safety_controller_k_vel}"
-            />
             <dynamics damping="${joint_damping}" friction="${joint_friction}"/>
         </joint>

File: lbr_description/urdf/med14/med14_description.urdf.xacro (robot description, xacro)
@@ -3,6 +3,4 @@
     <!-- some constants -->
     <xacro:property name="PI" value="3.1415926535897931"/>
-    <xacro:property name="safety_controller_k_pos" value="100"/>
-    <xacro:property name="safety_controller_k_vel" value="2"/>
     <xacro:property name="joint_damping" value="10.0"/>
     <xacro:property name="joint_friction" value="0.1"/>
@@ -43,12 +41,6 @@
             <parent link="${robot_name}_link_0"/>
             <child link="${robot_name}_link_1"/>
-            <axis xyz="0.0 0.0 0.01"/>
+            <axis xyz="0.0 0.0 1.0"/>
             <limit effort="${max_effort}" lower="${-170 * PI / 180}" upper="${170 * PI / 180}" velocity="${max_velocity}"/>
-            <safety_controller
-                soft_lower_limit="${-168 * PI / 180}"
-                soft_upper_limit="${168 * PI / 180}"
-                k_position="${safety_controller_k_pos}"
-                k_velocity="${safety_controller_k_vel}"
-            />
             <dynamics damping="${joint_damping}" friction="${joint_friction}"/>
         </joint>
@@ -77,12 +69,6 @@
             <parent link="${robot_name}_link_1"/>
             <child link="${robot_name}_link_2"/>
-            <axis xyz="0.0 0.01 0.0"/>
+            <axis xyz="0.0 1.0 0.0"/>
             <limit effort="${max_effort}" lower="${-120 * PI / 180}" upper="${120 * PI / 180}" velocity="${max_velocity}"/>
-            <safety_controller
-                soft_lower_limit="${-118 * PI / 180}"
-                soft_upper_limit="${118 * PI / 180}"
-                k_position="${safety_controller_k_pos}"
-                k_velocity="${safety_controller_k_vel}"
-            />
             <dynamics damping="${joint_damping}" friction="${joint_friction}"/>
         </joint>
@@ -111,12 +97,6 @@
             <parent link="${robot_name}_link_2"/>
             <child link="${robot_name}_link_3"/>
-            <axis xyz="0.0 0.0 0.01"/>
+            <axis xyz="0.0 0.0 1.0"/>
             <limit effort="${max_effort}" lower="${-170 * PI / 180}" upper="${170 * PI / 180}" velocity="${max_velocity}"/>
-            <safety_controller
-                soft_lower_limit="${-168 * PI / 180}"
-                soft_upper_limit="${168 * PI / 180}"
-                k_position="${safety_controller_k_pos}"
-                k_velocity="${safety_controller_k_vel}"
-            />
             <dynamics damping="${joint_damping}" friction="${joint_friction}"/>
         </joint>
@@ -145,12 +125,6 @@
             <parent link="${robot_name}_link_3"/>
             <child link="${robot_name}_link_4"/>
-            <axis xyz="0.0 -0.01 0.0"/>
+            <axis xyz="0.0 -1.0 0.0"/>
             <limit effort="${max_effort}" lower="${-120 * PI / 180}" upper="${120 * PI / 180}" velocity="${max_velocity}"/>
-            <safety_controller
-                soft_lower_limit="${-118 * PI / 180}"
-                soft_upper_limit="${118 * PI / 180}"
-                k_position="${safety_controller_k_pos}"
-                k_velocity="${safety_controller_k_vel}"
-            />
             <dynamics damping="${joint_damping}" friction="${joint_friction}"/>
         </joint>
@@ -179,12 +153,6 @@
             <parent link="${robot_name}_link_4"/>
             <child link="${robot_name}_link_5"/>
-            <axis xyz="0.0 0.0 0.01"/>
+            <axis xyz="0.0 0.0 1.0"/>
             <limit effort="${max_effort}" lower="${-170 * PI / 180}" upper="${170 * PI / 180}" velocity="${max_velocity}"/>
-            <safety_controller
-                soft_lower_limit="${-168 * PI / 180}"
-                soft_upper_limit="${168 * PI / 180}"
-                k_position="${safety_controller_k_pos}"
-                k_velocity="${safety_controller_k_vel}"
-            />
             <dynamics damping="${joint_damping}" friction="${joint_friction}"/>
         </joint>
@@ -213,12 +181,6 @@
             <parent link="${robot_name}_link_5"/>
             <child link="${robot_name}_link_6"/>
-            <axis xyz="0.0 0.01 0.0"/>
+            <axis xyz="0.0 1.0 0.0"/>
             <limit effort="${max_effort}" lower="${-120 * PI / 180}" upper="${120 * PI / 180}" velocity="${max_velocity}"/>
-            <safety_controller
-                soft_lower_limit="${-118 * PI / 180}"
-                soft_upper_limit="${118 * PI / 180}"
-                k_position="${safety_controller_k_pos}"
-                k_velocity="${safety_controller_k_vel}"
-            />
             <dynamics damping="${joint_damping}" friction="${joint_friction}"/>
         </joint>
@@ -247,12 +209,6 @@
             <parent link="${robot_name}_link_6"/>
             <child link="${robot_name}_link_7"/>
-            <axis xyz="0.0 0.0 0.01"/>
+            <axis xyz="0.0 0.0 1.0"/>
             <limit effort="${max_effort}" lower="${-175 * PI / 180}" upper="${175 * PI / 180}" velocity="${max_velocity}"/>
-            <safety_controller
-                soft_lower_limit="${-173 * PI / 180}"
-                soft_upper_limit="${173 * PI / 180}"
-                k_position="${safety_controller_k_pos}"
-                k_velocity="${safety_controller_k_vel}"
-            />
             <dynamics damping="${joint_damping}" friction="${joint_friction}"/>
         </joint>

File: lbr_description/urdf/med7/med7_description.urdf.xacro (robot description, xacro)
@@ -3,6 +3,4 @@
     <!-- some constants -->
     <xacro:property name="PI" value="3.1415926535897931"/>
-    <xacro:property name="safety_controller_k_pos" value="100"/>
-    <xacro:property name="safety_controller_k_vel" value="2"/>
     <xacro:property name="joint_damping" value="10.0"/>
     <xacro:property name="joint_friction" value="0.1"/>
@@ -43,12 +41,6 @@
             <parent link="${robot_name}_link_0"/>
             <child link="${robot_name}_link_1"/>
-            <axis xyz="0.0 0.0 0.01"/>
+            <axis xyz="0.0 0.0 1.0"/>
             <limit effort="${max_effort}" lower="${-170 * PI / 180}" upper="${170 * PI / 180}" velocity="${max_velocity}"/>
-            <safety_controller
-                soft_lower_limit="${-168 * PI / 180}"
-                soft_upper_limit="${168 * PI / 180}"
-                k_position="${safety_controller_k_pos}"
-                k_velocity="${safety_controller_k_vel}"
-            />
             <dynamics damping="${joint_damping}" friction="${joint_friction}"/>
         </joint>
@@ -77,12 +69,6 @@
             <parent link="${robot_name}_link_1"/>
             <child link="${robot_name}_link_2"/>
-            <axis xyz="0.0 0.01 0.0"/>
+            <axis xyz="0.0 1.0 0.0"/>
             <limit effort="${max_effort}" lower="${-120 * PI / 180}" upper="${120 * PI / 180}" velocity="${max_velocity}"/>
-            <safety_controller
-                soft_lower_limit="${-118 * PI / 180}"
-                soft_upper_limit="${118 * PI / 180}"
-                k_position="${safety_controller_k_pos}"
-                k_velocity="${safety_controller_k_vel}"
-            />
             <dynamics damping="${joint_damping}" friction="${joint_friction}"/>
         </joint>
@@ -111,12 +97,6 @@
             <parent link="${robot_name}_link_2"/>
             <child link="${robot_name}_link_3"/>
-            <axis xyz="0.0 0.0 0.01"/>
+            <axis xyz="0.0 0.0 1.0"/>
             <limit effort="${max_effort}" lower="${-170 * PI / 180}" upper="${170 * PI / 180}" velocity="${max_velocity}"/>
-            <safety_controller
-                soft_lower_limit="${-168 * PI / 180}"
-                soft_upper_limit="${168 * PI / 180}"
-                k_position="${safety_controller_k_pos}"
-                k_velocity="${safety_controller_k_vel}"
-            />
             <dynamics damping="${joint_damping}" friction="${joint_friction}"/>
         </joint>
@@ -145,12 +125,6 @@
             <parent link="${robot_name}_link_3"/>
             <child link="${robot_name}_link_4"/>
-            <axis xyz="0.0 -0.01 0.0"/>
+            <axis xyz="0.0 -1.0 0.0"/>
             <limit effort="${max_effort}" lower="${-120 * PI / 180}" upper="${120 * PI / 180}" velocity="${max_velocity}"/>
-            <safety_controller
-                soft_lower_limit="${-118 * PI / 180}"
-                soft_upper_limit="${118 * PI / 180}"
-                k_position="${safety_controller_k_pos}"
-                k_velocity="${safety_controller_k_vel}"
-            />
             <dynamics damping="${joint_damping}" friction="${joint_friction}"/>
         </joint>
@@ -179,12 +153,6 @@
             <parent link="${robot_name}_link_4"/>
             <child link="${robot_name}_link_5"/>
-            <axis xyz="0.0 0.0 0.01"/>
+            <axis xyz="0.0 0.0 1.0"/>
             <limit effort="${max_effort}" lower="${-170 * PI / 180}" upper="${170 * PI / 180}" velocity="${max_velocity}"/>
-            <safety_controller
-                soft_lower_limit="${-168 * PI / 180}"
-                soft_upper_limit="${168 * PI / 180}"
-                k_position="${safety_controller_k_pos}"
-                k_velocity="${safety_controller_k_vel}"
-            />
             <dynamics damping="${joint_damping}" friction="${joint_friction}"/>
         </joint>
@@ -213,12 +181,6 @@
             <parent link="${robot_name}_link_5"/>
             <child link="${robot_name}_link_6"/>
-            <axis xyz="0.0 0.01 0.0"/>
+            <axis xyz="0.0 1.0 0.0"/>
             <limit effort="${max_effort}" lower="${-120 * PI / 180}" upper="${120 * PI / 180}" velocity="${max_velocity}"/>
-            <safety_controller
-                soft_lower_limit="${-118 * PI / 180}"
-                soft_upper_limit="${118 * PI / 180}"
-                k_position="${safety_controller_k_pos}"
-                k_velocity="${safety_controller_k_vel}"
-            />
             <dynamics damping="${joint_damping}" friction="${joint_friction}"/>
         </joint>
@@ -247,12 +209,6 @@
             <parent link="${robot_name}_link_6"/>
             <child link="${robot_name}_link_7"/>
-            <axis xyz="0.0 0.0 0.01"/>
+            <axis xyz="0.0 0.0 1.0"/>
             <limit effort="${max_effort}" lower="${-175 * PI / 180}" upper="${175 * PI / 180}" velocity="${max_velocity}"/>
-            <safety_controller
-                soft_lower_limit="${-173 * PI / 180}"
-                soft_upper_limit="${173 * PI / 180}"
-                k_position="${safety_controller_k_pos}"
-                k_velocity="${safety_controller_k_vel}"
-            />
             <dynamics damping="${joint_damping}" friction="${joint_friction}"/>
         </joint>
