Commit message: updated velocity limits, re-factored urdf tests

File: lbr_description/urdf/iiwa14/iiwa14_description.urdf.xacro (robot description, xacro)
@@ -6,5 +6,4 @@
     <xacro:property name="joint_friction" value="0.1"/>
     <xacro:property name="max_effort" value="300"/>
-    <xacro:property name="max_velocity" value="10"/>
     <!-- includes -->
     <xacro:include filename="$(find lbr_description)/urdf/materials.urdf.xacro"/>
@@ -43,5 +42,5 @@
             <child link="${robot_name}_link_1"/>
             <axis xyz="0.0 0.0 1.0"/>
-            <limit effort="${max_effort}" lower="${-170 * PI / 180}" upper="${170 * PI / 180}" velocity="${max_velocity}"/>
+            <limit effort="${max_effort}" lower="${-170 * PI / 180}" upper="${170 * PI / 180}" velocity="${85 * PI / 180}"/>
             <dynamics damping="${joint_damping}" friction="${joint_friction}"/>
         </joint>
@@ -71,5 +70,5 @@
             <child link="${robot_name}_link_2"/>
             <axis xyz="0.0 1.0 0.0"/>
-            <limit effort="${max_effort}" lower="${-120 * PI / 180}" upper="${120 * PI / 180}" velocity="${max_velocity}"/>
+            <limit effort="${max_effort}" lower="${-120 * PI / 180}" upper="${120 * PI / 180}" velocity="${85 * PI / 180}"/>
             <dynamics damping="${joint_damping}" friction="${joint_friction}"/>
         </joint>
@@ -99,5 +98,5 @@
             <child link="${robot_name}_link_3"/>
             <axis xyz="0.0 0.0 1.0"/>
-            <limit effort="${max_effort}" lower="${-170 * PI / 180}" upper="${170 * PI / 180}" velocity="${max_velocity}"/>
+            <limit effort="${max_effort}" lower="${-170 * PI / 180}" upper="${170 * PI / 180}" velocity="${100 * PI / 180}"/>
             <dynamics damping="${joint_damping}" friction="${joint_friction}"/>
         </joint>
@@ -127,5 +126,5 @@
             <child link="${robot_name}_link_4"/>
             <axis xyz="0.0 -1.0 0.0"/>
-            <limit effort="${max_effort}" lower="${-120 * PI / 180}" upper="${120 * PI / 180}" velocity="${max_velocity}"/>
+            <limit effort="${max_effort}" lower="${-120 * PI / 180}" upper="${120 * PI / 180}" velocity="${75 * PI / 180}"/>
             <dynamics damping="${joint_damping}" friction="${joint_friction}"/>
         </joint>
@@ -155,5 +154,5 @@
             <child link="${robot_name}_link_5"/>
             <axis xyz="0.0 0.0 1.0"/>
-            <limit effort="${max_effort}" lower="${-170 * PI / 180}" upper="${170 * PI / 180}" velocity="${max_velocity}"/>
+            <limit effort="${max_effort}" lower="${-170 * PI / 180}" upper="${170 * PI / 180}" velocity="${130 * PI / 180}"/>
             <dynamics damping="${joint_damping}" friction="${joint_friction}"/>
         </joint>
@@ -183,5 +182,5 @@
             <child link="${robot_name}_link_6"/>
             <axis xyz="0.0 1.0 0.0"/>
-            <limit effort="${max_effort}" lower="${-120 * PI / 180}" upper="${120 * PI / 180}" velocity="${max_velocity}"/>
+            <limit effort="${max_effort}" lower="${-120 * PI / 180}" upper="${120 * PI / 180}" velocity="${135 * PI / 180}"/>
             <dynamics damping="${joint_damping}" friction="${joint_friction}"/>
         </joint>
@@ -211,5 +210,5 @@
             <child link="${robot_name}_link_7"/>
             <axis xyz="0.0 0.0 1.0"/>
-            <limit effort="${max_effort}" lower="${-175 * PI / 180}" upper="${175 * PI / 180}" velocity="${max_velocity}"/>
+            <limit effort="${max_effort}" lower="${-175 * PI / 180}" upper="${175 * PI / 180}" velocity="${135 * PI / 180}"/>
             <dynamics damping="${joint_damping}" friction="${joint_friction}"/>
         </joint>

File: lbr_description/urdf/iiwa7/iiwa7_description.urdf.xacro (robot description, xacro)
@@ -6,5 +6,4 @@
     <xacro:property name="joint_friction" value="0.1"/>
     <xacro:property name="max_effort" value="300"/>
-    <xacro:property name="max_velocity" value="10"/>
     <!-- includes -->
     <xacro:include filename="$(find lbr_description)/urdf/materials.urdf.xacro"/>
@@ -43,5 +42,5 @@
             <child link="${robot_name}_link_1"/>
             <axis xyz="0.0 0.0 1.0"/>
-            <limit effort="${max_effort}" lower="${-170 * PI / 180}" upper="${170 * PI / 180}" velocity="${max_velocity}"/>
+            <limit effort="${max_effort}" lower="${-170 * PI / 180}" upper="${170 * PI / 180}" velocity="${98 * PI / 180}"/>
             <dynamics damping="${joint_damping}" friction="${joint_friction}"/>
         </joint>
@@ -71,5 +70,5 @@
             <child link="${robot_name}_link_2"/>
             <axis xyz="0.0 1.0 0.0"/>
-            <limit effort="${max_effort}" lower="${-120 * PI / 180}" upper="${120 * PI / 180}" velocity="${max_velocity}"/>
+            <limit effort="${max_effort}" lower="${-120 * PI / 180}" upper="${120 * PI / 180}" velocity="${98 * PI / 180}"/>
             <dynamics damping="${joint_damping}" friction="${joint_friction}"/>
         </joint>
@@ -99,5 +98,5 @@
             <child link="${robot_name}_link_3"/>
             <axis xyz="0.0 0.0 1.0"/>
-            <limit effort="${max_effort}" lower="${-170 * PI / 180}" upper="${170 * PI / 180}" velocity="${max_velocity}"/>
+            <limit effort="${max_effort}" lower="${-170 * PI / 180}" upper="${170 * PI / 180}" velocity="${100 * PI / 180}"/>
             <dynamics damping="${joint_damping}" friction="${joint_friction}"/>
         </joint>
@@ -127,5 +126,5 @@
             <child link="${robot_name}_link_4"/>
             <axis xyz="0.0 -1.0 0.0"/>
-            <limit effort="${max_effort}" lower="${-120 * PI / 180}" upper="${120 * PI / 180}" velocity="${max_velocity}"/>
+            <limit effort="${max_effort}" lower="${-120 * PI / 180}" upper="${120 * PI / 180}" velocity="${130 * PI / 180}"/>
             <dynamics damping="${joint_damping}" friction="${joint_friction}"/>
         </joint>
@@ -155,5 +154,5 @@
             <child link="${robot_name}_link_5"/>
             <axis xyz="0.0 0.0 1.0"/>
-            <limit effort="${max_effort}" lower="${-170 * PI / 180}" upper="${170 * PI / 180}" velocity="${max_velocity}"/>
+            <limit effort="${max_effort}" lower="${-170 * PI / 180}" upper="${170 * PI / 180}" velocity="${140 * PI / 180}"/>
             <dynamics damping="${joint_damping}" friction="${joint_friction}"/>
         </joint>
@@ -183,5 +182,5 @@
             <child link="${robot_name}_link_6"/>
             <axis xyz="0.0 1.0 0.0"/>
-            <limit effort="${max_effort}" lower="${-120 * PI / 180}" upper="${120 * PI / 180}" velocity="${max_velocity}"/>
+            <limit effort="${max_effort}" lower="${-120 * PI / 180}" upper="${120 * PI / 180}" velocity="${180 * PI / 180}"/>
             <dynamics damping="${joint_damping}" friction="${joint_friction}"/>
         </joint>
@@ -211,5 +210,5 @@
             <child link="${robot_name}_link_7"/>
             <axis xyz="0.0 0.0 1.0"/>
-            <limit effort="${max_effort}" lower="${-175 * PI / 180}" upper="${175 * PI / 180}" velocity="${max_velocity}"/>
+            <limit effort="${max_effort}" lower="${-175 * PI / 180}" upper="${175 * PI / 180}" velocity="${180 * PI / 180}"/>
             <dynamics damping="${joint_damping}" friction="${joint_friction}"/>
         </joint>

File: lbr_description/urdf/med14/med14_description.urdf.xacro (robot description, xacro)
@@ -6,5 +6,4 @@
     <xacro:property name="joint_friction" value="0.1"/>
     <xacro:property name="max_effort" value="300"/>
-    <xacro:property name="max_velocity" value="10"/>
     <!-- includes -->
     <xacro:include filename="$(find lbr_description)/urdf/materials.urdf.xacro"/>
@@ -43,5 +42,5 @@
             <child link="${robot_name}_link_1"/>
             <axis xyz="0.0 0.0 1.0"/>
-            <limit effort="${max_effort}" lower="${-170 * PI / 180}" upper="${170 * PI / 180}" velocity="${max_velocity}"/>
+            <limit effort="${max_effort}" lower="${-170 * PI / 180}" upper="${170 * PI / 180}" velocity="${85 * PI / 180}"/>
             <dynamics damping="${joint_damping}" friction="${joint_friction}"/>
         </joint>
@@ -71,5 +70,5 @@
             <child link="${robot_name}_link_2"/>
             <axis xyz="0.0 1.0 0.0"/>
-            <limit effort="${max_effort}" lower="${-120 * PI / 180}" upper="${120 * PI / 180}" velocity="${max_velocity}"/>
+            <limit effort="${max_effort}" lower="${-120 * PI / 180}" upper="${120 * PI / 180}" velocity="${85 * PI / 180}"/>
             <dynamics damping="${joint_damping}" friction="${joint_friction}"/>
         </joint>
@@ -99,5 +98,5 @@
             <child link="${robot_name}_link_3"/>
             <axis xyz="0.0 0.0 1.0"/>
-            <limit effort="${max_effort}" lower="${-170 * PI / 180}" upper="${170 * PI / 180}" velocity="${max_velocity}"/>
+            <limit effort="${max_effort}" lower="${-170 * PI / 180}" upper="${170 * PI / 180}" velocity="${100 * PI / 180}"/>
             <dynamics damping="${joint_damping}" friction="${joint_friction}"/>
         </joint>
@@ -127,5 +126,5 @@
             <child link="${robot_name}_link_4"/>
             <axis xyz="0.0 -1.0 0.0"/>
-            <limit effort="${max_effort}" lower="${-120 * PI / 180}" upper="${120 * PI / 180}" velocity="${max_velocity}"/>
+            <limit effort="${max_effort}" lower="${-120 * PI / 180}" upper="${120 * PI / 180}" velocity="${75 * PI / 180}"/>
             <dynamics damping="${joint_damping}" friction="${joint_friction}"/>
         </joint>
@@ -155,5 +154,5 @@
             <child link="${robot_name}_link_5"/>
             <axis xyz="0.0 0.0 1.0"/>
-            <limit effort="${max_effort}" lower="${-170 * PI / 180}" upper="${170 * PI / 180}" velocity="${max_velocity}"/>
+            <limit effort="${max_effort}" lower="${-170 * PI / 180}" upper="${170 * PI / 180}" velocity="${130 * PI / 180}"/>
             <dynamics damping="${joint_damping}" friction="${joint_friction}"/>
         </joint>
@@ -183,5 +182,5 @@
             <child link="${robot_name}_link_6"/>
             <axis xyz="0.0 1.0 0.0"/>
-            <limit effort="${max_effort}" lower="${-120 * PI / 180}" upper="${120 * PI / 180}" velocity="${max_velocity}"/>
+            <limit effort="${max_effort}" lower="${-120 * PI / 180}" upper="${120 * PI / 180}" velocity="${135 * PI / 180}"/>
             <dynamics damping="${joint_damping}" friction="${joint_friction}"/>
         </joint>
@@ -211,5 +210,5 @@
             <child link="${robot_name}_link_7"/>
             <axis xyz="0.0 0.0 1.0"/>
-            <limit effort="${max_effort}" lower="${-175 * PI / 180}" upper="${175 * PI / 180}" velocity="${max_velocity}"/>
+            <limit effort="${max_effort}" lower="${-175 * PI / 180}" upper="${175 * PI / 180}" velocity="${135 * PI / 180}"/>
             <dynamics damping="${joint_damping}" friction="${joint_friction}"/>
         </joint>

File: lbr_description/urdf/med7/med7_description.urdf.xacro (robot description, xacro)
@@ -6,5 +6,4 @@
     <xacro:property name="joint_friction" value="0.1"/>
     <xacro:property name="max_effort" value="100"/>
-    <xacro:property name="max_velocity" value="10"/>
     <!-- includes -->
     <xacro:include filename="$(find lbr_description)/urdf/materials.urdf.xacro"/>
@@ -43,5 +42,5 @@
             <child link="${robot_name}_link_1"/>
             <axis xyz="0.0 0.0 1.0"/>
-            <limit effort="${max_effort}" lower="${-170 * PI / 180}" upper="${170 * PI / 180}" velocity="${max_velocity}"/>
+            <limit effort="${max_effort}" lower="${-170 * PI / 180}" upper="${170 * PI / 180}" velocity="${98 * PI / 180}"/>
             <dynamics damping="${joint_damping}" friction="${joint_friction}"/>
         </joint>
@@ -71,5 +70,5 @@
             <child link="${robot_name}_link_2"/>
             <axis xyz="0.0 1.0 0.0"/>
-            <limit effort="${max_effort}" lower="${-120 * PI / 180}" upper="${120 * PI / 180}" velocity="${max_velocity}"/>
+            <limit effort="${max_effort}" lower="${-120 * PI / 180}" upper="${120 * PI / 180}" velocity="${98 * PI / 180}"/>
             <dynamics damping="${joint_damping}" friction="${joint_friction}"/>
         </joint>
@@ -99,5 +98,5 @@
             <child link="${robot_name}_link_3"/>
             <axis xyz="0.0 0.0 1.0"/>
-            <limit effort="${max_effort}" lower="${-170 * PI / 180}" upper="${170 * PI / 180}" velocity="${max_velocity}"/>
+            <limit effort="${max_effort}" lower="${-170 * PI / 180}" upper="${170 * PI / 180}" velocity="${100 * PI / 180}"/>
             <dynamics damping="${joint_damping}" friction="${joint_friction}"/>
         </joint>
@@ -127,5 +126,5 @@
             <child link="${robot_name}_link_4"/>
             <axis xyz="0.0 -1.0 0.0"/>
-            <limit effort="${max_effort}" lower="${-120 * PI / 180}" upper="${120 * PI / 180}" velocity="${max_velocity}"/>
+            <limit effort="${max_effort}" lower="${-120 * PI / 180}" upper="${120 * PI / 180}" velocity="${130 * PI / 180}"/>
             <dynamics damping="${joint_damping}" friction="${joint_friction}"/>
         </joint>
@@ -155,5 +154,5 @@
             <child link="${robot_name}_link_5"/>
             <axis xyz="0.0 0.0 1.0"/>
-            <limit effort="${max_effort}" lower="${-170 * PI / 180}" upper="${170 * PI / 180}" velocity="${max_velocity}"/>
+            <limit effort="${max_effort}" lower="${-170 * PI / 180}" upper="${170 * PI / 180}" velocity="${140 * PI / 180}"/>
             <dynamics damping="${joint_damping}" friction="${joint_friction}"/>
         </joint>
@@ -183,5 +182,5 @@
             <child link="${robot_name}_link_6"/>
             <axis xyz="0.0 1.0 0.0"/>
-            <limit effort="${max_effort}" lower="${-120 * PI / 180}" upper="${120 * PI / 180}" velocity="${max_velocity}"/>
+            <limit effort="${max_effort}" lower="${-120 * PI / 180}" upper="${120 * PI / 180}" velocity="${180 * PI / 180}"/>
             <dynamics damping="${joint_damping}" friction="${joint_friction}"/>
         </joint>
@@ -211,5 +210,5 @@
             <child link="${robot_name}_link_7"/>
             <axis xyz="0.0 0.0 1.0"/>
-            <limit effort="${max_effort}" lower="${-175 * PI / 180}" upper="${175 * PI / 180}" velocity="${max_velocity}"/>
+            <limit effort="${max_effort}" lower="${-175 * PI / 180}" upper="${175 * PI / 180}" velocity="${180 * PI / 180}"/>
             <dynamics damping="${joint_damping}" friction="${joint_friction}"/>
         </joint>
