Commit message: removed unused friction / damping

File: lbr_description/urdf/iiwa14/iiwa14_description.urdf.xacro (robot description, xacro)
@@ -3,6 +3,4 @@
     <!-- some constants -->
     <xacro:property name="PI" value="3.1415926535897931"/>
-    <xacro:property name="joint_damping" value="10.0"/>
-    <xacro:property name="joint_friction" value="0.1"/>
     <xacro:property name="max_effort" value="300"/>
     <!-- includes -->
@@ -43,5 +41,4 @@
             <axis xyz="0.0 0.0 1.0"/>
             <limit effort="${max_effort}" lower="${-170 * PI / 180}" upper="${170 * PI / 180}" velocity="${85 * PI / 180}"/>
-            <dynamics damping="${joint_damping}" friction="${joint_friction}"/>
         </joint>
         <link name="${robot_name}_link_1">
@@ -71,5 +68,4 @@
             <axis xyz="0.0 1.0 0.0"/>
             <limit effort="${max_effort}" lower="${-120 * PI / 180}" upper="${120 * PI / 180}" velocity="${85 * PI / 180}"/>
-            <dynamics damping="${joint_damping}" friction="${joint_friction}"/>
         </joint>
         <link name="${robot_name}_link_2">
@@ -99,5 +95,4 @@
             <axis xyz="0.0 0.0 1.0"/>
             <limit effort="${max_effort}" lower="${-170 * PI / 180}" upper="${170 * PI / 180}" velocity="${100 * PI / 180}"/>
-            <dynamics damping="${joint_damping}" friction="${joint_friction}"/>
         </joint>
         <link name="${robot_name}_link_3">
@@ -127,5 +122,4 @@
             <axis xyz="0.0 -1.0 0.0"/>
             <limit effort="${max_effort}" lower="${-120 * PI / 180}" upper="${120 * PI / 180}" velocity="${75 * PI / 180}"/>
-            <dynamics damping="${joint_damping}" friction="${joint_friction}"/>
         </joint>
         <link name="${robot_name}_link_4">
@@ -155,5 +149,4 @@
             <axis xyz="0.0 0.0 1.0"/>
             <limit effort="${max_effort}" lower="${-170 * PI / 180}" upper="${170 * PI / 180}" velocity="${130 * PI / 180}"/>
-            <dynamics damping="${joint_damping}" friction="${joint_friction}"/>
         </joint>
         <link name="${robot_name}_link_5">
@@ -183,5 +176,4 @@
             <axis xyz="0.0 1.0 0.0"/>
             <limit effort="${max_effort}" lower="${-120 * PI / 180}" upper="${120 * PI / 180}" velocity="${135 * PI / 180}"/>
-            <dynamics damping="${joint_damping}" friction="${joint_friction}"/>
         </joint>
         <link name="${robot_name}_link_6">
@@ -211,5 +203,4 @@
             <axis xyz="0.0 0.0 1.0"/>
             <limit effort="${max_effort}" lower="${-175 * PI / 180}" upper="${175 * PI / 180}" velocity="${135 * PI / 180}"/>
-            <dynamics damping="${joint_damping}" friction="${joint_friction}"/>
         </joint>
         <link name="${robot_name}_link_7">

File: lbr_description/urdf/iiwa7/iiwa7_description.urdf.xacro (robot description, xacro)
@@ -43,5 +43,4 @@
             <axis xyz="0.0 0.0 1.0"/>
             <limit effort="${max_effort}" lower="${-170 * PI / 180}" upper="${170 * PI / 180}" velocity="${98 * PI / 180}"/>
-            <dynamics damping="${joint_damping}" friction="${joint_friction}"/>
         </joint>
         <link name="${robot_name}_link_1">
@@ -71,5 +70,4 @@
             <axis xyz="0.0 1.0 0.0"/>
             <limit effort="${max_effort}" lower="${-120 * PI / 180}" upper="${120 * PI / 180}" velocity="${98 * PI / 180}"/>
-            <dynamics damping="${joint_damping}" friction="${joint_friction}"/>
         </joint>
         <link name="${robot_name}_link_2">
@@ -99,5 +97,4 @@
             <axis xyz="0.0 0.0 1.0"/>
             <limit effort="${max_effort}" lower="${-170 * PI / 180}" upper="${170 * PI / 180}" velocity="${100 * PI / 180}"/>
-            <dynamics damping="${joint_damping}" friction="${joint_friction}"/>
         </joint>
         <link name="${robot_name}_link_3">
@@ -127,5 +124,4 @@
             <axis xyz="0.0 -1.0 0.0"/>
             <limit effort="${max_effort}" lower="${-120 * PI / 180}" upper="${120 * PI / 180}" velocity="${130 * PI / 180}"/>
-            <dynamics damping="${joint_damping}" friction="${joint_friction}"/>
         </joint>
         <link name="${robot_name}_link_4">
@@ -155,5 +151,4 @@
             <axis xyz="0.0 0.0 1.0"/>
             <limit effort="${max_effort}" lower="${-170 * PI / 180}" upper="${170 * PI / 180}" velocity="${140 * PI / 180}"/>
-            <dynamics damping="${joint_damping}" friction="${joint_friction}"/>
         </joint>
         <link name="${robot_name}_link_5">
@@ -183,5 +178,4 @@
             <axis xyz="0.0 1.0 0.0"/>
             <limit effort="${max_effort}" lower="${-120 * PI / 180}" upper="${120 * PI / 180}" velocity="${180 * PI / 180}"/>
-            <dynamics damping="${joint_damping}" friction="${joint_friction}"/>
         </joint>
         <link name="${robot_name}_link_6">
@@ -211,5 +205,4 @@
             <axis xyz="0.0 0.0 1.0"/>
             <limit effort="${max_effort}" lower="${-175 * PI / 180}" upper="${175 * PI / 180}" velocity="${180 * PI / 180}"/>
-            <dynamics damping="${joint_damping}" friction="${joint_friction}"/>
         </joint>
         <link name="${robot_name}_link_7">

File: lbr_description/urdf/med14/med14_description.urdf.xacro (robot description, xacro)
@@ -3,6 +3,4 @@
     <!-- some constants -->
     <xacro:property name="PI" value="3.1415926535897931"/>
-    <xacro:property name="joint_damping" value="10.0"/>
-    <xacro:property name="joint_friction" value="0.1"/>
     <xacro:property name="max_effort" value="300"/>
     <!-- includes -->
@@ -43,5 +41,4 @@
             <axis xyz="0.0 0.0 1.0"/>
             <limit effort="${max_effort}" lower="${-170 * PI / 180}" upper="${170 * PI / 180}" velocity="${85 * PI / 180}"/>
-            <dynamics damping="${joint_damping}" friction="${joint_friction}"/>
         </joint>
         <link name="${robot_name}_link_1">
@@ -71,5 +68,4 @@
             <axis xyz="0.0 1.0 0.0"/>
             <limit effort="${max_effort}" lower="${-120 * PI / 180}" upper="${120 * PI / 180}" velocity="${85 * PI / 180}"/>
-            <dynamics damping="${joint_damping}" friction="${joint_friction}"/>
         </joint>
         <link name="${robot_name}_link_2">
@@ -99,5 +95,4 @@
             <axis xyz="0.0 0.0 1.0"/>
             <limit effort="${max_effort}" lower="${-170 * PI / 180}" upper="${170 * PI / 180}" velocity="${100 * PI / 180}"/>
-            <dynamics damping="${joint_damping}" friction="${joint_friction}"/>
         </joint>
         <link name="${robot_name}_link_3">
@@ -127,5 +122,4 @@
             <axis xyz="0.0 -1.0 0.0"/>
             <limit effort="${max_effort}" lower="${-120 * PI / 180}" upper="${120 * PI / 180}" velocity="${75 * PI / 180}"/>
-            <dynamics damping="${joint_damping}" friction="${joint_friction}"/>
         </joint>
         <link name="${robot_name}_link_4">
@@ -155,5 +149,4 @@
             <axis xyz="0.0 0.0 1.0"/>
             <limit effort="${max_effort}" lower="${-170 * PI / 180}" upper="${170 * PI / 180}" velocity="${130 * PI / 180}"/>
-            <dynamics damping="${joint_damping}" friction="${joint_friction}"/>
         </joint>
         <link name="${robot_name}_link_5">
@@ -183,5 +176,4 @@
             <axis xyz="0.0 1.0 0.0"/>
             <limit effort="${max_effort}" lower="${-120 * PI / 180}" upper="${120 * PI / 180}" velocity="${135 * PI / 180}"/>
-            <dynamics damping="${joint_damping}" friction="${joint_friction}"/>
         </joint>
         <link name="${robot_name}_link_6">
@@ -211,5 +203,4 @@
             <axis xyz="0.0 0.0 1.0"/>
             <limit effort="${max_effort}" lower="${-175 * PI / 180}" upper="${175 * PI / 180}" velocity="${135 * PI / 180}"/>
-            <dynamics damping="${joint_damping}" friction="${joint_friction}"/>
         </joint>
         <link name="${robot_name}_link_7">

File: lbr_description/urdf/med7/med7_description.urdf.xacro (robot description, xacro)
@@ -3,6 +3,4 @@
     <!-- some constants -->
     <xacro:property name="PI" value="3.1415926535897931"/>
-    <xacro:property name="joint_damping" value="10.0"/>
-    <xacro:property name="joint_friction" value="0.1"/>
     <xacro:property name="max_effort" value="100"/>
     <!-- includes -->
@@ -43,5 +41,4 @@
             <axis xyz="0.0 0.0 1.0"/>
             <limit effort="${max_effort}" lower="${-170 * PI / 180}" upper="${170 * PI / 180}" velocity="${98 * PI / 180}"/>
-            <dynamics damping="${joint_damping}" friction="${joint_friction}"/>
         </joint>
         <link name="${robot_name}_link_1">
@@ -71,5 +68,4 @@
             <axis xyz="0.0 1.0 0.0"/>
             <limit effort="${max_effort}" lower="${-120 * PI / 180}" upper="${120 * PI / 180}" velocity="${98 * PI / 180}"/>
-            <dynamics damping="${joint_damping}" friction="${joint_friction}"/>
         </joint>
         <link name="${robot_name}_link_2">
@@ -99,5 +95,4 @@
             <axis xyz="0.0 0.0 1.0"/>
             <limit effort="${max_effort}" lower="${-170 * PI / 180}" upper="${170 * PI / 180}" velocity="${100 * PI / 180}"/>
-            <dynamics damping="${joint_damping}" friction="${joint_friction}"/>
         </joint>
         <link name="${robot_name}_link_3">
@@ -127,5 +122,4 @@
             <axis xyz="0.0 -1.0 0.0"/>
             <limit effort="${max_effort}" lower="${-120 * PI / 180}" upper="${120 * PI / 180}" velocity="${130 * PI / 180}"/>
-            <dynamics damping="${joint_damping}" friction="${joint_friction}"/>
         </joint>
         <link name="${robot_name}_link_4">
@@ -155,5 +149,4 @@
             <axis xyz="0.0 0.0 1.0"/>
             <limit effort="${max_effort}" lower="${-170 * PI / 180}" upper="${170 * PI / 180}" velocity="${140 * PI / 180}"/>
-            <dynamics damping="${joint_damping}" friction="${joint_friction}"/>
         </joint>
         <link name="${robot_name}_link_5">
@@ -183,5 +176,4 @@
             <axis xyz="0.0 1.0 0.0"/>
             <limit effort="${max_effort}" lower="${-120 * PI / 180}" upper="${120 * PI / 180}" velocity="${180 * PI / 180}"/>
-            <dynamics damping="${joint_damping}" friction="${joint_friction}"/>
         </joint>
         <link name="${robot_name}_link_6">
@@ -211,5 +203,4 @@
             <axis xyz="0.0 0.0 1.0"/>
             <limit effort="${max_effort}" lower="${-175 * PI / 180}" upper="${175 * PI / 180}" velocity="${180 * PI / 180}"/>
-            <dynamics damping="${joint_damping}" friction="${joint_friction}"/>
         </joint>
         <link name="${robot_name}_link_7">

Commit message: re-added dynamics term for simulation

File: lbr_description/urdf/iiwa14/iiwa14_description.urdf.xacro (robot description, xacro)
@@ -60,4 +60,5 @@
                 upper="${joint_0_position_limit * PI / 180}"
                 velocity="${joint_0_velocity_limit * PI / 180}" />
+            <dynamics damping="1.0" friction="1.0" />
         </joint>
         <link name="${robot_name}_link_1">
@@ -91,4 +92,5 @@
                 upper="${joint_1_position_limit * PI / 180}"
                 velocity="${joint_1_velocity_limit * PI / 180}" />
+            <dynamics damping="1.0" friction="1.0" />
         </joint>
         <link name="${robot_name}_link_2">
@@ -122,4 +124,5 @@
                 upper="${joint_2_position_limit * PI / 180}"
                 velocity="${joint_2_velocity_limit * PI / 180}" />
+            <dynamics damping="1.0" friction="1.0" />
         </joint>
         <link name="${robot_name}_link_3">
@@ -153,4 +156,5 @@
                 upper="${joint_3_position_limit * PI / 180}"
                 velocity="${joint_3_velocity_limit * PI / 180}" />
+            <dynamics damping="1.0" friction="1.0" />
         </joint>
         <link name="${robot_name}_link_4">
@@ -184,4 +188,5 @@
                 upper="${joint_4_position_limit * PI / 180}"
                 velocity="${joint_4_velocity_limit * PI / 180}" />
+            <dynamics damping="1.0" friction="1.0" />
         </joint>
         <link name="${robot_name}_link_5">
@@ -215,4 +220,5 @@
                 upper="${joint_5_position_limit * PI / 180}"
                 velocity="${joint_5_velocity_limit * PI / 180}" />
+            <dynamics damping="1.0" friction="1.0" />
         </joint>
         <link name="${robot_name}_link_6">
@@ -246,4 +252,5 @@
                 upper="${joint_6_position_limit * PI / 180}"
                 velocity="${joint_6_velocity_limit * PI / 180}" />
+            <dynamics damping="1.0" friction="1.0" />
         </joint>
         <link name="${robot_name}_link_7">

File: lbr_description/urdf/iiwa7/iiwa7_description.urdf.xacro (robot description, xacro)
@@ -60,4 +60,5 @@
                 upper="${joint_0_position_limit * PI / 180}"
                 velocity="${joint_0_velocity_limit * PI / 180}" />
+            <dynamics damping="1.0" friction="1.0" />
         </joint>
         <link name="${robot_name}_link_1">
@@ -91,4 +92,5 @@
                 upper="${joint_1_position_limit * PI / 180}"
                 velocity="${joint_1_velocity_limit * PI / 180}" />
+            <dynamics damping="1.0" friction="1.0" />
         </joint>
         <link name="${robot_name}_link_2">
@@ -122,4 +124,5 @@
                 upper="${joint_2_position_limit * PI / 180}"
                 velocity="${joint_2_velocity_limit * PI / 180}" />
+            <dynamics damping="1.0" friction="1.0" />
         </joint>
         <link name="${robot_name}_link_3">
@@ -153,4 +156,5 @@
                 upper="${joint_3_position_limit * PI / 180}"
                 velocity="${joint_3_velocity_limit * PI / 180}" />
+            <dynamics damping="1.0" friction="1.0" />
         </joint>
         <link name="${robot_name}_link_4">
@@ -184,4 +188,5 @@
                 upper="${joint_4_position_limit * PI / 180}"
                 velocity="${joint_4_velocity_limit * PI / 180}" />
+            <dynamics damping="1.0" friction="1.0" />
         </joint>
         <link name="${robot_name}_link_5">
@@ -215,4 +220,5 @@
                 upper="${joint_5_position_limit * PI / 180}"
                 velocity="${joint_5_velocity_limit * PI / 180}" />
+            <dynamics damping="1.0" friction="1.0" />
         </joint>
         <link name="${robot_name}_link_6">
@@ -246,4 +252,5 @@
                 upper="${joint_6_position_limit * PI / 180}"
                 velocity="${joint_6_velocity_limit * PI / 180}" />
+            <dynamics damping="1.0" friction="1.0" />
         </joint>
         <link name="${robot_name}_link_7">

File: lbr_description/urdf/med14/med14_description.urdf.xacro (robot description, xacro)
@@ -60,4 +60,5 @@
                 upper="${joint_0_position_limit * PI / 180}"
                 velocity="${joint_0_velocity_limit * PI / 180}" />
+            <dynamics damping="1.0" friction="1.0" />
         </joint>
         <link name="${robot_name}_link_1">
@@ -91,4 +92,5 @@
                 upper="${joint_1_position_limit * PI / 180}"
                 velocity="${joint_1_velocity_limit * PI / 180}" />
+            <dynamics damping="1.0" friction="1.0" />
         </joint>
         <link name="${robot_name}_link_2">
@@ -122,4 +124,5 @@
                 upper="${joint_2_position_limit * PI / 180}"
                 velocity="${joint_2_velocity_limit * PI / 180}" />
+            <dynamics damping="1.0" friction="1.0" />
         </joint>
         <link name="${robot_name}_link_3">
@@ -153,4 +156,5 @@
                 upper="${joint_3_position_limit * PI / 180}"
                 velocity="${joint_3_velocity_limit * PI / 180}" />
+            <dynamics damping="1.0" friction="1.0" />
         </joint>
         <link name="${robot_name}_link_4">
@@ -184,4 +188,5 @@
                 upper="${joint_4_position_limit * PI / 180}"
                 velocity="${joint_4_velocity_limit * PI / 180}" />
+            <dynamics damping="1.0" friction="1.0" />
         </joint>
         <link name="${robot_name}_link_5">
@@ -215,4 +220,5 @@
                 upper="${joint_5_position_limit * PI / 180}"
                 velocity="${joint_5_velocity_limit * PI / 180}" />
+            <dynamics damping="1.0" friction="1.0" />
         </joint>
         <link name="${robot_name}_link_6">
@@ -246,4 +252,5 @@
                 upper="${joint_6_position_limit * PI / 180}"
                 velocity="${joint_6_velocity_limit * PI / 180}" />
+            <dynamics damping="1.0" friction="1.0" />
         </joint>
         <link name="${robot_name}_link_7">

File: lbr_description/urdf/med7/med7_description.urdf.xacro (robot description, xacro)
@@ -59,4 +59,5 @@
                 upper="${joint_0_position_limit * PI / 180}"
                 velocity="${joint_0_velocity_limit * PI / 180}" />
+            <dynamics damping="1.0" friction="1.0" />
         </joint>
         <link name="${robot_name}_link_1">
@@ -90,4 +91,5 @@
                 upper="${joint_1_position_limit * PI / 180}"
                 velocity="${joint_1_velocity_limit * PI / 180}" />
+            <dynamics damping="1.0" friction="1.0" />
         </joint>
         <link name="${robot_name}_link_2">
@@ -121,4 +123,5 @@
                 upper="${joint_2_position_limit * PI / 180}"
                 velocity="${joint_2_velocity_limit * PI / 180}" />
+            <dynamics damping="1.0" friction="1.0" />
         </joint>
         <link name="${robot_name}_link_3">
@@ -152,4 +155,5 @@
                 upper="${joint_3_position_limit * PI / 180}"
                 velocity="${joint_3_velocity_limit * PI / 180}" />
+            <dynamics damping="1.0" friction="1.0" />
         </joint>
         <link name="${robot_name}_link_4">
@@ -183,4 +187,5 @@
                 upper="${joint_4_position_limit * PI / 180}"
                 velocity="${joint_4_velocity_limit * PI / 180}" />
+            <dynamics damping="1.0" friction="1.0" />
         </joint>
         <link name="${robot_name}_link_5">
@@ -214,4 +219,5 @@
                 upper="${joint_5_position_limit * PI / 180}"
                 velocity="${joint_5_velocity_limit * PI / 180}" />
+            <dynamics damping="1.0" friction="1.0" />
         </joint>
         <link name="${robot_name}_link_6">
@@ -245,4 +251,5 @@
                 upper="${joint_6_position_limit * PI / 180}"
                 velocity="${joint_6_velocity_limit * PI / 180}" />
+            <dynamics damping="1.0" friction="1.0" />
         </joint>
         <link name="${robot_name}_link_7">
