Commit message: updated friction

File: lbr_description/urdf/iiwa14/iiwa14_description.urdf.xacro (robot description, xacro)
@@ -3,4 +3,6 @@
     <!-- some constants -->
     <xacro:property name="PI" value="3.1415926535897931" />
+    <xacro:property name="joint_damping" value="10.0" />
+    <xacro:property name="joint_friction" value="0.1" />
     <xacro:property name="joint_0_position_limit" value="170" />
     <xacro:property name="joint_1_position_limit" value="120" />
@@ -24,6 +26,5 @@
     <!-- robot as extracted via https://github.com/syuntoku14/fusion2urdf -->
     <xacro:macro name="iiwa14" params="parent:=^|world robot_name:=^|lbr sim:=^|true">
-        <!--joint
-        between {parent} and link_0-->
+        <!--joint between {parent} and link_0-->
         <joint name="${parent}_${robot_name}_joint" type="fixed">
             <parent link="${parent}" />
@@ -60,5 +61,5 @@
                 upper="${joint_0_position_limit * PI / 180}"
                 velocity="${joint_0_velocity_limit * PI / 180}" />
-            <dynamics damping="1.0" friction="1.0" />
+            <dynamics damping="${joint_damping}" friction="${joint_friction}" />
         </joint>
         <link name="${robot_name}_link_1">
@@ -92,5 +93,5 @@
                 upper="${joint_1_position_limit * PI / 180}"
                 velocity="${joint_1_velocity_limit * PI / 180}" />
-            <dynamics damping="1.0" friction="1.0" />
+            <dynamics damping="${joint_damping}" friction="${joint_friction}" />
         </joint>
         <link name="${robot_name}_link_2">
@@ -124,5 +125,5 @@
                 upper="${joint_2_position_limit * PI / 180}"
                 velocity="${joint_2_velocity_limit * PI / 180}" />
-            <dynamics damping="1.0" friction="1.0" />
+            <dynamics damping="${joint_damping}" friction="${joint_friction}" />
         </joint>
         <link name="${robot_name}_link_3">
@@ -156,5 +157,5 @@
                 upper="${joint_3_position_limit * PI / 180}"
                 velocity="${joint_3_velocity_limit * PI / 180}" />
-            <dynamics damping="1.0" friction="1.0" />
+            <dynamics damping="${joint_damping}" friction="${joint_friction}" />
         </joint>
         <link name="${robot_name}_link_4">
@@ -188,5 +189,5 @@
                 upper="${joint_4_position_limit * PI / 180}"
                 velocity="${joint_4_velocity_limit * PI / 180}" />
-            <dynamics damping="1.0" friction="1.0" />
+            <dynamics damping="${joint_damping}" friction="${joint_friction}" />
         </joint>
         <link name="${robot_name}_link_5">
@@ -220,5 +221,5 @@
                 upper="${joint_5_position_limit * PI / 180}"
                 velocity="${joint_5_velocity_limit * PI / 180}" />
-            <dynamics damping="1.0" friction="1.0" />
+            <dynamics damping="${joint_damping}" friction="${joint_friction}" />
         </joint>
         <link name="${robot_name}_link_6">
@@ -252,5 +253,5 @@
                 upper="${joint_6_position_limit * PI / 180}"
                 velocity="${joint_6_velocity_limit * PI / 180}" />
-            <dynamics damping="1.0" friction="1.0" />
+            <dynamics damping="${joint_damping}" friction="${joint_friction}" />
         </joint>
         <link name="${robot_name}_link_7">

File: lbr_description/urdf/iiwa7/iiwa7_description.urdf.xacro (robot description, xacro)
@@ -3,4 +3,6 @@
     <!-- some constants -->
     <xacro:property name="PI" value="3.1415926535897931" />
+    <xacro:property name="joint_damping" value="10.0" />
+    <xacro:property name="joint_friction" value="0.1" />
     <xacro:property name="joint_0_position_limit" value="170" />
     <xacro:property name="joint_1_position_limit" value="120" />
@@ -24,6 +26,5 @@
     <!-- robot as extracted via https://github.com/syuntoku14/fusion2urdf -->
     <xacro:macro name="iiwa7" params="parent:=^|world robot_name:=^|lbr sim:=^|true">
-        <!--joint
-        between {parent} and link_0-->
+        <!--joint between {parent} and link_0-->
         <joint name="${parent}_${robot_name}_joint" type="fixed">
             <parent link="${parent}" />
@@ -60,5 +61,5 @@
                 upper="${joint_0_position_limit * PI / 180}"
                 velocity="${joint_0_velocity_limit * PI / 180}" />
-            <dynamics damping="1.0" friction="1.0" />
+            <dynamics damping="${joint_damping}" friction="${joint_friction}" />
         </joint>
         <link name="${robot_name}_link_1">
@@ -92,5 +93,5 @@
                 upper="${joint_1_position_limit * PI / 180}"
                 velocity="${joint_1_velocity_limit * PI / 180}" />
-            <dynamics damping="1.0" friction="1.0" />
+            <dynamics damping="${joint_damping}" friction="${joint_friction}" />
         </joint>
         <link name="${robot_name}_link_2">
@@ -124,5 +125,5 @@
                 upper="${joint_2_position_limit * PI / 180}"
                 velocity="${joint_2_velocity_limit * PI / 180}" />
-            <dynamics damping="1.0" friction="1.0" />
+            <dynamics damping="${joint_damping}" friction="${joint_friction}" />
         </joint>
         <link name="${robot_name}_link_3">
@@ -156,5 +157,5 @@
                 upper="${joint_3_position_limit * PI / 180}"
                 velocity="${joint_3_velocity_limit * PI / 180}" />
-            <dynamics damping="1.0" friction="1.0" />
+            <dynamics damping="${joint_damping}" friction="${joint_friction}" />
         </joint>
         <link name="${robot_name}_link_4">
@@ -188,5 +189,5 @@
                 upper="${joint_4_position_limit * PI / 180}"
                 velocity="${joint_4_velocity_limit * PI / 180}" />
-            <dynamics damping="1.0" friction="1.0" />
+            <dynamics damping="${joint_damping}" friction="${joint_friction}" />
         </joint>
         <link name="${robot_name}_link_5">
@@ -220,5 +221,5 @@
                 upper="${joint_5_position_limit * PI / 180}"
                 velocity="${joint_5_velocity_limit * PI / 180}" />
-            <dynamics damping="1.0" friction="1.0" />
+            <dynamics damping="${joint_damping}" friction="${joint_friction}" />
         </joint>
         <link name="${robot_name}_link_6">
@@ -252,5 +253,5 @@
                 upper="${joint_6_position_limit * PI / 180}"
                 velocity="${joint_6_velocity_limit * PI / 180}" />
-            <dynamics damping="1.0" friction="1.0" />
+            <dynamics damping="${joint_damping}" friction="${joint_friction}" />
         </joint>
         <link name="${robot_name}_link_7">

File: lbr_description/urdf/med14/med14_description.urdf.xacro (robot description, xacro)
@@ -3,4 +3,6 @@
     <!-- some constants -->
     <xacro:property name="PI" value="3.1415926535897931" />
+    <xacro:property name="joint_damping" value="10.0" />
+    <xacro:property name="joint_friction" value="0.1" />
     <xacro:property name="joint_0_position_limit" value="170" />
     <xacro:property name="joint_1_position_limit" value="120" />
@@ -24,6 +26,5 @@
     <!-- robot as extracted via https://github.com/syuntoku14/fusion2urdf -->
     <xacro:macro name="med14" params="parent:=^|world robot_name:=^|lbr sim:=^|true">
-        <!--joint
-        between {parent} and link_0-->
+        <!--joint between {parent} and link_0-->
         <joint name="${parent}_${robot_name}_joint" type="fixed">
             <parent link="${parent}" />
@@ -60,5 +61,5 @@
                 upper="${joint_0_position_limit * PI / 180}"
                 velocity="${joint_0_velocity_limit * PI / 180}" />
-            <dynamics damping="1.0" friction="1.0" />
+            <dynamics damping="${joint_damping}" friction="${joint_friction}" />
         </joint>
         <link name="${robot_name}_link_1">
@@ -92,5 +93,5 @@
                 upper="${joint_1_position_limit * PI / 180}"
                 velocity="${joint_1_velocity_limit * PI / 180}" />
-            <dynamics damping="1.0" friction="1.0" />
+            <dynamics damping="${joint_damping}" friction="${joint_friction}" />
         </joint>
         <link name="${robot_name}_link_2">
@@ -124,5 +125,5 @@
                 upper="${joint_2_position_limit * PI / 180}"
                 velocity="${joint_2_velocity_limit * PI / 180}" />
-            <dynamics damping="1.0" friction="1.0" />
+            <dynamics damping="${joint_damping}" friction="${joint_friction}" />
         </joint>
         <link name="${robot_name}_link_3">
@@ -156,5 +157,5 @@
                 upper="${joint_3_position_limit * PI / 180}"
                 velocity="${joint_3_velocity_limit * PI / 180}" />
-            <dynamics damping="1.0" friction="1.0" />
+            <dynamics damping="${joint_damping}" friction="${joint_friction}" />
         </joint>
         <link name="${robot_name}_link_4">
@@ -188,5 +189,5 @@
                 upper="${joint_4_position_limit * PI / 180}"
                 velocity="${joint_4_velocity_limit * PI / 180}" />
-            <dynamics damping="1.0" friction="1.0" />
+            <dynamics damping="${joint_damping}" friction="${joint_friction}" />
         </joint>
         <link name="${robot_name}_link_5">
@@ -220,5 +221,5 @@
                 upper="${joint_5_position_limit * PI / 180}"
                 velocity="${joint_5_velocity_limit * PI / 180}" />
-            <dynamics damping="1.0" friction="1.0" />
+            <dynamics damping="${joint_damping}" friction="${joint_friction}" />
         </joint>
         <link name="${robot_name}_link_6">
@@ -252,5 +253,5 @@
                 upper="${joint_6_position_limit * PI / 180}"
                 velocity="${joint_6_velocity_limit * PI / 180}" />
-            <dynamics damping="1.0" friction="1.0" />
+            <dynamics damping="${joint_damping}" friction="${joint_friction}" />
         </joint>
         <link name="${robot_name}_link_7">

File: lbr_description/urdf/med7/med7_description.urdf.xacro (robot description, xacro)
@@ -3,4 +3,6 @@
     <!-- some constants -->
     <xacro:property name="PI" value="3.1415926535897931" />
+    <xacro:property name="joint_damping" value="10.0" />
+    <xacro:property name="joint_friction" value="0.1" />
     <xacro:property name="joint_0_position_limit" value="170" />
     <xacro:property name="joint_1_position_limit" value="120" />
@@ -59,5 +61,5 @@
                 upper="${joint_0_position_limit * PI / 180}"
                 velocity="${joint_0_velocity_limit * PI / 180}" />
-            <dynamics damping="1.0" friction="1.0" />
+            <dynamics damping="${joint_damping}" friction="${joint_friction}" />
         </joint>
         <link name="${robot_name}_link_1">
@@ -91,5 +93,5 @@
                 upper="${joint_1_position_limit * PI / 180}"
                 velocity="${joint_1_velocity_limit * PI / 180}" />
-            <dynamics damping="1.0" friction="1.0" />
+            <dynamics damping="${joint_damping}" friction="${joint_friction}" />
         </joint>
         <link name="${robot_name}_link_2">
@@ -123,5 +125,5 @@
                 upper="${joint_2_position_limit * PI / 180}"
                 velocity="${joint_2_velocity_limit * PI / 180}" />
-            <dynamics damping="1.0" friction="1.0" />
+            <dynamics damping="${joint_damping}" friction="${joint_friction}" />
         </joint>
         <link name="${robot_name}_link_3">
@@ -155,5 +157,5 @@
                 upper="${joint_3_position_limit * PI / 180}"
                 velocity="${joint_3_velocity_limit * PI / 180}" />
-            <dynamics damping="1.0" friction="1.0" />
+            <dynamics damping="${joint_damping}" friction="${joint_friction}" />
         </joint>
         <link name="${robot_name}_link_4">
@@ -187,5 +189,5 @@
                 upper="${joint_4_position_limit * PI / 180}"
                 velocity="${joint_4_velocity_limit * PI / 180}" />
-            <dynamics damping="1.0" friction="1.0" />
+            <dynamics damping="${joint_damping}" friction="${joint_friction}" />
         </joint>
         <link name="${robot_name}_link_5">
@@ -219,5 +221,5 @@
                 upper="${joint_5_position_limit * PI / 180}"
                 velocity="${joint_5_velocity_limit * PI / 180}" />
-            <dynamics damping="1.0" friction="1.0" />
+            <dynamics damping="${joint_damping}" friction="${joint_friction}" />
         </joint>
         <link name="${robot_name}_link_6">
@@ -251,5 +253,5 @@
                 upper="${joint_6_position_limit * PI / 180}"
                 velocity="${joint_6_velocity_limit * PI / 180}" />
-            <dynamics damping="1.0" friction="1.0" />
+            <dynamics damping="${joint_damping}" friction="${joint_friction}" />
         </joint>
         <link name="${robot_name}_link_7">
