Commit message: removed robot name

File: lbr_description/urdf/iiwa14/iiwa14_description.urdf.xacro (robot description, xacro)
@@ -274,7 +274,6 @@
             <origin xyz="0 0 0.035" rpy="0 0 0" />
         </joint>
-        <link name="link_ee">
-        </link>
-        <xacro:lbr_gazebo robot_name="${robot_name}" />
+        <link name="link_ee" />
+        <xacro:lbr_gazebo />
         <!-- TODO: move modes to args, decouple urdf/gazebo/controls -->
         <xacro:lbr_hardware_interface

File: lbr_description/urdf/iiwa7/iiwa7_description.urdf.xacro (robot description, xacro)
@@ -274,7 +274,6 @@
             <origin xyz="0 0 0.035" rpy="0 0 0" />
         </joint>
-        <link name="link_ee">
-        </link>
-        <xacro:lbr_gazebo robot_name="${robot_name}" />
+        <link name="link_ee" />
+        <xacro:lbr_gazebo />
         <!-- TODO: move modes to args, decouple urdf/gazebo/controls -->
         <xacro:lbr_hardware_interface

File: lbr_description/urdf/med14/med14_description.urdf.xacro (robot description, xacro)
@@ -274,7 +274,6 @@
             <origin xyz="0 0 0.035" rpy="0 0 0" />
         </joint>
-        <link name="link_ee">
-        </link>
-        <xacro:lbr_gazebo robot_name="${robot_name}" />
+        <link name="link_ee" />
+        <xacro:lbr_gazebo />
         <!-- TODO: move modes to args, decouple urdf/gazebo/controls -->
         <xacro:lbr_hardware_interface

File: lbr_description/urdf/med7/med7_description.urdf.xacro (robot description, xacro)
@@ -274,7 +274,6 @@
             <origin xyz="0 0 0.035" rpy="0 0 0" />
         </joint>
-        <link name="link_ee">
-        </link>
-        <xacro:lbr_gazebo robot_name="${robot_name}" />
+        <link name="link_ee" />
+        <xacro:lbr_gazebo />
         <!-- TODO: move modes to args, decouple urdf/gazebo/controls -->
         <xacro:lbr_hardware_interface

Commit message: ee fix #125

File: lbr_description/urdf/iiwa14/iiwa14_description.urdf.xacro (robot description, xacro)
@@ -272,5 +272,5 @@
             <parent link="link_7" />
             <child link="link_ee" />
-            <origin xyz="0 0 0.035" rpy="0 0 0" />
+            <origin xyz="0 0 0.045" rpy="0 0 0" />
         </joint>
         <link name="link_ee">

File: lbr_description/urdf/med14/med14_description.urdf.xacro (robot description, xacro)
@@ -272,5 +272,5 @@
             <parent link="link_7" />
             <child link="link_ee" />
-            <origin xyz="0 0 0.035" rpy="0 0 0" />
+            <origin xyz="0 0 0.045" rpy="0 0 0" />
         </joint>
         <link name="link_ee">

Commit message: ee fix #125

File: lbr_description/urdf/iiwa14/iiwa14_description.urdf.xacro (robot description, xacro)
@@ -280,5 +280,5 @@
             <parent link="${robot_name}_link_7" />
             <child link="${robot_name}_link_ee" />
-            <origin xyz="0 0 0.035" rpy="0 0 0" />
+            <origin xyz="0 0 0.045" rpy="0 0 0" />
         </joint>
         <link name="${robot_name}_link_ee">

File: lbr_description/urdf/med14/med14_description.urdf.xacro (robot description, xacro)
@@ -280,5 +280,5 @@
             <parent link="${robot_name}_link_7" />
             <child link="${robot_name}_link_ee" />
-            <origin xyz="0 0 0.035" rpy="0 0 0" />
+            <origin xyz="0 0 0.045" rpy="0 0 0" />
         </joint>
         <link name="${robot_name}_link_ee">

Commit message: ee fix #125

File: lbr_description/urdf/iiwa14/iiwa14_description.urdf.xacro (robot description, xacro)
@@ -267,5 +267,5 @@
             <parent link="link_7" />
             <child link="link_ee" />
-            <origin xyz="0 0 0.035" rpy="0 0 0" />
+            <origin xyz="0 0 0.045" rpy="0 0 0" />
         </joint>
         <link name="link_ee">

File: lbr_description/urdf/med14/med14_description.urdf.xacro (robot description, xacro)
@@ -267,5 +267,5 @@
             <parent link="link_7" />
             <child link="link_ee" />
-            <origin xyz="0 0 0.035" rpy="0 0 0" />
+            <origin xyz="0 0 0.045" rpy="0 0 0" />
         </joint>
         <link name="link_ee">

Commit message: revert tf

File: lbr_description/urdf/iiwa14/iiwa14_description.urdf.xacro (robot description, xacro)
@@ -267,5 +267,5 @@
             <parent link="link_7" />
             <child link="link_ee" />
-            <origin xyz="0 0 0.045" rpy="0 0 0" />
+            <origin xyz="0 0 0.035" rpy="0 0 0" />
         </joint>
         <link name="link_ee">

File: lbr_description/urdf/med14/med14_description.urdf.xacro (robot description, xacro)
@@ -267,5 +267,5 @@
             <parent link="link_7" />
             <child link="link_ee" />
-            <origin xyz="0 0 0.045" rpy="0 0 0" />
+            <origin xyz="0 0 0.035" rpy="0 0 0" />
         </joint>
         <link name="link_ee">

Commit message: revert tf

File: lbr_description/urdf/iiwa14/iiwa14_description.urdf.xacro (robot description, xacro)
@@ -272,5 +272,5 @@
             <parent link="link_7" />
             <child link="link_ee" />
-            <origin xyz="0 0 0.045" rpy="0 0 0" />
+            <origin xyz="0 0 0.035" rpy="0 0 0" />
         </joint>
         <link name="link_ee">

File: lbr_description/urdf/med14/med14_description.urdf.xacro (robot description, xacro)
@@ -272,5 +272,5 @@
             <parent link="link_7" />
             <child link="link_ee" />
-            <origin xyz="0 0 0.045" rpy="0 0 0" />
+            <origin xyz="0 0 0.035" rpy="0 0 0" />
         </joint>
         <link name="link_ee">

Commit message: revert tf

File: lbr_description/urdf/iiwa14/iiwa14_description.urdf.xacro (robot description, xacro)
@@ -280,5 +280,5 @@
             <parent link="${robot_name}_link_7" />
             <child link="${robot_name}_link_ee" />
-            <origin xyz="0 0 0.045" rpy="0 0 0" />
+            <origin xyz="0 0 0.035" rpy="0 0 0" />
         </joint>
         <link name="${robot_name}_link_ee">

File: lbr_description/urdf/med14/med14_description.urdf.xacro (robot description, xacro)
@@ -280,5 +280,5 @@
             <parent link="${robot_name}_link_7" />
             <child link="${robot_name}_link_ee" />
-            <origin xyz="0 0 0.045" rpy="0 0 0" />
+            <origin xyz="0 0 0.035" rpy="0 0 0" />
         </joint>
         <link name="${robot_name}_link_ee">

Commit message: updated transforms

File: lbr_description/urdf/iiwa14/iiwa14_description.urdf.xacro (robot description, xacro)
@@ -79,5 +79,5 @@
         </link>
         <joint name="A2" type="revolute">
-            <origin rpy="0 0 0" xyz="0.0 -0.01 0.2125" />
+            <origin rpy="0 0 0" xyz="-0.0 -0.01 0.2125" />
             <parent link="link_1" />
             <child link="link_2" />
@@ -110,5 +110,5 @@
         </link>
         <joint name="A3" type="revolute">
-            <origin rpy="0 0 0" xyz="0.0 0.01 0.1945" />
+            <origin rpy="0 0 0" xyz="0.0 0.01 0.228" />
             <parent link="link_2" />
             <child link="link_3" />
@@ -128,5 +128,5 @@
             </inertial>
             <visual>
-                <origin rpy="0 0 0" xyz="-0.0 0.0 -0.5545" />
+                <origin rpy="0 0 0" xyz="0.0 -0.0 -0.588" />
                 <geometry>
                     <mesh filename="package://lbr_description/meshes/iiwa14/visual/link_3.dae" />
@@ -134,5 +134,5 @@
             </visual>
             <collision>
-                <origin rpy="0 0 0" xyz="-0.0 0.0 -0.5545" />
+                <origin rpy="0 0 0" xyz="0.0 -0.0 -0.588" />
                 <geometry>
                     <mesh filename="package://lbr_description/meshes/iiwa14/collision/link_3.stl" />
@@ -141,5 +141,5 @@
         </link>
         <joint name="A4" type="revolute">
-            <origin rpy="0 0 0" xyz="-0.0 0.0105 0.2255" />
+            <origin rpy="0 0 0" xyz="0.0 0.0105 0.192" />
             <parent link="link_3" />
             <child link="link_4" />
@@ -159,5 +159,5 @@
             </inertial>
             <visual>
-                <origin rpy="0 0 0" xyz="0.0 -0.0105 -0.78" />
+                <origin rpy="0 0 0" xyz="-0.0 -0.0105 -0.78" />
                 <geometry>
                     <mesh filename="package://lbr_description/meshes/iiwa14/visual/link_4.dae" />
@@ -165,5 +165,5 @@
             </visual>
             <collision>
-                <origin rpy="0 0 0" xyz="0.0 -0.0105 -0.78" />
+                <origin rpy="0 0 0" xyz="-0.0 -0.0105 -0.78" />
                 <geometry>
                     <mesh filename="package://lbr_description/meshes/iiwa14/collision/link_4.stl" />
@@ -172,5 +172,5 @@
         </link>
         <joint name="A5" type="revolute">
-            <origin rpy="0 0 0" xyz="0.0 -0.0105 0.1745" />
+            <origin rpy="0 0 0" xyz="-0.0 -0.0105 0.2075" />
             <parent link="link_4" />
             <child link="link_5" />
@@ -190,5 +190,5 @@
             </inertial>
             <visual>
-                <origin rpy="0 0 0" xyz="-0.0 0.0 -0.9545" />
+                <origin rpy="0 0 0" xyz="0.0 0.0 -0.9875" />
                 <geometry>
                     <mesh filename="package://lbr_description/meshes/iiwa14/visual/link_5.dae" />
@@ -196,5 +196,5 @@
             </visual>
             <collision>
-                <origin rpy="0 0 0" xyz="-0.0 0.0 -0.9545" />
+                <origin rpy="0 0 0" xyz="0.0 0.0 -0.9875" />
                 <geometry>
                     <mesh filename="package://lbr_description/meshes/iiwa14/collision/link_5.stl" />
@@ -203,5 +203,5 @@
         </link>
         <joint name="A6" type="revolute">
-            <origin rpy="0 0 0" xyz="-0.0 -0.0707 0.2255" />
+            <origin rpy="0 0 0" xyz="0.0 -0.0707 0.1925" />
             <parent link="link_5" />
             <child link="link_6" />
@@ -234,5 +234,5 @@
         </link>
         <joint name="A7" type="revolute">
-            <origin rpy="0 0 0" xyz="0.0 0.0707 0.0711" />
+            <origin rpy="0 0 0" xyz="0.0 0.0707 0.091" />
             <parent link="link_6" />
             <child link="link_7" />
@@ -252,5 +252,5 @@
             </inertial>
             <visual>
-                <origin rpy="0 0 0" xyz="0.0 0.0 -1.2511" />
+                <origin rpy="0 0 0" xyz="-0.0 0.0 -1.271" />
                 <geometry>
                     <mesh filename="package://lbr_description/meshes/iiwa14/visual/link_7.dae" />
@@ -258,5 +258,5 @@
             </visual>
             <collision>
-                <origin rpy="0 0 0" xyz="0.0 0.0 -1.2511" />
+                <origin rpy="0 0 0" xyz="-0.0 0.0 -1.271" />
                 <geometry>
                     <mesh filename="package://lbr_description/meshes/iiwa14/collision/link_7.stl" />

File: lbr_description/urdf/iiwa7/iiwa7_description.urdf.xacro (robot description, xacro)
@@ -79,5 +79,5 @@
         </link>
         <joint name="A2" type="revolute">
-            <origin rpy="0 0 0" xyz="-0.0 -0.0105 0.193" />
+            <origin rpy="0 0 0" xyz="-0.0 -0.0105 0.1925" />
             <parent link="link_1" />
             <child link="link_2" />
@@ -97,5 +97,5 @@
             </inertial>
             <visual>
-                <origin rpy="0 0 0" xyz="0.0 0.0105 -0.3405" />
+                <origin rpy="0 0 0" xyz="0.0 0.0105 -0.34" />
                 <geometry>
                     <mesh filename="package://lbr_description/meshes/iiwa7/visual/link_2.dae" />
@@ -103,5 +103,5 @@
             </visual>
             <collision>
-                <origin rpy="0 0 0" xyz="0.0 0.0105 -0.3405" />
+                <origin rpy="0 0 0" xyz="0.0 0.0105 -0.34" />
                 <geometry>
                     <mesh filename="package://lbr_description/meshes/iiwa7/collision/link_2.stl" />
@@ -110,5 +110,5 @@
         </link>
         <joint name="A3" type="revolute">
-            <origin rpy="0 0 0" xyz="0.0 0.0105 0.1745" />
+            <origin rpy="0 0 0" xyz="0.0 0.0105 0.2075" />
             <parent link="link_2" />
             <child link="link_3" />
@@ -128,5 +128,5 @@
             </inertial>
             <visual>
-                <origin rpy="0 0 0" xyz="0.0 0.0 -0.515" />
+                <origin rpy="0 0 0" xyz="0.0 -0.0 -0.5475" />
                 <geometry>
                     <mesh filename="package://lbr_description/meshes/iiwa7/visual/link_3.dae" />
@@ -134,5 +134,5 @@
             </visual>
             <collision>
-                <origin rpy="0 0 0" xyz="0.0 0.0 -0.515" />
+                <origin rpy="0 0 0" xyz="0.0 -0.0 -0.5475" />
                 <geometry>
                     <mesh filename="package://lbr_description/meshes/iiwa7/collision/link_3.stl" />
@@ -141,5 +141,5 @@
         </link>
         <joint name="A4" type="revolute">
-            <origin rpy="0 0 0" xyz="0.0 0.0105 0.2255" />
+            <origin rpy="0 0 0" xyz="0.0 0.0105 0.1925" />
             <parent link="link_3" />
             <child link="link_4" />
@@ -159,5 +159,5 @@
             </inertial>
             <visual>
-                <origin rpy="0 0 0" xyz="0.0 -0.0105 -0.7405" />
+                <origin rpy="0 0 0" xyz="-0.0 -0.0105 -0.74" />
                 <geometry>
                     <mesh filename="package://lbr_description/meshes/iiwa7/visual/link_4.dae" />
@@ -165,5 +165,5 @@
             </visual>
             <collision>
-                <origin rpy="0 0 0" xyz="0.0 -0.0105 -0.7405" />
+                <origin rpy="0 0 0" xyz="-0.0 -0.0105 -0.74" />
                 <geometry>
                     <mesh filename="package://lbr_description/meshes/iiwa7/collision/link_4.stl" />
@@ -172,5 +172,5 @@
         </link>
         <joint name="A5" type="revolute">
-            <origin rpy="0 0 0" xyz="0.0 -0.0105 0.1745" />
+            <origin rpy="0 0 0" xyz="-0.0 -0.0105 0.2075" />
             <parent link="link_4" />
             <child link="link_5" />
@@ -190,5 +190,5 @@
             </inertial>
             <visual>
-                <origin rpy="0 0 0" xyz="0.0 0.0 -0.915" />
+                <origin rpy="0 0 0" xyz="0.0 0.0 -0.9475" />
                 <geometry>
                     <mesh filename="package://lbr_description/meshes/iiwa7/visual/link_5.dae" />
@@ -196,5 +196,5 @@
             </visual>
             <collision>
-                <origin rpy="0 0 0" xyz="0.0 0.0 -0.915" />
+                <origin rpy="0 0 0" xyz="0.0 0.0 -0.9475" />
                 <geometry>
                     <mesh filename="package://lbr_description/meshes/iiwa7/collision/link_5.stl" />
@@ -203,5 +203,5 @@
         </link>
         <joint name="A6" type="revolute">
-            <origin rpy="0 0 0" xyz="0.0 -0.0707 0.2255" />
+            <origin rpy="0 0 0" xyz="0.0 -0.0707 0.1925" />
             <parent link="link_5" />
             <child link="link_6" />
@@ -221,5 +221,5 @@
             </inertial>
             <visual>
-                <origin rpy="0 0 0" xyz="0.0 0.0707 -1.1405" />
+                <origin rpy="0 0 0" xyz="0.0 0.0707 -1.14" />
                 <geometry>
                     <mesh filename="package://lbr_description/meshes/iiwa7/visual/link_6.dae" />
@@ -227,5 +227,5 @@
             </visual>
             <collision>
-                <origin rpy="0 0 0" xyz="0.0 0.0707 -1.1405" />
+                <origin rpy="0 0 0" xyz="0.0 0.0707 -1.14" />
                 <geometry>
                     <mesh filename="package://lbr_description/meshes/iiwa7/collision/link_6.stl" />
@@ -234,5 +234,5 @@
         </link>
         <joint name="A7" type="revolute">
-            <origin rpy="0 0 0" xyz="0.0 0.0705 0.0909" />
+            <origin rpy="0 0 0" xyz="0.0 0.0707 0.091" />
             <parent link="link_6" />
             <child link="link_7" />
@@ -252,5 +252,5 @@
             </inertial>
             <visual>
-                <origin rpy="0 0 0" xyz="0.0 0.0002 -1.2314" />
+                <origin rpy="0 0 0" xyz="-0.0 0.0 -1.231" />
                 <geometry>
                     <mesh filename="package://lbr_description/meshes/iiwa7/visual/link_7.dae" />
@@ -258,5 +258,5 @@
             </visual>
             <collision>
-                <origin rpy="0 0 0" xyz="0.0 0.0002 -1.2314" />
+                <origin rpy="0 0 0" xyz="-0.0 0.0 -1.231" />
                 <geometry>
                     <mesh filename="package://lbr_description/meshes/iiwa7/collision/link_7.stl" />

Commit message: updated masses

File: lbr_description/urdf/iiwa14/iiwa14_description.urdf.xacro (robot description, xacro)
@@ -30,5 +30,5 @@
                 <origin rpy="0 0 0"
                     xyz="-0.0128215344957798 -7.86364415362405e-08 0.07150661827888387" />
-                <mass value="7.039242" />
+                <mass value="7.05037793" />
                 <inertia ixx="0.031177" ixy="0.000000" ixz="0.000870" iyy="0.039634" iyz="0.000000"
                     izz="0.043034" />
@@ -61,5 +61,5 @@
                 <origin rpy="0 0 0"
                     xyz="9.307232415315581e-08 -0.03379543155079102 0.13240370669453902" />
-                <mass value="5.281174" />
+                <mass value="5.28952872" />
                 <inertia ixx="0.042394" ixy="-0.000000" ixz="-0.000000" iyy="0.042770"
                     iyz="0.006331" izz="0.015845" />
@@ -92,5 +92,5 @@
                 <origin rpy="0 0 0"
                     xyz="0.00015188022518878674 0.051987109728758904 0.05880129877994178" />
-                <mass value="5.079432" />
+                <mass value="5.68888779" />
                 <inertia ixx="0.039326" ixy="-0.000029" ixz="0.000042" iyy="0.039101" iyz="0.006282"
                     izz="0.014161" />
@@ -123,5 +123,5 @@
                 <origin rpy="0 0 0"
                     xyz="-5.974614313346012e-09 0.029563618732667742 0.13650341869763982" />
-                <mass value="4.0811177" />
+                <mass value="3.46124535" />
                 <inertia ixx="0.032236" ixy="-0.000000" ixz="0.000000" iyy="0.030602"
                     iyz="-0.006265" izz="0.009779" />
@@ -154,5 +154,5 @@
                 <origin rpy="0 0 0"
                     xyz="-2.09625967727708e-08 -0.04476439079596513 0.06741903952954653" />
-                <mass value="3.521230" />
+                <mass value="4.12299549" />
                 <inertia ixx="0.022114" ixy="-0.000000" ixz="-0.000000" iyy="0.021074"
                     iyz="-0.003660" izz="0.007890" />
@@ -185,5 +185,5 @@
                 <origin rpy="0 0 0"
                     xyz="-0.00012008657208039079 -0.021390023245727908 0.0854754261653966" />
-                <mass value="2.176916" />
+                <mass value="1.56375558" />
                 <inertia ixx="0.012955" ixy="0.000002" ixz="-0.000001" iyy="0.011185" iyz="0.003972"
                     izz="0.005744" />
@@ -216,5 +216,5 @@
                 <origin rpy="0 0 0"
                     xyz="-6.000032555678588e-08 0.07103825551434698 0.000565530522845803" />
-                <mass value="2.324906" />
+                <mass value="2.4578784" />
                 <inertia ixx="0.006292" ixy="-0.000000" ixz="-0.000000" iyy="0.006023"
                     iyz="0.000314" izz="0.004585" />
@@ -247,5 +247,5 @@
                 <origin rpy="0 0 0"
                     xyz="3.963019849314055e-06 -1.5392768444664745e-08 0.027186686478491096" />
-                <mass value="0.395984" />
+                <mass value="0.26533073" />
                 <inertia ixx="0.000281" ixy="-0.000000" ixz="-0.000000" iyy="0.000277"
                     iyz="0.000000" izz="0.000430" />

File: lbr_description/urdf/iiwa7/iiwa7_description.urdf.xacro (robot description, xacro)
@@ -30,5 +30,5 @@
                 <origin rpy="0 0 0"
                     xyz="-0.01283618494463161 4.904567390585061e-08 0.07010682239932087" />
-                <mass value="4.861279" />
+                <mass value="4.85565842" />
                 <inertia ixx="0.017901" ixy="0.000000" ixz="0.000771" iyy="0.022356" iyz="-0.000000"
                     izz="0.021346" />
@@ -61,5 +61,5 @@
                 <origin rpy="0 0 0"
                     xyz="4.9980243666546455e-08 -0.0347335291089292 0.12351608478142942" />
-                <mass value="3.400745" />
+                <mass value="3.39401127" />
                 <inertia ixx="0.021502" ixy="-0.000000" ixz="0.000000" iyy="0.020512" iyz="0.003828"
                     izz="0.007587" />
@@ -92,5 +92,5 @@
                 <origin rpy="0 0 0"
                     xyz="4.0558428502019873e-08 0.04491581578298656 0.06732515284873997" />
-                <mass value="3.430184" />
+                <mass value="4.03199094" />
                 <inertia ixx="0.021455" ixy="-0.000000" ixz="0.000000" iyy="0.020444" iyz="0.003570"
                     izz="0.007671" />
@@ -123,5 +123,5 @@
                 <origin rpy="0 0 0"
                     xyz="-5.881068064938613e-09 0.02956361869175564 0.1365034185434154" />
-                <mass value="3.995443" />
+                <mass value="3.39401127" />
                 <inertia ixx="0.031559" ixy="-0.000000" ixz="0.000000" iyy="0.029960"
                     iyz="-0.006133" izz="0.009574" />
@@ -154,5 +154,5 @@
                 <origin rpy="0 0 0"
                     xyz="-4.1344813497116265e-08 -0.044916218629510306 0.06732501840381" />
-                <mass value="3.430182" />
+                <mass value="4.03198902" />
                 <inertia ixx="0.021454" ixy="0.000000" ixz="-0.000000" iyy="0.020443"
                     iyz="-0.003570" izz="0.007670" />
@@ -185,5 +185,5 @@
                 <origin rpy="0 0 0"
                     xyz="2.416002990197734e-08 -0.021386601078580914 0.085468591256322" />
-                <mass value="2.131557" />
+                <mass value="1.52923896" />
                 <inertia ixx="0.012684" ixy="-0.000000" ixz="-0.000000" iyy="0.010952"
                     iyz="0.003889" izz="0.005624" />
@@ -216,5 +216,5 @@
                 <origin rpy="0 0 0"
                     xyz="-9.07120004240837e-08 0.0709871260349443 0.002115721730276743" />
-                <mass value="2.311862" />
+                <mass value="2.40362602" />
                 <inertia ixx="0.006412" ixy="-0.000000" ixz="-0.000000" iyy="0.006166"
                     iyz="0.000314" izz="0.004459" />
@@ -247,5 +247,5 @@
                 <origin rpy="0 0 0"
                     xyz="4.535378460217862e-06 -1.7615872956281168e-08 0.009883270430701696" />
-                <mass value="0.338747" />
+                <mass value="0.25947411" />
                 <inertia ixx="0.000250" ixy="-0.000000" ixz="-0.000000" iyy="0.000245"
                     iyz="0.000000" izz="0.000406" />
