Commit message: updated inertias

File: lbr_description/urdf/iiwa14/iiwa14_description.urdf.xacro (robot description, xacro)
@@ -30,7 +30,7 @@
                 <origin rpy="0 0 0"
                     xyz="-0.0128215344957798 -7.86364415362405e-08 0.07150661827888387" />
-                <mass value="7.05037793" />
-                <inertia ixx="0.031177" ixy="0.000000" ixz="0.000870" iyy="0.039634" iyz="0.000000"
-                    izz="0.043034" />
+                <mass value="7.050378" />
+                <inertia ixx="0.031226" ixy="0.0" ixz="0.000871" iyy="0.039697" iyz="0.0"
+                    izz="0.043102" />
             </inertial>
             <visual>
@@ -61,10 +61,10 @@
                 <origin rpy="0 0 0"
                     xyz="9.307232415315581e-08 -0.03379543155079102 0.13240370669453902" />
-                <mass value="5.28952872" />
-                <inertia ixx="0.042394" ixy="-0.000000" ixz="-0.000000" iyy="0.042770"
-                    iyz="0.006331" izz="0.015845" />
-            </inertial>
-            <visual>
-                <origin rpy="0 0 0" xyz="-0.0 0.0 -0.1475" />
+                <mass value="5.289529" />
+                <inertia ixx="0.042462" ixy="0.0" ixz="0.0" iyy="0.042838" iyz="0.006341"
+                    izz="0.01587" />
+            </inertial>
+            <visual>
+                <origin rpy="0 0 0" xyz="0.0 0.0 -0.1475" />
                 <geometry>
                     <mesh filename="package://lbr_description/meshes/iiwa14/visual/link_1.dae" />
@@ -72,5 +72,5 @@
             </visual>
             <collision>
-                <origin rpy="0 0 0" xyz="-0.0 0.0 -0.1475" />
+                <origin rpy="0 0 0" xyz="0.0 0.0 -0.1475" />
                 <geometry>
                     <mesh filename="package://lbr_description/meshes/iiwa14/collision/link_1.stl" />
@@ -79,5 +79,5 @@
         </link>
         <joint name="A2" type="revolute">
-            <origin rpy="0 0 0" xyz="-0.0 -0.01 0.2125" />
+            <origin rpy="0 0 0" xyz="0.0 -0.01 0.2125" />
             <parent link="link_1" />
             <child link="link_2" />
@@ -92,10 +92,10 @@
                 <origin rpy="0 0 0"
                     xyz="0.00015188022518878674 0.051987109728758904 0.05880129877994178" />
-                <mass value="5.68888779" />
-                <inertia ixx="0.039326" ixy="-0.000029" ixz="0.000042" iyy="0.039101" iyz="0.006282"
-                    izz="0.014161" />
-            </inertial>
-            <visual>
-                <origin rpy="0 0 0" xyz="-0.0 0.01 -0.36" />
+                <mass value="5.688888" />
+                <inertia ixx="0.055182" ixy="-3.3e-05" ixz="5.6e-05" iyy="0.053983" iyz="0.010034"
+                    izz="0.016523" />
+            </inertial>
+            <visual>
+                <origin rpy="0 0 0" xyz="0.0 0.01 -0.36" />
                 <geometry>
                     <mesh filename="package://lbr_description/meshes/iiwa14/visual/link_2.dae" />
@@ -103,5 +103,5 @@
             </visual>
             <collision>
-                <origin rpy="0 0 0" xyz="-0.0 0.01 -0.36" />
+                <origin rpy="0 0 0" xyz="0.0 0.01 -0.36" />
                 <geometry>
                     <mesh filename="package://lbr_description/meshes/iiwa14/collision/link_2.stl" />
@@ -123,10 +123,10 @@
                 <origin rpy="0 0 0"
                     xyz="-5.974614313346012e-09 0.029563618732667742 0.13650341869763982" />
-                <mass value="3.46124535" />
-                <inertia ixx="0.032236" ixy="-0.000000" ixz="0.000000" iyy="0.030602"
-                    iyz="-0.006265" izz="0.009779" />
-            </inertial>
-            <visual>
-                <origin rpy="0 0 0" xyz="0.0 -0.0 -0.588" />
+                <mass value="3.461245" />
+                <inertia ixx="0.02172" ixy="0.0" ixz="0.0" iyy="0.02073" iyz="-0.003845"
+                    izz="0.007701" />
+            </inertial>
+            <visual>
+                <origin rpy="0 0 0" xyz="0.0 0.0 -0.588" />
                 <geometry>
                     <mesh filename="package://lbr_description/meshes/iiwa14/visual/link_3.dae" />
@@ -134,5 +134,5 @@
             </visual>
             <collision>
-                <origin rpy="0 0 0" xyz="0.0 -0.0 -0.588" />
+                <origin rpy="0 0 0" xyz="0.0 0.0 -0.588" />
                 <geometry>
                     <mesh filename="package://lbr_description/meshes/iiwa14/collision/link_3.stl" />
@@ -154,10 +154,10 @@
                 <origin rpy="0 0 0"
                     xyz="-2.09625967727708e-08 -0.04476439079596513 0.06741903952954653" />
-                <mass value="4.12299549" />
-                <inertia ixx="0.022114" ixy="-0.000000" ixz="-0.000000" iyy="0.021074"
-                    iyz="-0.003660" izz="0.007890" />
-            </inertial>
-            <visual>
-                <origin rpy="0 0 0" xyz="-0.0 -0.0105 -0.78" />
+                <mass value="4.122995" />
+                <inertia ixx="0.03241" ixy="0.0" ixz="0.0" iyy="0.030758" iyz="-0.006022"
+                    izz="0.009883" />
+            </inertial>
+            <visual>
+                <origin rpy="0 0 0" xyz="0.0 -0.0105 -0.78" />
                 <geometry>
                     <mesh filename="package://lbr_description/meshes/iiwa14/visual/link_4.dae" />
@@ -165,5 +165,5 @@
             </visual>
             <collision>
-                <origin rpy="0 0 0" xyz="-0.0 -0.0105 -0.78" />
+                <origin rpy="0 0 0" xyz="0.0 -0.0105 -0.78" />
                 <geometry>
                     <mesh filename="package://lbr_description/meshes/iiwa14/collision/link_4.stl" />
@@ -172,5 +172,5 @@
         </link>
         <joint name="A5" type="revolute">
-            <origin rpy="0 0 0" xyz="-0.0 -0.0105 0.2075" />
+            <origin rpy="0 0 0" xyz="0.0 -0.0105 0.2075" />
             <parent link="link_4" />
             <child link="link_5" />
@@ -185,7 +185,7 @@
                 <origin rpy="0 0 0"
                     xyz="-0.00012008657208039079 -0.021390023245727908 0.0854754261653966" />
-                <mass value="1.56375558" />
-                <inertia ixx="0.012955" ixy="0.000002" ixz="-0.000001" iyy="0.011185" iyz="0.003972"
-                    izz="0.005744" />
+                <mass value="1.563756" />
+                <inertia ixx="0.008677" ixy="0.0" ixz="0.0" iyy="0.007297" iyz="0.002869"
+                    izz="0.003935" />
             </inertial>
             <visual>
@@ -216,7 +216,7 @@
                 <origin rpy="0 0 0"
                     xyz="-6.000032555678588e-08 0.07103825551434698 0.000565530522845803" />
-                <mass value="2.4578784" />
-                <inertia ixx="0.006292" ixy="-0.000000" ixz="-0.000000" iyy="0.006023"
-                    iyz="0.000314" izz="0.004585" />
+                <mass value="2.457878" />
+                <inertia ixx="0.007227" ixy="0.0" ixz="0.0" iyy="0.006958" iyz="0.000318"
+                    izz="0.004734" />
             </inertial>
             <visual>
@@ -247,10 +247,9 @@
                 <origin rpy="0 0 0"
                     xyz="3.963019849314055e-06 -1.5392768444664745e-08 0.027186686478491096" />
-                <mass value="0.26533073" />
-                <inertia ixx="0.000281" ixy="-0.000000" ixz="-0.000000" iyy="0.000277"
-                    iyz="0.000000" izz="0.000430" />
-            </inertial>
-            <visual>
-                <origin rpy="0 0 0" xyz="-0.0 0.0 -1.271" />
+                <mass value="0.265331" />
+                <inertia ixx="0.000175" ixy="0.0" ixz="0.0" iyy="0.000175" iyz="0.0" izz="0.000306" />
+            </inertial>
+            <visual>
+                <origin rpy="0 0 0" xyz="0.0 0.0 -1.271" />
                 <geometry>
                     <mesh filename="package://lbr_description/meshes/iiwa14/visual/link_7.dae" />
@@ -258,5 +257,5 @@
             </visual>
             <collision>
-                <origin rpy="0 0 0" xyz="-0.0 0.0 -1.271" />
+                <origin rpy="0 0 0" xyz="0.0 0.0 -1.271" />
                 <geometry>
                     <mesh filename="package://lbr_description/meshes/iiwa14/collision/link_7.stl" />

File: lbr_description/urdf/iiwa7/iiwa7_description.urdf.xacro (robot description, xacro)
@@ -30,7 +30,7 @@
                 <origin rpy="0 0 0"
                     xyz="-0.01283618494463161 4.904567390585061e-08 0.07010682239932087" />
-                <mass value="4.85565842" />
-                <inertia ixx="0.017901" ixy="0.000000" ixz="0.000771" iyy="0.022356" iyz="-0.000000"
-                    izz="0.021346" />
+                <mass value="4.855658" />
+                <inertia ixx="0.017839" ixy="0.0" ixz="0.000781" iyy="0.022294" iyz="0.0"
+                    izz="0.021334" />
             </inertial>
             <visual>
@@ -61,10 +61,10 @@
                 <origin rpy="0 0 0"
                     xyz="4.9980243666546455e-08 -0.0347335291089292 0.12351608478142942" />
-                <mass value="3.39401127" />
-                <inertia ixx="0.021502" ixy="-0.000000" ixz="0.000000" iyy="0.020512" iyz="0.003828"
-                    izz="0.007587" />
-            </inertial>
-            <visual>
-                <origin rpy="0 0 0" xyz="-0.0 0.0 -0.1475" />
+                <mass value="3.394011" />
+                <inertia ixx="0.021383" ixy="0.0" ixz="0.0" iyy="0.020403" iyz="0.003797"
+                    izz="0.007563" />
+            </inertial>
+            <visual>
+                <origin rpy="0 0 0" xyz="0.0 0.0 -0.1475" />
                 <geometry>
                     <mesh filename="package://lbr_description/meshes/iiwa7/visual/link_1.dae" />
@@ -72,5 +72,5 @@
             </visual>
             <collision>
-                <origin rpy="0 0 0" xyz="-0.0 0.0 -0.1475" />
+                <origin rpy="0 0 0" xyz="0.0 0.0 -0.1475" />
                 <geometry>
                     <mesh filename="package://lbr_description/meshes/iiwa7/collision/link_1.stl" />
@@ -79,5 +79,5 @@
         </link>
         <joint name="A2" type="revolute">
-            <origin rpy="0 0 0" xyz="-0.0 -0.0105 0.1925" />
+            <origin rpy="0 0 0" xyz="0.0 -0.0105 0.1925" />
             <parent link="link_1" />
             <child link="link_2" />
@@ -92,7 +92,7 @@
                 <origin rpy="0 0 0"
                     xyz="4.0558428502019873e-08 0.04491581578298656 0.06732515284873997" />
-                <mass value="4.03199094" />
-                <inertia ixx="0.021455" ixy="-0.000000" ixz="0.000000" iyy="0.020444" iyz="0.003570"
-                    izz="0.007671" />
+                <mass value="4.031991" />
+                <inertia ixx="0.031697" ixy="0.0" ixz="0.0" iyy="0.03008" iyz="0.005889"
+                    izz="0.009666" />
             </inertial>
             <visual>
@@ -123,10 +123,10 @@
                 <origin rpy="0 0 0"
                     xyz="-5.881068064938613e-09 0.02956361869175564 0.1365034185434154" />
-                <mass value="3.39401127" />
-                <inertia ixx="0.031559" ixy="-0.000000" ixz="0.000000" iyy="0.029960"
-                    iyz="-0.006133" izz="0.009574" />
-            </inertial>
-            <visual>
-                <origin rpy="0 0 0" xyz="0.0 -0.0 -0.5475" />
+                <mass value="3.394011" />
+                <inertia ixx="0.021383" ixy="0.0" ixz="0.0" iyy="0.020403" iyz="-0.003797"
+                    izz="0.007563" />
+            </inertial>
+            <visual>
+                <origin rpy="0 0 0" xyz="0.0 0.0 -0.5475" />
                 <geometry>
                     <mesh filename="package://lbr_description/meshes/iiwa7/visual/link_3.dae" />
@@ -134,5 +134,5 @@
             </visual>
             <collision>
-                <origin rpy="0 0 0" xyz="0.0 -0.0 -0.5475" />
+                <origin rpy="0 0 0" xyz="0.0 0.0 -0.5475" />
                 <geometry>
                     <mesh filename="package://lbr_description/meshes/iiwa7/collision/link_3.stl" />
@@ -154,10 +154,10 @@
                 <origin rpy="0 0 0"
                     xyz="-4.1344813497116265e-08 -0.044916218629510306 0.06732501840381" />
-                <mass value="4.03198902" />
-                <inertia ixx="0.021454" ixy="0.000000" ixz="-0.000000" iyy="0.020443"
-                    iyz="-0.003570" izz="0.007670" />
-            </inertial>
-            <visual>
-                <origin rpy="0 0 0" xyz="-0.0 -0.0105 -0.74" />
+                <mass value="4.031989" />
+                <inertia ixx="0.031695" ixy="0.0" ixz="0.0" iyy="0.030079" iyz="-0.005889"
+                    izz="0.009665" />
+            </inertial>
+            <visual>
+                <origin rpy="0 0 0" xyz="0.0 -0.0105 -0.74" />
                 <geometry>
                     <mesh filename="package://lbr_description/meshes/iiwa7/visual/link_4.dae" />
@@ -165,5 +165,5 @@
             </visual>
             <collision>
-                <origin rpy="0 0 0" xyz="-0.0 -0.0105 -0.74" />
+                <origin rpy="0 0 0" xyz="0.0 -0.0105 -0.74" />
                 <geometry>
                     <mesh filename="package://lbr_description/meshes/iiwa7/collision/link_4.stl" />
@@ -172,5 +172,5 @@
         </link>
         <joint name="A5" type="revolute">
-            <origin rpy="0 0 0" xyz="-0.0 -0.0105 0.2075" />
+            <origin rpy="0 0 0" xyz="0.0 -0.0105 0.2075" />
             <parent link="link_4" />
             <child link="link_5" />
@@ -185,7 +185,7 @@
                 <origin rpy="0 0 0"
                     xyz="2.416002990197734e-08 -0.021386601078580914 0.085468591256322" />
-                <mass value="1.52923896" />
-                <inertia ixx="0.012684" ixy="-0.000000" ixz="-0.000000" iyy="0.010952"
-                    iyz="0.003889" izz="0.005624" />
+                <mass value="1.529239" />
+                <inertia ixx="0.008485" ixy="0.0" ixz="0.0" iyy="0.007136" iyz="0.002806"
+                    izz="0.003848" />
             </inertial>
             <visual>
@@ -216,7 +216,7 @@
                 <origin rpy="0 0 0"
                     xyz="-9.07120004240837e-08 0.0709871260349443 0.002115721730276743" />
-                <mass value="2.40362602" />
-                <inertia ixx="0.006412" ixy="-0.000000" ixz="-0.000000" iyy="0.006166"
-                    iyz="0.000314" izz="0.004459" />
+                <mass value="2.403626" />
+                <inertia ixx="0.007067" ixy="0.0" ixz="0.0" iyy="0.006804" iyz="0.000311"
+                    izz="0.004629" />
             </inertial>
             <visual>
@@ -247,10 +247,9 @@
                 <origin rpy="0 0 0"
                     xyz="4.535378460217862e-06 -1.7615872956281168e-08 0.009883270430701696" />
-                <mass value="0.25947411" />
-                <inertia ixx="0.000250" ixy="-0.000000" ixz="-0.000000" iyy="0.000245"
-                    iyz="0.000000" izz="0.000406" />
-            </inertial>
-            <visual>
-                <origin rpy="0 0 0" xyz="-0.0 0.0 -1.231" />
+                <mass value="0.259474" />
+                <inertia ixx="0.000171" ixy="0.0" ixz="0.0" iyy="0.000171" iyz="0.0" izz="0.000299" />
+            </inertial>
+            <visual>
+                <origin rpy="0 0 0" xyz="0.0 0.0 -1.231" />
                 <geometry>
                     <mesh filename="package://lbr_description/meshes/iiwa7/visual/link_7.dae" />
@@ -258,5 +257,5 @@
             </visual>
             <collision>
-                <origin rpy="0 0 0" xyz="-0.0 0.0 -1.231" />
+                <origin rpy="0 0 0" xyz="0.0 0.0 -1.231" />
                 <geometry>
                     <mesh filename="package://lbr_description/meshes/iiwa7/collision/link_7.stl" />
