Commit message: updated inertias

File: lbr_description/urdf/med14/med14_description.urdf.xacro (robot description, xacro)
@@ -30,7 +30,7 @@
                 <origin rpy="0 0 0"
                     xyz="-0.0018642104260720833 -9.120393625716289e-09 0.07751683665104403" />
-                <mass value="8.146350" />
-                <inertia ixx="0.044603" ixy="-0.000000" ixz="-0.000788" iyy="0.045465"
-                    iyz="0.000000" izz="0.061903" />
+                <mass value="8.146413" />
+                <inertia ixx="0.044604" ixy="0.0" ixz="-0.000788" iyy="0.045465" iyz="0.0"
+                    izz="0.061904" />
             </inertial>
             <visual>
@@ -61,10 +61,10 @@
                 <origin rpy="0 0 0"
                     xyz="9.307232415315581e-08 -0.033795431550791004 0.13240370669453896" />
-                <mass value="5.591386" />
-                <inertia ixx="0.044885" ixy="-0.000000" ixz="-0.000000" iyy="0.045283"
-                    iyz="0.006703" izz="0.016775" />
-            </inertial>
-            <visual>
-                <origin rpy="0 0 0" xyz="-0.0 -0.0 -0.147" />
+                <mass value="5.591419" />
+                <inertia ixx="0.044885" ixy="0.0" ixz="0.0" iyy="0.045283" iyz="0.006703"
+                    izz="0.016776" />
+            </inertial>
+            <visual>
+                <origin rpy="0 0 0" xyz="0.0 0.0 -0.147" />
                 <geometry>
                     <mesh filename="package://lbr_description/meshes/med14/visual/link_1.dae" />
@@ -72,5 +72,5 @@
             </visual>
             <collision>
-                <origin rpy="0 0 0" xyz="-0.0 -0.0 -0.147" />
+                <origin rpy="0 0 0" xyz="0.0 0.0 -0.147" />
                 <geometry>
                     <mesh filename="package://lbr_description/meshes/med14/collision/link_1.stl" />
@@ -92,10 +92,10 @@
                 <origin rpy="0 0 0"
                     xyz="0.0001358226533474577 0.0475476440926152 0.07632205850106144" />
-                <mass value="6.013539" />
-                <inertia ixx="0.058332" ixy="-0.000035" ixz="0.000059" iyy="0.057063" iyz="0.010606"
+                <mass value="6.013411" />
+                <inertia ixx="0.05833" ixy="-3.5e-05" ixz="5.9e-05" iyy="0.057062" iyz="0.010605"
                     izz="0.017466" />
             </inertial>
             <visual>
-                <origin rpy="0 0 0" xyz="-0.0 0.01 -0.3595" />
+                <origin rpy="0 0 0" xyz="0.0 0.01 -0.3595" />
                 <geometry>
                     <mesh filename="package://lbr_description/meshes/med14/visual/link_2.dae" />
@@ -103,5 +103,5 @@
             </visual>
             <collision>
-                <origin rpy="0 0 0" xyz="-0.0 0.01 -0.3595" />
+                <origin rpy="0 0 0" xyz="0.0 0.01 -0.3595" />
                 <geometry>
                     <mesh filename="package://lbr_description/meshes/med14/collision/link_2.stl" />
@@ -110,5 +110,5 @@
         </link>
         <joint name="A3" type="revolute">
-            <origin rpy="0 0 0" xyz="-0.0 0.01 0.228" />
+            <origin rpy="0 0 0" xyz="0.0 0.01 0.228" />
             <parent link="link_2" />
             <child link="link_3" />
@@ -123,10 +123,10 @@
                 <origin rpy="0 0 0"
                     xyz="5.689213978259012e-08 0.03491265072974692 0.12310820658934007" />
-                <mass value="3.658768" />
-                <inertia ixx="0.022960" ixy="-0.000000" ixz="0.000000" iyy="0.021913"
-                    iyz="-0.004065" izz="0.008140" />
-            </inertial>
-            <visual>
-                <origin rpy="0 0 0" xyz="0.0 -0.0 -0.5875" />
+                <mass value="3.65879" />
+                <inertia ixx="0.02296" ixy="0.0" ixz="0.0" iyy="0.021913" iyz="-0.004065"
+                    izz="0.00814" />
+            </inertial>
+            <visual>
+                <origin rpy="0 0 0" xyz="0.0 0.0 -0.5875" />
                 <geometry>
                     <mesh filename="package://lbr_description/meshes/med14/visual/link_3.dae" />
@@ -134,5 +134,5 @@
             </visual>
             <collision>
-                <origin rpy="0 0 0" xyz="0.0 -0.0 -0.5875" />
+                <origin rpy="0 0 0" xyz="0.0 0.0 -0.5875" />
                 <geometry>
                     <mesh filename="package://lbr_description/meshes/med14/collision/link_3.stl" />
@@ -154,7 +154,7 @@
                 <origin rpy="0 0 0"
                     xyz="-3.025185496951432e-08 -0.03979329512420171 0.08694364647762443" />
-                <mass value="4.358282" />
-                <inertia ixx="0.034259" ixy="-0.000000" ixz="-0.000000" iyy="0.032514"
-                    iyz="-0.006365" izz="0.010447" />
+                <mass value="4.358267" />
+                <inertia ixx="0.034255" ixy="0.0" ixz="0.0" iyy="0.032512" iyz="-0.006365"
+                    izz="0.010444" />
             </inertial>
             <visual>
@@ -185,10 +185,10 @@
                 <origin rpy="0 0 0"
                     xyz="3.8871741664391765e-08 -0.029824284088761824 0.07626701716135809" />
-                <mass value="1.652994" />
-                <inertia ixx="0.009172" ixy="0.000000" ixz="-0.000000" iyy="0.007714" iyz="0.003033"
-                    izz="0.004159" />
-            </inertial>
-            <visual>
-                <origin rpy="0 0 0" xyz="-0.0 0.0 -0.987" />
+                <mass value="1.653015" />
+                <inertia ixx="0.009172" ixy="0.0" ixz="0.0"
+                    iyy="0.007714" iyz="0.003033" izz="0.004159" />
+            </inertial>
+            <visual>
+                <origin rpy="0 0 0" xyz="0.0 0.0 -0.987" />
                 <geometry>
                     <mesh filename="package://lbr_description/meshes/med14/visual/link_5.dae" />
@@ -196,5 +196,5 @@
             </visual>
             <collision>
-                <origin rpy="0 0 0" xyz="-0.0 0.0 -0.987" />
+                <origin rpy="0 0 0" xyz="0.0 0.0 -0.987" />
                 <geometry>
                     <mesh filename="package://lbr_description/meshes/med14/collision/link_5.stl" />
@@ -216,10 +216,10 @@
                 <origin rpy="0 0 0"
                     xyz="-7.073221484902805e-07 0.07101990943401978 0.004952526180380223" />
-                <mass value="2.598208" />
-                <inertia ixx="0.007640" ixy="-0.000000" ixz="0.000000" iyy="0.007355" iyz="0.000336"
+                <mass value="2.598211" />
+                <inertia ixx="0.00764" ixy="0.0" ixz="0.0" iyy="0.007355" iyz="0.000336"
                     izz="0.005004" />
             </inertial>
             <visual>
-                <origin rpy="0 0 0" xyz="-0.0 0.0707 -1.1795" />
+                <origin rpy="0 0 0" xyz="0.0 0.0707 -1.1795" />
                 <geometry>
                     <mesh filename="package://lbr_description/meshes/med14/visual/link_6.dae" />
@@ -227,5 +227,5 @@
             </visual>
             <collision>
-                <origin rpy="0 0 0" xyz="-0.0 0.0707 -1.1795" />
+                <origin rpy="0 0 0" xyz="0.0 0.0707 -1.1795" />
                 <geometry>
                     <mesh filename="package://lbr_description/meshes/med14/collision/link_6.stl" />
@@ -247,10 +247,9 @@
                 <origin rpy="0 0 0"
                     xyz="3.121827460016089e-06 -1.635815563460264e-06 0.0137822955218736" />
-                <mass value="0.280472" />
-                <inertia ixx="0.000185" ixy="0.000000" ixz="-0.000000" iyy="0.000185" iyz="0.000000"
-                    izz="0.000323" />
-            </inertial>
-            <visual>
-                <origin rpy="0 0 0" xyz="-0.0 -0.0 -1.2705" />
+                <mass value="0.280474" />
+                <inertia ixx="0.000185" ixy="0.0" ixz="0.0" iyy="0.000185" iyz="0.0" izz="0.000323" />
+            </inertial>
+            <visual>
+                <origin rpy="0 0 0" xyz="0.0 0.0 -1.2705" />
                 <geometry>
                     <mesh filename="package://lbr_description/meshes/med14/visual/link_7.dae" />
@@ -258,5 +257,5 @@
             </visual>
             <collision>
-                <origin rpy="0 0 0" xyz="-0.0 -0.0 -1.2705" />
+                <origin rpy="0 0 0" xyz="0.0 0.0 -1.2705" />
                 <geometry>
                     <mesh filename="package://lbr_description/meshes/med14/collision/link_7.stl" />

File: lbr_description/urdf/med7/med7_description.urdf.xacro (robot description, xacro)
@@ -30,7 +30,7 @@
                 <origin rpy="0 0 0"
                     xyz="-0.0018958727522859222 -8.736009549202623e-09 0.07626305487275586" />
-                <mass value="7.143078" />
-                <inertia ixx="0.038693" ixy="-0.000000" ixz="-0.000686" iyy="0.039461"
-                    iyz="-0.000000" izz="0.054387" />
+                <mass value="7.143112" />
+                <inertia ixx="0.038694" ixy="0.0" ixz="-0.000686" iyy="0.039461" iyz="0.0"
+                    izz="0.054387" />
             </inertial>
             <visual>
@@ -61,10 +61,10 @@
                 <origin rpy="0 0 0"
                     xyz="5.010328793588479e-08 -0.03481903813472808 0.12329857163085542" />
-                <mass value="3.271492" />
-                <inertia ixx="0.020611" ixy="-0.000000" ixz="0.000000" iyy="0.019667" iyz="0.003660"
-                    izz="0.007290" />
-            </inertial>
-            <visual>
-                <origin rpy="0 0 0" xyz="-0.0 0.0 -0.1475" />
+                <mass value="3.271499" />
+                <inertia ixx="0.020611" ixy="0.0" ixz="0.0" iyy="0.019667" iyz="0.00366"
+                    izz="0.00729" />
+            </inertial>
+            <visual>
+                <origin rpy="0 0 0" xyz="0.0 0.0 -0.1475" />
                 <geometry>
                     <mesh filename="package://lbr_description/meshes/med7/visual/link_1.dae" />
@@ -72,5 +72,5 @@
             </visual>
             <collision>
-                <origin rpy="0 0 0" xyz="-0.0 0.0 -0.1475" />
+                <origin rpy="0 0 0" xyz="0.0 0.0 -0.1475" />
                 <geometry>
                     <mesh filename="package://lbr_description/meshes/med7/collision/link_1.stl" />
@@ -79,5 +79,5 @@
         </link>
         <joint name="A2" type="revolute">
-            <origin rpy="0 0 0" xyz="-0.0 -0.0105 0.1925" />
+            <origin rpy="0 0 0" xyz="0.0 -0.0105 0.1925" />
             <parent link="link_1" />
             <child link="link_2" />
@@ -92,6 +92,6 @@
                 <origin rpy="0 0 0"
                     xyz="2.958275959973659e-08 0.03979295468456965 0.08694361150855662" />
-                <mass value="3.886440" />
-                <inertia ixx="0.030552" ixy="-0.000000" ixz="0.000000" iyy="0.028995" iyz="0.005676"
+                <mass value="3.886413" />
+                <inertia ixx="0.030552" ixy="0.0" ixz="0.0" iyy="0.028995" iyz="0.005676"
                     izz="0.009317" />
             </inertial>
@@ -123,10 +123,10 @@
                 <origin rpy="0 0 0"
                     xyz="-5.010330962930412e-08 0.03481903813473644 0.1232985716309013" />
-                <mass value="3.271492" />
-                <inertia ixx="0.020611" ixy="-0.000000" ixz="-0.000000" iyy="0.019667"
-                    iyz="-0.003660" izz="0.007290" />
-            </inertial>
-            <visual>
-                <origin rpy="0 0 0" xyz="0.0 -0.0 -0.5475" />
+                <mass value="3.271499" />
+                <inertia ixx="0.020611" ixy="0.0" ixz="0.0" iyy="0.019667" iyz="-0.00366"
+                    izz="0.00729" />
+            </inertial>
+            <visual>
+                <origin rpy="0 0 0" xyz="0.0 0.0 -0.5475" />
                 <geometry>
                     <mesh filename="package://lbr_description/meshes/med7/visual/link_3.dae" />
@@ -134,5 +134,5 @@
             </visual>
             <collision>
-                <origin rpy="0 0 0" xyz="0.0 -0.0 -0.5475" />
+                <origin rpy="0 0 0" xyz="0.0 0.0 -0.5475" />
                 <geometry>
                     <mesh filename="package://lbr_description/meshes/med7/collision/link_3.stl" />
@@ -154,10 +154,10 @@
                 <origin rpy="0 0 0"
                     xyz="-3.025230048709993e-08 -0.03979329512443697 0.08694363375610437" />
-                <mass value="3.886439" />
-                <inertia ixx="0.030551" ixy="-0.000000" ixz="-0.000000" iyy="0.028993"
-                    iyz="-0.005676" izz="0.009316" />
-            </inertial>
-            <visual>
-                <origin rpy="0 0 0" xyz="-0.0 -0.0105 -0.74" />
+                <mass value="3.886411" />
+                <inertia ixx="0.030547" ixy="0.0" ixz="0.0" iyy="0.028993" iyz="-0.005676"
+                    izz="0.009313" />
+            </inertial>
+            <visual>
+                <origin rpy="0 0 0" xyz="0.0 -0.0105 -0.74" />
                 <geometry>
                     <mesh filename="package://lbr_description/meshes/med7/visual/link_4.dae" />
@@ -165,5 +165,5 @@
             </visual>
             <collision>
-                <origin rpy="0 0 0" xyz="-0.0 -0.0105 -0.74" />
+                <origin rpy="0 0 0" xyz="0.0 -0.0105 -0.74" />
                 <geometry>
                     <mesh filename="package://lbr_description/meshes/med7/collision/link_4.stl" />
@@ -172,5 +172,5 @@
         </link>
         <joint name="A5" type="revolute">
-            <origin rpy="0 0 0" xyz="-0.0 -0.0105 0.2075" />
+            <origin rpy="0 0 0" xyz="0.0 -0.0105 0.2075" />
             <parent link="link_4" />
             <child link="link_5" />
@@ -185,6 +185,6 @@
                 <origin rpy="0 0 0"
                     xyz="3.887174133882675e-08 -0.02982428408876193 0.07626701716135398" />
-                <mass value="1.474035" />
-                <inertia ixx="0.008179" ixy="0.000000" ixz="-0.000000" iyy="0.006879" iyz="0.002704"
+                <mass value="1.474048" />
+                <inertia ixx="0.008179" ixy="0.0" ixz="0.0" iyy="0.006879" iyz="0.002704"
                     izz="0.003709" />
             </inertial>
@@ -216,6 +216,6 @@
                 <origin rpy="0 0 0"
                     xyz="-7.073221144775636e-07 0.07101990943401648 0.004952526180360017" />
-                <mass value="2.316917" />
-                <inertia ixx="0.006813" ixy="-0.000000" ixz="0.000000" iyy="0.006559" iyz="0.000300"
+                <mass value="2.316911" />
+                <inertia ixx="0.006813" ixy="0.0" ixz="0.0" iyy="0.006559" iyz="0.0003"
                     izz="0.004462" />
             </inertial>
@@ -247,10 +247,9 @@
                 <origin rpy="0 0 0"
                     xyz="3.1218274599808524e-06 -1.6358155634513969e-06 0.013782295521067356" />
-                <mass value="0.250107" />
-                <inertia ixx="0.000165" ixy="0.000000" ixz="-0.000000" iyy="0.000165" iyz="0.000000"
-                    izz="0.000288" />
-            </inertial>
-            <visual>
-                <origin rpy="0 0 0" xyz="-0.0 -0.0 -1.231" />
+                <mass value="0.250108" />
+                <inertia ixx="0.000165" ixy="0.0" ixz="0.0" iyy="0.000165" iyz="0.0" izz="0.000288" />
+            </inertial>
+            <visual>
+                <origin rpy="0 0 0" xyz="0.0 0.0 -1.231" />
                 <geometry>
                     <mesh filename="package://lbr_description/meshes/med7/visual/link_7.dae" />
@@ -258,5 +257,5 @@
             </visual>
             <collision>
-                <origin rpy="0 0 0" xyz="-0.0 -0.0 -1.231" />
+                <origin rpy="0 0 0" xyz="0.0 0.0 -1.231" />
                 <geometry>
                     <mesh filename="package://lbr_description/meshes/med7/collision/link_7.stl" />
