Commit message: updated origins

File: lbr_description/urdf/iiwa14/iiwa14_description.urdf.xacro (robot description, xacro)
@@ -28,6 +28,5 @@
         <link name="link_0">
             <inertial>
-                <origin rpy="0 0 0"
-                    xyz="-0.0128215344957798 -7.86364415362405e-08 0.07150661827888387" />
+                <origin rpy="0 0 0" xyz="-0.012822 0.0 0.071507" />
                 <mass value="7.050378" />
                 <inertia ixx="0.031226" ixy="0.0" ixz="0.000871" iyy="0.039697" iyz="0.0"
@@ -59,6 +58,5 @@
         <link name="link_1">
             <inertial>
-                <origin rpy="0 0 0"
-                    xyz="9.307232415315581e-08 -0.03379543155079102 0.13240370669453902" />
+                <origin rpy="0 0 0" xyz="0.0 -0.033795 0.132404" />
                 <mass value="5.289529" />
                 <inertia ixx="0.042462" ixy="0.0" ixz="0.0" iyy="0.042838" iyz="0.006341"
@@ -90,6 +88,5 @@
         <link name="link_2">
             <inertial>
-                <origin rpy="0 0 0"
-                    xyz="0.00015188022518878674 0.051987109728758904 0.05880129877994178" />
+                <origin rpy="0 0 0" xyz="0.000136 0.047548 0.076322" />
                 <mass value="5.688888" />
                 <inertia ixx="0.055182" ixy="-3.3e-05" ixz="5.6e-05" iyy="0.053983" iyz="0.010034"
@@ -121,6 +118,5 @@
         <link name="link_3">
             <inertial>
-                <origin rpy="0 0 0"
-                    xyz="-5.974614313346012e-09 0.029563618732667742 0.13650341869763982" />
+                <origin rpy="0 0 0" xyz="0.0 0.034913 0.123108" />
                 <mass value="3.461245" />
                 <inertia ixx="0.02172" ixy="0.0" ixz="0.0" iyy="0.02073" iyz="-0.003845"
@@ -152,6 +148,5 @@
         <link name="link_4">
             <inertial>
-                <origin rpy="0 0 0"
-                    xyz="-2.09625967727708e-08 -0.04476439079596513 0.06741903952954653" />
+                <origin rpy="0 0 0" xyz="0.0 -0.039793 0.086944" />
                 <mass value="4.122995" />
                 <inertia ixx="0.03241" ixy="0.0" ixz="0.0" iyy="0.030758" iyz="-0.006022"
@@ -183,6 +178,5 @@
         <link name="link_5">
             <inertial>
-                <origin rpy="0 0 0"
-                    xyz="-0.00012008657208039079 -0.021390023245727908 0.0854754261653966" />
+                <origin rpy="0 0 0" xyz="0.0 -0.029824 0.076267" />
                 <mass value="1.563756" />
                 <inertia ixx="0.008677" ixy="0.0" ixz="0.0" iyy="0.007297" iyz="0.002869"
@@ -214,6 +208,5 @@
         <link name="link_6">
             <inertial>
-                <origin rpy="0 0 0"
-                    xyz="-6.000032555678588e-08 0.07103825551434698 0.000565530522845803" />
+                <origin rpy="0 0 0" xyz="0.0 0.07102 0.00495" />
                 <mass value="2.457878" />
                 <inertia ixx="0.007227" ixy="0.0" ixz="0.0" iyy="0.006958" iyz="0.000318"
@@ -245,6 +238,5 @@
         <link name="link_7">
             <inertial>
-                <origin rpy="0 0 0"
-                    xyz="3.963019849314055e-06 -1.5392768444664745e-08 0.027186686478491096" />
+                <origin rpy="0 0 0" xyz="3.0000e-06 -2.0000e-06 1.3782e-02" />
                 <mass value="0.265331" />
                 <inertia ixx="0.000175" ixy="0.0" ixz="0.0" iyy="0.000175" iyz="0.0" izz="0.000306" />

File: lbr_description/urdf/iiwa7/iiwa7_description.urdf.xacro (robot description, xacro)
@@ -28,6 +28,5 @@
         <link name="link_0">
             <inertial>
-                <origin rpy="0 0 0"
-                    xyz="-0.01283618494463161 4.904567390585061e-08 0.07010682239932087" />
+                <origin rpy="0 0 0" xyz="-0.012857 0.0 0.069964" />
                 <mass value="4.855658" />
                 <inertia ixx="0.017839" ixy="0.0" ixz="0.000781" iyy="0.022294" iyz="0.0"
@@ -59,6 +58,5 @@
         <link name="link_1">
             <inertial>
-                <origin rpy="0 0 0"
-                    xyz="4.9980243666546455e-08 -0.0347335291089292 0.12351608478142942" />
+                <origin rpy="0 0 0" xyz="0.0 -0.034819 0.123299" />
                 <mass value="3.394011" />
                 <inertia ixx="0.021383" ixy="0.0" ixz="0.0" iyy="0.020403" iyz="0.003797"
@@ -90,6 +88,5 @@
         <link name="link_2">
             <inertial>
-                <origin rpy="0 0 0"
-                    xyz="4.0558428502019873e-08 0.04491581578298656 0.06732515284873997" />
+                <origin rpy="0 0 0" xyz="0.0 0.039793 0.086944" />
                 <mass value="4.031991" />
                 <inertia ixx="0.031697" ixy="0.0" ixz="0.0" iyy="0.03008" iyz="0.005889"
@@ -121,6 +118,5 @@
         <link name="link_3">
             <inertial>
-                <origin rpy="0 0 0"
-                    xyz="-5.881068064938613e-09 0.02956361869175564 0.1365034185434154" />
+                <origin rpy="0 0 0" xyz="0.0 0.034819 0.123299" />
                 <mass value="3.394011" />
                 <inertia ixx="0.021383" ixy="0.0" ixz="0.0" iyy="0.020403" iyz="-0.003797"
@@ -152,6 +148,5 @@
         <link name="link_4">
             <inertial>
-                <origin rpy="0 0 0"
-                    xyz="-4.1344813497116265e-08 -0.044916218629510306 0.06732501840381" />
+                <origin rpy="0 0 0" xyz="0.0 -0.039793 0.086944" />
                 <mass value="4.031989" />
                 <inertia ixx="0.031695" ixy="0.0" ixz="0.0" iyy="0.030079" iyz="-0.005889"
@@ -183,6 +178,5 @@
         <link name="link_5">
             <inertial>
-                <origin rpy="0 0 0"
-                    xyz="2.416002990197734e-08 -0.021386601078580914 0.085468591256322" />
+                <origin rpy="0 0 0" xyz="0.0 -0.029824 0.076267" />
                 <mass value="1.529239" />
                 <inertia ixx="0.008485" ixy="0.0" ixz="0.0" iyy="0.007136" iyz="0.002806"
@@ -214,6 +208,5 @@
         <link name="link_6">
             <inertial>
-                <origin rpy="0 0 0"
-                    xyz="-9.07120004240837e-08 0.0709871260349443 0.002115721730276743" />
+                <origin rpy="0 0 0" xyz="0.0 0.07102 0.00495" />
                 <mass value="2.403626" />
                 <inertia ixx="0.007067" ixy="0.0" ixz="0.0" iyy="0.006804" iyz="0.000311"
@@ -245,6 +238,5 @@
         <link name="link_7">
             <inertial>
-                <origin rpy="0 0 0"
-                    xyz="4.535378460217862e-06 -1.7615872956281168e-08 0.009883270430701696" />
+                <origin rpy="0 0 0" xyz="3.0000e-06 -2.0000e-06 1.3782e-02" />
                 <mass value="0.259474" />
                 <inertia ixx="0.000171" ixy="0.0" ixz="0.0" iyy="0.000171" iyz="0.0" izz="0.000299" />

File: lbr_description/urdf/med14/med14_description.urdf.xacro (robot description, xacro)
@@ -28,6 +28,5 @@
         <link name="link_0">
             <inertial>
-                <origin rpy="0 0 0"
-                    xyz="-0.0018642104260720833 -9.120393625716289e-09 0.07751683665104403" />
+                <origin rpy="0 0 0" xyz="-0.001864 0.0 0.077517" />
                 <mass value="8.146413" />
                 <inertia ixx="0.044604" ixy="0.0" ixz="-0.000788" iyy="0.045465" iyz="0.0"
@@ -59,6 +58,5 @@
         <link name="link_1">
             <inertial>
-                <origin rpy="0 0 0"
-                    xyz="9.307232415315581e-08 -0.033795431550791004 0.13240370669453896" />
+                <origin rpy="0 0 0" xyz="0.0 -0.033795  0.132404" />
                 <mass value="5.591419" />
                 <inertia ixx="0.044885" ixy="0.0" ixz="0.0" iyy="0.045283" iyz="0.006703"
@@ -90,6 +88,5 @@
         <link name="link_2">
             <inertial>
-                <origin rpy="0 0 0"
-                    xyz="0.0001358226533474577 0.0475476440926152 0.07632205850106144" />
+                <origin rpy="0 0 0" xyz="0.000136 0.047546 0.076324" />
                 <mass value="6.013411" />
                 <inertia ixx="0.05833" ixy="-3.5e-05" ixz="5.9e-05" iyy="0.057062" iyz="0.010605"
@@ -121,6 +118,5 @@
         <link name="link_3">
             <inertial>
-                <origin rpy="0 0 0"
-                    xyz="5.689213978259012e-08 0.03491265072974692 0.12310820658934007" />
+                <origin rpy="0 0 0" xyz="0.0 0.034913 0.123108" />
                 <mass value="3.65879" />
                 <inertia ixx="0.02296" ixy="0.0" ixz="0.0" iyy="0.021913" iyz="-0.004065"
@@ -152,6 +148,5 @@
         <link name="link_4">
             <inertial>
-                <origin rpy="0 0 0"
-                    xyz="-3.025185496951432e-08 -0.03979329512420171 0.08694364647762443" />
+                <origin rpy="0 0 0" xyz="0.0 -0.039793  0.086944" />
                 <mass value="4.358267" />
                 <inertia ixx="0.034255" ixy="0.0" ixz="0.0" iyy="0.032512" iyz="-0.006365"
@@ -183,6 +178,5 @@
         <link name="link_5">
             <inertial>
-                <origin rpy="0 0 0"
-                    xyz="3.8871741664391765e-08 -0.029824284088761824 0.07626701716135809" />
+                <origin rpy="0 0 0" xyz="0.0 -0.029824  0.076267" />
                 <mass value="1.653015" />
                 <inertia ixx="0.009172" ixy="0.0" ixz="0.0"
@@ -214,6 +208,5 @@
         <link name="link_6">
             <inertial>
-                <origin rpy="0 0 0"
-                    xyz="-7.073221484902805e-07 0.07101990943401978 0.004952526180380223" />
+                <origin rpy="0 0 0" xyz="-1.000e-06 7.102e-02 4.953e-03" />
                 <mass value="2.598211" />
                 <inertia ixx="0.00764" ixy="0.0" ixz="0.0" iyy="0.007355" iyz="0.000336"
@@ -245,6 +238,5 @@
         <link name="link_7">
             <inertial>
-                <origin rpy="0 0 0"
-                    xyz="3.121827460016089e-06 -1.635815563460264e-06 0.0137822955218736" />
+                <origin rpy="0 0 0" xyz="3.0000e-06 -2.0000e-06 1.3782e-02" />
                 <mass value="0.280474" />
                 <inertia ixx="0.000185" ixy="0.0" ixz="0.0" iyy="0.000185" iyz="0.0" izz="0.000323" />

File: lbr_description/urdf/med7/med7_description.urdf.xacro (robot description, xacro)
@@ -28,6 +28,5 @@
         <link name="link_0">
             <inertial>
-                <origin rpy="0 0 0"
-                    xyz="-0.0018958727522859222 -8.736009549202623e-09 0.07626305487275586" />
+                <origin rpy="0 0 0" xyz="-0.001896 0.0 0.076263" />
                 <mass value="7.143112" />
                 <inertia ixx="0.038694" ixy="0.0" ixz="-0.000686" iyy="0.039461" iyz="0.0"
@@ -59,6 +58,5 @@
         <link name="link_1">
             <inertial>
-                <origin rpy="0 0 0"
-                    xyz="5.010328793588479e-08 -0.03481903813472808 0.12329857163085542" />
+                <origin rpy="0 0 0" xyz="0.0 -0.034819  0.123299" />
                 <mass value="3.271499" />
                 <inertia ixx="0.020611" ixy="0.0" ixz="0.0" iyy="0.019667" iyz="0.00366"
@@ -90,6 +88,5 @@
         <link name="link_2">
             <inertial>
-                <origin rpy="0 0 0"
-                    xyz="2.958275959973659e-08 0.03979295468456965 0.08694361150855662" />
+                <origin rpy="0 0 0" xyz="0.0 0.039793 0.086944" />
                 <mass value="3.886413" />
                 <inertia ixx="0.030552" ixy="0.0" ixz="0.0" iyy="0.028995" iyz="0.005676"
@@ -121,6 +118,5 @@
         <link name="link_3">
             <inertial>
-                <origin rpy="0 0 0"
-                    xyz="-5.010330962930412e-08 0.03481903813473644 0.1232985716309013" />
+                <origin rpy="0 0 0" xyz="0.0 0.034819  0.123299" />
                 <mass value="3.271499" />
                 <inertia ixx="0.020611" ixy="0.0" ixz="0.0" iyy="0.019667" iyz="-0.00366"
@@ -152,6 +148,5 @@
         <link name="link_4">
             <inertial>
-                <origin rpy="0 0 0"
-                    xyz="-3.025230048709993e-08 -0.03979329512443697 0.08694363375610437" />
+                <origin rpy="0 0 0" xyz="0.0 -0.039793  0.086944" />
                 <mass value="3.886411" />
                 <inertia ixx="0.030547" ixy="0.0" ixz="0.0" iyy="0.028993" iyz="-0.005676"
@@ -183,6 +178,5 @@
         <link name="link_5">
             <inertial>
-                <origin rpy="0 0 0"
-                    xyz="3.887174133882675e-08 -0.02982428408876193 0.07626701716135398" />
+                <origin rpy="0 0 0" xyz="0.0 -0.029824 0.076267" />
                 <mass value="1.474048" />
                 <inertia ixx="0.008179" ixy="0.0" ixz="0.0" iyy="0.006879" iyz="0.002704"
@@ -214,6 +208,5 @@
         <link name="link_6">
             <inertial>
-                <origin rpy="0 0 0"
-                    xyz="-7.073221144775636e-07 0.07101990943401648 0.004952526180360017" />
+                <origin rpy="0 0 0" xyz="-1.000e-06 7.102e-02 4.953e-03" />
                 <mass value="2.316911" />
                 <inertia ixx="0.006813" ixy="0.0" ixz="0.0" iyy="0.006559" iyz="0.0003"
@@ -245,6 +238,5 @@
         <link name="link_7">
             <inertial>
-                <origin rpy="0 0 0"
-                    xyz="3.1218274599808524e-06 -1.6358155634513969e-06 0.013782295521067356" />
+                <origin rpy="0 0 0" xyz="3.0000e-06 -2.0000e-06 1.3782e-02" />
                 <mass value="0.250108" />
                 <inertia ixx="0.000165" ixy="0.0" ixz="0.0" iyy="0.000165" iyz="0.0" izz="0.000288" />
