Commit message: re-named velocity limits

File: lbr_description/urdf/iiwa14/iiwa14_description.urdf.xacro (robot description, xacro)
@@ -12,11 +12,11 @@
     <xacro:property name="A6_position_limit" value="120" />
     <xacro:property name="A7_position_limit" value="175" />
-    <xacro:property name="joint_0_velocity_limit" value="85" />
-    <xacro:property name="joint_1_velocity_limit" value="85" />
-    <xacro:property name="joint_2_velocity_limit" value="100" />
-    <xacro:property name="joint_3_velocity_limit" value="75" />
-    <xacro:property name="joint_4_velocity_limit" value="130" />
-    <xacro:property name="joint_5_velocity_limit" value="135" />
-    <xacro:property name="joint_6_velocity_limit" value="135" />
+    <xacro:property name="A1_velocity_limit" value="85" />
+    <xacro:property name="A2_velocity_limit" value="85" />
+    <xacro:property name="A3_velocity_limit" value="100" />
+    <xacro:property name="A4_velocity_limit" value="75" />
+    <xacro:property name="A5_velocity_limit" value="130" />
+    <xacro:property name="A6_velocity_limit" value="135" />
+    <xacro:property name="A7_velocity_limit" value="135" />
     <xacro:property name="effort_limit" value="200" />
     <!-- includes -->
@@ -53,5 +53,5 @@
             <limit effort="${effort_limit}" lower="${-A1_position_limit * PI / 180}"
                 upper="${A1_position_limit * PI / 180}"
-                velocity="${joint_0_velocity_limit * PI / 180}" />
+                velocity="${A1_velocity_limit * PI / 180}" />
             <dynamics damping="${joint_damping}" friction="${joint_friction}" />
         </joint>
@@ -83,5 +83,5 @@
             <limit effort="${effort_limit}" lower="${-A2_position_limit * PI / 180}"
                 upper="${A2_position_limit * PI / 180}"
-                velocity="${joint_1_velocity_limit * PI / 180}" />
+                velocity="${A2_velocity_limit * PI / 180}" />
             <dynamics damping="${joint_damping}" friction="${joint_friction}" />
         </joint>
@@ -113,5 +113,5 @@
             <limit effort="${effort_limit}" lower="${-A3_position_limit * PI / 180}"
                 upper="${A3_position_limit * PI / 180}"
-                velocity="${joint_2_velocity_limit * PI / 180}" />
+                velocity="${A3_velocity_limit * PI / 180}" />
             <dynamics damping="${joint_damping}" friction="${joint_friction}" />
         </joint>
@@ -143,5 +143,5 @@
             <limit effort="${effort_limit}" lower="${-A4_position_limit * PI / 180}"
                 upper="${A4_position_limit * PI / 180}"
-                velocity="${joint_3_velocity_limit * PI / 180}" />
+                velocity="${A4_velocity_limit * PI / 180}" />
             <dynamics damping="${joint_damping}" friction="${joint_friction}" />
         </joint>
@@ -173,5 +173,5 @@
             <limit effort="${effort_limit}" lower="${-A5_position_limit * PI / 180}"
                 upper="${A5_position_limit * PI / 180}"
-                velocity="${joint_4_velocity_limit * PI / 180}" />
+                velocity="${A5_velocity_limit * PI / 180}" />
             <dynamics damping="${joint_damping}" friction="${joint_friction}" />
         </joint>
@@ -203,5 +203,5 @@
             <limit effort="${effort_limit}" lower="${-A6_position_limit * PI / 180}"
                 upper="${A6_position_limit * PI / 180}"
-                velocity="${joint_5_velocity_limit * PI / 180}" />
+                velocity="${A6_velocity_limit * PI / 180}" />
             <dynamics damping="${joint_damping}" friction="${joint_friction}" />
         </joint>
@@ -233,5 +233,5 @@
             <limit effort="${effort_limit}" lower="${-A7_position_limit * PI / 180}"
                 upper="${A7_position_limit * PI / 180}"
-                velocity="${joint_6_velocity_limit * PI / 180}" />
+                velocity="${A7_velocity_limit * PI / 180}" />
             <dynamics damping="${joint_damping}" friction="${joint_friction}" />
         </joint>

File: lbr_description/urdf/iiwa7/iiwa7_description.urdf.xacro (robot description, xacro)
@@ -12,11 +12,11 @@
     <xacro:property name="A6_position_limit" value="120" />
     <xacro:property name="A7_position_limit" value="175" />
-    <xacro:property name="joint_0_velocity_limit" value="98" />
-    <xacro:property name="joint_1_velocity_limit" value="98" />
-    <xacro:property name="joint_2_velocity_limit" value="100" />
-    <xacro:property name="joint_3_velocity_limit" value="130" />
-    <xacro:property name="joint_4_velocity_limit" value="140" />
-    <xacro:property name="joint_5_velocity_limit" value="180" />
-    <xacro:property name="joint_6_velocity_limit" value="180" />
+    <xacro:property name="A1_velocity_limit" value="98" />
+    <xacro:property name="A2_velocity_limit" value="98" />
+    <xacro:property name="A3_velocity_limit" value="100" />
+    <xacro:property name="A4_velocity_limit" value="130" />
+    <xacro:property name="A5_velocity_limit" value="140" />
+    <xacro:property name="A6_velocity_limit" value="180" />
+    <xacro:property name="A7_velocity_limit" value="180" />
     <xacro:property name="effort_limit" value="200" />
     <!-- includes -->
@@ -53,5 +53,5 @@
             <limit effort="${effort_limit}" lower="${-A1_position_limit * PI / 180}"
                 upper="${A1_position_limit * PI / 180}"
-                velocity="${joint_0_velocity_limit * PI / 180}" />
+                velocity="${A1_velocity_limit * PI / 180}" />
             <dynamics damping="${joint_damping}" friction="${joint_friction}" />
         </joint>
@@ -83,5 +83,5 @@
             <limit effort="${effort_limit}" lower="${-A2_position_limit * PI / 180}"
                 upper="${A2_position_limit * PI / 180}"
-                velocity="${joint_1_velocity_limit * PI / 180}" />
+                velocity="${A2_velocity_limit * PI / 180}" />
             <dynamics damping="${joint_damping}" friction="${joint_friction}" />
         </joint>
@@ -113,5 +113,5 @@
             <limit effort="${effort_limit}" lower="${-A3_position_limit * PI / 180}"
                 upper="${A3_position_limit * PI / 180}"
-                velocity="${joint_2_velocity_limit * PI / 180}" />
+                velocity="${A3_velocity_limit * PI / 180}" />
             <dynamics damping="${joint_damping}" friction="${joint_friction}" />
         </joint>
@@ -143,5 +143,5 @@
             <limit effort="${effort_limit}" lower="${-A4_position_limit * PI / 180}"
                 upper="${A4_position_limit * PI / 180}"
-                velocity="${joint_3_velocity_limit * PI / 180}" />
+                velocity="${A4_velocity_limit * PI / 180}" />
             <dynamics damping="${joint_damping}" friction="${joint_friction}" />
         </joint>
@@ -173,5 +173,5 @@
             <limit effort="${effort_limit}" lower="${-A5_position_limit * PI / 180}"
                 upper="${A5_position_limit * PI / 180}"
-                velocity="${joint_4_velocity_limit * PI / 180}" />
+                velocity="${A5_velocity_limit * PI / 180}" />
             <dynamics damping="${joint_damping}" friction="${joint_friction}" />
         </joint>
@@ -203,5 +203,5 @@
             <limit effort="${effort_limit}" lower="${-A6_position_limit * PI / 180}"
                 upper="${A6_position_limit * PI / 180}"
-                velocity="${joint_5_velocity_limit * PI / 180}" />
+                velocity="${A6_velocity_limit * PI / 180}" />
             <dynamics damping="${joint_damping}" friction="${joint_friction}" />
         </joint>
@@ -233,5 +233,5 @@
             <limit effort="${effort_limit}" lower="${-A7_position_limit * PI / 180}"
                 upper="${A7_position_limit * PI / 180}"
-                velocity="${joint_6_velocity_limit * PI / 180}" />
+                velocity="${A7_velocity_limit * PI / 180}" />
             <dynamics damping="${joint_damping}" friction="${joint_friction}" />
         </joint>

File: lbr_description/urdf/med14/med14_description.urdf.xacro (robot description, xacro)
@@ -12,11 +12,11 @@
     <xacro:property name="A6_position_limit" value="120" />
     <xacro:property name="A7_position_limit" value="175" />
-    <xacro:property name="joint_0_velocity_limit" value="85" />
-    <xacro:property name="joint_1_velocity_limit" value="85" />
-    <xacro:property name="joint_2_velocity_limit" value="100" />
-    <xacro:property name="joint_3_velocity_limit" value="75" />
-    <xacro:property name="joint_4_velocity_limit" value="130" />
-    <xacro:property name="joint_5_velocity_limit" value="135" />
-    <xacro:property name="joint_6_velocity_limit" value="135" />
+    <xacro:property name="A1_velocity_limit" value="85" />
+    <xacro:property name="A2_velocity_limit" value="85" />
+    <xacro:property name="A3_velocity_limit" value="100" />
+    <xacro:property name="A4_velocity_limit" value="75" />
+    <xacro:property name="A5_velocity_limit" value="130" />
+    <xacro:property name="A6_velocity_limit" value="135" />
+    <xacro:property name="A7_velocity_limit" value="135" />
     <xacro:property name="effort_limit" value="200" />
     <!-- includes -->
@@ -53,5 +53,5 @@
             <limit effort="${effort_limit}" lower="${-A1_position_limit * PI / 180}"
                 upper="${A1_position_limit * PI / 180}"
-                velocity="${joint_0_velocity_limit * PI / 180}" />
+                velocity="${A1_velocity_limit * PI / 180}" />
             <dynamics damping="${joint_damping}" friction="${joint_friction}" />
         </joint>
@@ -83,5 +83,5 @@
             <limit effort="${effort_limit}" lower="${-A2_position_limit * PI / 180}"
                 upper="${A2_position_limit * PI / 180}"
-                velocity="${joint_1_velocity_limit * PI / 180}" />
+                velocity="${A2_velocity_limit * PI / 180}" />
             <dynamics damping="${joint_damping}" friction="${joint_friction}" />
         </joint>
@@ -113,5 +113,5 @@
             <limit effort="${effort_limit}" lower="${-A3_position_limit * PI / 180}"
                 upper="${A3_position_limit * PI / 180}"
-                velocity="${joint_2_velocity_limit * PI / 180}" />
+                velocity="${A3_velocity_limit * PI / 180}" />
             <dynamics damping="${joint_damping}" friction="${joint_friction}" />
         </joint>
@@ -143,5 +143,5 @@
             <limit effort="${effort_limit}" lower="${-A4_position_limit * PI / 180}"
                 upper="${A4_position_limit * PI / 180}"
-                velocity="${joint_3_velocity_limit * PI / 180}" />
+                velocity="${A4_velocity_limit * PI / 180}" />
             <dynamics damping="${joint_damping}" friction="${joint_friction}" />
         </joint>
@@ -173,5 +173,5 @@
             <limit effort="${effort_limit}" lower="${-A5_position_limit * PI / 180}"
                 upper="${A5_position_limit * PI / 180}"
-                velocity="${joint_4_velocity_limit * PI / 180}" />
+                velocity="${A5_velocity_limit * PI / 180}" />
             <dynamics damping="${joint_damping}" friction="${joint_friction}" />
         </joint>
@@ -203,5 +203,5 @@
             <limit effort="${effort_limit}" lower="${-A6_position_limit * PI / 180}"
                 upper="${A6_position_limit * PI / 180}"
-                velocity="${joint_5_velocity_limit * PI / 180}" />
+                velocity="${A6_velocity_limit * PI / 180}" />
             <dynamics damping="${joint_damping}" friction="${joint_friction}" />
         </joint>
@@ -233,5 +233,5 @@
             <limit effort="${effort_limit}" lower="${-A7_position_limit * PI / 180}"
                 upper="${A7_position_limit * PI / 180}"
-                velocity="${joint_6_velocity_limit * PI / 180}" />
+                velocity="${A7_velocity_limit * PI / 180}" />
             <dynamics damping="${joint_damping}" friction="${joint_friction}" />
         </joint>

File: lbr_description/urdf/med7/med7_description.urdf.xacro (robot description, xacro)
@@ -12,11 +12,11 @@
     <xacro:property name="A6_position_limit" value="120" />
     <xacro:property name="A7_position_limit" value="175" />
-    <xacro:property name="joint_0_velocity_limit" value="98" />
-    <xacro:property name="joint_1_velocity_limit" value="98" />
-    <xacro:property name="joint_2_velocity_limit" value="100" />
-    <xacro:property name="joint_3_velocity_limit" value="130" />
-    <xacro:property name="joint_4_velocity_limit" value="140" />
-    <xacro:property name="joint_5_velocity_limit" value="180" />
-    <xacro:property name="joint_6_velocity_limit" value="180" />
+    <xacro:property name="A1_velocity_limit" value="98" />
+    <xacro:property name="A2_velocity_limit" value="98" />
+    <xacro:property name="A3_velocity_limit" value="100" />
+    <xacro:property name="A4_velocity_limit" value="130" />
+    <xacro:property name="A5_velocity_limit" value="140" />
+    <xacro:property name="A6_velocity_limit" value="180" />
+    <xacro:property name="A7_velocity_limit" value="180" />
     <xacro:property name="effort_limit" value="200" />
     <!-- includes -->
@@ -53,5 +53,5 @@
             <limit effort="${effort_limit}" lower="${-A1_position_limit * PI / 180}"
                 upper="${A1_position_limit * PI / 180}"
-                velocity="${joint_0_velocity_limit * PI / 180}" />
+                velocity="${A1_velocity_limit * PI / 180}" />
             <dynamics damping="${joint_damping}" friction="${joint_friction}" />
         </joint>
@@ -83,5 +83,5 @@
             <limit effort="${effort_limit}" lower="${-A2_position_limit * PI / 180}"
                 upper="${A2_position_limit * PI / 180}"
-                velocity="${joint_1_velocity_limit * PI / 180}" />
+                velocity="${A2_velocity_limit * PI / 180}" />
             <dynamics damping="${joint_damping}" friction="${joint_friction}" />
         </joint>
@@ -113,5 +113,5 @@
             <limit effort="${effort_limit}" lower="${-A3_position_limit * PI / 180}"
                 upper="${A3_position_limit * PI / 180}"
-                velocity="${joint_2_velocity_limit * PI / 180}" />
+                velocity="${A3_velocity_limit * PI / 180}" />
             <dynamics damping="${joint_damping}" friction="${joint_friction}" />
         </joint>
@@ -143,5 +143,5 @@
             <limit effort="${effort_limit}" lower="${-A4_position_limit * PI / 180}"
                 upper="${A4_position_limit * PI / 180}"
-                velocity="${joint_3_velocity_limit * PI / 180}" />
+                velocity="${A4_velocity_limit * PI / 180}" />
             <dynamics damping="${joint_damping}" friction="${joint_friction}" />
         </joint>
@@ -173,5 +173,5 @@
             <limit effort="${effort_limit}" lower="${-A5_position_limit * PI / 180}"
                 upper="${A5_position_limit * PI / 180}"
-                velocity="${joint_4_velocity_limit * PI / 180}" />
+                velocity="${A5_velocity_limit * PI / 180}" />
             <dynamics damping="${joint_damping}" friction="${joint_friction}" />
         </joint>
@@ -203,5 +203,5 @@
             <limit effort="${effort_limit}" lower="${-A6_position_limit * PI / 180}"
                 upper="${A6_position_limit * PI / 180}"
-                velocity="${joint_5_velocity_limit * PI / 180}" />
+                velocity="${A6_velocity_limit * PI / 180}" />
             <dynamics damping="${joint_damping}" friction="${joint_friction}" />
         </joint>
@@ -233,5 +233,5 @@
             <limit effort="${effort_limit}" lower="${-A7_position_limit * PI / 180}"
                 upper="${A7_position_limit * PI / 180}"
-                velocity="${joint_6_velocity_limit * PI / 180}" />
+                velocity="${A7_velocity_limit * PI / 180}" />
             <dynamics damping="${joint_damping}" friction="${joint_friction}" />
         </joint>
