Commit message: added moveit

File: lbr_description/urdf/iiwa14/iiwa14.urdf.xacro (robot description, xacro)
@@ -7,12 +7,8 @@
     <xacro:include filename="$(find lbr_description)/urdf/iiwa14/iiwa14_description.urdf.xacro"/>
     <xacro:arg name="robot_name" default="lbr"/>
-    <xacro:arg name="origin_xyz" default="0 0 0"/>
-    <xacro:arg name="origin_rpy" default="0 0 0"/>
     <xacro:arg name="sim" default="true"/>
     <!-- fix to world -->
     <link name="world"/>
     <!-- iiwa -->
-    <xacro:iiwa14 parent="world" robot_name="$(arg robot_name)" sim="$(arg sim)">
-        <origin xyz="$(arg origin_xyz)" rpy="$(arg origin_rpy)" />
-    </xacro:iiwa14>
+    <xacro:iiwa14 parent="world" robot_name="$(arg robot_name)" sim="$(arg sim)"/>
 </robot>

File: lbr_description/urdf/iiwa14/iiwa14_description.urdf.xacro (robot description, xacro)
@@ -13,8 +13,7 @@
     <xacro:include filename="$(find lbr_description)/ros2_control/lbr.ros2_control.xacro"/>
     <!-- robot as extracted via https://github.com/syuntoku14/fusion2urdf -->
-    <xacro:macro name="iiwa14" params="*origin parent:=^|world robot_name:=^|lbr sim:=^|true">
+    <xacro:macro name="iiwa14" params="parent:=^|world robot_name:=^|lbr sim:=^|true">
         <!--joint between {parent} and link_0-->
         <joint name="${parent}_${robot_name}_joint" type="fixed">
-            <xacro:insert_block name="origin"/>
             <parent link="${parent}"/>
             <child link="${robot_name}_link_0"/>

File: lbr_description/urdf/iiwa7/iiwa7.urdf.xacro (robot description, xacro)
@@ -7,12 +7,8 @@
     <xacro:include filename="$(find lbr_description)/urdf/iiwa7/iiwa7_description.urdf.xacro"/>
     <xacro:arg name="robot_name" default="lbr"/>
-    <xacro:arg name="origin_xyz" default="0 0 0"/>
-    <xacro:arg name="origin_rpy" default="0 0 0"/>
     <xacro:arg name="sim" default="true"/>
     <!-- fix to world -->
     <link name="world"/>
     <!-- iiwa -->
-    <xacro:iiwa7 parent="world" robot_name="$(arg robot_name)" sim="$(arg sim)">
-        <origin xyz="$(arg origin_xyz)" rpy="$(arg origin_rpy)" />
-    </xacro:iiwa7>
+    <xacro:iiwa7 parent="world" robot_name="$(arg robot_name)" sim="$(arg sim)"/>
 </robot>

File: lbr_description/urdf/iiwa7/iiwa7_description.urdf.xacro (robot description, xacro)
@@ -13,8 +13,7 @@
     <xacro:include filename="$(find lbr_description)/ros2_control/lbr.ros2_control.xacro"/>
     <!-- robot as extracted via https://github.com/syuntoku14/fusion2urdf -->
-    <xacro:macro name="iiwa7" params="*origin parent:=^|world robot_name:=^|lbr sim:=^|true">
+    <xacro:macro name="iiwa7" params="parent:=^|world robot_name:=^|lbr sim:=^|true">
         <!--joint between {parent} and link_0-->
         <joint name="${parent}_${robot_name}_joint" type="fixed">
-            <xacro:insert_block name="origin"/>
             <parent link="${parent}"/>
             <child link="${robot_name}_link_0"/>

File: lbr_description/urdf/med14/med14.urdf.xacro (robot description, xacro)
@@ -7,12 +7,8 @@
     <xacro:include filename="$(find lbr_description)/urdf/med14/med14_description.urdf.xacro"/>
     <xacro:arg name="robot_name" default="lbr"/>
-    <xacro:arg name="origin_xyz" default="0 0 0"/>
-    <xacro:arg name="origin_rpy" default="0 0 0"/>
     <xacro:arg name="sim" default="true"/>
     <!-- fix to world -->
     <link name="world"/>
     <!-- med -->
-    <xacro:med14 parent="world" robot_name="$(arg robot_name)" sim="$(arg sim)">
-        <origin xyz="$(arg origin_xyz)" rpy="$(arg origin_rpy)" />
-    </xacro:med14>
+    <xacro:med14 parent="world" robot_name="$(arg robot_name)" sim="$(arg sim)"/>
 </robot>

File: lbr_description/urdf/med14/med14_description.urdf.xacro (robot description, xacro)
@@ -13,8 +13,7 @@
     <xacro:include filename="$(find lbr_description)/ros2_control/lbr.ros2_control.xacro"/>
     <!-- robot as extracted via https://github.com/syuntoku14/fusion2urdf -->
-    <xacro:macro name="med14" params="*origin parent:=^|world robot_name:=^|lbr sim:=^|true">
+    <xacro:macro name="med14" params="parent:=^|world robot_name:=^|lbr sim:=^|true">
         <!--joint between {parent} and link_0-->
         <joint name="${parent}_${robot_name}_joint" type="fixed">
-            <xacro:insert_block name="origin"/>
             <parent link="${parent}"/>
             <child link="${robot_name}_link_0"/>

File: lbr_description/urdf/med7/med7.urdf.xacro (robot description, xacro)
@@ -13,6 +13,4 @@
     <link name="world"/>
     <!-- med -->
-    <xacro:med7 parent="world" robot_name="$(arg robot_name)" sim="$(arg sim)">
-        <origin xyz="$(arg origin_xyz)" rpy="$(arg origin_rpy)" />
-    </xacro:med7>
+    <xacro:med7 parent="world" robot_name="$(arg robot_name)" sim="$(arg sim)"/>
 </robot>

File: lbr_description/urdf/med7/med7_description.urdf.xacro (robot description, xacro)
@@ -13,8 +13,7 @@
     <xacro:include filename="$(find lbr_description)/ros2_control/lbr.ros2_control.xacro"/>
     <!-- robot as extracted via https://github.com/syuntoku14/fusion2urdf -->
-    <xacro:macro name="med7" params="*origin parent:=^|world robot_name:=^|lbr sim:=^|true">
+    <xacro:macro name="med7" params="parent:=^|world robot_name:=^|lbr sim:=^|true">
         <!--joint between {parent} and link_0-->
         <joint name="${parent}_${robot_name}_joint" type="fixed">
-            <xacro:insert_block name="origin"/>
             <parent link="${parent}"/>
             <child link="${robot_name}_link_0"/>=

Commit message: formatted xml

File: lbr_description/urdf/iiwa14/iiwa14.urdf.xacro (robot description, xacro)
@@ -3,10 +3,10 @@
 <robot name="iiwa14" xmlns:xacro="http://www.ros.org/wiki/xacro">
     <!-- include the lbr iiwa macro -->
-    <xacro:include filename="$(find lbr_description)/urdf/iiwa14/iiwa14_description.urdf.xacro"/>
-    <xacro:arg name="robot_name" default="lbr"/>
-    <xacro:arg name="sim" default="true"/>
+    <xacro:include filename="$(find lbr_description)/urdf/iiwa14/iiwa14_description.urdf.xacro" />
+    <xacro:arg name="robot_name" default="lbr" />
+    <xacro:arg name="sim" default="true" />
     <!-- fix to world -->
-    <link name="world"/>
+    <link name="world" />
     <!-- iiwa -->
-    <xacro:iiwa14 parent="world" robot_name="$(arg robot_name)" sim="$(arg sim)"/>
+    <xacro:iiwa14 parent="world" robot_name="$(arg robot_name)" sim="$(arg sim)" />
 </robot>

File: lbr_description/urdf/iiwa7/iiwa7.urdf.xacro (robot description, xacro)
@@ -3,10 +3,10 @@
 <robot name="iiwa7" xmlns:xacro="http://www.ros.org/wiki/xacro">
     <!-- include the lbr iiwa macro -->
-    <xacro:include filename="$(find lbr_description)/urdf/iiwa7/iiwa7_description.urdf.xacro"/>
-    <xacro:arg name="robot_name" default="lbr"/>
-    <xacro:arg name="sim" default="true"/>
+    <xacro:include filename="$(find lbr_description)/urdf/iiwa7/iiwa7_description.urdf.xacro" />
+    <xacro:arg name="robot_name" default="lbr" />
+    <xacro:arg name="sim" default="true" />
     <!-- fix to world -->
-    <link name="world"/>
+    <link name="world" />
     <!-- iiwa -->
-    <xacro:iiwa7 parent="world" robot_name="$(arg robot_name)" sim="$(arg sim)"/>
+    <xacro:iiwa7 parent="world" robot_name="$(arg robot_name)" sim="$(arg sim)" />
 </robot>

File: lbr_description/urdf/materials.urdf.xacro (robot description, xacro)
@@ -2,11 +2,11 @@
 <robot>
     <material name="orange">
-        <color rgba="1.0 0.42 0.04 1.0"/>
+        <color rgba="1.0 0.42 0.04 1.0" />
     </material>
     <material name="white">
-        <color rgba="1.0 1.0 1.0 1.0"/>
+        <color rgba="1.0 1.0 1.0 1.0" />
     </material>
     <material name="silver">
-        <color rgba="0.7 0.7 0.7 1.0"/>
+        <color rgba="0.7 0.7 0.7 1.0" />
     </material>
 </robot>

File: lbr_description/urdf/med14/med14.urdf.xacro (robot description, xacro)
@@ -3,10 +3,10 @@
 <robot name="med14" xmlns:xacro="http://www.ros.org/wiki/xacro">
     <!-- include the lbr med macro -->
-    <xacro:include filename="$(find lbr_description)/urdf/med14/med14_description.urdf.xacro"/>
-    <xacro:arg name="robot_name" default="lbr"/>
-    <xacro:arg name="sim" default="true"/>
+    <xacro:include filename="$(find lbr_description)/urdf/med14/med14_description.urdf.xacro" />
+    <xacro:arg name="robot_name" default="lbr" />
+    <xacro:arg name="sim" default="true" />
     <!-- fix to world -->
-    <link name="world"/>
+    <link name="world" />
     <!-- med -->
-    <xacro:med14 parent="world" robot_name="$(arg robot_name)" sim="$(arg sim)"/>
+    <xacro:med14 parent="world" robot_name="$(arg robot_name)" sim="$(arg sim)" />
 </robot>

File: lbr_description/urdf/med7/med7.urdf.xacro (robot description, xacro)
@@ -3,10 +3,10 @@
 <robot name="med7" xmlns:xacro="http://www.ros.org/wiki/xacro">
     <!-- include the lbr med macro -->
-    <xacro:include filename="$(find lbr_description)/urdf/med7/med7_description.urdf.xacro"/>
-    <xacro:arg name="robot_name" default="lbr"/>
-    <xacro:arg name="sim" default="true"/>
+    <xacro:include filename="$(find lbr_description)/urdf/med7/med7_description.urdf.xacro" />
+    <xacro:arg name="robot_name" default="lbr" />
+    <xacro:arg name="sim" default="true" />
     <!-- fix to world -->
-    <link name="world"/>
+    <link name="world" />
     <!-- med -->
-    <xacro:med7 parent="world" robot_name="$(arg robot_name)" sim="$(arg sim)"/>
+    <xacro:med7 parent="world" robot_name="$(arg robot_name)" sim="$(arg sim)" />
 </robot>

Commit message: added configurable base frame

File: lbr_description/urdf/iiwa14/iiwa14.urdf.xacro (robot description, xacro)
@@ -6,7 +6,8 @@
     <xacro:arg name="robot_name" default="lbr" />
     <xacro:arg name="sim" default="true" />
-    <!-- fix to world -->
-    <link name="world" />
+    <xacro:arg name="base_frame" default="world" />
+    <!-- fix to base_frame -->
+    <link name="$(arg base_frame)" />
     <!-- iiwa -->
-    <xacro:iiwa14 parent="world" robot_name="$(arg robot_name)" sim="$(arg sim)" />
+    <xacro:iiwa14 base_frame="$(arg base_frame)" robot_name="$(arg robot_name)" sim="$(arg sim)" />
 </robot>

File: lbr_description/urdf/iiwa14/iiwa14_description.urdf.xacro (robot description, xacro)
@@ -25,8 +25,9 @@
     <xacro:include filename="$(find lbr_description)/ros2_control/lbr.ros2_control.xacro" />
     <!-- robot as extracted via https://github.com/syuntoku14/fusion2urdf -->
-    <xacro:macro name="iiwa14" params="parent:=^|world robot_name:=^|lbr sim:=^|true">
-        <!--joint between {parent} and link_0-->
-        <joint name="${parent}_${robot_name}_joint" type="fixed">
-            <parent link="${parent}" />
+    <xacro:macro name="iiwa14" params="base_frame:=^|world robot_name:=^|lbr sim:=^|true">
+        <!--joint
+        between {base_frame} and link_0-->
+        <joint name="${base_frame}_${robot_name}_joint" type="fixed">
+            <parent link="${base_frame}" />
             <child link="${robot_name}_link_0" />
         </joint>

File: lbr_description/urdf/iiwa7/iiwa7.urdf.xacro (robot description, xacro)
@@ -6,7 +6,8 @@
     <xacro:arg name="robot_name" default="lbr" />
     <xacro:arg name="sim" default="true" />
-    <!-- fix to world -->
-    <link name="world" />
+    <xacro:arg name="base_frame" default="world" />
+    <!-- fix to base_frame -->
+    <link name="$(arg base_frame)" />
     <!-- iiwa -->
-    <xacro:iiwa7 parent="world" robot_name="$(arg robot_name)" sim="$(arg sim)" />
+    <xacro:iiwa7 base_frame="$(arg base_frame)" robot_name="$(arg robot_name)" sim="$(arg sim)" />
 </robot>

File: lbr_description/urdf/iiwa7/iiwa7_description.urdf.xacro (robot description, xacro)
@@ -25,8 +25,9 @@
     <xacro:include filename="$(find lbr_description)/ros2_control/lbr.ros2_control.xacro" />
     <!-- robot as extracted via https://github.com/syuntoku14/fusion2urdf -->
-    <xacro:macro name="iiwa7" params="parent:=^|world robot_name:=^|lbr sim:=^|true">
-        <!--joint between {parent} and link_0-->
-        <joint name="${parent}_${robot_name}_joint" type="fixed">
-            <parent link="${parent}" />
+    <xacro:macro name="iiwa7" params="base_frame:=^|world robot_name:=^|lbr sim:=^|true">
+        <!--joint
+        between {base_frame} and link_0-->
+        <joint name="${base_frame}_${robot_name}_joint" type="fixed">
+            <parent link="${base_frame}" />
             <child link="${robot_name}_link_0" />
         </joint>

File: lbr_description/urdf/med14/med14.urdf.xacro (robot description, xacro)
@@ -6,7 +6,8 @@
     <xacro:arg name="robot_name" default="lbr" />
     <xacro:arg name="sim" default="true" />
-    <!-- fix to world -->
-    <link name="world" />
+    <xacro:arg name="base_frame" default="world" />
+    <!-- fix to base_frame -->
+    <link name="$(arg base_frame)" />
     <!-- med -->
-    <xacro:med14 parent="world" robot_name="$(arg robot_name)" sim="$(arg sim)" />
+    <xacro:med14 base_frame="$(arg base_frame)" robot_name="$(arg robot_name)" sim="$(arg sim)" />
 </robot>

File: lbr_description/urdf/med14/med14_description.urdf.xacro (robot description, xacro)
@@ -25,8 +25,9 @@
     <xacro:include filename="$(find lbr_description)/ros2_control/lbr.ros2_control.xacro" />
     <!-- robot as extracted via https://github.com/syuntoku14/fusion2urdf -->
-    <xacro:macro name="med14" params="parent:=^|world robot_name:=^|lbr sim:=^|true">
-        <!--joint between {parent} and link_0-->
-        <joint name="${parent}_${robot_name}_joint" type="fixed">
-            <parent link="${parent}" />
+    <xacro:macro name="med14" params="base_frame:=^|world robot_name:=^|lbr sim:=^|true">
+        <!--joint
+        between {base_frame} and link_0-->
+        <joint name="${base_frame}_${robot_name}_joint" type="fixed">
+            <parent link="${base_frame}" />
             <child link="${robot_name}_link_0" />
         </joint>

File: lbr_description/urdf/med7/med7.urdf.xacro (robot description, xacro)
@@ -6,7 +6,8 @@
     <xacro:arg name="robot_name" default="lbr" />
     <xacro:arg name="sim" default="true" />
-    <!-- fix to world -->
-    <link name="world" />
+    <xacro:arg name="base_frame" default="world" />
+    <!-- fix to base_frame -->
+    <link name="$(arg base_frame)" />
     <!-- med -->
-    <xacro:med7 parent="world" robot_name="$(arg robot_name)" sim="$(arg sim)" />
+    <xacro:med7 base_frame="$(arg base_frame)" robot_name="$(arg robot_name)" sim="$(arg sim)" />
 </robot>

File: lbr_description/urdf/med7/med7_description.urdf.xacro (robot description, xacro)
@@ -25,8 +25,9 @@
     <xacro:include filename="$(find lbr_description)/ros2_control/lbr.ros2_control.xacro" />
     <!-- robot as extracted via https://github.com/syuntoku14/fusion2urdf -->
-    <xacro:macro name="med7" params="parent:=^|world robot_name:=^|lbr sim:=^|true">
-        <!--joint between {parent} and link_0-->
-        <joint name="${parent}_${robot_name}_joint" type="fixed">
-            <parent link="${parent}" />
+    <xacro:macro name="med7" params="base_frame:=^|world robot_name:=^|lbr sim:=^|true">
+        <!--joint
+        between {base_frame} and link_0-->
+        <joint name="${base_frame}_${robot_name}_joint" type="fixed">
+            <parent link="${base_frame}" />
             <child link="${robot_name}_link_0" />
         </joint>

Commit message: added port id to urdf

File: lbr_description/urdf/iiwa14/iiwa14.urdf.xacro (robot description, xacro)
@@ -4,10 +4,12 @@
     <!-- include the lbr iiwa macro -->
     <xacro:include filename="$(find lbr_description)/urdf/iiwa14/iiwa14_description.urdf.xacro" />
+    <xacro:arg name="base_frame" default="world" />
     <xacro:arg name="robot_name" default="lbr" />
+    <xacro:arg name="port_id" default="30200" />
     <xacro:arg name="sim" default="true" />
-    <xacro:arg name="base_frame" default="world" />
     <!-- fix to base_frame -->
     <link name="$(arg base_frame)" />
     <!-- iiwa -->
-    <xacro:iiwa14 base_frame="$(arg base_frame)" robot_name="$(arg robot_name)" sim="$(arg sim)" />
+    <xacro:iiwa14 base_frame="$(arg base_frame)" robot_name="$(arg robot_name)"
+        port_id="$(arg port_id)" sim="$(arg sim)" />
 </robot>

File: lbr_description/urdf/iiwa14/iiwa14_description.urdf.xacro (robot description, xacro)
@@ -24,5 +24,6 @@
     <xacro:include filename="$(find lbr_description)/ros2_control/lbr.ros2_control.xacro" />
     <!-- robot as extracted via https://github.com/syuntoku14/fusion2urdf -->
-    <xacro:macro name="iiwa14" params="base_frame:=^|world robot_name:=^|lbr sim:=^|true">
+    <xacro:macro name="iiwa14"
+        params="base_frame:=^|world robot_name:=^|lbr port_id:=^|30200 sim:=^|true">
         <!--joint
         between {base_frame} and link_0-->
@@ -287,5 +288,5 @@
             joint_6_position_limit="${joint_6_position_limit * PI / 180}"
             effort_limit="${effort_limit}"
-            sim="${sim}" remote_host="INADDR_ANY" port_id="30200" />
+            sim="${sim}" remote_host="INADDR_ANY" port_id="${port_id}" />
     </xacro:macro>
 </robot>

File: lbr_description/urdf/iiwa7/iiwa7.urdf.xacro (robot description, xacro)
@@ -4,10 +4,12 @@
     <!-- include the lbr iiwa macro -->
     <xacro:include filename="$(find lbr_description)/urdf/iiwa7/iiwa7_description.urdf.xacro" />
+    <xacro:arg name="base_frame" default="world" />
     <xacro:arg name="robot_name" default="lbr" />
+    <xacro:arg name="port_id" default="30200" />
     <xacro:arg name="sim" default="true" />
-    <xacro:arg name="base_frame" default="world" />
     <!-- fix to base_frame -->
     <link name="$(arg base_frame)" />
     <!-- iiwa -->
-    <xacro:iiwa7 base_frame="$(arg base_frame)" robot_name="$(arg robot_name)" sim="$(arg sim)" />
+    <xacro:iiwa7 base_frame="$(arg base_frame)" robot_name="$(arg robot_name)"
+        port_id="$(arg port_id)" sim="$(arg sim)" />
 </robot>

File: lbr_description/urdf/iiwa7/iiwa7_description.urdf.xacro (robot description, xacro)
@@ -24,5 +24,6 @@
     <xacro:include filename="$(find lbr_description)/ros2_control/lbr.ros2_control.xacro" />
     <!-- robot as extracted via https://github.com/syuntoku14/fusion2urdf -->
-    <xacro:macro name="iiwa7" params="base_frame:=^|world robot_name:=^|lbr sim:=^|true">
+    <xacro:macro name="iiwa7"
+        params="base_frame:=^|world robot_name:=^|lbr port_id:=^|30200 sim:=^|true">
         <!--joint
         between {base_frame} and link_0-->
@@ -287,5 +288,5 @@
             joint_6_position_limit="${joint_6_position_limit * PI / 180}"
             effort_limit="${effort_limit}"
-            sim="${sim}" remote_host="INADDR_ANY" port_id="30200" />
+            sim="${sim}" remote_host="INADDR_ANY" port_id="${port_id}" />
     </xacro:macro>
 </robot>

File: lbr_description/urdf/med14/med14.urdf.xacro (robot description, xacro)
@@ -4,10 +4,12 @@
     <!-- include the lbr med macro -->
     <xacro:include filename="$(find lbr_description)/urdf/med14/med14_description.urdf.xacro" />
+    <xacro:arg name="base_frame" default="world" />
     <xacro:arg name="robot_name" default="lbr" />
+    <xacro:arg name="port_id" default="30200" />
     <xacro:arg name="sim" default="true" />
-    <xacro:arg name="base_frame" default="world" />
     <!-- fix to base_frame -->
     <link name="$(arg base_frame)" />
     <!-- med -->
-    <xacro:med14 base_frame="$(arg base_frame)" robot_name="$(arg robot_name)" sim="$(arg sim)" />
+    <xacro:med14 base_frame="$(arg base_frame)" robot_name="$(arg robot_name)"
+        port_id="$(arg port_id)" sim="$(arg sim)" />
 </robot>

File: lbr_description/urdf/med14/med14_description.urdf.xacro (robot description, xacro)
@@ -24,5 +24,6 @@
     <xacro:include filename="$(find lbr_description)/ros2_control/lbr.ros2_control.xacro" />
     <!-- robot as extracted via https://github.com/syuntoku14/fusion2urdf -->
-    <xacro:macro name="med14" params="base_frame:=^|world robot_name:=^|lbr sim:=^|true">
+    <xacro:macro name="med14"
+        params="base_frame:=^|world robot_name:=^|lbr port_id:=^|30200 sim:=^|true">
         <!--joint
         between {base_frame} and link_0-->
@@ -287,5 +288,5 @@
             joint_6_position_limit="${joint_6_position_limit * PI / 180}"
             effort_limit="${effort_limit}"
-            sim="${sim}" remote_host="INADDR_ANY" port_id="30200" />
+            sim="${sim}" remote_host="INADDR_ANY" port_id="${port_id}" />
     </xacro:macro>
 </robot>

File: lbr_description/urdf/med7/med7.urdf.xacro (robot description, xacro)
@@ -4,10 +4,12 @@
     <!-- include the lbr med macro -->
     <xacro:include filename="$(find lbr_description)/urdf/med7/med7_description.urdf.xacro" />
+    <xacro:arg name="base_frame" default="world" />
     <xacro:arg name="robot_name" default="lbr" />
+    <xacro:arg name="port_id" default="30200" />
     <xacro:arg name="sim" default="true" />
-    <xacro:arg name="base_frame" default="world" />
     <!-- fix to base_frame -->
     <link name="$(arg base_frame)" />
     <!-- med -->
-    <xacro:med7 base_frame="$(arg base_frame)" robot_name="$(arg robot_name)" sim="$(arg sim)" />
+    <xacro:med7 base_frame="$(arg base_frame)" robot_name="$(arg robot_name)"
+        port_id="$(arg port_id)" sim="$(arg sim)" />
 </robot>

File: lbr_description/urdf/med7/med7_description.urdf.xacro (robot description, xacro)
@@ -24,5 +24,6 @@
     <xacro:include filename="$(find lbr_description)/ros2_control/lbr.ros2_control.xacro" />
     <!-- robot as extracted via https://github.com/syuntoku14/fusion2urdf -->
-    <xacro:macro name="med7" params="base_frame:=^|world robot_name:=^|lbr sim:=^|true">
+    <xacro:macro name="med7"
+        params="base_frame:=^|world robot_name:=^|lbr port_id:=^|30200 sim:=^|true">
         <!--joint
         between {base_frame} and link_0-->
@@ -287,5 +288,5 @@
             joint_6_position_limit="${joint_6_position_limit * PI / 180}"
             effort_limit="${effort_limit}"
-            sim="${sim}" remote_host="INADDR_ANY" port_id="30200" />
+            sim="${sim}" remote_host="INADDR_ANY" port_id="${port_id}" />
     </xacro:macro>
 </robot>
