Commit message: de-couple base frame from urdf

File: lbr_description/urdf/iiwa14/iiwa14.urdf.xacro (robot description, xacro)
@@ -8,8 +8,13 @@
     <xacro:arg name="port_id" default="30200" />
     <xacro:arg name="sim" default="true" />
-    <!-- fix to base_frame -->
+    <!-- fixed to base_frame -->
     <link name="$(arg base_frame)" />
+    <!--joint
+        between {base_frame} and link_0-->
+    <joint name="$(arg base_frame)_joint" type="fixed">
+        <parent link="$(arg base_frame)" />
+        <child link="link_0" />
+    </joint>
     <!-- iiwa -->
-    <xacro:iiwa14 base_frame="$(arg base_frame)" robot_name="$(arg robot_name)"
-        port_id="$(arg port_id)" sim="$(arg sim)" />
+    <xacro:iiwa14 robot_name="$(arg robot_name)" port_id="$(arg port_id)" sim="$(arg sim)" />
 </robot>

File: lbr_description/urdf/iiwa14/iiwa14_description.urdf.xacro (robot description, xacro)
@@ -25,11 +25,5 @@
     <!-- robot as extracted via https://github.com/syuntoku14/fusion2urdf -->
     <xacro:macro name="iiwa14"
-        params="base_frame:=^|world robot_name:=^|lbr port_id:=^|30200 sim:=^|true">
-        <!--joint
-        between {base_frame} and link_0-->
-        <joint name="${base_frame}_joint" type="fixed">
-            <parent link="${base_frame}" />
-            <child link="link_0" />
-        </joint>
+        params="robot_name:=^|lbr port_id:=^|30200 sim:=^|true">
         <link name="link_0">
             <inertial>

File: lbr_description/urdf/iiwa7/iiwa7.urdf.xacro (robot description, xacro)
@@ -8,8 +8,13 @@
     <xacro:arg name="port_id" default="30200" />
     <xacro:arg name="sim" default="true" />
-    <!-- fix to base_frame -->
+    <!-- fixed to base_frame -->
     <link name="$(arg base_frame)" />
+    <!--joint
+        between {base_frame} and link_0-->
+    <joint name="$(arg base_frame)_joint" type="fixed">
+        <parent link="$(arg base_frame)" />
+        <child link="link_0" />
+    </joint>
     <!-- iiwa -->
-    <xacro:iiwa7 base_frame="$(arg base_frame)" robot_name="$(arg robot_name)"
-        port_id="$(arg port_id)" sim="$(arg sim)" />
+    <xacro:iiwa7 robot_name="$(arg robot_name)" port_id="$(arg port_id)" sim="$(arg sim)" />
 </robot>

File: lbr_description/urdf/iiwa7/iiwa7_description.urdf.xacro (robot description, xacro)
@@ -25,11 +25,5 @@
     <!-- robot as extracted via https://github.com/syuntoku14/fusion2urdf -->
     <xacro:macro name="iiwa7"
-        params="base_frame:=^|world robot_name:=^|lbr port_id:=^|30200 sim:=^|true">
-        <!--joint
-        between {base_frame} and link_0-->
-        <joint name="${base_frame}_joint" type="fixed">
-            <parent link="${base_frame}" />
-            <child link="link_0" />
-        </joint>
+        params="robot_name:=^|lbr port_id:=^|30200 sim:=^|true">
         <link name="link_0">
             <inertial>

File: lbr_description/urdf/med14/med14.urdf.xacro (robot description, xacro)
@@ -8,8 +8,13 @@
     <xacro:arg name="port_id" default="30200" />
     <xacro:arg name="sim" default="true" />
-    <!-- fix to base_frame -->
+    <!-- fixed to base_frame -->
     <link name="$(arg base_frame)" />
+    <!--joint
+        between {base_frame} and link_0-->
+    <joint name="$(arg base_frame)_joint" type="fixed">
+        <parent link="$(arg base_frame)" />
+        <child link="link_0" />
+    </joint>
     <!-- med -->
-    <xacro:med14 base_frame="$(arg base_frame)" robot_name="$(arg robot_name)"
-        port_id="$(arg port_id)" sim="$(arg sim)" />
+    <xacro:med14 robot_name="$(arg robot_name)" port_id="$(arg port_id)" sim="$(arg sim)" />
 </robot>

File: lbr_description/urdf/med14/med14_description.urdf.xacro (robot description, xacro)
@@ -25,11 +25,5 @@
     <!-- robot as extracted via https://github.com/syuntoku14/fusion2urdf -->
     <xacro:macro name="med14"
-        params="base_frame:=^|world robot_name:=^|lbr port_id:=^|30200 sim:=^|true">
-        <!--joint
-        between {base_frame} and link_0-->
-        <joint name="${base_frame}_joint" type="fixed">
-            <parent link="${base_frame}" />
-            <child link="link_0" />
-        </joint>
+        params="robot_name:=^|lbr port_id:=^|30200 sim:=^|true">
         <link name="link_0">
             <inertial>

File: lbr_description/urdf/med7/med7.urdf.xacro (robot description, xacro)
@@ -8,8 +8,13 @@
     <xacro:arg name="port_id" default="30200" />
     <xacro:arg name="sim" default="true" />
-    <!-- fix to base_frame -->
+    <!-- fixed to base_frame -->
     <link name="$(arg base_frame)" />
+    <!--joint
+        between {base_frame} and link_0-->
+    <joint name="$(arg base_frame)_joint" type="fixed">
+        <parent link="$(arg base_frame)" />
+        <child link="link_0" />
+    </joint>
     <!-- med -->
-    <xacro:med7 base_frame="$(arg base_frame)" robot_name="$(arg robot_name)"
-        port_id="$(arg port_id)" sim="$(arg sim)" />
+    <xacro:med7 robot_name="$(arg robot_name)" port_id="$(arg port_id)" sim="$(arg sim)" />
 </robot>

File: lbr_description/urdf/med7/med7_description.urdf.xacro (robot description, xacro)
@@ -25,11 +25,5 @@
     <!-- robot as extracted via https://github.com/syuntoku14/fusion2urdf -->
     <xacro:macro name="med7"
-        params="base_frame:=^|world robot_name:=^|lbr port_id:=^|30200 sim:=^|true">
-        <!--joint
-        between {base_frame} and link_0-->
-        <joint name="${base_frame}_joint" type="fixed">
-            <parent link="${base_frame}" />
-            <child link="link_0" />
-        </joint>
+        params="robot_name:=^|lbr port_id:=^|30200 sim:=^|true">
         <link name="link_0">
             <inertial>

Commit message: removed base frame #129

File: lbr_description/urdf/iiwa14/iiwa14.urdf.xacro (robot description, xacro)
@@ -4,14 +4,13 @@
     <!-- include the lbr iiwa macro -->
     <xacro:include filename="$(find lbr_description)/urdf/iiwa14/iiwa14_description.urdf.xacro" />
-    <xacro:arg name="base_frame" default="base_frame" />
     <xacro:arg name="robot_name" default="lbr" />
     <xacro:arg name="port_id" default="30200" />
     <xacro:arg name="sim" default="true" />
-    <!-- fixed to base_frame -->
-    <link name="$(arg base_frame)" />
+    <!-- fixed to world, see http://classic.gazebosim.org/tutorials?tut=ros_urdf&cat=connect_ros -->
+    <link name="world" />
     <!--joint
-        between {base_frame} and link_0-->
-    <joint name="$(arg base_frame)_joint" type="fixed">
-        <parent link="$(arg base_frame)" />
+        between world and link_0-->
+    <joint name="world_joint" type="fixed">
+        <parent link="world" />
         <child link="link_0" />
     </joint>

File: lbr_description/urdf/iiwa7/iiwa7.urdf.xacro (robot description, xacro)
@@ -4,14 +4,13 @@
     <!-- include the lbr iiwa macro -->
     <xacro:include filename="$(find lbr_description)/urdf/iiwa7/iiwa7_description.urdf.xacro" />
-    <xacro:arg name="base_frame" default="base_frame" />
     <xacro:arg name="robot_name" default="lbr" />
     <xacro:arg name="port_id" default="30200" />
     <xacro:arg name="sim" default="true" />
-    <!-- fixed to base_frame -->
-    <link name="$(arg base_frame)" />
+    <!-- fixed to world, see http://classic.gazebosim.org/tutorials?tut=ros_urdf&cat=connect_ros -->
+    <link name="world" />
     <!--joint
-        between {base_frame} and link_0-->
-    <joint name="$(arg base_frame)_joint" type="fixed">
-        <parent link="$(arg base_frame)" />
+        between world and link_0-->
+    <joint name="world_joint" type="fixed">
+        <parent link="world" />
         <child link="link_0" />
     </joint>

File: lbr_description/urdf/med14/med14.urdf.xacro (robot description, xacro)
@@ -4,14 +4,13 @@
     <!-- include the lbr med macro -->
     <xacro:include filename="$(find lbr_description)/urdf/med14/med14_description.urdf.xacro" />
-    <xacro:arg name="base_frame" default="base_frame" />
     <xacro:arg name="robot_name" default="lbr" />
     <xacro:arg name="port_id" default="30200" />
     <xacro:arg name="sim" default="true" />
-    <!-- fixed to base_frame -->
-    <link name="$(arg base_frame)" />
+    <!-- fixed to world, see http://classic.gazebosim.org/tutorials?tut=ros_urdf&cat=connect_ros -->
+    <link name="world" />
     <!--joint
-        between {base_frame} and link_0-->
-    <joint name="$(arg base_frame)_joint" type="fixed">
-        <parent link="$(arg base_frame)" />
+        between world and link_0-->
+    <joint name="world_joint" type="fixed">
+        <parent link="world" />
         <child link="link_0" />
     </joint>

File: lbr_description/urdf/med7/med7.urdf.xacro (robot description, xacro)
@@ -4,14 +4,13 @@
     <!-- include the lbr med macro -->
     <xacro:include filename="$(find lbr_description)/urdf/med7/med7_description.urdf.xacro" />
-    <xacro:arg name="base_frame" default="base_frame" />
     <xacro:arg name="robot_name" default="lbr" />
     <xacro:arg name="port_id" default="30200" />
     <xacro:arg name="sim" default="true" />
-    <!-- fixed to base_frame -->
-    <link name="$(arg base_frame)" />
+    <!-- fixed to world, see http://classic.gazebosim.org/tutorials?tut=ros_urdf&cat=connect_ros -->
+    <link name="world" />
     <!--joint
-        between {base_frame} and link_0-->
-    <joint name="$(arg base_frame)_joint" type="fixed">
-        <parent link="$(arg base_frame)" />
+        between world and link_0-->
+    <joint name="world_joint" type="fixed">
+        <parent link="world" />
         <child link="link_0" />
     </joint>
