Commit message: system_parameters_path -> ros2_control xacro

File: lbr_description/urdf/iiwa14/iiwa14_description.xacro (robot description, xacro)
@@ -11,7 +11,4 @@
             value="$(find lbr_description)/urdf/iiwa14/joint_limits.yaml" />
         <xacro:property name="joint_limits" value="${xacro.load_yaml(joint_limits_path)}" />
-        <!-- system parameters via yaml -->
-        <xacro:property name="system_parameters"
-            value="${xacro.load_yaml(system_parameters_path)}" />
         <!-- constants -->
         <xacro:property name="PI" value="3.1415926535897931" />
@@ -23,5 +20,5 @@
             sim="${sim}"
             joint_limits="${joint_limits}"
-            system_parameters="${system_parameters}" />
+            system_parameters_path="${system_parameters_path}" />
         <link name="link_0">
             <inertial>

File: lbr_description/urdf/iiwa7/iiwa7_description.xacro (robot description, xacro)
@@ -11,7 +11,4 @@
             value="$(find lbr_description)/urdf/iiwa7/joint_limits.yaml" />
         <xacro:property name="joint_limits" value="${xacro.load_yaml(joint_limits_path)}" />
-        <!-- system parameters via yaml -->
-        <xacro:property name="system_parameters"
-            value="${xacro.load_yaml(system_parameters_path)}" />
         <!-- constants -->
         <xacro:property name="PI" value="3.1415926535897931" />
@@ -23,5 +20,5 @@
             sim="${sim}"
             joint_limits="${joint_limits}"
-            system_parameters="${system_parameters}" />
+            system_parameters_path="${system_parameters_path}" />
         <link name="link_0">
             <inertial>

File: lbr_description/urdf/med14/med14_description.xacro (robot description, xacro)
@@ -11,7 +11,4 @@
             value="$(find lbr_description)/urdf/med14/joint_limits.yaml" />
         <xacro:property name="joint_limits" value="${xacro.load_yaml(joint_limits_path)}" />
-        <!-- system parameters via yaml -->
-        <xacro:property name="system_parameters"
-            value="${xacro.load_yaml(system_parameters_path)}" />
         <!-- constants -->
         <xacro:property name="PI" value="3.1415926535897931" />
@@ -23,5 +20,5 @@
             sim="${sim}"
             joint_limits="${joint_limits}"
-            system_parameters="${system_parameters}" />
+            system_parameters_path="${system_parameters_path}" />
         <link name="link_0">
             <inertial>

File: lbr_description/urdf/med7/med7_description.xacro (robot description, xacro)
@@ -11,7 +11,4 @@
             value="$(find lbr_description)/urdf/med7/joint_limits.yaml" />
         <xacro:property name="joint_limits" value="${xacro.load_yaml(joint_limits_path)}" />
-        <!-- system parameters via yaml -->
-        <xacro:property name="system_parameters"
-            value="${xacro.load_yaml(system_parameters_path)}" />
         <!-- constants -->
         <xacro:property name="PI" value="3.1415926535897931" />
@@ -23,5 +20,5 @@
             sim="${sim}"
             joint_limits="${joint_limits}"
-            system_parameters="${system_parameters}" />
+            system_parameters_path="${system_parameters_path}" />
         <!-- properties -->
         <link name="link_0">

File: lbr_ros2_control/config/lbr_system_interface.xacro (robot description, xacro)
@@ -2,5 +2,8 @@
 <robot xmlns:xacro="http://www.ros.org/wiki/xacro">
     <xacro:macro name="lbr_system_interface"
-        params="sim joint_limits system_parameters">
+        params="sim joint_limits system_parameters_path">
+        <!-- load system parameters via yaml -->
+        <xacro:property name="system_parameters"
+            value="${xacro.load_yaml(system_parameters_path)}" />
         <ros2_control name="lbr_system_interface" type="system">
             <!-- define hardware including parameters, also gazebo -->

Commit message: added prefix (#189)

File: lbr_description/urdf/iiwa14/iiwa14_description.xacro (robot description, xacro)
@@ -265,5 +265,5 @@
             </collision>
         </link>
-        <joint name="joint_ee" type="fixed">
+        <joint name="${robot_name}_joint_ee" type="fixed">
             <parent link="${robot_name}_link_7" />
             <child link="${robot_name}_link_ee" />

File: lbr_description/urdf/iiwa7/iiwa7_description.xacro (robot description, xacro)
@@ -265,5 +265,5 @@
             </collision>
         </link>
-        <joint name="joint_ee" type="fixed">
+        <joint name="${robot_name}_joint_ee" type="fixed">
             <parent link="${robot_name}_link_7" />
             <child link="${robot_name}_link_ee" />

File: lbr_description/urdf/med14/med14_description.xacro (robot description, xacro)
@@ -265,5 +265,5 @@
             </collision>
         </link>
-        <joint name="joint_ee" type="fixed">
+        <joint name="${robot_name}_joint_ee" type="fixed">
             <parent link="${robot_name}_link_7" />
             <child link="${robot_name}_link_ee" />

File: lbr_description/urdf/med7/med7_description.xacro (robot description, xacro)
@@ -266,5 +266,5 @@
             </collision>
         </link>
-        <joint name="joint_ee" type="fixed">
+        <joint name="${robot_name}_joint_ee" type="fixed">
             <parent link="${robot_name}_link_7" />
             <child link="${robot_name}_link_ee" />
