Commit message: added a floating link with name prefix (#189)

File: lbr_description/urdf/iiwa14/iiwa14.xacro (robot description, xacro)
@@ -9,10 +9,10 @@
         name="system_config_path"
         default="$(find lbr_description)/ros2_control/lbr_system_config.yaml" />
-    <!-- fixed to world, see http://classic.gazebosim.org/tutorials?tut=ros_urdf&cat=connect_ros -->
-    <link name="world" />
+    <!-- KDL requires a link without inertia -->
+    <link name="$(arg robot_name)_floating_link" />
     <!--joint
-        between world and link_0-->
-    <joint name="world_joint" type="fixed">
-        <parent link="world" />
+        between <robot_name>_floating_link and robot_name_link_0-->
+    <joint name="$(arg robot_name)_floating_joint" type="fixed">
+        <parent link="$(arg robot_name)_floating_link" />
         <child link="$(arg robot_name)_link_0" />
     </joint>

File: lbr_description/urdf/iiwa7/iiwa7.xacro (robot description, xacro)
@@ -9,10 +9,10 @@
         name="system_config_path"
         default="$(find lbr_description)/ros2_control/lbr_system_config.yaml" />
-    <!-- fixed to world, see http://classic.gazebosim.org/tutorials?tut=ros_urdf&cat=connect_ros -->
-    <link name="world" />
+    <!-- KDL requires a link without inertia -->
+    <link name="$(arg robot_name)_floating_link" />
     <!--joint
-        between world and link_0-->
-    <joint name="world_joint" type="fixed">
-        <parent link="world" />
+        between <robot_name>_floating_link and robot_name_link_0-->
+    <joint name="$(arg robot_name)_floating_joint" type="fixed">
+        <parent link="$(arg robot_name)_floating_link" />
         <child link="$(arg robot_name)_link_0" />
     </joint>

File: lbr_description/urdf/med14/med14.xacro (robot description, xacro)
@@ -9,10 +9,10 @@
         name="system_config_path"
         default="$(find lbr_description)/ros2_control/lbr_system_config.yaml" />
-    <!-- fixed to world, see http://classic.gazebosim.org/tutorials?tut=ros_urdf&cat=connect_ros -->
-    <link name="world" />
+    <!-- KDL requires a link without inertia -->
+    <link name="$(arg robot_name)_floating_link" />
     <!--joint
-        between world and link_0-->
-    <joint name="world_joint" type="fixed">
-        <parent link="world" />
+        between <robot_name>_floating_link and robot_name_link_0-->
+    <joint name="$(arg robot_name)_floating_joint" type="fixed">
+        <parent link="$(arg robot_name)_floating_link" />
         <child link="$(arg robot_name)_link_0" />
     </joint>

File: lbr_description/urdf/med7/med7.xacro (robot description, xacro)
@@ -9,10 +9,10 @@
         name="system_config_path"
         default="$(find lbr_description)/ros2_control/lbr_system_config.yaml" />
-    <!-- fixed to world, see http://classic.gazebosim.org/tutorials?tut=ros_urdf&cat=connect_ros -->
-    <link name="world" />
+    <!-- KDL requires a link without inertia -->
+    <link name="$(arg robot_name)_floating_link" />
     <!--joint
-        between world and link_0-->
-    <joint name="world_joint" type="fixed">
-        <parent link="world" />
+        between <robot_name>_floating_link and robot_name_link_0-->
+    <joint name="$(arg robot_name)_floating_joint" type="fixed">
+        <parent link="$(arg robot_name)_floating_link" />
         <child link="$(arg robot_name)_link_0" />
     </joint>

Commit message: added configurable joint limits path (#333)

File: lbr_description/urdf/iiwa14/iiwa14.xacro (robot description, xacro)
@@ -9,4 +9,7 @@
         name="system_config_path"
         default="$(find lbr_description)/ros2_control/lbr_system_config.yaml" />
+    <xacro:arg
+        name="joint_limits_path"
+        default="$(find lbr_description)/urdf/iiwa14/joint_limits.yaml" />
     <xacro:arg
         name="initial_joint_positions_path"
@@ -26,4 +29,5 @@
         mode="$(arg mode)"
         system_config_path="$(arg system_config_path)"
+        joint_limits_path="$(arg joint_limits_path)"
         initial_joint_positions_path="$(arg initial_joint_positions_path)" />
 </robot>

File: lbr_description/urdf/iiwa14/iiwa14_description.xacro (robot description, xacro)
@@ -3,11 +3,9 @@
     <!-- robot as extracted via https://github.com/syuntoku14/fusion2urdf -->
     <xacro:macro name="iiwa14"
-        params="robot_name:=^|lbr mode:=^|mock system_config_path:=^|'$(find lbr_description)/ros2_control/lbr_system_config.yaml' initial_joint_positions_path:=^|'$(find lbr_description)/ros2_control/initial_joint_positions.yaml'">
+        params="robot_name:=^|lbr mode:=^|mock system_config_path:=^|'$(find lbr_description)/ros2_control/lbr_system_config.yaml' joint_limits_path:=^|'$(find lbr_description)/urdf/iiwa14/joint_limits.yaml' initial_joint_positions_path:=^|'$(find lbr_description)/ros2_control/initial_joint_positions.yaml'">
         <!-- includes -->
         <xacro:include filename="$(find lbr_description)/gazebo/lbr_gazebo.xacro" />
         <xacro:include filename="$(find lbr_description)/ros2_control/lbr_system_interface.xacro" />
         <!-- joint limits via yaml -->
-        <xacro:property name="joint_limits_path"
-            value="$(find lbr_description)/urdf/iiwa14/joint_limits.yaml" />
         <xacro:property name="joint_limits" value="${xacro.load_yaml(joint_limits_path)}" />
         <!-- constants -->

File: lbr_description/urdf/iiwa7/iiwa7.xacro (robot description, xacro)
@@ -9,4 +9,7 @@
         name="system_config_path"
         default="$(find lbr_description)/ros2_control/lbr_system_config.yaml" />
+    <xacro:arg
+        name="joint_limits_path"
+        default="$(find lbr_description)/urdf/iiwa7/joint_limits.yaml" />
     <xacro:arg
         name="initial_joint_positions_path"
@@ -26,4 +29,5 @@
         mode="$(arg mode)"
         system_config_path="$(arg system_config_path)"
+        joint_limits_path="$(arg joint_limits_path)"
         initial_joint_positions_path="$(arg initial_joint_positions_path)" />
 </robot>

File: lbr_description/urdf/iiwa7/iiwa7_description.xacro (robot description, xacro)
@@ -3,11 +3,9 @@
     <!-- robot as extracted via https://github.com/syuntoku14/fusion2urdf -->
     <xacro:macro name="iiwa7"
-        params="robot_name:=^|lbr mode:=^|mock system_config_path:=^|'$(find lbr_description)/ros2_control/lbr_system_config.yaml' initial_joint_positions_path:=^|'$(find lbr_description)/ros2_control/initial_joint_positions.yaml'">
+        params="robot_name:=^|lbr mode:=^|mock system_config_path:=^|'$(find lbr_description)/ros2_control/lbr_system_config.yaml' joint_limits_path:=^|'$(find lbr_description)/urdf/iiwa7/joint_limits.yaml' initial_joint_positions_path:=^|'$(find lbr_description)/ros2_control/initial_joint_positions.yaml'">
         <!-- includes -->
         <xacro:include filename="$(find lbr_description)/gazebo/lbr_gazebo.xacro" />
         <xacro:include filename="$(find lbr_description)/ros2_control/lbr_system_interface.xacro" />
         <!-- joint limits via yaml -->
-        <xacro:property name="joint_limits_path"
-            value="$(find lbr_description)/urdf/iiwa7/joint_limits.yaml" />
         <xacro:property name="joint_limits" value="${xacro.load_yaml(joint_limits_path)}" />
         <!-- constants -->

File: lbr_description/urdf/med14/med14.xacro (robot description, xacro)
@@ -9,4 +9,7 @@
         name="system_config_path"
         default="$(find lbr_description)/ros2_control/lbr_system_config.yaml" />
+    <xacro:arg
+        name="joint_limits_path"
+        default="$(find lbr_description)/urdf/med14/joint_limits.yaml" />
     <xacro:arg
         name="initial_joint_positions_path"
@@ -26,4 +29,5 @@
         mode="$(arg mode)"
         system_config_path="$(arg system_config_path)"
+        joint_limits_path="$(arg joint_limits_path)"
         initial_joint_positions_path="$(arg initial_joint_positions_path)" />
 </robot>

File: lbr_description/urdf/med14/med14_description.xacro (robot description, xacro)
@@ -3,11 +3,9 @@
     <!-- robot as extracted via https://github.com/syuntoku14/fusion2urdf -->
     <xacro:macro name="med14"
-        params="robot_name:=^|lbr mode:=^|mock system_config_path:=^|'$(find lbr_description)/ros2_control/lbr_system_config.yaml' initial_joint_positions_path:=^|'$(find lbr_description)/ros2_control/initial_joint_positions.yaml'">
+        params="robot_name:=^|lbr mode:=^|mock system_config_path:=^|'$(find lbr_description)/ros2_control/lbr_system_config.yaml' joint_limits_path:=^|'$(find lbr_description)/urdf/med14/joint_limits.yaml' initial_joint_positions_path:=^|'$(find lbr_description)/ros2_control/initial_joint_positions.yaml'">
         <!-- includes -->
         <xacro:include filename="$(find lbr_description)/gazebo/lbr_gazebo.xacro" />
         <xacro:include filename="$(find lbr_description)/ros2_control/lbr_system_interface.xacro" />
         <!-- joint limits via yaml -->
-        <xacro:property name="joint_limits_path"
-            value="$(find lbr_description)/urdf/med14/joint_limits.yaml" />
         <xacro:property name="joint_limits" value="${xacro.load_yaml(joint_limits_path)}" />
         <!-- constants -->

File: lbr_description/urdf/med7/med7.xacro (robot description, xacro)
@@ -9,4 +9,7 @@
         name="system_config_path"
         default="$(find lbr_description)/ros2_control/lbr_system_config.yaml" />
+    <xacro:arg
+        name="joint_limits_path"
+        default="$(find lbr_description)/urdf/med7/joint_limits.yaml" />
     <xacro:arg
         name="initial_joint_positions_path"
@@ -26,4 +29,5 @@
         mode="$(arg mode)"
         system_config_path="$(arg system_config_path)"
+        joint_limits_path="$(arg joint_limits_path)"
         initial_joint_positions_path="$(arg initial_joint_positions_path)" />
 </robot>

File: lbr_description/urdf/med7/med7_description.xacro (robot description, xacro)
@@ -3,11 +3,9 @@
     <!-- robot as extracted via https://github.com/syuntoku14/fusion2urdf -->
     <xacro:macro name="med7"
-        params="robot_name:=^|lbr mode:=^|mock system_config_path:=^|'$(find lbr_description)/ros2_control/lbr_system_config.yaml' initial_joint_positions_path:=^|'$(find lbr_description)/ros2_control/initial_joint_positions.yaml'">
+        params="robot_name:=^|lbr mode:=^|mock system_config_path:=^|'$(find lbr_description)/ros2_control/lbr_system_config.yaml' joint_limits_path:=^|'$(find lbr_description)/urdf/med7/joint_limits.yaml' initial_joint_positions_path:=^|'$(find lbr_description)/ros2_control/initial_joint_positions.yaml'">
         <!-- includes -->
         <xacro:include filename="$(find lbr_description)/gazebo/lbr_gazebo.xacro" />
         <xacro:include filename="$(find lbr_description)/ros2_control/lbr_system_interface.xacro" />
         <!-- joint limits via yaml -->
-        <xacro:property name="joint_limits_path"
-            value="$(find lbr_description)/urdf/med7/joint_limits.yaml" />
         <xacro:property name="joint_limits" value="${xacro.load_yaml(joint_limits_path)}" />
         <!-- constants -->
